Commit message: refactor tianji arm

File: m6_srs_description/xacro/arm.xacro (robot description, xacro)
@@ -4,5 +4,5 @@
 	<xacro:macro name="M6_SRS" params="name:='' direction:=1 collider:=convex">
 		<xacro:property name="prefix" value="${name + '_' if name else ''}"/>
-		<!-- Base Link -->
+		<!-- Base link -->
 		<link name="${prefix}base_link">
 			<inertial>
@@ -15,17 +15,14 @@
 			<visual>
 				<geometry>
-					<mesh filename="package://m6_srs_description/meshes/Base.STL"/>
-				</geometry>
-				<material name="">
-					<color rgba="1 0 0 1"/>
-				</material>
-			</visual>
-			<collision>
-				<geometry>
-					<mesh filename="package://m6_srs_description/meshes/Base.STL"/>
-				</geometry>
-			</collision>
-		</link>
-		<!-- Link 1 -->
+					<mesh filename="file://$(find m6_srs_description)/meshes/base.obj"/>
+				</geometry>
+			</visual>
+			<collision>
+				<geometry>
+					<mesh filename="file://$(find m6_srs_description)/meshes/base.obj"/>
+				</geometry>
+			</collision>
+		</link>
+		<!-- link 1 -->
 		<link name="${prefix}link1">
 			<inertial>
@@ -38,13 +35,10 @@
 			<visual>
 				<geometry>
-					<mesh filename="package://m6_srs_description/meshes/Link1.STL"/>
-				</geometry>
-				<material name="">
-					<color rgba="0 1 0 1"/>
-				</material>
-			</visual>
-			<collision>
-				<geometry>
-					<mesh filename="package://m6_srs_description/meshes/Link1.STL"/>
+					<mesh filename="file://$(find m6_srs_description)/meshes/link1.obj"/>
+				</geometry>
+			</visual>
+			<collision>
+				<geometry>
+					<mesh filename="file://$(find m6_srs_description)/meshes/link1.obj"/>
 				</geometry>
 			</collision>
@@ -57,5 +51,5 @@
 			<limit lower="-3.1067" upper="3.1067" effort="108" velocity="3.1416"/>
 		</joint>
-		<!-- Link 2 -->
+		<!-- link 2 -->
 		<link name="${prefix}link2">
 			<inertial>
@@ -68,13 +62,10 @@
 			<visual>
 				<geometry>
-					<mesh filename="package://m6_srs_description/meshes/Link2.STL"/>
-				</geometry>
-				<material name="">
-					<color rgba="0 0 1 1"/>
-				</material>
-			</visual>
-			<collision>
-				<geometry>
-					<mesh filename="package://m6_srs_description/meshes/Link2.STL"/>
+					<mesh filename="file://$(find m6_srs_description)/meshes/link2.obj"/>
+				</geometry>
+			</visual>
+			<collision>
+				<geometry>
+					<mesh filename="file://$(find m6_srs_description)/meshes/link2.obj"/>
 				</geometry>
 			</collision>
@@ -88,5 +79,5 @@
 			<limit lower="-2.0944" upper="2.0944" effort="108" velocity="3.1416"/>
 		</joint>
-		<!-- Link 3 -->
+		<!-- link 3 -->
 		<link name="${prefix}link3">
 			<inertial>
@@ -99,13 +90,10 @@
 			<visual>
 				<geometry>
-					<mesh filename="package://m6_srs_description/meshes/Link3.STL"/>
-				</geometry>
-				<material name="">
-					<color rgba="1 0 0 1"/>
-				</material>
-			</visual>
-			<collision>
-				<geometry>
-					<mesh filename="package://m6_srs_description/meshes/Link3.STL"/>
+					<mesh filename="file://$(find m6_srs_description)/meshes/link3.obj"/>
+				</geometry>
+			</visual>
+			<collision>
+				<geometry>
+					<mesh filename="file://$(find m6_srs_description)/meshes/link3.obj"/>
 				</geometry>
 			</collision>
@@ -119,5 +107,5 @@
 			<limit lower="-3.1067" upper="3.1067" effort="66" velocity="3.1416"/>
 		</joint>
-		<!-- Link 4 -->
+		<!-- link 4 -->
 		<link name="${prefix}link4">
 			<inertial>
@@ -130,13 +118,10 @@
 			<visual>
 				<geometry>
-					<mesh filename="package://m6_srs_description/meshes/Link4.STL"/>
-				</geometry>
-				<material name="">
-					<color rgba="0 1 0 1"/>
-				</material>
-			</visual>
-			<collision>
-				<geometry>
-					<mesh filename="package://m6_srs_description/meshes/Link4.STL"/>
+					<mesh filename="file://$(find m6_srs_description)/meshes/link4.obj"/>
+				</geometry>
+			</visual>
+			<collision>
+				<geometry>
+					<mesh filename="file://$(find m6_srs_description)/meshes/link4.obj"/>
 				</geometry>
 			</collision>
@@ -150,5 +135,5 @@
 			<limit lower="-2.5307" upper="1.0472" effort="66" velocity="3.1416"/>
 		</joint>
-		<!-- Link 5 -->
+		<!-- link 5 -->
 		<link name="${prefix}link5">
 			<inertial>
@@ -161,13 +146,10 @@
 			<visual>
 				<geometry>
-					<mesh filename="package://m6_srs_description/meshes/Link5.STL"/>
-				</geometry>
-				<material name="">
-					<color rgba="0 0 1 1"/>
-				</material>
-			</visual>
-			<collision>
-				<geometry>
-					<mesh filename="package://m6_srs_description/meshes/Link5.STL"/>
+					<mesh filename="file://$(find m6_srs_description)/meshes/link5.obj"/>
+				</geometry>
+			</visual>
+			<collision>
+				<geometry>
+					<mesh filename="file://$(find m6_srs_description)/meshes/link5.obj"/>
 				</geometry>
 			</collision>
@@ -181,5 +163,5 @@
 			<limit lower="-3.1067" upper="3.1067" effort="18" velocity="3.1416"/>
 		</joint>
-		<!-- Link 6 -->
+		<!-- link 6 -->
 		<link name="${prefix}link6">
 			<inertial>
@@ -192,5 +174,5 @@
 			<visual>
 				<geometry>
-					<mesh filename="package://m6_srs_description/meshes/Link6.STL"/>
+					<mesh filename="file://$(find m6_srs_description)/meshes/link6.obj"/>
 				</geometry>
 				<material name="">
@@ -200,5 +182,5 @@
 			<collision>
 				<geometry>
-					<mesh filename="package://m6_srs_description/meshes/Link6.STL"/>
+					<mesh filename="file://$(find m6_srs_description)/meshes/link6.obj"/>
 				</geometry>
 			</collision>
@@ -212,5 +194,5 @@
 			<limit lower="-1.9199" upper="1.9199" effort="18" velocity="3.1416"/>
 		</joint>
-		<!-- Link 7 -->
+		<!-- link 7 -->
 		<link name="${prefix}link7">
 			<inertial>
@@ -223,5 +205,5 @@
 			<visual>
 				<geometry>
-					<mesh filename="package://m6_srs_description/meshes/Link7.STL" scale="1 ${direction} 1"/>
+					<mesh filename="file://$(find m6_srs_description)/meshes/link7.obj" scale="1 ${direction} 1"/>
 				</geometry>
 				<material name="">
@@ -231,5 +213,5 @@
 			<collision>
 				<geometry>
-					<mesh filename="package://m6_srs_description/meshes/Link7.STL" scale="1 ${direction} 1"/>
+					<mesh filename="file://$(find m6_srs_description)/meshes/link7.obj" scale="1 ${direction} 1"/>
 				</geometry>
 			</collision>

File: m6_srs_description/xacro/ros2_control/interfaces.xacro (robot description, xacro)
@@ -1,5 +1,5 @@
 <?xml version="1.0"?>
 <robot xmlns:xacro="http://www.ros.org/wiki/xacro">
-	<xacro:macro name="ar5_interfaces" params="name">
+	<xacro:macro name="m6_interfaces" params="name">
 		<xacro:property name="prefix" value="${name + '_' if name else ''}"/>
 		<!-- 关节接口定义 -->

File: m6_srs_description/xacro/ros2_control/robot.xacro (robot description, xacro)
@@ -1,4 +1,4 @@
 <?xml version="1.0"?>
-<robot xmlns:xacro="http://www.ros.org/wiki/xacro" name="AR5">
+<robot xmlns:xacro="http://www.ros.org/wiki/xacro" name="M6 SRS">
   <xacro:arg name="ros2_control_hardware_type" default="mock_components"/>
   <link name="world"/>
@@ -8,7 +8,7 @@
     <origin/>
   </joint>
-  <xacro:include filename="$(find rokae_ar5_description)/xacro/robot.xacro"/>
-  <xacro:include filename="$(find rokae_ar5_description)/xacro/ros2_control/interfaces.xacro"/>
-  <ros2_control name="ar5System" type="system">
+  <xacro:include filename="$(find m6_srs_description)/xacro/robot.xacro"/>
+  <xacro:include filename="$(find m6_srs_description)/xacro/ros2_control/interfaces.xacro"/>
+  <ros2_control name="m6System" type="system">
     <hardware>
       <xacro:if value="${'$(arg ros2_control_hardware_type)' == 'gz'}">
@@ -25,10 +25,6 @@
         <param name="initialize_commands_from_state">true</param>
       </xacro:if>
-      <xacro:if value="${'$(arg ros2_control_hardware_type)' == 'real'}">
-        <plugin>rokae_ros2_control/RokaeHardware</plugin>
-        <param name="arm_ip">192.168.2.160</param>
-      </xacro:if>
     </hardware>
-    <xacro:ar5_interfaces name=""/>
+    <xacro:m6_interfaces name=""/>
   </ros2_control>
   <xacro:arg name="gazebo" default="false"/>
@@ -37,8 +33,8 @@
       <plugin filename="gz_ros2_control-system" name="gz_ros2_control::GazeboSimROS2ControlPlugin">
         <xacro:if value="${'$(arg type)' == 'left'}">
-          <parameters>$(find rokae_ar5_description)/config/ros2_control/ros2_controllers.yaml</parameters>
+          <parameters>$(find m6_srs_description)/config/ros2_control/ros2_controllers.yaml</parameters>
         </xacro:if>
         <xacro:if value="${'$(arg type)' == 'right'}">
-          <parameters>$(find rokae_ar5_description)/config/ros2_control/right.yaml</parameters>
+          <parameters>$(find m6_srs_description)/config/ros2_control/right.yaml</parameters>
         </xacro:if>
       </plugin>
