Commit message: update m6 usb scene configuration

File: m6_ccs_description/urdf/m6_ccs_usb-90c.urdf (robot description, URDF)
Before this commit: robot DobotCR5, 23 links, 22 joints
Joints:
- joint base_joint: origin rpy=0 0 -1.5707963267948966 -> rpy=0 0 0

File: m6_ccs_description/xacro/robot.xacro (robot description, xacro)
@@ -39,5 +39,5 @@
 			<parent link="base_link"/>
 			<child link="base"/>
-			<origin rpy="0 0 -${PI/2}"/>
+			<origin rpy="0 0 0"/>
 		</joint>
 		<link name="base">

File: m6_ccs_description/xacro/ros2_control/robot.xacro (robot description, xacro)
@@ -34,7 +34,10 @@
 						<param name="left_right_arm">0</param>
 					</xacro:if>
-					<xacro:unless value="${'$(arg type)' == 'left'}">
-						<param name="left_right_arm">1</param>
-					</xacro:unless>
+					<xacro:if value="${'$(arg type)' == 'usb-90c'}">
+						<param name="left_right_arm">0</param>
+					</xacro:if>
+					<xacro:if value="${'$(arg type)' == 'right'}">
+						<param name="left_right_arm">0</param>
+					</xacro:if>
 				</xacro:unless>
 			</xacro:if>
