Commit message: fixed dual arm config

File: m6_ccs_description/urdf/m6_ccs_dual_rg75.urdf (robot description, URDF)
Before this commit: robot DobotCR5, 34 links, 33 joints
Joints:
- joint left_gripper_base_joint: origin xyz=0 0 -0.0045 rpy=1.5707963267948966 0 0 -> rpy=-1.5707963267948966 0 3.141592653589793
- joint right_gripper_base_joint: origin xyz=0 0 -0.0045 rpy=1.5707963267948966 0 0 -> rpy=1.5707963267948966 0 0

File: m6_ccs_description/xacro/robot.xacro (robot description, xacro)
@@ -1,4 +1,4 @@
 <?xml version="1.0"?>
-<robot name="DobotCR5" xmlns:xacro="http://www.ros.org/wiki/xacro">
+<robot name="M6_CCS" xmlns:xacro="http://www.ros.org/wiki/xacro">
 	<xacro:arg name="collider" default="convex"/>
 	<xacro:arg name="type" default="left"/>
@@ -58,10 +58,10 @@
 			<xacro:RG75-300 name="right" use_flange="true"/>
 			<joint name="left_gripper_base_joint" type="fixed">
-				<origin xyz="0 0 -0.0045" rpy="${PI/2} 0 0"/>
+				<origin rpy="${-PI/2} 0 ${PI}"/>
 				<parent link="left_tcp"/>
 				<child link="left_flange"/>
 			</joint>
 			<joint name="right_gripper_base_joint" type="fixed">
-				<origin xyz="0 0 -0.0045" rpy="${PI/2} 0 0"/>
+				<origin rpy="${PI/2} 0 0"/>
 				<parent link="right_tcp"/>
 				<child link="right_flange"/>

Commit message: update dual.info

File: m6_ccs_description/urdf/m6_ccs_dual_rg75.urdf (robot description, URDF)
Before this commit: robot M6_CCS, 34 links, 33 joints
Links:
- link arm_base: geometry collision box size=0.2000 0.3 0.4029
- link left_link3: geometry collision cylinder length=0.117016 radius=0.049964; visual mesh filename=package://m6_ccs_description/meshes/link3.obj
- link right_link3: geometry collision cylinder length=0.117016 radius=0.049964; visual mesh filename=package://m6_ccs_description/meshes/link3.obj
