Commit message: add tianji desktop dual 90c

File: m6_ccs_description/urdf/m6_ccs_dual_desktop.urdf (robot description, URDF)
Before this commit: robot DobotCR5, 21 links, 20 joints
Links:
- added link arm_base; collision box size=0.10045 0.100398 0.648662; visual mesh filename=package://m6_ccs_description/meshes/dual_base.obj
- link base_link: geometry 
- link left_link3: geometry collision cylinder length=0.117016 radius=0.049964; visual mesh filename=package://m6_ccs_description/meshes/link3.obj
- link right_link3: geometry collision cylinder length=0.117016 radius=0.049964; visual mesh filename=package://m6_ccs_description/meshes/link3.obj
Joints:
- added joint arm_base_joint: type fixed, parent base_link, child arm_base
- joint left_arm_base_joint: parent base_link -> arm_base
- joint left_tcp_joint: origin xyz=0 -0.095 0 rpy=1.5707963267948966 1.5707963267948966 0 -> xyz=0 -0.095 0 rpy=1.5707963267948966 -1.5707963267948966 0
- joint right_arm_base_joint: parent base_link -> arm_base
- joint right_tcp_joint: origin xyz=0 -0.095 0 rpy=1.5707963267948966 1.5707963267948966 0 -> xyz=0 -0.095 0 rpy=1.5707963267948966 -1.5707963267948966 0

File: m6_ccs_description/xacro/robot.xacro (robot description, xacro)
@@ -24,10 +24,10 @@
 	<xacro:if value="${type_arg == 'usb-90c'}">
 		<xacro:property name="selected_arm_config" value="left"/>
-		<xacro:property name="selected_gripper_type" value="ag2f90"/>
+		<xacro:property name="selected_gripper_type" value="ag2f90c"/>
 		<xacro:property name="selected_scene" value="usb-90c"/>
 	</xacro:if>
 	<!-- 双臂配置 -->
-	<xacro:if value="${type_arg == 'dual_ag2f90'}">
-		<xacro:property name="selected_gripper_type" value="ag2f90"/>
+	<xacro:if value="${type_arg == 'dual_ag2f90c'}">
+		<xacro:property name="selected_gripper_type" value="ag2f90c"/>
 	</xacro:if>
 	<xacro:if value="${type_arg == 'dual_rg75'}">
@@ -36,4 +36,8 @@
 	<xacro:if value="${type_arg == 'dual_desktop'}">
 		<xacro:property name="selected_scene" value="desktop"/>
+	</xacro:if>
+	<xacro:if value="${type_arg == 'dual_desktop_90c'}">
+		<xacro:property name="selected_scene" value="desktop"/>
+		<xacro:property name="selected_gripper_type" value="ag2f90c"/>
 	</xacro:if>
 	<xacro:include filename="$(find m6_ccs_description)/xacro/arm.xacro"/>
@@ -58,6 +62,6 @@
 		<!-- Base link 和 arm_base 根据 scene 设置 -->
 		<xacro:if value="${selected_scene == 'desktop'}">
-			<!-- Desktop 场景：base_link 有视觉和碰撞，没有 arm_base -->
-			<link name="base_link">
+			<link name="base_link"/>
+			<link name="arm_base">
 				<visual>
 					<geometry>
@@ -72,7 +76,11 @@
 				</collision>
 			</link>
+			<joint name="arm_base_joint" type="fixed">
+				<parent link="base_link"/>
+				<child link="arm_base"/>
+			</joint>
 			<!-- Left Arm -->
 			<joint name="left_arm_base_joint" type="fixed">
-				<parent link="base_link"/>
+				<parent link="arm_base"/>
 				<child link="left_base_link"/>
 				<origin rpy="-${PI/2} 0 0" xyz="0.0 0.12 0.701"/>
@@ -80,8 +88,20 @@
 			<!-- Right Arm -->
 			<joint name="right_arm_base_joint" type="fixed">
-				<parent link="base_link"/>
+				<parent link="arm_base"/>
 				<child link="right_base_link"/>
 				<origin rpy="${PI/2} 0 0" xyz="0.0 -0.12 0.701"/>
 			</joint>
+			<xacro:if value="${selected_gripper_type == 'none'}">
+				<link name="right_eef"/>
+				<joint name="right_eef_joint" type="fixed">
+					<parent link="right_tcp"/>
+					<child link="right_eef"/>
+				</joint>
+				<link name="left_eef"/>
+				<joint name="left_eef_joint" type="fixed">
+					<parent link="left_tcp"/>
+					<child link="left_eef"/>
+				</joint>
+			</xacro:if>
 		</xacro:if>
 		<xacro:unless value="${selected_scene == 'desktop'}">
@@ -117,5 +137,5 @@
 		<xacro:M6_CCS name="right" direction="-1" collider="$(arg collider)"/>
 		<!-- 双臂末端执行器 -->
-		<xacro:if value="${selected_gripper_type == 'ag2f90'}">
+		<xacro:if value="${selected_gripper_type == 'ag2f90c'}">
 			<xacro:include filename="$(find changingtek_description)/xacro/AG2F90-C.xacro"/>
 			<xacro:AG2F90-C name="left" use_flange="true"/>
@@ -176,5 +196,5 @@
 		<xacro:M6_CCS name="left" collider="$(arg collider)"/>
 		<!-- USB-90C 默认使用 AG2F90 末端 -->
-		<xacro:if value="${selected_gripper_type == 'ag2f90' or selected_gripper_type == 'none'}">
+		<xacro:if value="${selected_gripper_type == 'ag2f90c' or selected_gripper_type == 'none'}">
 			<xacro:include filename="$(find changingtek_description)/xacro/AG2F90-C.xacro"/>
 			<xacro:AG2F90-C name="" use_flange="true"/>

File: m6_ccs_description/xacro/ros2_control/robot.xacro (robot description, xacro)
@@ -42,5 +42,5 @@
 			<xacro:m6_interfaces name="left"/>
 			<xacro:m6_interfaces name="right"/>
-			<xacro:if value="${selected_gripper_type == 'ag2f90'}">
+			<xacro:if value="${selected_gripper_type == 'ag2f90c'}">
 				<xacro:include filename="$(find changingtek_description)/xacro/ros2_control/AG2F90-C.xacro"/>
 				<xacro:ag2f90c_interfaces name="left"/>
@@ -57,5 +57,5 @@
 			<xacro:if value="${selected_arm_config == 'left'}">
 				<xacro:m6_interfaces name=""/>
-				<xacro:if value="${selected_gripper_type == 'ag2f90'}">
+				<xacro:if value="${selected_gripper_type == 'ag2f90c'}">
 					<xacro:include filename="$(find changingtek_description)/xacro/ros2_control/AG2F90-C.xacro"/>
 					<xacro:ag2f90c_interfaces name=""/>
