Commit message: add m6 ccs dual

File: m6_ccs_description/urdf/m6_ccs_dual_ag2f90_c.urdf (robot description, URDF)
Before this commit: robot M6_CCS, 46 links, 45 joints
Links:
- link left_link3: geometry collision cylinder length=0.117016 radius=0.049964; visual mesh filename=package://m6_ccs_description/meshes/link3.obj
- link right_link3: geometry collision cylinder length=0.117016 radius=0.049964; visual mesh filename=package://m6_ccs_description/meshes/link3.obj

File: m6_ccs_description/xacro/robot.xacro (robot description, xacro)
@@ -24,11 +24,19 @@
 	<xacro:if value="${type_arg == 'usb-90c'}">
 		<xacro:property name="selected_arm_config" value="left"/>
-		<xacro:property name="selected_gripper_type" value="ag2f90c"/>
+		<xacro:property name="selected_gripper_type" value="ag2f90_c"/>
 		<xacro:property name="selected_scene" value="usb-90c"/>
 	</xacro:if>
 	<!-- 双臂配置 -->
-	<xacro:if value="${type_arg == 'dual_ag2f90c'}">
-		<xacro:property name="selected_gripper_type" value="ag2f90c"/>
-	</xacro:if>
+	<!-- 适用于人形机器人的配置 -->
+	<xacro:if value="${type_arg == 'dual_ag2f90'}">
+		<xacro:property name="selected_gripper_type" value="ag2f90d"/>
+	</xacro:if>
+	<xacro:if value="${type_arg == 'dual_ag2f90_c'}">
+		<xacro:property name="selected_gripper_type" value="ag2f90_c"/>
+	</xacro:if>
+	<xacro:if value="${type_arg == 'dual_ag2f90_d'}">
+		<xacro:property name="selected_gripper_type" value="ag2f90_d"/>
+	</xacro:if>
+	<!-- 适用纯双臂演示场景的配置 -->
 	<xacro:if value="${type_arg == 'dual_rg75'}">
 		<xacro:property name="selected_gripper_type" value="rg75"/>
@@ -39,5 +47,5 @@
 	<xacro:if value="${type_arg == 'dual_desktop_90c'}">
 		<xacro:property name="selected_scene" value="desktop"/>
-		<xacro:property name="selected_gripper_type" value="ag2f90c"/>
+		<xacro:property name="selected_gripper_type" value="ag2f90_c"/>
 	</xacro:if>
 	<xacro:include filename="$(find m6_ccs_description)/xacro/arm.xacro"/>
@@ -137,5 +145,5 @@
 		<xacro:M6_CCS name="right" direction="-1" collider="$(arg collider)"/>
 		<!-- 双臂末端执行器 -->
-		<xacro:if value="${selected_gripper_type == 'ag2f90c'}">
+		<xacro:if value="${selected_gripper_type == 'ag2f90_c' or selected_gripper_type == 'ag2f90_d'}">
 			<xacro:include filename="$(find changingtek_description)/xacro/AG2F90-C.xacro"/>
 			<xacro:AG2F90-C name="left" use_flange="true"/>
@@ -173,5 +181,4 @@
 			<parent link="base_link"/>
 			<child link="base"/>
-			<origin rpy="0 0 0"/>
 		</joint>
 		<link name="base">
@@ -195,14 +202,11 @@
 		</joint>
 		<xacro:M6_CCS name="left" collider="$(arg collider)"/>
-		<!-- USB-90C 默认使用 AG2F90 末端 -->
-		<xacro:if value="${selected_gripper_type == 'ag2f90c' or selected_gripper_type == 'none'}">
-			<xacro:include filename="$(find changingtek_description)/xacro/AG2F90-C.xacro"/>
-			<xacro:AG2F90-C name="" use_flange="true"/>
-			<joint name="gripper_fix" type="fixed">
-				<parent link="left_link7"/>
-				<child link="flange"/>
-				<origin xyz="0 -0.0995 0" rpy=" ${PI/2} 0 0"/>
-			</joint>
-		</xacro:if>
+		<xacro:include filename="$(find changingtek_description)/xacro/AG2F90-C.xacro"/>
+		<xacro:AG2F90-C name="" use_flange="true"/>
+		<joint name="gripper_fix" type="fixed">
+			<parent link="left_link7"/>
+			<child link="flange"/>
+			<origin xyz="0 -0.0995 0" rpy=" ${PI/2} 0 0"/>
+		</joint>
 	</xacro:if>
 </robot>

File: m6_ccs_description/xacro/ros2_control/robot.xacro (robot description, xacro)
@@ -42,5 +42,5 @@
 			<xacro:m6_interfaces name="left"/>
 			<xacro:m6_interfaces name="right"/>
-			<xacro:if value="${selected_gripper_type == 'ag2f90c'}">
+			<xacro:if value="${selected_gripper_type == 'ag2f90_c' or selected_gripper_type == 'ag2f90_d'}">
 				<xacro:include filename="$(find changingtek_description)/xacro/ros2_control/AG2F90-C.xacro"/>
 				<xacro:ag2f90c_interfaces name="left"/>
@@ -62,5 +62,5 @@
 					<xacro:m6_interfaces name=""/>
 				</xacro:unless>
-				<xacro:if value="${selected_gripper_type == 'ag2f90c'}">
+				<xacro:if value="${selected_gripper_type == 'ag2f90_c' or selected_gripper_type == 'ag2f90_d'}">
 					<xacro:include filename="$(find changingtek_description)/xacro/ros2_control/AG2F90-C.xacro"/>
 					<xacro:ag2f90c_interfaces name=""/>
