Commit message: add tianji dual base

File: m6_ccs_description/urdf/m6_ccs_dual.urdf (robot description, URDF)
Before this commit: robot DobotCR5, 17 links, 16 joints
Links:
- link base_link: geometry visual mesh filename=package://m6_ccs_description/meshes/dual_base.obj
Joints:
- joint left_arm_base_joint: origin xyz=0.0 0.05 0 rpy=-1.5708 1.5708 0 -> xyz=0.0 0.12 0.701 rpy=-1.5708 0 0
- joint right_arm_base_joint: origin xyz=0.0 -0.05 0 rpy=1.5708 1.5708 0 -> xyz=0.0 -0.12 0.701 rpy=1.5708 0 0

File: m6_ccs_description/xacro/robot.xacro (robot description, xacro)
@@ -22,5 +22,5 @@
 			<parent link="base_link"/>
 			<child link="left_base_link"/>
-			<origin rpy="-1.5708 1.5708 0" xyz="0.0 0.12 0.701"/>
+			<origin rpy="-1.5708 0 0" xyz="0.0 0.12 0.701"/>
 		</joint>
 		<!-- Right Arm -->
@@ -28,5 +28,5 @@
 			<parent link="base_link"/>
 			<child link="right_base_link"/>
-			<origin rpy="1.5708 1.5708 0" xyz="0.0 -0.12 0.701"/>
+			<origin rpy="1.5708 0 0" xyz="0.0 -0.12 0.701"/>
 		</joint>
 		<xacro:M6_CCS name="left"/>

Commit message: 添加m6_ccs碰撞体和自碰撞检测

File: m6_ccs_description/urdf/m6_ccs_dual.urdf (robot description, URDF)
Before this commit: robot DobotCR5, 17 links, 16 joints
Links:
- added link left_eef
- added link right_eef
- link base_link: geometry collision box size=0.10045 0.100398 0.648662; visual mesh filename=package://m6_ccs_description/meshes/dual_base.obj
- link left_base_link: geometry collision cylinder length=0.083664 radius=0.051277; visual mesh filename=package://m6_ccs_description/meshes/base.obj
- link left_link1: geometry collision cylinder length=0.125958 radius=0.057588; visual mesh filename=package://m6_ccs_description/meshes/link1.obj
- link left_link2: geometry collision cylinder length=0.078386 radius=0.046717; visual mesh filename=package://m6_ccs_description/meshes/link2.obj
- link left_link3: geometry collision cylinder length=0.089056 radius=0.046717; collision cylinder length=0.117016 radius=0.049964
- link left_link4: geometry collision cylinder length=0.080203 radius=0.041759; visual mesh filename=package://m6_ccs_description/meshes/link4.obj
- link left_link5: geometry collision cylinder length=0.14268 radius=0.056747; visual mesh filename=package://m6_ccs_description/meshes/link5.obj scale=1 1 1
- link left_link6: geometry collision cylinder length=0.108046 radius=0.038348; visual mesh filename=package://m6_ccs_description/meshes/link6.obj
- link left_link7: geometry collision cylinder length=0.038392 radius=0.041707; visual mesh filename=package://m6_ccs_description/meshes/link7.obj
- link right_base_link: geometry collision cylinder length=0.083664 radius=0.051277; visual mesh filename=package://m6_ccs_description/meshes/base.obj
- link right_link1: geometry collision cylinder length=0.125958 radius=0.057588; visual mesh filename=package://m6_ccs_description/meshes/link1.obj
- link right_link2: geometry collision cylinder length=0.078386 radius=0.046717; visual mesh filename=package://m6_ccs_description/meshes/link2.obj
- link right_link3: geometry collision cylinder length=0.089056 radius=0.046717; collision cylinder length=0.117016 radius=0.049964
- link right_link4: geometry collision cylinder length=0.080203 radius=0.041759; visual mesh filename=package://m6_ccs_description/meshes/link4.obj
- link right_link5: geometry collision cylinder length=0.14268 radius=0.056747; visual mesh filename=package://m6_ccs_description/meshes/link5.obj scale=1 -1 1
- link right_link6: geometry collision cylinder length=0.108046 radius=0.038348; visual mesh filename=package://m6_ccs_description/meshes/link6.obj
- link right_link7: geometry collision cylinder length=0.038392 radius=0.041707; visual mesh filename=package://m6_ccs_description/meshes/link7_r.obj
Joints:
- added joint left_eef_joint: type fixed, parent left_link7, child left_eef, origin xyz=0 -0.095296 0 rpy=0 0 0
- added joint right_eef_joint: type fixed, parent right_link7, child right_eef, origin xyz=0 -0.095296 0 rpy=0 0 0

File: m6_ccs_description/xacro/arm.xacro (robot description, xacro)
@@ -18,9 +18,19 @@
 				</geometry>
 			</visual>
-			<collision>
-				<geometry>
-					<mesh filename="file://$(find m6_ccs_description)/meshes/base.obj"/>
-				</geometry>
-			</collision>
+			<xacro:if value="${collider == 'convex'}">
+				<collision>
+					<geometry>
+						<mesh filename="file://$(find m6_ccs_description)/meshes/base.obj"/>
+					</geometry>
+				</collision>
+			</xacro:if>
+			<xacro:if value="${collider == 'simple'}">
+				<collision>
+					<origin xyz="0 0 0.041832"/>
+					<geometry>
+						<cylinder length="0.083664" radius="0.051277"/>
+					</geometry>
+				</collision>
+			</xacro:if>
 		</link>
 		<!-- Link 1 -->
@@ -38,9 +48,19 @@
 				</geometry>
 			</visual>
-			<collision>
-				<geometry>
-					<mesh filename="file://$(find m6_ccs_description)/meshes/link1.obj"/>
-				</geometry>
-			</collision>
+			<xacro:if value="${collider == 'convex'}">
+				<collision>
+					<geometry>
+						<mesh filename="file://$(find m6_ccs_description)/meshes/link1.obj"/>
+					</geometry>
+				</collision>
+			</xacro:if>
+			<xacro:if value="${collider == 'simple'}">
+				<collision>
+					<origin rpy="1.5708 0 0"/>
+					<geometry>
+						<cylinder length="0.125958" radius="0.057588"/>
+					</geometry>
+				</collision>
+			</xacro:if>
 		</link>
 		<!-- Joint 1 -->
@@ -66,9 +86,19 @@
 				</geometry>
 			</visual>
-			<collision>
-				<geometry>
-					<mesh filename="file://$(find m6_ccs_description)/meshes/link2.obj"/>
-				</geometry>
-			</collision>
+			<xacro:if value="${collider == 'convex'}">
+				<collision>
+					<geometry>
+						<mesh filename="file://$(find m6_ccs_description)/meshes/link2.obj"/>
+					</geometry>
+				</collision>
+			</xacro:if>
+			<xacro:if value="${collider == 'simple'}">
+				<collision>
+					<origin xyz="0 0.099087 0" rpy="1.5708 0 0"/>
+					<geometry>
+						<cylinder length="0.078386" radius="0.046717"/>
+					</geometry>
+				</collision>
+			</xacro:if>
 		</link>
 		<!-- Joint 2 -->
@@ -94,9 +124,25 @@
 				</geometry>
 			</visual>
-			<collision>
-				<geometry>
-					<mesh filename="file://$(find m6_ccs_description)/meshes/link3.obj"/>
-				</geometry>
-			</collision>
+			<xacro:if value="${collider == 'convex'}">
+				<collision>
+					<geometry>
+						<mesh filename="file://$(find m6_ccs_description)/meshes/link3.obj"/>
+					</geometry>
+				</collision>
+			</xacro:if>
+			<xacro:if value="${collider == 'simple'}">
+				<collision>
+					<origin xyz="0 0 -0.098932"/>
+					<geometry>
+						<cylinder length="0.089056" radius="0.046717"/>
+					</geometry>
+				</collision>
+				<collision>
+					<origin xyz="0.018119 0 0" rpy="1.5708 0 0"/>
+					<geometry>
+						<cylinder length="0.117016" radius="0.049964"/>
+					</geometry>
+				</collision>
+			</xacro:if>
 		</link>
 		<!-- Joint 3 -->
@@ -122,9 +168,19 @@
 				</geometry>
 			</visual>
-			<collision>
-				<geometry>
-					<mesh filename="file://$(find m6_ccs_description)/meshes/link4.obj"/>
-				</geometry>
-			</collision>
+			<xacro:if value="${collider == 'convex'}">
+				<collision>
+					<geometry>
+						<mesh filename="file://$(find m6_ccs_description)/meshes/link4.obj"/>
+					</geometry>
+				</collision>
+			</xacro:if>
+			<xacro:if value="${collider == 'simple'}">
+				<collision>
+					<origin xyz="0.017721 -0.079733 0" rpy="1.5708 0 0"/>
+					<geometry>
+						<cylinder length="0.080203" radius="0.041759"/>
+					</geometry>
+				</collision>
+			</xacro:if>
 		</link>
 		<!-- Joint 4 -->
@@ -150,9 +206,19 @@
 				</geometry>
 			</visual>
-			<collision>
-				<geometry>
-					<mesh filename="file://$(find m6_ccs_description)/meshes/link5.obj" scale="1 ${direction} 1"/>
-				</geometry>
-			</collision>
+			<xacro:if value="${collider == 'convex'}">
+				<collision>
+					<geometry>
+						<mesh filename="file://$(find m6_ccs_description)/meshes/link5.obj" scale="1 ${direction} 1"/>
+					</geometry>
+				</collision>
+			</xacro:if>
+			<xacro:if value="${collider == 'simple'}">
+				<collision>
+					<origin xyz="0 0 -0.117153"/>
+					<geometry>
+						<cylinder length="0.14268" radius="0.056747"/>
+					</geometry>
+				</collision>
+			</xacro:if>
 		</link>
 		<!-- Joint 5 -->
@@ -178,9 +244,19 @@
 				</geometry>
 			</visual>
-			<collision>
-				<geometry>
-					<mesh filename="file://$(find m6_ccs_description)/meshes/link6.obj"/>
-				</geometry>
-			</collision>
+			<xacro:if value="${collider == 'convex'}">
+				<collision>
+					<geometry>
+						<mesh filename="file://$(find m6_ccs_description)/meshes/link6.obj"/>
+					</geometry>
+				</collision>
+			</xacro:if>
+			<xacro:if value="${collider == 'simple'}">
+				<collision>
+					<origin xyz="0 0 0" rpy="1.5708 0 0"/>
+					<geometry>
+						<cylinder length="0.108046" radius="0.038348"/>
+					</geometry>
+				</collision>
+			</xacro:if>
 		</link>
 		<!-- Joint 6 -->
@@ -211,14 +287,19 @@
 				</geometry>
 			</visual>
-			<collision>
-				<geometry>
-					<xacro:if value="${direction == 1}">
+			<xacro:if value="${collider == 'convex'}">
+				<collision>
+					<geometry>
 						<mesh filename="file://$(find m6_ccs_description)/meshes/link7.obj"/>
-					</xacro:if>
-					<xacro:if value="${direction == -1}">
-						<mesh filename="file://$(find m6_ccs_description)/meshes/link7_r.obj"/>
-					</xacro:if>
-				</geometry>
-			</collision>
+					</geometry>
+				</collision>
+			</xacro:if>
+			<xacro:if value="${collider == 'simple'}">
+				<collision>
+					<origin xyz="0 -0.075732 0" rpy="1.5708 0 0"/>
+					<geometry>
+						<cylinder length="0.038392" radius="0.041707"/>
+					</geometry>
+				</collision>
+			</xacro:if>
 		</link>
 		<!-- Joint 7 -->
@@ -230,4 +311,10 @@
 			<limit lower="-1.5708" upper="1.5708" effort="18" velocity="3.1416"/>
 		</joint>
+		<link name="${prefix}eef"/>
+		<joint name="${prefix}eef_joint" type="fixed">
+			<origin rpy="0 0 0" xyz="0 -0.095296 0"/>
+			<parent link="${prefix}link7"/>
+			<child link="${prefix}eef"/>
+		</joint>
 	</xacro:macro>
 </robot>

File: m6_ccs_description/xacro/robot.xacro (robot description, xacro)
@@ -5,8 +5,8 @@
 	<xacro:include filename="$(find m6_ccs_description)/xacro/arm.xacro"/>
 	<xacro:if value="${'$(arg type)' == 'left'}">
-		<xacro:M6_CCS/>
+		<xacro:M6_CCS collider="$(arg collider)"/>
 	</xacro:if>
 	<xacro:if value="${'$(arg type)' == 'right'}">
-		<xacro:M6_CCS direction="-1"/>
+		<xacro:M6_CCS direction="-1" collider="$(arg collider)"/>
 	</xacro:if>
 	<xacro:if value="${'$(arg type)' == 'dual'}">
@@ -17,4 +17,10 @@
 				</geometry>
 			</visual>
+			<collision>
+				<origin xyz="0 0 0.324331"/>
+				<geometry>
+					<box size="0.10045 0.100398 0.648662"/>
+				</geometry>
+			</collision>
 		</link>
 		<!-- Left Arm -->
@@ -30,6 +36,6 @@
 			<origin rpy="1.5708 0 0" xyz="0.0 -0.12 0.701"/>
 		</joint>
-		<xacro:M6_CCS name="left"/>
-		<xacro:M6_CCS name="right" direction="-1"/>
+		<xacro:M6_CCS name="left" collider="$(arg collider)"/>
+		<xacro:M6_CCS name="right" direction="-1" collider="$(arg collider)"/>
 	</xacro:if>
 	<xacro:if value="${'$(arg type)' == 'usb-90c'}">
@@ -47,4 +53,10 @@
 				</geometry>
 			</visual>
+			<collision>
+				<origin xyz="0 0 0.324331"/>
+				<geometry>
+					<box size="0.10045 0.100398 0.648662"/>
+				</geometry>
+			</collision>
 		</link>
 		<!-- Left Arm -->
@@ -54,5 +66,5 @@
 			<origin rpy="-${PI/2} 0 0" xyz="0.0 0.12 0.701"/>
 		</joint>
-		<xacro:M6_CCS name="left"/>
+		<xacro:M6_CCS name="left" collider="$(arg collider)"/>
 		<xacro:include filename="$(find changingtek_description)/xacro/AG2F90-C.xacro"/>
 		<xacro:AG2F90-C name="" use_flange="true"/>

Commit message: update param set

File: m6_ccs_description/urdf/m6_ccs_dual.urdf (robot description, URDF)
Before this commit: robot M6_CCS, 22 links, 21 joints
Links:
- link left_link3: geometry collision cylinder length=0.117016 radius=0.049964; visual mesh filename=package://m6_ccs_description/meshes/link3.obj
- link right_link3: geometry collision cylinder length=0.117016 radius=0.049964; visual mesh filename=package://m6_ccs_description/meshes/link3.obj

File: m6_ccs_description/xacro/ros2_control/robot.xacro (robot description, xacro)
@@ -31,8 +31,15 @@
 				<plugin>marvin_ros2_control/MarvinHardware</plugin>
 				<param name="arm_type">${selected_arm_config}</param>
-				<param name="ctrl_mode">position</param>
 				<param name="gripper_type">${selected_gripper_type}</param>
-				<param name="max_velocity">40</param>
-				<param name="max_acceleration">10</param>
+				<param name="max_joint_speed">50</param>
+				<param name="max_joint_acceleration">30</param>
+				<xacro:if value="${selected_scene == 'desktop'}">
+					<param name="device_ip">192.168.10.190</param>
+					<param name="ctrl_mode">JOINT_IMPEDANCE</param>
+				</xacro:if>
+				<xacro:if value="${selected_scene == 'usb-90c'}">
+					<param name="device_ip">192.168.10.190</param>
+					<param name="ctrl_mode">CART_IMPEDANCE</param>
+				</xacro:if>
 			</xacro:if>
 		</hardware>

Commit message: update body collision

File: m6_ccs_description/urdf/m6_ccs_dual.urdf (robot description, URDF)
Before this commit: robot M6_CCS, 22 links, 21 joints
Links:
- link arm_base: geometry collision box size=0.2000 0.3 0.4029

File: m6_ccs_description/urdf/m6_ccs_dual_ag2f90_c.urdf (robot description, URDF)
Before this commit: robot M6_CCS, 46 links, 45 joints
Links:
- link arm_base: geometry collision box size=0.2000 0.3 0.4029

File: m6_ccs_description/xacro/robot.xacro (robot description, xacro)
@@ -118,7 +118,7 @@
 			<link name="arm_base">
 				<collision>
-					<origin xyz="0.0091 0 -0.2"/>
+					<origin xyz="0.0091 0 -0.25"/>
 					<geometry>
-						<box size="0.2000 0.32 0.5029"/>
+						<box size="0.2000 0.3 0.4029"/>
 					</geometry>
 				</collision>

Commit message: update urdf arm collision

File: m6_ccs_description/urdf/m6_ccs_dual.urdf (robot description, URDF)
Before this commit: robot M6_CCS, 22 links, 21 joints
Links:
- link left_link3: geometry collision cylinder length=0.089056 radius=0.046717; collision cylinder length=0.117016 radius=0.049964
- link right_link3: geometry collision cylinder length=0.089056 radius=0.046717; collision cylinder length=0.117016 radius=0.049964

File: m6_ccs_description/urdf/m6_ccs_dual_ag2f90_c.urdf (robot description, URDF)
Before this commit: robot M6_CCS, 46 links, 45 joints
Links:
- link left_link3: geometry collision cylinder length=0.089056 radius=0.046717; collision cylinder length=0.117016 radius=0.049964
- link right_link3: geometry collision cylinder length=0.089056 radius=0.046717; collision cylinder length=0.117016 radius=0.049964

File: m6_ccs_description/urdf/m6_ccs_dual_rg75.urdf (robot description, URDF)
Before this commit: robot M6_CCS, 34 links, 33 joints
Links:
- link left_link3: geometry collision cylinder length=0.089056 radius=0.046717; collision cylinder length=0.117016 radius=0.049964
- link right_link3: geometry collision cylinder length=0.089056 radius=0.046717; collision cylinder length=0.117016 radius=0.049964
