Commit message: add planning urdf publish in ocs2 arm controller

File: m6_ccs_description/urdf/m6_ccs_desktop.urdf (robot description, URDF)
Before this commit: robot M6_CCS, 22 links, 21 joints
Links:
- link arm_base: geometry collision box size=0.10045 0.100398 0.648662; visual mesh filename=package://m6_ccs_description/meshes/desktop_base.glb
- link left_link3: geometry collision cylinder length=0.089056 radius=0.046717; collision cylinder length=0.117016 radius=0.049964
- link right_link3: geometry collision cylinder length=0.089056 radius=0.046717; collision cylinder length=0.117016 radius=0.049964
Joints:
- joint left_joint5: limit lower=-3.1067 upper=3.1067 effort=18 velocity=3.141592653589793 -> lower=-2.9321531433504737 upper=2.9321531433504737 effort=18 velocity=3.141592653589793
- joint right_joint5: limit lower=-3.1067 upper=3.1067 effort=18 velocity=3.141592653589793 -> lower=-2.9321531433504737 upper=2.9321531433504737 effort=18 velocity=3.141592653589793

File: m6_ccs_description/urdf/m6_ccs_desktop_90c.urdf (robot description, URDF)
Before this commit: robot M6_CCS, 46 links, 45 joints
Links:
- link arm_base: geometry collision box size=0.10045 0.100398 0.648662; visual mesh filename=package://m6_ccs_description/meshes/desktop_base.glb
- link left_gripper_base: geometry visual mesh filename=package://changingtek_description/meshes/AG2F90-C/visual/gr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
- link left_left_1_link: geometry visual mesh filename=package://changingtek_description/meshes/AG2F90-C/visual/li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
- link left_left_2_link: geometry visual mesh filename=package://changingtek_description/meshes/AG2F90-C/visual/li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
- link left_left_Pad_link: geometry visual mesh filename=package://changingtek_description/meshes/AG2F90-C/visual/pa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
- link left_left_in_link: geometry visual mesh filename=package://changingtek_description/meshes/AG2F90-C/visual/in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
- link left_left_up_link: geometry visual mesh filename=package://changingtek_description/meshes/AG2F90-C/visual/up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
- link left_link7: geometry collision cylinder length=0.038392 radius=0.041707; collision cylinder length=0.08 radius=0.021707
- link left_right_1_link: geometry visual mesh filename=package://changingtek_description/meshes/AG2F90-C/visual/li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
- link left_right_2_link: geometry visual mesh filename=package://changingtek_description/meshes/AG2F90-C/visual/li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
- link left_right_Pad_link: geometry visual mesh filename=package://changingtek_description/meshes/AG2F90-C/visual/pa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
- link left_right_in_link: geometry visual mesh filename=package://changingtek_description/meshes/AG2F90-C/visual/in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
- link left_right_up_link: geometry visual mesh filename=package://changingtek_description/meshes/AG2F90-C/visual/up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
- link right_gripper_base: geometry visual mesh filename=package://changingtek_description/meshes/AG2F90-C/visual/gr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
- link right_left_1_link: geometry visual mesh filename=package://changingtek_description/meshes/AG2F90-C/visual/li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
- link right_left_2_link: geometry visual mesh filename=package://changingtek_description/meshes/AG2F90-C/visual/li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
- link right_left_Pad_link: geometry visual mesh filename=package://changingtek_description/meshes/AG2F90-C/visual/pa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
- link right_left_in_link: geometry visual mesh filename=package://changingtek_description/meshes/AG2F90-C/visual/in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
- link right_left_up_link: geometry visual mesh filename=package://changingtek_description/meshes/AG2F90-C/visual/up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
- link right_link7: geometry collision cylinder length=0.038392 radius=0.041707; collision cylinder length=0.08 radius=0.021707
- link right_right_1_link: geometry visual mesh filename=package://changingtek_description/meshes/AG2F90-C/visual/li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
- link right_right_2_link: geometry visual mesh filename=package://changingtek_description/meshes/AG2F90-C/visual/li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
- link right_right_Pad_link: geometry visual mesh filename=package://changingtek_description/meshes/AG2F90-C/visual/pa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
- link right_right_in_link: geometry visual mesh filename=package://changingtek_description/meshes/AG2F90-C/visual/in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
- link right_right_up_link: geometry visual mesh filename=package://changingtek_description/meshes/AG2F90-C/visual/up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
Joints:
- joint left_right_2_Joint: mimic joint=left_left_2_Joint -> joint=left_gripper_joint
- joint left_right_in_Joint: mimic joint=left_right_1_Joint multiplier=0.1 offset=0 -> joint=left_gripper_joint multiplier=0.1 offset=0
- joint left_right_up_Joint: mimic joint=left_right_1_Joint -> joint=left_gripper_joint
- joint right_right_2_Joint: mimic joint=right_left_2_Joint -> joint=right_gripper_joint
- joint right_right_in_Joint: mimic joint=right_right_1_Joint multiplier=0.1 offset=0 -> joint=right_gripper_joint multiplier=0.1 offset=0
- joint right_right_up_Joint: mimic joint=right_right_1_Joint -> joint=right_gripper_joint
