Commit message: 更新 m6_ccs_description: 修改控制器配置和 URDF 碰撞模型

File: m6_ccs_description/urdf/m6_ccs.urdf (robot description, URDF)
Before this commit: robot M6_CCS, 8 links, 7 joints
Links:
- added link eef
- link base_link: geometry collision cylinder length=0.083664 radius=0.051277; visual mesh filename=package://m6_ccs_description/meshes/base.obj
- link link1: geometry collision cylinder length=0.125958 radius=0.057588; visual mesh filename=package://m6_ccs_description/meshes/link1.obj
- link link2: geometry collision cylinder length=0.078386 radius=0.046717; visual mesh filename=package://m6_ccs_description/meshes/link2.obj
- link link3: geometry collision cylinder length=0.089056 radius=0.046717; collision cylinder length=0.117016 radius=0.049964
- link link4: geometry collision cylinder length=0.080203 radius=0.041759; visual mesh filename=package://m6_ccs_description/meshes/link4.obj
- link link5: geometry collision cylinder length=0.14268 radius=0.056747; visual mesh filename=package://m6_ccs_description/meshes/link5.obj scale=1 1 1
- link link6: geometry collision cylinder length=0.108046 radius=0.038348; visual mesh filename=package://m6_ccs_description/meshes/link6.obj
- link link7: geometry collision cylinder length=0.038392 radius=0.041707; visual mesh filename=package://m6_ccs_description/meshes/link7.obj
Joints:
- added joint eef_joint: type fixed, parent link7, child eef, origin xyz=0 -0.095296 0 rpy=0 0 0
- joint joint2: origin xyz=0 0 0 rpy=1.5708 0 0 -> rpy=1.5708 0 0
- joint joint6: origin xyz=0 0 0 rpy=1.5708 -1.5708 0 -> rpy=1.5708 -1.5708 0
- joint joint7: origin xyz=0 0 0 rpy=1.5708 -1.5708 0 -> rpy=1.5708 -1.5708 0

Commit message: update m6 ccs to used high precision pi

File: m6_ccs_description/urdf/m6_ccs.urdf (robot description, URDF)
Before this commit: robot DobotCR5, 9 links, 8 joints
Joints:
- joint joint1: limit lower=-3.1067 upper=3.1067 effort=108 velocity=3.1416 -> lower=-3.1067 upper=3.1067 effort=108 velocity=3.141592653589793
- joint joint2: limit lower=-2.0944 upper=2.0944 effort=108 velocity=3.1416 -> lower=-2.0944 upper=2.0944 effort=108 velocity=3.141592653589793; origin rpy=1.5708 0 0 -> rpy=1.5707963267948966 0 0
- joint joint3: limit lower=-3.1067 upper=3.1067 effort=66 velocity=3.1416 -> lower=-3.1067 upper=3.1067 effort=66 velocity=3.141592653589793; origin xyz=0 0.287 0 rpy=-1.5708 0 0 -> xyz=0 0.287 0 rpy=-1.5707963267948966 0 0
- joint joint4: limit lower=-2.5307 upper=1.0472 effort=66 velocity=3.1416 -> lower=-2.5307 upper=1.0472 effort=66 velocity=3.141592653589793; origin xyz=0.018 0 0 rpy=-1.5708 0 3.1416 -> xyz=0.018 0 0 rpy=-1.5707963267948966 0 3.141592653589793
- joint joint5: limit lower=-3.1067 upper=3.1067 effort=18 velocity=3.1416 -> lower=-3.1067 upper=3.1067 effort=18 velocity=3.141592653589793; origin xyz=0.018 -0.314 0 rpy=-1.5708 0 3.1416 -> xyz=0.018 -0.314 0 rpy=-1.5707963267948966 0 3.141592653589793
- joint joint6: limit lower=-1.0472 upper=1.0472 effort=18 velocity=3.1416 -> lower=-1.0472 upper=1.0472 effort=18 velocity=3.141592653589793; origin rpy=1.5708 -1.5708 0 -> rpy=1.5707963267948966 -1.5707963267948966 0
- joint joint7: limit lower=-1.5708 upper=1.5708 effort=18 velocity=3.1416 -> lower=-1.5707963267948966 upper=1.5707963267948966 effort=18 velocity=3.141592653589793; origin rpy=1.5708 -1.5708 0 -> rpy=1.5707963267948966 -1.5707963267948966 0

File: m6_ccs_description/urdf/m6_ccs_dual.urdf (robot description, URDF)
Before this commit: robot DobotCR5, 20 links, 19 joints
Links:
- link arm_base: geometry collision box size=0.2000 0.32 0.5029
- link left_base_link: geometry collision cylinder length=0.083664 radius=0.051277; visual mesh filename=package://m6_ccs_description/meshes/base.obj
- link left_link1: geometry collision cylinder length=0.125958 radius=0.057588; visual mesh filename=package://m6_ccs_description/meshes/link1.obj
- link left_link2: geometry collision cylinder length=0.078386 radius=0.046717; visual mesh filename=package://m6_ccs_description/meshes/link2.obj
- link left_link3: geometry collision cylinder length=0.089056 radius=0.046717; collision cylinder length=0.117016 radius=0.049964
- link left_link4: geometry collision cylinder length=0.080203 radius=0.041759; visual mesh filename=package://m6_ccs_description/meshes/link4.obj
- link left_link5: geometry collision cylinder length=0.14268 radius=0.056747; visual mesh filename=package://m6_ccs_description/meshes/link5.obj scale=1 1 1
- link left_link6: geometry collision cylinder length=0.108046 radius=0.038348; visual mesh filename=package://m6_ccs_description/meshes/link6.obj
- link left_link7: geometry collision cylinder length=0.038392 radius=0.041707; visual mesh filename=package://m6_ccs_description/meshes/link7.obj
- link right_base_link: geometry collision cylinder length=0.083664 radius=0.051277; visual mesh filename=package://m6_ccs_description/meshes/base.obj
- link right_link1: geometry collision cylinder length=0.125958 radius=0.057588; visual mesh filename=package://m6_ccs_description/meshes/link1.obj
- link right_link2: geometry collision cylinder length=0.078386 radius=0.046717; visual mesh filename=package://m6_ccs_description/meshes/link2.obj
- link right_link3: geometry collision cylinder length=0.089056 radius=0.046717; collision cylinder length=0.117016 radius=0.049964
- link right_link4: geometry collision cylinder length=0.080203 radius=0.041759; visual mesh filename=package://m6_ccs_description/meshes/link4.obj
- link right_link5: geometry collision cylinder length=0.14268 radius=0.056747; visual mesh filename=package://m6_ccs_description/meshes/link5.obj scale=1 -1 1
- link right_link6: geometry collision cylinder length=0.108046 radius=0.038348; visual mesh filename=package://m6_ccs_description/meshes/link6.obj
- link right_link7: geometry collision cylinder length=0.038392 radius=0.041707; visual mesh filename=package://m6_ccs_description/meshes/link7_r.obj
Joints:
- joint left_arm_base_joint: origin xyz=0.0 0.062 0 rpy=-1.5708 0 0 -> xyz=0.0 0.062 0 rpy=-1.5707963267948966 0 0
- joint left_joint1: limit lower=-3.1067 upper=3.1067 effort=108 velocity=3.1416 -> lower=-3.1067 upper=3.1067 effort=108 velocity=3.141592653589793
- joint left_joint2: limit lower=-2.0944 upper=2.0944 effort=108 velocity=3.1416 -> lower=-2.0944 upper=2.0944 effort=108 velocity=3.141592653589793; origin rpy=1.5708 0 0 -> rpy=1.5707963267948966 0 0
- joint left_joint3: limit lower=-3.1067 upper=3.1067 effort=66 velocity=3.1416 -> lower=-3.1067 upper=3.1067 effort=66 velocity=3.141592653589793; origin xyz=0 0.287 0 rpy=-1.5708 0 0 -> xyz=0 0.287 0 rpy=-1.5707963267948966 0 0
- joint left_joint4: limit lower=-2.5307 upper=1.0472 effort=66 velocity=3.1416 -> lower=-2.5307 upper=1.0472 effort=66 velocity=3.141592653589793; origin xyz=0.018 0 0 rpy=-1.5708 0 3.1416 -> xyz=0.018 0 0 rpy=-1.5707963267948966 0 3.141592653589793
- joint left_joint5: limit lower=-3.1067 upper=3.1067 effort=18 velocity=3.1416 -> lower=-3.1067 upper=3.1067 effort=18 velocity=3.141592653589793; origin xyz=0.018 -0.314 0 rpy=-1.5708 0 3.1416 -> xyz=0.018 -0.314 0 rpy=-1.5707963267948966 0 3.141592653589793
- joint left_joint6: limit lower=-1.0472 upper=1.0472 effort=18 velocity=3.1416 -> lower=-1.0472 upper=1.0472 effort=18 velocity=3.141592653589793; origin rpy=1.5708 -1.5708 0 -> rpy=1.5707963267948966 -1.5707963267948966 0
- joint left_joint7: limit lower=-1.5708 upper=1.5708 effort=18 velocity=3.1416 -> lower=-1.5707963267948966 upper=1.5707963267948966 effort=18 velocity=3.141592653589793; origin rpy=1.5708 -1.5708 0 -> rpy=1.5707963267948966 -1.5707963267948966 0
- joint right_arm_base_joint: origin xyz=0 -0.062 0 rpy=1.5708 0 0 -> xyz=0 -0.062 0 rpy=1.5707963267948966 0 0
- joint right_joint1: limit lower=-3.1067 upper=3.1067 effort=108 velocity=3.1416 -> lower=-3.1067 upper=3.1067 effort=108 velocity=3.141592653589793
- joint right_joint2: limit lower=-2.0944 upper=2.0944 effort=108 velocity=3.1416 -> lower=-2.0944 upper=2.0944 effort=108 velocity=3.141592653589793; origin rpy=1.5708 0 0 -> rpy=1.5707963267948966 0 0
- joint right_joint3: limit lower=-3.1067 upper=3.1067 effort=66 velocity=3.1416 -> lower=-3.1067 upper=3.1067 effort=66 velocity=3.141592653589793; origin xyz=0 0.287 0 rpy=-1.5708 0 0 -> xyz=0 0.287 0 rpy=-1.5707963267948966 0 0
- joint right_joint4: limit lower=-2.5307 upper=1.0472 effort=66 velocity=3.1416 -> lower=-2.5307 upper=1.0472 effort=66 velocity=3.141592653589793; origin xyz=0.018 0 0 rpy=-1.5708 0 3.1416 -> xyz=0.018 0 0 rpy=-1.5707963267948966 0 3.141592653589793
- joint right_joint5: limit lower=-3.1067 upper=3.1067 effort=18 velocity=3.1416 -> lower=-3.1067 upper=3.1067 effort=18 velocity=3.141592653589793; origin xyz=0.018 -0.314 0 rpy=-1.5708 0 3.1416 -> xyz=0.018 -0.314 0 rpy=-1.5707963267948966 0 3.141592653589793
- joint right_joint6: limit lower=-1.0472 upper=1.0472 effort=18 velocity=3.1416 -> lower=-1.0472 upper=1.0472 effort=18 velocity=3.141592653589793; origin rpy=1.5708 -1.5708 0 -> rpy=1.5707963267948966 -1.5707963267948966 0
- joint right_joint7: limit lower=-1.5708 upper=1.5708 effort=18 velocity=3.1416 -> lower=-1.5707963267948966 upper=1.5707963267948966 effort=18 velocity=3.141592653589793; origin rpy=1.5708 -1.5708 0 -> rpy=1.5707963267948966 -1.5707963267948966 0

File: m6_ccs_description/urdf/m6_ccs_dual_desktop.urdf (robot description, URDF)
Before this commit: robot DobotCR5, 19 links, 18 joints
Joints:
- joint left_arm_base_joint: origin xyz=0.0 0.12 0.701 rpy=-1.5708 0 0 -> xyz=0.0 0.12 0.701 rpy=-1.5707963267948966 0 0
- joint left_joint1: limit lower=-3.1067 upper=3.1067 effort=108 velocity=3.1416 -> lower=-3.1067 upper=3.1067 effort=108 velocity=3.141592653589793
- joint left_joint2: limit lower=-2.0944 upper=2.0944 effort=108 velocity=3.1416 -> lower=-2.0944 upper=2.0944 effort=108 velocity=3.141592653589793; origin rpy=1.5708 0 0 -> rpy=1.5707963267948966 0 0
- joint left_joint3: limit lower=-3.1067 upper=3.1067 effort=66 velocity=3.1416 -> lower=-3.1067 upper=3.1067 effort=66 velocity=3.141592653589793; origin xyz=0 0.287 0 rpy=-1.5708 0 0 -> xyz=0 0.287 0 rpy=-1.5707963267948966 0 0
- joint left_joint4: limit lower=-2.5307 upper=1.0472 effort=66 velocity=3.1416 -> lower=-2.5307 upper=1.0472 effort=66 velocity=3.141592653589793; origin xyz=0.018 0 0 rpy=-1.5708 0 3.1416 -> xyz=0.018 0 0 rpy=-1.5707963267948966 0 3.141592653589793
- joint left_joint5: limit lower=-3.1067 upper=3.1067 effort=18 velocity=3.1416 -> lower=-3.1067 upper=3.1067 effort=18 velocity=3.141592653589793; origin xyz=0.018 -0.314 0 rpy=-1.5708 0 3.1416 -> xyz=0.018 -0.314 0 rpy=-1.5707963267948966 0 3.141592653589793
- joint left_joint6: limit lower=-1.0472 upper=1.0472 effort=18 velocity=3.1416 -> lower=-1.0472 upper=1.0472 effort=18 velocity=3.141592653589793; origin rpy=1.5708 -1.5708 0 -> rpy=1.5707963267948966 -1.5707963267948966 0
- joint left_joint7: limit lower=-1.5708 upper=1.5708 effort=18 velocity=3.1416 -> lower=-1.5707963267948966 upper=1.5707963267948966 effort=18 velocity=3.141592653589793; origin rpy=1.5708 -1.5708 0 -> rpy=1.5707963267948966 -1.5707963267948966 0
- joint right_arm_base_joint: origin xyz=0.0 -0.12 0.701 rpy=1.5708 0 0 -> xyz=0.0 -0.12 0.701 rpy=1.5707963267948966 0 0
- joint right_joint1: limit lower=-3.1067 upper=3.1067 effort=108 velocity=3.1416 -> lower=-3.1067 upper=3.1067 effort=108 velocity=3.141592653589793
- joint right_joint2: limit lower=-2.0944 upper=2.0944 effort=108 velocity=3.1416 -> lower=-2.0944 upper=2.0944 effort=108 velocity=3.141592653589793; origin rpy=1.5708 0 0 -> rpy=1.5707963267948966 0 0
- joint right_joint3: limit lower=-3.1067 upper=3.1067 effort=66 velocity=3.1416 -> lower=-3.1067 upper=3.1067 effort=66 velocity=3.141592653589793; origin xyz=0 0.287 0 rpy=-1.5708 0 0 -> xyz=0 0.287 0 rpy=-1.5707963267948966 0 0
- joint right_joint4: limit lower=-2.5307 upper=1.0472 effort=66 velocity=3.1416 -> lower=-2.5307 upper=1.0472 effort=66 velocity=3.141592653589793; origin xyz=0.018 0 0 rpy=-1.5708 0 3.1416 -> xyz=0.018 0 0 rpy=-1.5707963267948966 0 3.141592653589793
- joint right_joint5: limit lower=-3.1067 upper=3.1067 effort=18 velocity=3.1416 -> lower=-3.1067 upper=3.1067 effort=18 velocity=3.141592653589793; origin xyz=0.018 -0.314 0 rpy=-1.5708 0 3.1416 -> xyz=0.018 -0.314 0 rpy=-1.5707963267948966 0 3.141592653589793
- joint right_joint6: limit lower=-1.0472 upper=1.0472 effort=18 velocity=3.1416 -> lower=-1.0472 upper=1.0472 effort=18 velocity=3.141592653589793; origin rpy=1.5708 -1.5708 0 -> rpy=1.5707963267948966 -1.5707963267948966 0
- joint right_joint7: limit lower=-1.5708 upper=1.5708 effort=18 velocity=3.1416 -> lower=-1.5707963267948966 upper=1.5707963267948966 effort=18 velocity=3.141592653589793; origin rpy=1.5708 -1.5708 0 -> rpy=1.5707963267948966 -1.5707963267948966 0

File: m6_ccs_description/urdf/m6_ccs_usb-90c.urdf (robot description, URDF)
Before this commit: robot DobotCR5, 23 links, 22 joints
Links:
- added link left_eef
- link base: geometry collision box size=0.10045 0.100398 0.648662; visual mesh filename=package://m6_ccs_description/meshes/dual_base.obj
- link left_base_link: geometry collision cylinder length=0.083664 radius=0.051277; visual mesh filename=package://m6_ccs_description/meshes/base.obj
- link left_link1: geometry collision cylinder length=0.125958 radius=0.057588; visual mesh filename=package://m6_ccs_description/meshes/link1.obj
- link left_link2: geometry collision cylinder length=0.078386 radius=0.046717; visual mesh filename=package://m6_ccs_description/meshes/link2.obj
- link left_link3: geometry collision cylinder length=0.089056 radius=0.046717; collision cylinder length=0.117016 radius=0.049964
- link left_link4: geometry collision cylinder length=0.080203 radius=0.041759; visual mesh filename=package://m6_ccs_description/meshes/link4.obj
- link left_link5: geometry collision cylinder length=0.14268 radius=0.056747; visual mesh filename=package://m6_ccs_description/meshes/link5.obj scale=1 1 1
- link left_link6: geometry collision cylinder length=0.108046 radius=0.038348; visual mesh filename=package://m6_ccs_description/meshes/link6.obj
- link left_link7: geometry collision cylinder length=0.038392 radius=0.041707; visual mesh filename=package://m6_ccs_description/meshes/link7.obj
Joints:
- added joint left_eef_joint: type fixed, parent left_link7, child left_eef, origin xyz=0 -0.095296 0 rpy=0 0 0
- joint left_joint1: limit lower=-3.1067 upper=3.1067 effort=108 velocity=3.1416 -> lower=-3.1067 upper=3.1067 effort=108 velocity=3.141592653589793
- joint left_joint2: limit lower=-2.0944 upper=2.0944 effort=108 velocity=3.1416 -> lower=-2.0944 upper=2.0944 effort=108 velocity=3.141592653589793; origin rpy=1.5708 0 0 -> rpy=1.5707963267948966 0 0
- joint left_joint3: limit lower=-3.1067 upper=3.1067 effort=66 velocity=3.1416 -> lower=-3.1067 upper=3.1067 effort=66 velocity=3.141592653589793; origin xyz=0 0.287 0 rpy=-1.5708 0 0 -> xyz=0 0.287 0 rpy=-1.5707963267948966 0 0
- joint left_joint4: limit lower=-2.5307 upper=1.0472 effort=66 velocity=3.1416 -> lower=-2.5307 upper=1.0472 effort=66 velocity=3.141592653589793; origin xyz=0.018 0 0 rpy=-1.5708 0 3.1416 -> xyz=0.018 0 0 rpy=-1.5707963267948966 0 3.141592653589793
- joint left_joint5: limit lower=-3.1067 upper=3.1067 effort=18 velocity=3.1416 -> lower=-3.1067 upper=3.1067 effort=18 velocity=3.141592653589793; origin xyz=0.018 -0.314 0 rpy=-1.5708 0 3.1416 -> xyz=0.018 -0.314 0 rpy=-1.5707963267948966 0 3.141592653589793
- joint left_joint6: limit lower=-1.0472 upper=1.0472 effort=18 velocity=3.1416 -> lower=-1.0472 upper=1.0472 effort=18 velocity=3.141592653589793; origin rpy=1.5708 -1.5708 0 -> rpy=1.5707963267948966 -1.5707963267948966 0
- joint left_joint7: limit lower=-1.5708 upper=1.5708 effort=18 velocity=3.1416 -> lower=-1.5707963267948966 upper=1.5707963267948966 effort=18 velocity=3.141592653589793; origin rpy=1.5708 -1.5708 0 -> rpy=1.5707963267948966 -1.5707963267948966 0

Commit message: dual arm config with gripper

File: m6_ccs_description/urdf/m6_ccs.urdf (robot description, URDF)
Before this commit: robot DobotCR5, 9 links, 8 joints
Links:
- removed link eef
- added link tcp
Joints:
- removed joint eef_joint
- added joint tcp_joint: type fixed, parent link7, child tcp, origin xyz=0 -0.095296 0 rpy=0 0 0

File: m6_ccs_description/urdf/m6_ccs_dual.urdf (robot description, URDF)
Before this commit: robot DobotCR5, 20 links, 19 joints
Links:
- added link left_tcp
- added link right_tcp
Joints:
- added joint left_tcp_joint: type fixed, parent left_link7, child left_tcp, origin xyz=0 -0.095296 0 rpy=0 0 0
- added joint right_tcp_joint: type fixed, parent right_link7, child right_tcp, origin xyz=0 -0.095296 0 rpy=0 0 0
- joint left_eef_joint: origin xyz=0 -0.095296 0 rpy=0 0 0 -> (none); parent left_link7 -> left_tcp
- joint right_eef_joint: origin xyz=0 -0.095296 0 rpy=0 0 0 -> (none); parent right_link7 -> right_tcp

File: m6_ccs_description/urdf/m6_ccs_dual_desktop.urdf (robot description, URDF)
Before this commit: robot DobotCR5, 19 links, 18 joints
Links:
- added link left_tcp
- added link right_tcp
Joints:
- added joint left_tcp_joint: type fixed, parent left_link7, child left_tcp, origin xyz=0 -0.095296 0 rpy=0 0 0
- added joint right_tcp_joint: type fixed, parent right_link7, child right_tcp, origin xyz=0 -0.095296 0 rpy=0 0 0
- joint left_eef_joint: origin xyz=0 -0.095296 0 rpy=0 0 0 -> (none); parent left_link7 -> left_tcp
- joint right_eef_joint: origin xyz=0 -0.095296 0 rpy=0 0 0 -> (none); parent right_link7 -> right_tcp

File: m6_ccs_description/urdf/m6_ccs_usb-90c.urdf (robot description, URDF)
Before this commit: robot DobotCR5, 24 links, 23 joints
Links:
- removed link left_eef
- added link left_tcp
Joints:
- removed joint left_eef_joint
- added joint left_tcp_joint: type fixed, parent left_link7, child left_tcp, origin xyz=0 -0.095296 0 rpy=0 0 0

File: m6_ccs_description/xacro/arm.xacro (robot description, xacro)
@@ -311,9 +311,9 @@
 			<limit lower="-${PI/2}" upper="${PI/2}" effort="18" velocity="${PI}"/>
 		</joint>
-		<link name="${prefix}eef"/>
-		<joint name="${prefix}eef_joint" type="fixed">
+		<link name="${prefix}tcp"/>
+		<joint name="${prefix}tcp_joint" type="fixed">
 			<origin rpy="0 0 0" xyz="0 -0.095296 0"/>
 			<parent link="${prefix}link7"/>
-			<child link="${prefix}eef"/>
+			<child link="${prefix}tcp"/>
 		</joint>
 	</xacro:macro>

File: m6_ccs_description/xacro/robot.xacro (robot description, xacro)
@@ -10,5 +10,5 @@
 		<xacro:M6_CCS direction="-1" collider="$(arg collider)"/>
 	</xacro:if>
-	<xacro:if value="${'$(arg type)' == 'dual'}">
+	<xacro:if value="${'$(arg type)' == 'dual' or '$(arg type)' == 'dual_ag2f90' or '$(arg type)' == 'dual_rg75'}">
 		<link name="base_link"/>
 		<link name="arm_base">
@@ -38,4 +38,19 @@
 		<xacro:M6_CCS name="left" collider="$(arg collider)"/>
 		<xacro:M6_CCS name="right" direction="-1" collider="$(arg collider)"/>
+		<xacro:if value="${'$(arg type)' == 'dual_ag2f90'}">
+			<xacro:include filename="$(find changingtek_description)/xacro/AG2F90-C.xacro"/>
+			<xacro:AG2F90-C name="left" use_flange="true"/>
+			<joint name="left_gripper_fix" type="fixed">
+				<parent link="left_link7"/>
+				<child link="left_flange"/>
+				<origin xyz="0 -0.0995 0" rpy=" ${PI/2} 0 0"/>
+			</joint>
+			<xacro:AG2F90-C name="right" use_flange="true"/>
+			<joint name="right_gripper_fix" type="fixed">
+				<parent link="right_link7"/>
+				<child link="right_flange"/>
+				<origin xyz="0 -0.0995 0" rpy=" ${PI/2} 0 0"/>
+			</joint>
+		</xacro:if>
 	</xacro:if>
 	<xacro:if value="${'$(arg type)' == 'dual_desktop'}">

File: m6_ccs_description/xacro/ros2_control/robot.xacro (robot description, xacro)
@@ -28,5 +28,5 @@
 			<xacro:if value="${'$(arg ros2_control_hardware_type)' == 'real'}">
 				<plugin>marvin_ros2_control/MarvinHardware</plugin>
-				<xacro:if value="${'$(arg type)' == 'dual'}">
+				<xacro:if value="${'$(arg type)' == 'dual' or '$(arg type)' == 'dual_ag2f90'}">
 					<param name="left_right_arm">2</param>
 				</xacro:if>
@@ -43,21 +43,26 @@
 				</xacro:unless>
 			</xacro:if>
-       <xacro:if value="${'$(arg ctrl_mode)' == 'position'}">
-          <param name="ctrl_mode">2</param>
-        </xacro:if>
-        <xacro:unless value="${'$(arg ctrl_mode)' == 'position'}">
-          <xacro:if value="${'$(arg ctrl_mode)' == 'joint_imp'}">
-            <param name="ctrl_mode">3</param>
-          </xacro:if>
-          <xacro:unless value="${'$(arg ctrl_mode)' == 'joint_imp'}">
-            <param name="ctrl_mode">4</param>
-          </xacro:unless>
-        </xacro:unless>
+			<xacro:if value="${'$(arg ctrl_mode)' == 'position'}">
+				<param name="ctrl_mode">2</param>
+			</xacro:if>
+			<xacro:unless value="${'$(arg ctrl_mode)' == 'position'}">
+				<xacro:if value="${'$(arg ctrl_mode)' == 'joint_imp'}">
+					<param name="ctrl_mode">3</param>
+				</xacro:if>
+				<xacro:unless value="${'$(arg ctrl_mode)' == 'joint_imp'}">
+					<param name="ctrl_mode">4</param>
+				</xacro:unless>
+			</xacro:unless>
 		</hardware>
-		<xacro:if value="${'$(arg type)' == 'dual'}">
+		<xacro:if value="${'$(arg type)' == 'dual' or '$(arg type)' == 'dual_ag2f90'}">
 			<xacro:m6_interfaces name="left"/>
 			<xacro:m6_interfaces name="right"/>
+			<xacro:if value="${'$(arg type)' == 'dual_ag2f90'}">
+				<xacro:include filename="$(find changingtek_description)/xacro/ros2_control/AG2F90-C.xacro"/>
+				<xacro:ag2f90c_interfaces name="left"/>
+				<xacro:ag2f90c_interfaces name="right"/>
+			</xacro:if>
 		</xacro:if>
-		<xacro:unless value="${'$(arg type)' == 'dual'}">
+		<xacro:unless value="${'$(arg type)' == 'dual' or '$(arg type)' == 'dual_ag2f90'}">
 			<xacro:if value="${'$(arg type)' == 'usb-90c'}">
 				<xacro:m6_interfaces name="left"/>
