Commit message: fix m6 ccs urdf param

File: m6_ccs_description/urdf/m6_ccs.urdf (robot description, URDF)
Before this commit: robot DobotCR5, 9 links, 8 joints
Joints:
- joint tcp_joint: origin xyz=0 -0.095296 0 rpy=0 0 0 -> xyz=0 -0.095 0 rpy=1.5707963267948966 -1.5707963267948966 0

File: m6_ccs_description/urdf/m6_ccs_dual.urdf (robot description, URDF)
Before this commit: robot DobotCR5, 22 links, 21 joints
Joints:
- joint left_tcp_joint: origin xyz=0 -0.095296 0 rpy=0 0 0 -> xyz=0 -0.095 0 rpy=1.5707963267948966 -1.5707963267948966 0
- joint right_tcp_joint: origin xyz=0 -0.095296 0 rpy=0 0 0 -> xyz=0 -0.095 0 rpy=1.5707963267948966 -1.5707963267948966 0

File: m6_ccs_description/urdf/m6_ccs_dual_ag2f90.urdf (robot description, URDF)
Before this commit: robot DobotCR5, 46 links, 45 joints
Joints:
- joint left_gripper_fix: origin xyz=0 -0.0995 0 rpy= 1.5707963267948966 0 0 -> xyz=0 0 0.0045; parent left_link7 -> left_tcp
- joint left_tcp_joint: origin xyz=0 -0.095296 0 rpy=0 0 0 -> xyz=0 -0.095 0 rpy=1.5707963267948966 -1.5707963267948966 0
- joint right_gripper_fix: origin xyz=0 -0.0995 0 rpy= 1.5707963267948966 0 0 -> xyz=0 0 0.0045; parent right_link7 -> right_tcp
- joint right_tcp_joint: origin xyz=0 -0.095296 0 rpy=0 0 0 -> xyz=0 -0.095 0 rpy=1.5707963267948966 -1.5707963267948966 0

File: m6_ccs_description/urdf/m6_ccs_dual_desktop.urdf (robot description, URDF)
Before this commit: robot DobotCR5, 21 links, 20 joints
Joints:
- joint left_tcp_joint: origin xyz=0 -0.095296 0 rpy=0 0 0 -> xyz=0 -0.095 0 rpy=1.5707963267948966 1.5707963267948966 0
- joint right_tcp_joint: origin xyz=0 -0.095296 0 rpy=0 0 0 -> xyz=0 -0.095 0 rpy=1.5707963267948966 1.5707963267948966 0

File: m6_ccs_description/urdf/m6_ccs_dual_rg75.urdf (robot description, URDF)
Before this commit: robot DobotCR5, 34 links, 33 joints
Joints:
- joint left_gripper_base_joint: origin rpy=-1.5707963267948966 0 3.141592653589793 -> (none)
- joint left_tcp_joint: origin xyz=0 -0.095296 0 rpy=0 0 0 -> xyz=0 -0.095 0 rpy=1.5707963267948966 -1.5707963267948966 0
- joint right_gripper_base_joint: origin rpy=1.5707963267948966 0 0 -> (none)
- joint right_tcp_joint: origin xyz=0 -0.095296 0 rpy=0 0 0 -> xyz=0 -0.095 0 rpy=1.5707963267948966 -1.5707963267948966 0

File: m6_ccs_description/urdf/m6_ccs_usb-90c.urdf (robot description, URDF)
Before this commit: robot DobotCR5, 24 links, 23 joints
Joints:
- joint gripper_fix: origin xyz=0 -0.0995 0 rpy= 1.5707963267948966 0 0 -> xyz=0 -0.0995 0 rpy=1.5707963267948966 0 0
- joint left_tcp_joint: origin xyz=0 -0.095296 0 rpy=0 0 0 -> xyz=0 -0.095 0 rpy=1.5707963267948966 -1.5707963267948966 0

File: m6_ccs_description/xacro/arm.xacro (robot description, xacro)
@@ -313,5 +313,5 @@
 		<link name="${prefix}tcp"/>
 		<joint name="${prefix}tcp_joint" type="fixed">
-			<origin rpy="0 0 0" xyz="0 -0.095296 0"/>
+			<origin rpy="${PI/2} -${PI/2} 0" xyz="0 -0.095 0"/>
 			<parent link="${prefix}link7"/>
 			<child link="${prefix}tcp"/>

File: m6_ccs_description/xacro/robot.xacro (robot description, xacro)
@@ -42,13 +42,13 @@
 			<xacro:AG2F90-C name="left" use_flange="true"/>
 			<joint name="left_gripper_fix" type="fixed">
-				<parent link="left_link7"/>
+				<parent link="left_tcp"/>
 				<child link="left_flange"/>
-				<origin xyz="0 -0.0995 0" rpy=" ${PI/2} 0 0"/>
+				<origin xyz="0 0 0.0045"/>
 			</joint>
 			<xacro:AG2F90-C name="right" use_flange="true"/>
 			<joint name="right_gripper_fix" type="fixed">
-				<parent link="right_link7"/>
+				<parent link="right_tcp"/>
 				<child link="right_flange"/>
-				<origin xyz="0 -0.0995 0" rpy=" ${PI/2} 0 0"/>
+				<origin xyz="0 0 0.0045"/>
 			</joint>
 		</xacro:if>
@@ -58,10 +58,8 @@
 			<xacro:RG75-300 name="right" use_flange="true"/>
 			<joint name="left_gripper_base_joint" type="fixed">
-				<origin rpy="${-PI/2} 0 ${PI}"/>
 				<parent link="left_tcp"/>
 				<child link="left_flange"/>
 			</joint>
 			<joint name="right_gripper_base_joint" type="fixed">
-				<origin rpy="${PI/2} 0 0"/>
 				<parent link="right_tcp"/>
 				<child link="right_flange"/>

Commit message: update joint limit

File: m6_ccs_description/urdf/m6_ccs.urdf (robot description, URDF)
Before this commit: robot M6_CCS, 9 links, 8 joints
Joints:
- joint joint1: limit lower=-3.1067 upper=3.1067 effort=108 velocity=3.141592653589793 -> lower=-3.106686068549907 upper=3.106686068549907 effort=108 velocity=3.141592653589793
- joint joint2: limit lower=-2.0944 upper=2.0944 effort=108 velocity=3.141592653589793 -> lower=-2.0594885173533086 upper=2.0594885173533086 effort=108 velocity=3.141592653589793
- joint joint3: limit lower=-3.1067 upper=3.1067 effort=66 velocity=3.141592653589793 -> lower=-2.9321531433504737 upper=2.9321531433504737 effort=66 velocity=3.141592653589793
- joint joint4: limit lower=-2.5307 upper=1.0472 effort=66 velocity=3.141592653589793 -> lower=-2.4958208303518914 upper=1.0122909661567112 effort=66 velocity=3.141592653589793
- joint joint5: limit lower=-3.1067 upper=3.1067 effort=18 velocity=3.141592653589793 -> lower=-2.9321531433504737 upper=2.9321531433504737 effort=18 velocity=3.141592653589793
- joint joint6: limit lower=-1.0472 upper=1.0472 effort=18 velocity=3.141592653589793 -> lower=-1.0122909661567112 upper=1.0122909661567112 effort=18 velocity=3.141592653589793
- joint joint7: limit lower=-1.5707963267948966 upper=1.5707963267948966 effort=18 velocity=3.141592653589793 -> lower=-1.361356816555577 upper=1.361356816555577 effort=18 velocity=3.141592653589793

File: m6_ccs_description/urdf/m6_ccs_dual.urdf (robot description, URDF)
Before this commit: robot M6_CCS, 22 links, 21 joints
Joints:
- joint left_joint1: limit lower=-3.1067 upper=3.1067 effort=108 velocity=3.141592653589793 -> lower=-3.106686068549907 upper=3.106686068549907 effort=108 velocity=3.141592653589793
- joint left_joint2: limit lower=-2.0944 upper=2.0944 effort=108 velocity=3.141592653589793 -> lower=-2.0594885173533086 upper=2.0594885173533086 effort=108 velocity=3.141592653589793
- joint left_joint3: limit lower=-3.1067 upper=3.1067 effort=66 velocity=3.141592653589793 -> lower=-2.9321531433504737 upper=2.9321531433504737 effort=66 velocity=3.141592653589793
- joint left_joint4: limit lower=-2.5307 upper=1.0472 effort=66 velocity=3.141592653589793 -> lower=-2.4958208303518914 upper=1.0122909661567112 effort=66 velocity=3.141592653589793
- joint left_joint6: limit lower=-1.0472 upper=1.0472 effort=18 velocity=3.141592653589793 -> lower=-1.0122909661567112 upper=1.0122909661567112 effort=18 velocity=3.141592653589793
- joint left_joint7: limit lower=-1.5707963267948966 upper=1.5707963267948966 effort=18 velocity=3.141592653589793 -> lower=-1.361356816555577 upper=1.361356816555577 effort=18 velocity=3.141592653589793
- joint right_joint1: limit lower=-3.1067 upper=3.1067 effort=108 velocity=3.141592653589793 -> lower=-3.106686068549907 upper=3.106686068549907 effort=108 velocity=3.141592653589793
- joint right_joint2: limit lower=-2.0944 upper=2.0944 effort=108 velocity=3.141592653589793 -> lower=-2.0594885173533086 upper=2.0594885173533086 effort=108 velocity=3.141592653589793
- joint right_joint3: limit lower=-3.1067 upper=3.1067 effort=66 velocity=3.141592653589793 -> lower=-2.9321531433504737 upper=2.9321531433504737 effort=66 velocity=3.141592653589793
- joint right_joint4: limit lower=-2.5307 upper=1.0472 effort=66 velocity=3.141592653589793 -> lower=-2.4958208303518914 upper=1.0122909661567112 effort=66 velocity=3.141592653589793
- joint right_joint6: limit lower=-1.0472 upper=1.0472 effort=18 velocity=3.141592653589793 -> lower=-1.0122909661567112 upper=1.0122909661567112 effort=18 velocity=3.141592653589793
- joint right_joint7: limit lower=-1.5707963267948966 upper=1.5707963267948966 effort=18 velocity=3.141592653589793 -> lower=-1.361356816555577 upper=1.361356816555577 effort=18 velocity=3.141592653589793

File: m6_ccs_description/urdf/m6_ccs_dual_ag2f90_c.urdf (robot description, URDF)
Before this commit: robot M6_CCS, 46 links, 45 joints
Joints:
- joint left_joint1: limit lower=-3.1067 upper=3.1067 effort=108 velocity=3.141592653589793 -> lower=-3.106686068549907 upper=3.106686068549907 effort=108 velocity=3.141592653589793
- joint left_joint2: limit lower=-2.0944 upper=2.0944 effort=108 velocity=3.141592653589793 -> lower=-2.0594885173533086 upper=2.0594885173533086 effort=108 velocity=3.141592653589793
- joint left_joint3: limit lower=-3.1067 upper=3.1067 effort=66 velocity=3.141592653589793 -> lower=-2.9321531433504737 upper=2.9321531433504737 effort=66 velocity=3.141592653589793
- joint left_joint4: limit lower=-2.5307 upper=1.0472 effort=66 velocity=3.141592653589793 -> lower=-2.4958208303518914 upper=1.0122909661567112 effort=66 velocity=3.141592653589793
- joint left_joint6: limit lower=-1.0472 upper=1.0472 effort=18 velocity=3.141592653589793 -> lower=-1.0122909661567112 upper=1.0122909661567112 effort=18 velocity=3.141592653589793
- joint left_joint7: limit lower=-1.5707963267948966 upper=1.5707963267948966 effort=18 velocity=3.141592653589793 -> lower=-1.361356816555577 upper=1.361356816555577 effort=18 velocity=3.141592653589793
- joint right_joint1: limit lower=-3.1067 upper=3.1067 effort=108 velocity=3.141592653589793 -> lower=-3.106686068549907 upper=3.106686068549907 effort=108 velocity=3.141592653589793
- joint right_joint2: limit lower=-2.0944 upper=2.0944 effort=108 velocity=3.141592653589793 -> lower=-2.0594885173533086 upper=2.0594885173533086 effort=108 velocity=3.141592653589793
- joint right_joint3: limit lower=-3.1067 upper=3.1067 effort=66 velocity=3.141592653589793 -> lower=-2.9321531433504737 upper=2.9321531433504737 effort=66 velocity=3.141592653589793
- joint right_joint4: limit lower=-2.5307 upper=1.0472 effort=66 velocity=3.141592653589793 -> lower=-2.4958208303518914 upper=1.0122909661567112 effort=66 velocity=3.141592653589793
- joint right_joint6: limit lower=-1.0472 upper=1.0472 effort=18 velocity=3.141592653589793 -> lower=-1.0122909661567112 upper=1.0122909661567112 effort=18 velocity=3.141592653589793
- joint right_joint7: limit lower=-1.5707963267948966 upper=1.5707963267948966 effort=18 velocity=3.141592653589793 -> lower=-1.361356816555577 upper=1.361356816555577 effort=18 velocity=3.141592653589793

File: m6_ccs_description/urdf/m6_ccs_dual_desktop.urdf (robot description, URDF)
Before this commit: robot M6_CCS, 22 links, 21 joints
Joints:
- joint left_joint1: limit lower=-3.1067 upper=3.1067 effort=108 velocity=3.141592653589793 -> lower=-3.106686068549907 upper=3.106686068549907 effort=108 velocity=3.141592653589793
- joint left_joint2: limit lower=-2.0944 upper=2.0944 effort=108 velocity=3.141592653589793 -> lower=-2.0594885173533086 upper=2.0594885173533086 effort=108 velocity=3.141592653589793
- joint left_joint3: limit lower=-3.1067 upper=3.1067 effort=66 velocity=3.141592653589793 -> lower=-2.9321531433504737 upper=2.9321531433504737 effort=66 velocity=3.141592653589793
- joint left_joint4: limit lower=-2.5307 upper=1.0472 effort=66 velocity=3.141592653589793 -> lower=-2.4958208303518914 upper=1.0122909661567112 effort=66 velocity=3.141592653589793
- joint left_joint6: limit lower=-1.0472 upper=1.0472 effort=18 velocity=3.141592653589793 -> lower=-1.0122909661567112 upper=1.0122909661567112 effort=18 velocity=3.141592653589793
- joint left_joint7: limit lower=-1.5707963267948966 upper=1.5707963267948966 effort=18 velocity=3.141592653589793 -> lower=-1.361356816555577 upper=1.361356816555577 effort=18 velocity=3.141592653589793
- joint right_joint1: limit lower=-3.1067 upper=3.1067 effort=108 velocity=3.141592653589793 -> lower=-3.106686068549907 upper=3.106686068549907 effort=108 velocity=3.141592653589793
- joint right_joint2: limit lower=-2.0944 upper=2.0944 effort=108 velocity=3.141592653589793 -> lower=-2.0594885173533086 upper=2.0594885173533086 effort=108 velocity=3.141592653589793
- joint right_joint3: limit lower=-3.1067 upper=3.1067 effort=66 velocity=3.141592653589793 -> lower=-2.9321531433504737 upper=2.9321531433504737 effort=66 velocity=3.141592653589793
- joint right_joint4: limit lower=-2.5307 upper=1.0472 effort=66 velocity=3.141592653589793 -> lower=-2.4958208303518914 upper=1.0122909661567112 effort=66 velocity=3.141592653589793
- joint right_joint6: limit lower=-1.0472 upper=1.0472 effort=18 velocity=3.141592653589793 -> lower=-1.0122909661567112 upper=1.0122909661567112 effort=18 velocity=3.141592653589793
- joint right_joint7: limit lower=-1.5707963267948966 upper=1.5707963267948966 effort=18 velocity=3.141592653589793 -> lower=-1.361356816555577 upper=1.361356816555577 effort=18 velocity=3.141592653589793

File: m6_ccs_description/urdf/m6_ccs_dual_desktop_90c.urdf (robot description, URDF)
Before this commit: robot M6_CCS, 46 links, 45 joints
Joints:
- joint left_joint1: limit lower=-3.1067 upper=3.1067 effort=108 velocity=3.141592653589793 -> lower=-3.106686068549907 upper=3.106686068549907 effort=108 velocity=3.141592653589793
- joint left_joint2: limit lower=-2.0944 upper=2.0944 effort=108 velocity=3.141592653589793 -> lower=-2.0594885173533086 upper=2.0594885173533086 effort=108 velocity=3.141592653589793
- joint left_joint3: limit lower=-3.1067 upper=3.1067 effort=66 velocity=3.141592653589793 -> lower=-2.9321531433504737 upper=2.9321531433504737 effort=66 velocity=3.141592653589793
- joint left_joint4: limit lower=-2.5307 upper=1.0472 effort=66 velocity=3.141592653589793 -> lower=-2.4958208303518914 upper=1.0122909661567112 effort=66 velocity=3.141592653589793
- joint left_joint6: limit lower=-1.0472 upper=1.0472 effort=18 velocity=3.141592653589793 -> lower=-1.0122909661567112 upper=1.0122909661567112 effort=18 velocity=3.141592653589793
- joint left_joint7: limit lower=-1.5707963267948966 upper=1.5707963267948966 effort=18 velocity=3.141592653589793 -> lower=-1.361356816555577 upper=1.361356816555577 effort=18 velocity=3.141592653589793
- joint right_joint1: limit lower=-3.1067 upper=3.1067 effort=108 velocity=3.141592653589793 -> lower=-3.106686068549907 upper=3.106686068549907 effort=108 velocity=3.141592653589793
- joint right_joint2: limit lower=-2.0944 upper=2.0944 effort=108 velocity=3.141592653589793 -> lower=-2.0594885173533086 upper=2.0594885173533086 effort=108 velocity=3.141592653589793
- joint right_joint3: limit lower=-3.1067 upper=3.1067 effort=66 velocity=3.141592653589793 -> lower=-2.9321531433504737 upper=2.9321531433504737 effort=66 velocity=3.141592653589793
- joint right_joint4: limit lower=-2.5307 upper=1.0472 effort=66 velocity=3.141592653589793 -> lower=-2.4958208303518914 upper=1.0122909661567112 effort=66 velocity=3.141592653589793
- joint right_joint6: limit lower=-1.0472 upper=1.0472 effort=18 velocity=3.141592653589793 -> lower=-1.0122909661567112 upper=1.0122909661567112 effort=18 velocity=3.141592653589793
- joint right_joint7: limit lower=-1.5707963267948966 upper=1.5707963267948966 effort=18 velocity=3.141592653589793 -> lower=-1.361356816555577 upper=1.361356816555577 effort=18 velocity=3.141592653589793

File: m6_ccs_description/urdf/m6_ccs_dual_rg75.urdf (robot description, URDF)
Before this commit: robot M6_CCS, 34 links, 33 joints
Joints:
- joint left_joint1: limit lower=-3.1067 upper=3.1067 effort=108 velocity=3.141592653589793 -> lower=-3.106686068549907 upper=3.106686068549907 effort=108 velocity=3.141592653589793
- joint left_joint2: limit lower=-2.0944 upper=2.0944 effort=108 velocity=3.141592653589793 -> lower=-2.0594885173533086 upper=2.0594885173533086 effort=108 velocity=3.141592653589793
- joint left_joint3: limit lower=-3.1067 upper=3.1067 effort=66 velocity=3.141592653589793 -> lower=-2.9321531433504737 upper=2.9321531433504737 effort=66 velocity=3.141592653589793
- joint left_joint4: limit lower=-2.5307 upper=1.0472 effort=66 velocity=3.141592653589793 -> lower=-2.4958208303518914 upper=1.0122909661567112 effort=66 velocity=3.141592653589793
- joint left_joint6: limit lower=-1.0472 upper=1.0472 effort=18 velocity=3.141592653589793 -> lower=-1.0122909661567112 upper=1.0122909661567112 effort=18 velocity=3.141592653589793
- joint left_joint7: limit lower=-1.5707963267948966 upper=1.5707963267948966 effort=18 velocity=3.141592653589793 -> lower=-1.361356816555577 upper=1.361356816555577 effort=18 velocity=3.141592653589793
- joint right_joint1: limit lower=-3.1067 upper=3.1067 effort=108 velocity=3.141592653589793 -> lower=-3.106686068549907 upper=3.106686068549907 effort=108 velocity=3.141592653589793
- joint right_joint2: limit lower=-2.0944 upper=2.0944 effort=108 velocity=3.141592653589793 -> lower=-2.0594885173533086 upper=2.0594885173533086 effort=108 velocity=3.141592653589793
- joint right_joint3: limit lower=-3.1067 upper=3.1067 effort=66 velocity=3.141592653589793 -> lower=-2.9321531433504737 upper=2.9321531433504737 effort=66 velocity=3.141592653589793
- joint right_joint4: limit lower=-2.5307 upper=1.0472 effort=66 velocity=3.141592653589793 -> lower=-2.4958208303518914 upper=1.0122909661567112 effort=66 velocity=3.141592653589793
- joint right_joint6: limit lower=-1.0472 upper=1.0472 effort=18 velocity=3.141592653589793 -> lower=-1.0122909661567112 upper=1.0122909661567112 effort=18 velocity=3.141592653589793
- joint right_joint7: limit lower=-1.5707963267948966 upper=1.5707963267948966 effort=18 velocity=3.141592653589793 -> lower=-1.361356816555577 upper=1.361356816555577 effort=18 velocity=3.141592653589793

File: m6_ccs_description/urdf/m6_ccs_usb-90c.urdf (robot description, URDF)
Before this commit: robot DobotCR5, 24 links, 23 joints
Joints:
- joint left_joint1: limit lower=-3.1067 upper=3.1067 effort=108 velocity=3.141592653589793 -> lower=-3.106686068549907 upper=3.106686068549907 effort=108 velocity=3.141592653589793
- joint left_joint2: limit lower=-2.0944 upper=2.0944 effort=108 velocity=3.141592653589793 -> lower=-2.0594885173533086 upper=2.0594885173533086 effort=108 velocity=3.141592653589793
- joint left_joint3: limit lower=-3.1067 upper=3.1067 effort=66 velocity=3.141592653589793 -> lower=-2.9321531433504737 upper=2.9321531433504737 effort=66 velocity=3.141592653589793
- joint left_joint4: limit lower=-2.5307 upper=1.0472 effort=66 velocity=3.141592653589793 -> lower=-2.4958208303518914 upper=1.0122909661567112 effort=66 velocity=3.141592653589793
- joint left_joint6: limit lower=-1.0472 upper=1.0472 effort=18 velocity=3.141592653589793 -> lower=-1.0122909661567112 upper=1.0122909661567112 effort=18 velocity=3.141592653589793
- joint left_joint7: limit lower=-1.5707963267948966 upper=1.5707963267948966 effort=18 velocity=3.141592653589793 -> lower=-1.361356816555577 upper=1.361356816555577 effort=18 velocity=3.141592653589793

File: m6_ccs_description/xacro/arm.xacro (robot description, xacro)
@@ -70,5 +70,5 @@
 			<child link="${prefix}link1"/>
 			<axis xyz="0 0 1"/>
-			<limit lower="-3.1067" upper="3.1067" effort="108" velocity="${PI}"/>
+			<limit lower="-${PI*178/180}" upper="${PI*178/180}" effort="108" velocity="${PI}"/>
 		</joint>
 		<!-- Link 2 -->
@@ -108,5 +108,5 @@
 			<child link="${prefix}link2"/>
 			<axis xyz="0 0 1"/>
-			<limit lower="-2.0944" upper="2.0944" effort="108" velocity="${PI}"/>
+			<limit lower="-${PI*118/180}" upper="${PI*118/180}" effort="108" velocity="${PI}"/>
 		</joint>
 		<!-- Link 3 -->
@@ -152,5 +152,5 @@
 			<child link="${prefix}link3"/>
 			<axis xyz="0 0 1"/>
-			<limit lower="-3.1067" upper="3.1067" effort="66" velocity="${PI}"/>
+			<limit lower="-${PI*168/180}" upper="${PI*168/180}" effort="66" velocity="${PI}"/>
 		</joint>
 		<!-- Link 4 -->
@@ -190,5 +190,5 @@
 			<child link="${prefix}link4"/>
 			<axis xyz="0 0 1"/>
-			<limit lower="-2.5307" upper="1.0472" effort="66" velocity="${PI}"/>
+			<limit lower="-${PI*143/180}" upper="${PI*58/180}" effort="66" velocity="${PI}"/>
 		</joint>
 		<!-- Link 5 - Mirrored COM and partial inertia -->
@@ -228,5 +228,5 @@
 			<child link="${prefix}link5"/>
 			<axis xyz="0 0 1"/>
-			<limit lower="-3.1067" upper="3.1067" effort="18" velocity="${PI}"/>
+			<limit lower="-${PI*168/180}" upper="${PI*168/180}" effort="18" velocity="${PI}"/>
 		</joint>
 		<!-- Link 6 - Partially mirrored COM and inertia -->
@@ -253,5 +253,5 @@
 			<xacro:if value="${collider == 'simple'}">
 				<collision>
-					<origin xyz="0 0 0" rpy="${PI/2} 0 0"/>
+					<origin rpy="${PI/2} 0 0"/>
 					<geometry>
 						<cylinder length="0.108046" radius="0.038348"/>
@@ -266,5 +266,5 @@
 			<child link="${prefix}link6"/>
 			<axis xyz="0 0 1"/>
-			<limit lower="-1.0472" upper="1.0472" effort="18" velocity="${PI}"/>
+			<limit lower="-${PI*58/180}" upper="${PI*58/180}" effort="18" velocity="${PI}"/>
 		</joint>
 		<!-- Link 7 -->
@@ -309,5 +309,5 @@
 			<child link="${prefix}link7"/>
 			<axis xyz="0 0 1"/>
-			<limit lower="-${PI/2}" upper="${PI/2}" effort="18" velocity="${PI}"/>
+			<limit lower="-${PI*78/180}" upper="${PI*78/180}" effort="18" velocity="${PI}"/>
 		</joint>
 		<link name="${prefix}tcp"/>
