Commit message: migrate to glb mesh

File: m6_ccs_description/urdf/m6_ccs.urdf (robot description, URDF)
Before this commit: robot M6_CCS, 9 links, 8 joints
Links:
- link base_link: geometry collision cylinder length=0.083664 radius=0.051277; visual mesh filename=package://m6_ccs_description/meshes/base.glb
- link link1: geometry collision cylinder length=0.125958 radius=0.057588; visual mesh filename=package://m6_ccs_description/meshes/link1.glb
- link link2: geometry collision cylinder length=0.078386 radius=0.046717; visual mesh filename=package://m6_ccs_description/meshes/link2.glb
- link link3: geometry collision cylinder length=0.089056 radius=0.046717; collision cylinder length=0.117016 radius=0.049964
- link link4: geometry collision cylinder length=0.080203 radius=0.041759; visual mesh filename=package://m6_ccs_description/meshes/link4.glb
- link link5: geometry collision cylinder length=0.14268 radius=0.056747; visual mesh filename=package://m6_ccs_description/meshes/link5.glb scale=1 1 1
- link link6: geometry collision cylinder length=0.108046 radius=0.038348; visual mesh filename=package://m6_ccs_description/meshes/link6.glb
- link link7: geometry collision cylinder length=0.038392 radius=0.041707; visual mesh filename=package://m6_ccs_description/meshes/link7.glb

File: m6_ccs_description/urdf/m6_ccs_dual.urdf (robot description, URDF)
Before this commit: robot M6_CCS, 22 links, 21 joints
Links:
- link left_base_link: geometry collision cylinder length=0.083664 radius=0.051277; visual mesh filename=package://m6_ccs_description/meshes/base.glb
- link left_link1: geometry collision cylinder length=0.125958 radius=0.057588; visual mesh filename=package://m6_ccs_description/meshes/link1.glb
- link left_link2: geometry collision cylinder length=0.078386 radius=0.046717; visual mesh filename=package://m6_ccs_description/meshes/link2.glb
- link left_link3: geometry collision cylinder length=0.089056 radius=0.046717; collision cylinder length=0.117016 radius=0.049964
- link left_link4: geometry collision cylinder length=0.080203 radius=0.041759; visual mesh filename=package://m6_ccs_description/meshes/link4.glb
- link left_link5: geometry collision cylinder length=0.14268 radius=0.056747; visual mesh filename=package://m6_ccs_description/meshes/link5.glb scale=1 1 1
- link left_link6: geometry collision cylinder length=0.108046 radius=0.038348; visual mesh filename=package://m6_ccs_description/meshes/link6.glb
- link left_link7: geometry collision cylinder length=0.038392 radius=0.041707; visual mesh filename=package://m6_ccs_description/meshes/link7.glb
- link right_base_link: geometry collision cylinder length=0.083664 radius=0.051277; visual mesh filename=package://m6_ccs_description/meshes/base.glb
- link right_link1: geometry collision cylinder length=0.125958 radius=0.057588; visual mesh filename=package://m6_ccs_description/meshes/link1.glb
- link right_link2: geometry collision cylinder length=0.078386 radius=0.046717; visual mesh filename=package://m6_ccs_description/meshes/link2.glb
- link right_link3: geometry collision cylinder length=0.089056 radius=0.046717; collision cylinder length=0.117016 radius=0.049964
- link right_link4: geometry collision cylinder length=0.080203 radius=0.041759; visual mesh filename=package://m6_ccs_description/meshes/link4.glb
- link right_link5: geometry collision cylinder length=0.14268 radius=0.056747; visual mesh filename=package://m6_ccs_description/meshes/link5.glb scale=1 -1 1
- link right_link6: geometry collision cylinder length=0.108046 radius=0.038348; visual mesh filename=package://m6_ccs_description/meshes/link6.glb
- link right_link7: geometry collision cylinder length=0.038392 radius=0.041707; visual mesh filename=package://m6_ccs_description/meshes/link7_r.glb

File: m6_ccs_description/urdf/m6_ccs_dual_ag2f90_c.urdf (robot description, URDF)
Before this commit: robot M6_CCS, 46 links, 45 joints
Links:
- link left_base_link: geometry collision cylinder length=0.083664 radius=0.051277; visual mesh filename=package://m6_ccs_description/meshes/base.glb
- link left_link1: geometry collision cylinder length=0.125958 radius=0.057588; visual mesh filename=package://m6_ccs_description/meshes/link1.glb
- link left_link2: geometry collision cylinder length=0.078386 radius=0.046717; visual mesh filename=package://m6_ccs_description/meshes/link2.glb
- link left_link3: geometry collision cylinder length=0.089056 radius=0.046717; collision cylinder length=0.117016 radius=0.049964
- link left_link4: geometry collision cylinder length=0.080203 radius=0.041759; visual mesh filename=package://m6_ccs_description/meshes/link4.glb
- link left_link5: geometry collision cylinder length=0.14268 radius=0.056747; visual mesh filename=package://m6_ccs_description/meshes/link5.glb scale=1 1 1
- link left_link6: geometry collision cylinder length=0.108046 radius=0.038348; visual mesh filename=package://m6_ccs_description/meshes/link6.glb
- link left_link7: geometry collision cylinder length=0.038392 radius=0.041707; visual mesh filename=package://m6_ccs_description/meshes/link7.glb
- link right_base_link: geometry collision cylinder length=0.083664 radius=0.051277; visual mesh filename=package://m6_ccs_description/meshes/base.glb
- link right_link1: geometry collision cylinder length=0.125958 radius=0.057588; visual mesh filename=package://m6_ccs_description/meshes/link1.glb
- link right_link2: geometry collision cylinder length=0.078386 radius=0.046717; visual mesh filename=package://m6_ccs_description/meshes/link2.glb
- link right_link3: geometry collision cylinder length=0.089056 radius=0.046717; collision cylinder length=0.117016 radius=0.049964
- link right_link4: geometry collision cylinder length=0.080203 radius=0.041759; visual mesh filename=package://m6_ccs_description/meshes/link4.glb
- link right_link5: geometry collision cylinder length=0.14268 radius=0.056747; visual mesh filename=package://m6_ccs_description/meshes/link5.glb scale=1 -1 1
- link right_link6: geometry collision cylinder length=0.108046 radius=0.038348; visual mesh filename=package://m6_ccs_description/meshes/link6.glb
- link right_link7: geometry collision cylinder length=0.038392 radius=0.041707; visual mesh filename=package://m6_ccs_description/meshes/link7_r.glb

File: m6_ccs_description/urdf/m6_ccs_dual_desktop.urdf (robot description, URDF)
Before this commit: robot M6_CCS, 22 links, 21 joints
Links:
- link arm_base: geometry collision box size=0.10045 0.100398 0.648662; visual mesh filename=package://m6_ccs_description/meshes/dual_base.glb
- link left_base_link: geometry collision cylinder length=0.083664 radius=0.051277; visual mesh filename=package://m6_ccs_description/meshes/base.glb
- link left_link1: geometry collision cylinder length=0.125958 radius=0.057588; visual mesh filename=package://m6_ccs_description/meshes/link1.glb
- link left_link2: geometry collision cylinder length=0.078386 radius=0.046717; visual mesh filename=package://m6_ccs_description/meshes/link2.glb
- link left_link3: geometry collision cylinder length=0.117016 radius=0.049964; visual mesh filename=package://m6_ccs_description/meshes/link3.glb
- link left_link4: geometry collision cylinder length=0.080203 radius=0.041759; visual mesh filename=package://m6_ccs_description/meshes/link4.glb
- link left_link5: geometry collision cylinder length=0.14268 radius=0.056747; visual mesh filename=package://m6_ccs_description/meshes/link5.glb scale=1 1 1
- link left_link6: geometry collision cylinder length=0.108046 radius=0.038348; visual mesh filename=package://m6_ccs_description/meshes/link6.glb
- link left_link7: geometry collision cylinder length=0.038392 radius=0.041707; visual mesh filename=package://m6_ccs_description/meshes/link7.glb
- link right_base_link: geometry collision cylinder length=0.083664 radius=0.051277; visual mesh filename=package://m6_ccs_description/meshes/base.glb
- link right_link1: geometry collision cylinder length=0.125958 radius=0.057588; visual mesh filename=package://m6_ccs_description/meshes/link1.glb
- link right_link2: geometry collision cylinder length=0.078386 radius=0.046717; visual mesh filename=package://m6_ccs_description/meshes/link2.glb
- link right_link3: geometry collision cylinder length=0.117016 radius=0.049964; visual mesh filename=package://m6_ccs_description/meshes/link3.glb
- link right_link4: geometry collision cylinder length=0.080203 radius=0.041759; visual mesh filename=package://m6_ccs_description/meshes/link4.glb
- link right_link5: geometry collision cylinder length=0.14268 radius=0.056747; visual mesh filename=package://m6_ccs_description/meshes/link5.glb scale=1 -1 1
- link right_link6: geometry collision cylinder length=0.108046 radius=0.038348; visual mesh filename=package://m6_ccs_description/meshes/link6.glb
- link right_link7: geometry collision cylinder length=0.038392 radius=0.041707; visual mesh filename=package://m6_ccs_description/meshes/link7_r.glb

File: m6_ccs_description/urdf/m6_ccs_dual_desktop_90c.urdf (robot description, URDF)
Before this commit: robot M6_CCS, 46 links, 45 joints
Links:
- link arm_base: geometry collision box size=0.10045 0.100398 0.648662; visual mesh filename=package://m6_ccs_description/meshes/dual_base.glb
- link left_base_link: geometry collision cylinder length=0.083664 radius=0.051277; visual mesh filename=package://m6_ccs_description/meshes/base.glb
- link left_link1: geometry collision cylinder length=0.125958 radius=0.057588; visual mesh filename=package://m6_ccs_description/meshes/link1.glb
- link left_link2: geometry collision cylinder length=0.078386 radius=0.046717; visual mesh filename=package://m6_ccs_description/meshes/link2.glb
- link left_link3: geometry collision cylinder length=0.117016 radius=0.049964; visual mesh filename=package://m6_ccs_description/meshes/link3.glb
- link left_link4: geometry collision cylinder length=0.080203 radius=0.041759; visual mesh filename=package://m6_ccs_description/meshes/link4.glb
- link left_link5: geometry collision cylinder length=0.14268 radius=0.056747; visual mesh filename=package://m6_ccs_description/meshes/link5.glb scale=1 1 1
- link left_link6: geometry collision cylinder length=0.108046 radius=0.038348; visual mesh filename=package://m6_ccs_description/meshes/link6.glb
- link left_link7: geometry collision cylinder length=0.038392 radius=0.041707; visual mesh filename=package://m6_ccs_description/meshes/link7.glb
- link right_base_link: geometry collision cylinder length=0.083664 radius=0.051277; visual mesh filename=package://m6_ccs_description/meshes/base.glb
- link right_link1: geometry collision cylinder length=0.125958 radius=0.057588; visual mesh filename=package://m6_ccs_description/meshes/link1.glb
- link right_link2: geometry collision cylinder length=0.078386 radius=0.046717; visual mesh filename=package://m6_ccs_description/meshes/link2.glb
- link right_link3: geometry collision cylinder length=0.117016 radius=0.049964; visual mesh filename=package://m6_ccs_description/meshes/link3.glb
- link right_link4: geometry collision cylinder length=0.080203 radius=0.041759; visual mesh filename=package://m6_ccs_description/meshes/link4.glb
- link right_link5: geometry collision cylinder length=0.14268 radius=0.056747; visual mesh filename=package://m6_ccs_description/meshes/link5.glb scale=1 -1 1
- link right_link6: geometry collision cylinder length=0.108046 radius=0.038348; visual mesh filename=package://m6_ccs_description/meshes/link6.glb
- link right_link7: geometry collision cylinder length=0.038392 radius=0.041707; visual mesh filename=package://m6_ccs_description/meshes/link7_r.glb

File: m6_ccs_description/urdf/m6_ccs_dual_desktop_90c_soft.urdf (robot description, URDF)
Before this commit: robot M6_CCS, 46 links, 45 joints
Links:
- link arm_base: geometry collision box size=0.10045 0.100398 0.648662; visual mesh filename=package://m6_ccs_description/meshes/dual_base.glb
- link left_base_link: geometry collision cylinder length=0.083664 radius=0.051277; visual mesh filename=package://m6_ccs_description/meshes/base.glb
- link left_link1: geometry collision cylinder length=0.125958 radius=0.057588; visual mesh filename=package://m6_ccs_description/meshes/link1.glb
- link left_link2: geometry collision cylinder length=0.078386 radius=0.046717; visual mesh filename=package://m6_ccs_description/meshes/link2.glb
- link left_link3: geometry collision cylinder length=0.089056 radius=0.046717; collision cylinder length=0.117016 radius=0.049964
- link left_link4: geometry collision cylinder length=0.080203 radius=0.041759; visual mesh filename=package://m6_ccs_description/meshes/link4.glb
- link left_link5: geometry collision cylinder length=0.14268 radius=0.056747; visual mesh filename=package://m6_ccs_description/meshes/link5.glb scale=1 1 1
- link left_link6: geometry collision cylinder length=0.108046 radius=0.038348; visual mesh filename=package://m6_ccs_description/meshes/link6.glb
- link left_link7: geometry collision cylinder length=0.038392 radius=0.041707; visual mesh filename=package://m6_ccs_description/meshes/link7.glb
- link right_base_link: geometry collision cylinder length=0.083664 radius=0.051277; visual mesh filename=package://m6_ccs_description/meshes/base.glb
- link right_link1: geometry collision cylinder length=0.125958 radius=0.057588; visual mesh filename=package://m6_ccs_description/meshes/link1.glb
- link right_link2: geometry collision cylinder length=0.078386 radius=0.046717; visual mesh filename=package://m6_ccs_description/meshes/link2.glb
- link right_link3: geometry collision cylinder length=0.089056 radius=0.046717; collision cylinder length=0.117016 radius=0.049964
- link right_link4: geometry collision cylinder length=0.080203 radius=0.041759; visual mesh filename=package://m6_ccs_description/meshes/link4.glb
- link right_link5: geometry collision cylinder length=0.14268 radius=0.056747; visual mesh filename=package://m6_ccs_description/meshes/link5.glb scale=1 -1 1
- link right_link6: geometry collision cylinder length=0.108046 radius=0.038348; visual mesh filename=package://m6_ccs_description/meshes/link6.glb
- link right_link7: geometry collision cylinder length=0.038392 radius=0.041707; visual mesh filename=package://m6_ccs_description/meshes/link7_r.glb

File: m6_ccs_description/urdf/m6_ccs_dual_rg75.urdf (robot description, URDF)
Before this commit: robot M6_CCS, 34 links, 33 joints
Links:
- link left_base_link: geometry collision cylinder length=0.083664 radius=0.051277; visual mesh filename=package://m6_ccs_description/meshes/base.glb
- link left_flange: geometry collision mesh filename=package://jodell_description/meshes/RG75/flange.glb; visual mesh filename=package://jodell_description/meshes/RG75/flange.glb
- link left_gripper_base: geometry collision mesh filename=package://jodell_description/meshes/RG75/base.glb; visual mesh filename=package://jodell_description/meshes/RG75/base.glb
- link left_left_finger: geometry collision mesh filename=package://jodell_description/meshes/RG75/finger.glb; visual mesh filename=package://jodell_description/meshes/RG75/finger.glb
- link left_left_finger_pad: geometry collision mesh filename=package://jodell_description/meshes/RG75/pad_fiveages.glb; visual mesh filename=package://jodell_description/meshes/RG75/pad_fiveages.glb
- link left_link1: geometry collision cylinder length=0.125958 radius=0.057588; visual mesh filename=package://m6_ccs_description/meshes/link1.glb
- link left_link2: geometry collision cylinder length=0.078386 radius=0.046717; visual mesh filename=package://m6_ccs_description/meshes/link2.glb
- link left_link3: geometry collision cylinder length=0.089056 radius=0.046717; collision cylinder length=0.117016 radius=0.049964
- link left_link4: geometry collision cylinder length=0.080203 radius=0.041759; visual mesh filename=package://m6_ccs_description/meshes/link4.glb
- link left_link5: geometry collision cylinder length=0.14268 radius=0.056747; visual mesh filename=package://m6_ccs_description/meshes/link5.glb scale=1 1 1
- link left_link6: geometry collision cylinder length=0.108046 radius=0.038348; visual mesh filename=package://m6_ccs_description/meshes/link6.glb
- link left_link7: geometry collision cylinder length=0.038392 radius=0.041707; visual mesh filename=package://m6_ccs_description/meshes/link7.glb
- link left_right_finger: geometry collision mesh filename=package://jodell_description/meshes/RG75/finger.glb scale=-1 -1 1; visual mesh filename=package://jodell_description/meshes/RG75/finger.glb scale=-1 -1 1
- link left_right_finger_pad: geometry collision mesh filename=package://jodell_description/meshes/RG75/pad_fiveages.glb scale=1 -1 1; visual mesh filename=package://jodell_description/meshes/RG75/pad_fiveages.glb scale=1 -1 1
- link right_base_link: geometry collision cylinder length=0.083664 radius=0.051277; visual mesh filename=package://m6_ccs_description/meshes/base.glb
- link right_flange: geometry collision mesh filename=package://jodell_description/meshes/RG75/flange.glb; visual mesh filename=package://jodell_description/meshes/RG75/flange.glb
- link right_gripper_base: geometry collision mesh filename=package://jodell_description/meshes/RG75/base.glb; visual mesh filename=package://jodell_description/meshes/RG75/base.glb
- link right_left_finger: geometry collision mesh filename=package://jodell_description/meshes/RG75/finger.glb; visual mesh filename=package://jodell_description/meshes/RG75/finger.glb
- link right_left_finger_pad: geometry collision mesh filename=package://jodell_description/meshes/RG75/pad_fiveages.glb; visual mesh filename=package://jodell_description/meshes/RG75/pad_fiveages.glb
- link right_link1: geometry collision cylinder length=0.125958 radius=0.057588; visual mesh filename=package://m6_ccs_description/meshes/link1.glb
- link right_link2: geometry collision cylinder length=0.078386 radius=0.046717; visual mesh filename=package://m6_ccs_description/meshes/link2.glb
- link right_link3: geometry collision cylinder length=0.089056 radius=0.046717; collision cylinder length=0.117016 radius=0.049964
- link right_link4: geometry collision cylinder length=0.080203 radius=0.041759; visual mesh filename=package://m6_ccs_description/meshes/link4.glb
- link right_link5: geometry collision cylinder length=0.14268 radius=0.056747; visual mesh filename=package://m6_ccs_description/meshes/link5.glb scale=1 -1 1
- link right_link6: geometry collision cylinder length=0.108046 radius=0.038348; visual mesh filename=package://m6_ccs_description/meshes/link6.glb
- link right_link7: geometry collision cylinder length=0.038392 radius=0.041707; visual mesh filename=package://m6_ccs_description/meshes/link7_r.glb
- link right_right_finger: geometry collision mesh filename=package://jodell_description/meshes/RG75/finger.glb scale=-1 -1 1; visual mesh filename=package://jodell_description/meshes/RG75/finger.glb scale=-1 -1 1
- link right_right_finger_pad: geometry collision mesh filename=package://jodell_description/meshes/RG75/pad_fiveages.glb scale=1 -1 1; visual mesh filename=package://jodell_description/meshes/RG75/pad_fiveages.glb scale=1 -1 1

File: m6_ccs_description/urdf/m6_ccs_usb-90c.urdf (robot description, URDF)
Before this commit: robot DobotCR5, 24 links, 23 joints
Links:
- link base: geometry collision box size=0.10045 0.100398 0.648662; visual mesh filename=package://m6_ccs_description/meshes/dual_base.glb
- link left_base_link: geometry collision cylinder length=0.083664 radius=0.051277; visual mesh filename=package://m6_ccs_description/meshes/base.glb
- link left_link1: geometry collision cylinder length=0.125958 radius=0.057588; visual mesh filename=package://m6_ccs_description/meshes/link1.glb
- link left_link2: geometry collision cylinder length=0.078386 radius=0.046717; visual mesh filename=package://m6_ccs_description/meshes/link2.glb
- link left_link3: geometry collision cylinder length=0.089056 radius=0.046717; collision cylinder length=0.117016 radius=0.049964
- link left_link4: geometry collision cylinder length=0.080203 radius=0.041759; visual mesh filename=package://m6_ccs_description/meshes/link4.glb
- link left_link5: geometry collision cylinder length=0.14268 radius=0.056747; visual mesh filename=package://m6_ccs_description/meshes/link5.glb scale=1 1 1
- link left_link6: geometry collision cylinder length=0.108046 radius=0.038348; visual mesh filename=package://m6_ccs_description/meshes/link6.glb
- link left_link7: geometry collision cylinder length=0.038392 radius=0.041707; visual mesh filename=package://m6_ccs_description/meshes/link7.glb
