Commit message: migrate to glb mesh

File: m6_ccs_description/xacro/arm.xacro (robot description, xacro)
@@ -15,11 +15,11 @@
 			<visual>
 				<geometry>
-					<mesh filename="file://$(find m6_ccs_description)/meshes/base.obj"/>
-				</geometry>
-			</visual>
-			<xacro:if value="${collider == 'convex'}">
-				<collision>
-					<geometry>
-						<mesh filename="file://$(find m6_ccs_description)/meshes/base.obj"/>
+					<mesh filename="file://$(find m6_ccs_description)/meshes/base.glb"/>
+				</geometry>
+			</visual>
+			<xacro:if value="${collider == 'convex'}">
+				<collision>
+					<geometry>
+						<mesh filename="file://$(find m6_ccs_description)/meshes/base.glb"/>
 					</geometry>
 				</collision>
@@ -45,11 +45,11 @@
 			<visual>
 				<geometry>
-					<mesh filename="file://$(find m6_ccs_description)/meshes/link1.obj"/>
-				</geometry>
-			</visual>
-			<xacro:if value="${collider == 'convex'}">
-				<collision>
-					<geometry>
-						<mesh filename="file://$(find m6_ccs_description)/meshes/link1.obj"/>
+					<mesh filename="file://$(find m6_ccs_description)/meshes/link1.glb"/>
+				</geometry>
+			</visual>
+			<xacro:if value="${collider == 'convex'}">
+				<collision>
+					<geometry>
+						<mesh filename="file://$(find m6_ccs_description)/meshes/link1.glb"/>
 					</geometry>
 				</collision>
@@ -83,11 +83,11 @@
 			<visual>
 				<geometry>
-					<mesh filename="file://$(find m6_ccs_description)/meshes/link2.obj"/>
-				</geometry>
-			</visual>
-			<xacro:if value="${collider == 'convex'}">
-				<collision>
-					<geometry>
-						<mesh filename="file://$(find m6_ccs_description)/meshes/link2.obj"/>
+					<mesh filename="file://$(find m6_ccs_description)/meshes/link2.glb"/>
+				</geometry>
+			</visual>
+			<xacro:if value="${collider == 'convex'}">
+				<collision>
+					<geometry>
+						<mesh filename="file://$(find m6_ccs_description)/meshes/link2.glb"/>
 					</geometry>
 				</collision>
@@ -121,11 +121,11 @@
 			<visual>
 				<geometry>
-					<mesh filename="file://$(find m6_ccs_description)/meshes/link3.obj"/>
-				</geometry>
-			</visual>
-			<xacro:if value="${collider == 'convex'}">
-				<collision>
-					<geometry>
-						<mesh filename="file://$(find m6_ccs_description)/meshes/link3.obj"/>
+					<mesh filename="file://$(find m6_ccs_description)/meshes/link3.glb"/>
+				</geometry>
+			</visual>
+			<xacro:if value="${collider == 'convex'}">
+				<collision>
+					<geometry>
+						<mesh filename="file://$(find m6_ccs_description)/meshes/link3.glb"/>
 					</geometry>
 				</collision>
@@ -165,11 +165,11 @@
 			<visual>
 				<geometry>
-					<mesh filename="file://$(find m6_ccs_description)/meshes/link4.obj"/>
-				</geometry>
-			</visual>
-			<xacro:if value="${collider == 'convex'}">
-				<collision>
-					<geometry>
-						<mesh filename="file://$(find m6_ccs_description)/meshes/link4.obj"/>
+					<mesh filename="file://$(find m6_ccs_description)/meshes/link4.glb"/>
+				</geometry>
+			</visual>
+			<xacro:if value="${collider == 'convex'}">
+				<collision>
+					<geometry>
+						<mesh filename="file://$(find m6_ccs_description)/meshes/link4.glb"/>
 					</geometry>
 				</collision>
@@ -203,11 +203,11 @@
 			<visual>
 				<geometry>
-					<mesh filename="file://$(find m6_ccs_description)/meshes/link5.obj" scale="1 ${direction} 1"/>
-				</geometry>
-			</visual>
-			<xacro:if value="${collider == 'convex'}">
-				<collision>
-					<geometry>
-						<mesh filename="file://$(find m6_ccs_description)/meshes/link5.obj" scale="1 ${direction} 1"/>
+					<mesh filename="file://$(find m6_ccs_description)/meshes/link5.glb" scale="1 ${direction} 1"/>
+				</geometry>
+			</visual>
+			<xacro:if value="${collider == 'convex'}">
+				<collision>
+					<geometry>
+						<mesh filename="file://$(find m6_ccs_description)/meshes/link5.glb"/>
 					</geometry>
 				</collision>
@@ -241,11 +241,11 @@
 			<visual>
 				<geometry>
-					<mesh filename="file://$(find m6_ccs_description)/meshes/link6.obj"/>
-				</geometry>
-			</visual>
-			<xacro:if value="${collider == 'convex'}">
-				<collision>
-					<geometry>
-						<mesh filename="file://$(find m6_ccs_description)/meshes/link6.obj"/>
+					<mesh filename="file://$(find m6_ccs_description)/meshes/link6.glb"/>
+				</geometry>
+			</visual>
+			<xacro:if value="${collider == 'convex'}">
+				<collision>
+					<geometry>
+						<mesh filename="file://$(find m6_ccs_description)/meshes/link6.glb"/>
 					</geometry>
 				</collision>
@@ -280,8 +280,8 @@
 				<geometry>
 					<xacro:if value="${direction == 1}">
-						<mesh filename="file://$(find m6_ccs_description)/meshes/link7.obj"/>
+						<mesh filename="file://$(find m6_ccs_description)/meshes/link7.glb"/>
 					</xacro:if>
 					<xacro:if value="${direction == -1}">
-						<mesh filename="file://$(find m6_ccs_description)/meshes/link7_r.obj"/>
+						<mesh filename="file://$(find m6_ccs_description)/meshes/link7_r.glb"/>
 					</xacro:if>
 				</geometry>
@@ -290,5 +290,5 @@
 				<collision>
 					<geometry>
-						<mesh filename="file://$(find m6_ccs_description)/meshes/link7.obj"/>
+						<mesh filename="file://$(find m6_ccs_description)/meshes/link7.glb"/>
 					</geometry>
 				</collision>

File: m6_ccs_description/xacro/robot.xacro (robot description, xacro)
@@ -80,5 +80,5 @@
 				<visual>
 					<geometry>
-						<mesh filename="file://$(find m6_ccs_description)/meshes/dual_base.obj"/>
+						<mesh filename="file://$(find m6_ccs_description)/meshes/desktop_base.glb"/>
 					</geometry>
 				</visual>
@@ -191,5 +191,5 @@
 			<visual>
 				<geometry>
-					<mesh filename="file://$(find m6_ccs_description)/meshes/dual_base.obj"/>
+					<mesh filename="file://$(find m6_ccs_description)/meshes/desktop_base.glb"/>
 				</geometry>
 			</visual>
