Commit message: add planning urdf publish in ocs2 arm controller

File: m6_ccs_description/urdf/m6_ccs.urdf (robot description, URDF)
Before this commit: robot M6_CCS, 9 links, 8 joints
Links:
- removed link link1
- removed link link2
- removed link link3
- removed link link4
- removed link link5
- removed link link6
- removed link link7
- removed link tcp
- added link arm_base; collision box size=0.2000 0.3 0.4029
- added link left_base_link, mass 1.1962; collision cylinder length=0.083664 radius=0.051277; visual mesh filename=package://m6_ccs_description/meshes/base.glb
- added link left_eef
- added link left_link1, mass 1.9705; collision cylinder length=0.125958 radius=0.057588; visual mesh filename=package://m6_ccs_description/meshes/link1.glb
- added link left_link2, mass 2.24398; collision cylinder length=0.078386 radius=0.046717; visual mesh filename=package://m6_ccs_description/meshes/link2.glb
- added link left_link3, mass 1.9242; collision cylinder length=0.089056 radius=0.046717; collision cylinder length=0.117016 radius=0.049964
- added link left_link4, mass 1.6085; collision cylinder length=0.080203 radius=0.041759; visual mesh filename=package://m6_ccs_description/meshes/link4.glb
- added link left_link5, mass 2.0883; collision cylinder length=0.14268 radius=0.056747; visual mesh filename=package://m6_ccs_description/meshes/link5.glb scale=1 1 1
- added link left_link6, mass 0.72496; collision cylinder length=0.108046 radius=0.038348; visual mesh filename=package://m6_ccs_description/meshes/link6.glb
- added link left_link7, mass 0.68606; collision cylinder length=0.038392 radius=0.041707; visual mesh filename=package://m6_ccs_description/meshes/link7.glb
- added link left_tcp
- added link right_base_link, mass 1.1962; collision cylinder length=0.083664 radius=0.051277; visual mesh filename=package://m6_ccs_description/meshes/base.glb
- added link right_eef
- added link right_link1, mass 1.9705; collision cylinder length=0.125958 radius=0.057588; visual mesh filename=package://m6_ccs_description/meshes/link1.glb
- added link right_link2, mass 2.24398; collision cylinder length=0.078386 radius=0.046717; visual mesh filename=package://m6_ccs_description/meshes/link2.glb
- added link right_link3, mass 1.9242; collision cylinder length=0.089056 radius=0.046717; collision cylinder length=0.117016 radius=0.049964
- added link right_link4, mass 1.6085; collision cylinder length=0.080203 radius=0.041759; visual mesh filename=package://m6_ccs_description/meshes/link4.glb
- added link right_link5, mass 2.0883; collision cylinder length=0.14268 radius=0.056747; visual mesh filename=package://m6_ccs_description/meshes/link5.glb scale=1 -1 1
- added link right_link6, mass 0.72496; collision cylinder length=0.108046 radius=0.038348; visual mesh filename=package://m6_ccs_description/meshes/link6.glb
- added link right_link7, mass 0.68606; collision cylinder length=0.038392 radius=0.041707; visual mesh filename=package://m6_ccs_description/meshes/link7_r.glb
- added link right_tcp
- link base_link: mass 1.1962 -> None; geometry 
Joints:
- removed joint joint1
- removed joint joint2
- removed joint joint3
- removed joint joint4
- removed joint joint5
- removed joint joint6
- removed joint joint7
- removed joint tcp_joint
- added joint arm_base_joint: type fixed, parent base_link, child arm_base
- added joint left_arm_base_joint: type fixed, parent arm_base, child left_base_link, origin xyz=0.0 0.062 0 rpy=-1.5707963267948966 0 0
- added joint left_eef_joint: type fixed, parent left_tcp, child left_eef
- added joint left_joint1: type revolute, parent left_base_link, child left_link1, origin xyz=0 0 0.1745 rpy=0 0 0, axis 0 0 1, limit lower=-3.106686068549907 upper=3.106686068549907 effort=108 velocity=3.141592653589793
- added joint left_joint2: type revolute, parent left_link1, child left_link2, origin rpy=1.5707963267948966 0 0, axis 0 0 1, limit lower=-2.0594885173533086 upper=2.0594885173533086 effort=108 velocity=3.141592653589793
- added joint left_joint3: type revolute, parent left_link2, child left_link3, origin xyz=0 0.287 0 rpy=-1.5707963267948966 0 0, axis 0 0 1, limit lower=-2.9321531433504737 upper=2.9321531433504737 effort=66 velocity=3.141592653589793
- added joint left_joint4: type revolute, parent left_link3, child left_link4, origin xyz=0.018 0 0 rpy=-1.5707963267948966 0 3.141592653589793, axis 0 0 1, limit lower=-2.4958208303518914 upper=1.0122909661567112 effort=66 velocity=3.141592653589793
- added joint left_joint5: type revolute, parent left_link4, child left_link5, origin xyz=0.018 -0.314 0 rpy=-1.5707963267948966 0 3.141592653589793, axis 0 0 1, limit lower=-3.1067 upper=3.1067 effort=18 velocity=3.141592653589793
- added joint left_joint6: type revolute, parent left_link5, child left_link6, origin rpy=1.5707963267948966 -1.5707963267948966 0, axis 0 0 1, limit lower=-1.0122909661567112 upper=1.0122909661567112 effort=18 velocity=3.141592653589793
- added joint left_joint7: type revolute, parent left_link6, child left_link7, origin rpy=1.5707963267948966 -1.5707963267948966 0, axis 0 0 1, limit lower=-1.361356816555577 upper=1.361356816555577 effort=18 velocity=3.141592653589793
- added joint left_tcp_joint: type fixed, parent left_link7, child left_tcp, origin xyz=0 -0.095 0 rpy=1.5707963267948966 -1.5707963267948966 0
- added joint right_arm_base_joint: type fixed, parent arm_base, child right_base_link, origin xyz=0 -0.062 0 rpy=1.5707963267948966 0 0
- added joint right_eef_joint: type fixed, parent right_tcp, child right_eef
- added joint right_joint1: type revolute, parent right_base_link, child right_link1, origin xyz=0 0 0.1745 rpy=0 0 0, axis 0 0 1, limit lower=-3.106686068549907 upper=3.106686068549907 effort=108 velocity=3.141592653589793
- added joint right_joint2: type revolute, parent right_link1, child right_link2, origin rpy=1.5707963267948966 0 0, axis 0 0 1, limit lower=-2.0594885173533086 upper=2.0594885173533086 effort=108 velocity=3.141592653589793
- added joint right_joint3: type revolute, parent right_link2, child right_link3, origin xyz=0 0.287 0 rpy=-1.5707963267948966 0 0, axis 0 0 1, limit lower=-2.9321531433504737 upper=2.9321531433504737 effort=66 velocity=3.141592653589793
- added joint right_joint4: type revolute, parent right_link3, child right_link4, origin xyz=0.018 0 0 rpy=-1.5707963267948966 0 3.141592653589793, axis 0 0 1, limit lower=-2.4958208303518914 upper=1.0122909661567112 effort=66 velocity=3.141592653589793
- added joint right_joint5: type revolute, parent right_link4, child right_link5, origin xyz=0.018 -0.314 0 rpy=-1.5707963267948966 0 3.141592653589793, axis 0 0 1, limit lower=-3.1067 upper=3.1067 effort=18 velocity=3.141592653589793
- added joint right_joint6: type revolute, parent right_link5, child right_link6, origin rpy=1.5707963267948966 -1.5707963267948966 0, axis 0 0 1, limit lower=-1.0122909661567112 upper=1.0122909661567112 effort=18 velocity=3.141592653589793
- added joint right_joint7: type revolute, parent right_link6, child right_link7, origin rpy=1.5707963267948966 -1.5707963267948966 0, axis 0 0 1, limit lower=-1.361356816555577 upper=1.361356816555577 effort=18 velocity=3.141592653589793
- added joint right_tcp_joint: type fixed, parent right_link7, child right_tcp, origin xyz=0 -0.095 0 rpy=1.5707963267948966 -1.5707963267948966 0

File: m6_ccs_description/urdf/m6_ccs_ag2f90.urdf (robot description, URDF)
Before this commit: robot M6_CCS, 46 links, 45 joints
Links:
- link arm_base: geometry collision box size=0.2000 0.3 0.4029
- link left_gripper_base: geometry visual mesh filename=package://changingtek_description/meshes/AG2F90-C/visual/gr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
- link left_left_1_link: geometry visual mesh filename=package://changingtek_description/meshes/AG2F90-C/visual/li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
- link left_left_2_link: geometry visual mesh filename=package://changingtek_description/meshes/AG2F90-C/visual/li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
- link left_left_Pad_link: geometry visual mesh filename=package://changingtek_description/meshes/AG2F90-C/visual/pa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
- link left_left_in_link: geometry visual mesh filename=package://changingtek_description/meshes/AG2F90-C/visual/in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
- link left_left_up_link: geometry visual mesh filename=package://changingtek_description/meshes/AG2F90-C/visual/up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
- link left_link3: geometry collision cylinder length=0.089056 radius=0.046717; collision cylinder length=0.117016 radius=0.049964
- link left_link7: geometry collision cylinder length=0.038392 radius=0.041707; collision cylinder length=0.08 radius=0.021707
- link left_right_1_link: geometry visual mesh filename=package://changingtek_description/meshes/AG2F90-C/visual/li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
- link left_right_2_link: geometry visual mesh filename=package://changingtek_description/meshes/AG2F90-C/visual/li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
- link left_right_Pad_link: geometry visual mesh filename=package://changingtek_description/meshes/AG2F90-C/visual/pa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
- link left_right_in_link: geometry visual mesh filename=package://changingtek_description/meshes/AG2F90-C/visual/in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
- link left_right_up_link: geometry visual mesh filename=package://changingtek_description/meshes/AG2F90-C/visual/up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
- link right_gripper_base: geometry visual mesh filename=package://changingtek_description/meshes/AG2F90-C/visual/gr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
- link right_left_1_link: geometry visual mesh filename=package://changingtek_description/meshes/AG2F90-C/visual/li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
- link right_left_2_link: geometry visual mesh filename=package://changingtek_description/meshes/AG2F90-C/visual/li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
- link right_left_Pad_link: geometry visual mesh filename=package://changingtek_description/meshes/AG2F90-C/visual/pa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
- link right_left_in_link: geometry visual mesh filename=package://changingtek_description/meshes/AG2F90-C/visual/in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
- link right_left_up_link: geometry visual mesh filename=package://changingtek_description/meshes/AG2F90-C/visual/up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
- link right_link3: geometry collision cylinder length=0.089056 radius=0.046717; collision cylinder length=0.117016 radius=0.049964
- link right_link7: geometry collision cylinder length=0.038392 radius=0.041707; collision cylinder length=0.08 radius=0.021707
- link right_right_1_link: geometry visual mesh filename=package://changingtek_description/meshes/AG2F90-C/visual/li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
- link right_right_2_link: geometry visual mesh filename=package://changingtek_description/meshes/AG2F90-C/visual/li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
- link right_right_Pad_link: geometry visual mesh filename=package://changingtek_description/meshes/AG2F90-C/visual/pa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
- link right_right_in_link: geometry visual mesh filename=package://changingtek_description/meshes/AG2F90-C/visual/in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
- link right_right_up_link: geometry visual mesh filename=package://changingtek_description/meshes/AG2F90-C/visual/up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
Joints:
- joint left_arm_base_joint: origin xyz=0.0 0.12 0.701 rpy=-1.5707963267948966 0 0 -> xyz=0.0 0.062 0 rpy=-1.5707963267948966 0 0
- joint left_joint5: limit lower=-3.1067 upper=3.1067 effort=18 velocity=3.141592653589793 -> lower=-2.9321531433504737 upper=2.9321531433504737 effort=18 velocity=3.141592653589793
- joint left_right_2_Joint: mimic joint=left_left_2_Joint -> joint=left_gripper_joint
- joint left_right_in_Joint: mimic joint=left_right_1_Joint multiplier=0.1 offset=0 -> joint=left_gripper_joint multiplier=0.1 offset=0
- joint left_right_up_Joint: mimic joint=left_right_1_Joint -> joint=left_gripper_joint
- joint right_arm_base_joint: origin xyz=0.0 -0.12 0.701 rpy=1.5707963267948966 0 0 -> xyz=0 -0.062 0 rpy=1.5707963267948966 0 0
- joint right_joint5: limit lower=-3.1067 upper=3.1067 effort=18 velocity=3.141592653589793 -> lower=-2.9321531433504737 upper=2.9321531433504737 effort=18 velocity=3.141592653589793
- joint right_right_2_Joint: mimic joint=right_left_2_Joint -> joint=right_gripper_joint
- joint right_right_in_Joint: mimic joint=right_right_1_Joint multiplier=0.1 offset=0 -> joint=right_gripper_joint multiplier=0.1 offset=0
- joint right_right_up_Joint: mimic joint=right_right_1_Joint -> joint=right_gripper_joint

File: m6_ccs_description/urdf/m6_ccs_rg75.urdf (robot description, URDF)
Before this commit: robot M6_CCS, 34 links, 33 joints
Links:
- link left_flange: geometry visual mesh filename=package://jodell_description/meshes/RG75/flange.glb
- link left_gripper_base: geometry visual mesh filename=package://jodell_description/meshes/RG75/base.glb
- link left_left_finger: geometry visual mesh filename=package://jodell_description/meshes/RG75/finger.glb
- link left_left_finger_pad: geometry visual mesh filename=package://jodell_description/meshes/RG75/pad_fiveages.glb
- link left_link7: geometry collision cylinder length=0.038392 radius=0.041707; collision cylinder length=0.08 radius=0.021707
- link left_right_finger: geometry visual mesh filename=package://jodell_description/meshes/RG75/finger.glb scale=-1 -1 1
- link left_right_finger_pad: geometry visual mesh filename=package://jodell_description/meshes/RG75/pad_fiveages.glb scale=1 -1 1
- link right_flange: geometry visual mesh filename=package://jodell_description/meshes/RG75/flange.glb
- link right_gripper_base: geometry visual mesh filename=package://jodell_description/meshes/RG75/base.glb
- link right_left_finger: geometry visual mesh filename=package://jodell_description/meshes/RG75/finger.glb
- link right_left_finger_pad: geometry visual mesh filename=package://jodell_description/meshes/RG75/pad_fiveages.glb
- link right_link7: geometry collision cylinder length=0.038392 radius=0.041707; collision cylinder length=0.08 radius=0.021707
- link right_right_finger: geometry visual mesh filename=package://jodell_description/meshes/RG75/finger.glb scale=-1 -1 1
- link right_right_finger_pad: geometry visual mesh filename=package://jodell_description/meshes/RG75/pad_fiveages.glb scale=1 -1 1
Joints:
- joint left_joint5: limit lower=-3.1067 upper=3.1067 effort=18 velocity=3.141592653589793 -> lower=-2.9321531433504737 upper=2.9321531433504737 effort=18 velocity=3.141592653589793
- joint right_joint5: limit lower=-3.1067 upper=3.1067 effort=18 velocity=3.141592653589793 -> lower=-2.9321531433504737 upper=2.9321531433504737 effort=18 velocity=3.141592653589793

File: m6_ccs_description/xacro/arm.xacro (robot description, xacro)
@@ -1,6 +1,8 @@
 <?xml version="1.0"?>
 <robot xmlns:xacro="http://www.ros.org/wiki/xacro">
+	<xacro:arg name="collider" default="convex"/>
 	<xacro:property name="PI" value="3.1415926535897931"/>
-	<xacro:macro name="M6_CCS" params="name:='' direction:=1 collider:=convex">
+	<xacro:property name="collider_type" value="$(arg collider)"/>
+	<xacro:macro name="M6_CCS" params="name:='' direction:=1">
 		<xacro:property name="prefix" value="${name + '_' if name else ''}"/>
 		<!-- Base Link -->
@@ -18,5 +20,5 @@
 				</geometry>
 			</visual>
-			<xacro:if value="${collider == 'convex'}">
+			<xacro:if value="${collider_type == 'convex'}">
 				<collision>
 					<geometry>
@@ -25,5 +27,5 @@
 				</collision>
 			</xacro:if>
-			<xacro:if value="${collider == 'simple'}">
+			<xacro:if value="${collider_type == 'simple'}">
 				<collision>
 					<origin xyz="0 0 0.041832"/>
@@ -48,5 +50,5 @@
 				</geometry>
 			</visual>
-			<xacro:if value="${collider == 'convex'}">
+			<xacro:if value="${collider_type == 'convex'}">
 				<collision>
 					<geometry>
@@ -55,5 +57,5 @@
 				</collision>
 			</xacro:if>
-			<xacro:if value="${collider == 'simple'}">
+			<xacro:if value="${collider_type == 'simple'}">
 				<collision>
 					<origin rpy="${PI/2} 0 0"/>
@@ -86,5 +88,5 @@
 				</geometry>
 			</visual>
-			<xacro:if value="${collider == 'convex'}">
+			<xacro:if value="${collider_type == 'convex'}">
 				<collision>
 					<geometry>
@@ -93,5 +95,5 @@
 				</collision>
 			</xacro:if>
-			<xacro:if value="${collider == 'simple'}">
+			<xacro:if value="${collider_type == 'simple'}">
 				<collision>
 					<origin xyz="0 0.099087 0" rpy="${PI/2} 0 0"/>
@@ -124,5 +126,5 @@
 				</geometry>
 			</visual>
-			<xacro:if value="${collider == 'convex'}">
+			<xacro:if value="${collider_type == 'convex'}">
 				<collision>
 					<geometry>
@@ -131,5 +133,5 @@
 				</collision>
 			</xacro:if>
-			<xacro:if value="${collider == 'simple'}">
+			<xacro:if value="${collider_type == 'simple'}">
 				<collision>
 					<origin xyz="0 0 -0.098932"/>
@@ -168,5 +170,5 @@
 				</geometry>
 			</visual>
-			<xacro:if value="${collider == 'convex'}">
+			<xacro:if value="${collider_type == 'convex'}">
 				<collision>
 					<geometry>
@@ -175,5 +177,5 @@
 				</collision>
 			</xacro:if>
-			<xacro:if value="${collider == 'simple'}">
+			<xacro:if value="${collider_type == 'simple'}">
 				<collision>
 					<origin xyz="0.017721 -0.079733 0" rpy="${PI/2} 0 0"/>
@@ -206,5 +208,5 @@
 				</geometry>
 			</visual>
-			<xacro:if value="${collider == 'convex'}">
+			<xacro:if value="${collider_type == 'convex'}">
 				<collision>
 					<geometry>
@@ -213,5 +215,5 @@
 				</collision>
 			</xacro:if>
-			<xacro:if value="${collider == 'simple'}">
+			<xacro:if value="${collider_type == 'simple'}">
 				<collision>
 					<origin xyz="0 0 -0.117153"/>
@@ -244,5 +246,5 @@
 				</geometry>
 			</visual>
-			<xacro:if value="${collider == 'convex'}">
+			<xacro:if value="${collider_type == 'convex'}">
 				<collision>
 					<geometry>
@@ -251,5 +253,5 @@
 				</collision>
 			</xacro:if>
-			<xacro:if value="${collider == 'simple'}">
+			<xacro:if value="${collider_type == 'simple'}">
 				<collision>
 					<origin rpy="${PI/2} 0 0"/>
@@ -287,5 +289,5 @@
 				</geometry>
 			</visual>
-			<xacro:if value="${collider == 'convex'}">
+			<xacro:if value="${collider_type == 'convex'}">
 				<collision>
 					<geometry>
@@ -294,5 +296,5 @@
 				</collision>
 			</xacro:if>
-			<xacro:if value="${collider == 'simple'}">
+			<xacro:if value="${collider_type == 'simple'}">
 				<collision>
 					<origin xyz="0 -0.075732 0" rpy="${PI/2} 0 0"/>
@@ -301,4 +303,32 @@
 					</geometry>
 				</collision>
+				<xacro:if value="${selected_gripper_type == 'rg75'}">
+					<collision>
+						<origin xyz="0 -0.175732 0" rpy="${PI/2} 0 0"/>
+						<geometry>
+							<cylinder length="0.138392" radius="0.05"/>
+						</geometry>
+					</collision>
+					<collision>
+						<origin xyz="0 -0.28 0" rpy="${PI/2} 0 0"/>
+						<geometry>
+							<cylinder length="0.08" radius="0.021707"/>
+						</geometry>
+					</collision>
+				</xacro:if>
+				<xacro:if value="${selected_gripper_type == 'ag2f90_c' or selected_gripper_type == 'ag2f90_d'}">
+					<collision>
+						<origin xyz="0 -0.175732 0" rpy="${PI/2} 0 0"/>
+						<geometry>
+							<cylinder length="0.138392" radius="0.041707"/>
+						</geometry>
+					</collision>
+					<collision>
+						<origin xyz="0 -0.28 0" rpy="${PI/2} 0 0"/>
+						<geometry>
+							<cylinder length="0.08" radius="0.021707"/>
+						</geometry>
+					</collision>
+				</xacro:if>
 			</xacro:if>
 		</link>

File: m6_ccs_description/xacro/robot.xacro (robot description, xacro)
@@ -2,5 +2,5 @@
 <robot name="M6_CCS" xmlns:xacro="http://www.ros.org/wiki/xacro">
 	<xacro:arg name="collider" default="convex"/>
-	<xacro:arg name="type" default="left"/>
+	<xacro:arg name="type" default="dual"/>
 	<xacro:arg name="scene" default=""/>
 	<!-- 从 type 参数解析出 arm_config、gripper_type 和 scene -->
@@ -16,8 +16,4 @@
 		<xacro:property name="selected_arm_config" value="left"/>
 	</xacro:if>
-	<xacro:if value="${type_arg == 'rg75'}">
-		<xacro:property name="selected_arm_config" value="left"/>
-		<xacro:property name="selected_gripper_type" value="rg75"/>
-	</xacro:if>
 	<xacro:if value="${type_arg == 'right'}">
 		<xacro:property name="selected_arm_config" value="right"/>
@@ -30,25 +26,21 @@
 	<!-- 双臂配置 -->
 	<!-- 适用于人形机器人的配置 -->
-	<xacro:if value="${type_arg == 'dual_ag2f90'}">
-		<xacro:property name="selected_gripper_type" value="ag2f90d"/>
-	</xacro:if>
-	<xacro:if value="${type_arg == 'dual_ag2f90_c'}">
+	<xacro:if value="${type_arg == 'ag2f90'}">
+		<xacro:property name="selected_gripper_type" value="ag2f90_d"/>
+	</xacro:if>
+	<xacro:if value="${type_arg == 'ag2f90_c'}">
 		<xacro:property name="selected_gripper_type" value="ag2f90_c"/>
 	</xacro:if>
-	<xacro:if value="${type_arg == 'dual_ag2f90_d'}">
+	<xacro:if value="${type_arg == 'ag2f90_d'}">
 		<xacro:property name="selected_gripper_type" value="ag2f90_d"/>
 	</xacro:if>
+	<xacro:if value="${type_arg == 'rg75'}">
+		<xacro:property name="selected_gripper_type" value="rg75"/>
+	</xacro:if>
 	<!-- 适用纯双臂演示场景的配置 -->
-	<xacro:if value="${type_arg == 'dual_rg75'}">
-		<xacro:property name="selected_gripper_type" value="rg75"/>
-	</xacro:if>
-	<xacro:if value="${type_arg == 'dual_desktop'}">
+	<xacro:if value="${type_arg == 'desktop'}">
 		<xacro:property name="selected_scene" value="desktop"/>
 	</xacro:if>
-	<xacro:if value="${type_arg == 'dual_desktop_90c'}">
-		<xacro:property name="selected_scene" value="desktop"/>
-		<xacro:property name="selected_gripper_type" value="ag2f90_c"/>
-	</xacro:if>
-	<xacro:if value="${type_arg == 'dual_desktop_90c_soft'}">
+	<xacro:if value="${type_arg == 'desktop_90c'}">
 		<xacro:property name="selected_scene" value="desktop"/>
 		<xacro:property name="selected_gripper_type" value="ag2f90_c"/>
@@ -58,5 +50,5 @@
 	<!-- 单左臂（不包括 usb-90c 场景） -->
 	<xacro:if value="${selected_arm_config == 'left' and selected_scene != 'usb-90c'}">
-		<xacro:M6_CCS collider="$(arg collider)"/>
+		<xacro:M6_CCS/>
 		<xacro:if value="${selected_gripper_type == 'rg75'}">
 			<xacro:include filename="$(find jodell_description)/xacro/RG75-300.xacro"/>
@@ -70,5 +62,5 @@
 	<!-- 单右臂 -->
 	<xacro:if value="${selected_arm_config == 'right'}">
-		<xacro:M6_CCS direction="-1" collider="$(arg collider)"/>
+		<xacro:M6_CCS direction="-1"/>
 	</xacro:if>
 	<!-- 双臂配置 -->
@@ -148,6 +140,6 @@
 		</xacro:unless>
 		<!-- 双臂和末端执行器（两种场景共用） -->
-		<xacro:M6_CCS name="left" collider="$(arg collider)"/>
-		<xacro:M6_CCS name="right" direction="-1" collider="$(arg collider)"/>
+		<xacro:M6_CCS name="left"/>
+		<xacro:M6_CCS name="right" direction="-1"/>
 		<!-- 双臂末端执行器 -->
 		<xacro:if value="${selected_gripper_type == 'ag2f90_c' or selected_gripper_type == 'ag2f90_d'}">
@@ -207,5 +199,5 @@
 			<origin rpy="-${PI/2} 0 0" xyz="0.0 0.12 0.701"/>
 		</joint>
-		<xacro:M6_CCS name="left" collider="$(arg collider)"/>
+		<xacro:M6_CCS name="left"/>
 		<xacro:include filename="$(find changingtek_description)/xacro/AG2F90-C.xacro"/>
 		<xacro:AG2F90-C name="" use_flange="true"/>
