Commit message: modified hardware param

File: m6_ccs_description/urdf/m6_ccs.urdf (robot description, URDF)
Before this commit: robot M6_CCS, 22 links, 21 joints
Joints:
- joint left_joint7: limit lower=-1.361356816555577 upper=1.361356816555577 effort=18 velocity=3.141592653589793 -> lower=-0.661356816555577 upper=0.661356816555577 effort=18 velocity=3.141592653589793
- joint right_joint7: limit lower=-1.361356816555577 upper=1.361356816555577 effort=18 velocity=3.141592653589793 -> lower=-0.661356816555577 upper=0.661356816555577 effort=18 velocity=3.141592653589793

File: m6_ccs_description/xacro/ros2_control/robot.xacro (robot description, xacro)
@@ -32,6 +32,6 @@
 				<param name="arm_type">${selected_arm_config}</param>
 				<param name="gripper_type">${selected_gripper_type}</param>
-				<param name="max_joint_speed">50</param>
-				<param name="max_joint_acceleration">30</param>
+				<param name="max_joint_speed">100</param>
+				<param name="max_joint_acceleration">100</param>
 				<xacro:if value="${selected_scene == 'desktop'}">
 					<param name="device_ip">192.168.10.190</param>
