Commit message: modified ocs2 dual arm param for tianji

File: m6_ccs_description/urdf/m6_ccs_ag2f90.urdf (robot description, URDF)
Before this commit: robot M6_CCS, 46 links, 45 joints
Joints:
- joint left_joint6: limit lower=-1.0122909661567112 upper=1.0122909661567112 effort=18 velocity=3.141592653589793 -> lower=-0.5 upper=0.5 effort=18 velocity=3.141592653589793
- joint right_joint6: limit lower=-1.0122909661567112 upper=1.0122909661567112 effort=18 velocity=3.141592653589793 -> lower=-0.5 upper=0.5 effort=18 velocity=3.141592653589793

Commit message: modified ocs2 dual arm param for tianji

File: m6_ccs_description/urdf/m6_ccs_ag2f90.urdf (robot description, URDF)
Before this commit: robot M6_CCS, 46 links, 45 joints
Joints:
- joint left_joint6: limit lower=-0.5 upper=0.5 effort=18 velocity=3.141592653589793 -> lower=-0.8 upper=0.8 effort=18 velocity=3.141592653589793
- joint right_joint6: limit lower=-0.5 upper=0.5 effort=18 velocity=3.141592653589793 -> lower=-0.8 upper=0.8 effort=18 velocity=3.141592653589793
