Commit message: Add chain controller interface for admittance control

File: m6_ccs_description/xacro/ros2_control/interfaces.xacro (robot description, xacro)
@@ -47,3 +47,14 @@
 		</joint>
 	</xacro:macro>
+	<!-- Force-torque sensor semantic-component interfaces -->
+	<xacro:macro name="m6_ft_sensor_interfaces" params="sensor_name">
+		<sensor name="${sensor_name}">
+			<state_interface name="force.x"/>
+			<state_interface name="force.y"/>
+			<state_interface name="force.z"/>
+			<state_interface name="torque.x"/>
+			<state_interface name="torque.y"/>
+			<state_interface name="torque.z"/>
+		</sensor>
+	</xacro:macro>
 </robot>

File: m6_ccs_description/xacro/ros2_control/robot.xacro (robot description, xacro)
@@ -34,4 +34,8 @@
 				<param name="max_joint_speed">50</param>
 				<param name="max_joint_acceleration">30</param>
+				<!-- Virtual FT sensor wrench topics (geometry_msgs/WrenchStamped) -->
+				<!-- dual-arm -->
+				<param name="left_wrench_topic">/left_arm_external_wrench</param>
+				<param name="right_wrench_topic">/right_arm_external_wrench</param>
 				<xacro:if value="${selected_scene == 'desktop'}">
 					<param name="device_ip">192.168.10.190</param>
@@ -51,4 +55,7 @@
 			<xacro:m6_interfaces name="left"/>
 			<xacro:m6_interfaces name="right"/>
+			<!-- Virtual FT sensors (wrench estimated from joint external torques) -->
+			<xacro:m6_ft_sensor_interfaces sensor_name="left_ft_sensor"/>
+			<xacro:m6_ft_sensor_interfaces sensor_name="right_ft_sensor"/>
 			<xacro:if value="${selected_gripper_type == 'ag2f90_c' or selected_gripper_type == 'ag2f90_d'}">
 				<xacro:include filename="$(find changingtek_description)/xacro/ros2_control/AG2F90-C.xacro"/>
@@ -71,4 +78,5 @@
 					<xacro:m6_interfaces name=""/>
 				</xacro:unless>
+				<xacro:m6_ft_sensor_interfaces sensor_name="ft_sensor"/>
 				<xacro:if value="${selected_gripper_type == 'ag2f90_c' or selected_gripper_type == 'ag2f90_d'}">
 					<xacro:include filename="$(find changingtek_description)/xacro/ros2_control/AG2F90-C.xacro"/>
