Commit message: update hardware configuration and drive type specifications in README and Xacro files

File: m6_ccs_description/xacro/ros2_control/robot.xacro (robot description, xacro)
@@ -7,6 +7,6 @@
 	<xacro:arg name="left_ee_drive_type" default=""/>
 	<xacro:arg name="right_ee_drive_type" default=""/>
-	<xacro:property name="is_real_hardware" value="${'$(arg ros2_control_hardware_type)' == 'real' or '$(arg ros2_control_hardware_type)' == 'real_usb'}"/>
-	<xacro:property name="ee_drive_type" value="${'usb' if '$(arg ros2_control_hardware_type)' == 'real_usb' else ('marvin' if '$(arg ros2_control_hardware_type)' == 'real' else '')}"/>
+	<xacro:property name="is_real_hardware" value="${'$(arg ros2_control_hardware_type)' == 'real'}"/>
+	<xacro:property name="ee_drive_type" value="${'marvin' if is_real_hardware else ''}"/>
 	<xacro:property name="left_drive_type" value="${'$(arg left_ee_drive_type)' if '$(arg left_ee_drive_type)' != '' else ee_drive_type}"/>
 	<xacro:property name="right_drive_type" value="${'$(arg right_ee_drive_type)' if '$(arg right_ee_drive_type)' != '' else ee_drive_type}"/>

File: marvin_pro_description/xacro/ros2_control/robot.xacro (robot description, xacro)
@@ -14,5 +14,5 @@
   <xacro:include filename="$(find robot_common_launch)/xacro/ros2_control/simulation_hardware.xacro"/>
   <xacro:include filename="$(find m6_ccs_description)/xacro/ros2_control/end_effector_interfaces.xacro"/>
-  <xacro:property name="is_real_hardware" value="${'$(arg ros2_control_hardware_type)' == 'real' or '$(arg ros2_control_hardware_type)' == 'real_usb'}"/>
+  <xacro:property name="is_real_hardware" value="${'$(arg ros2_control_hardware_type)' == 'real'}"/>
   <xacro:property name="ee_block_mode" value="${'real' if is_real_hardware else 'sim'}"/>
   <ros2_control name="Marvin_Pro_System" type="system">
