Commit message: 增加kwr75传感器的485模式

File: m6_ccs_description/xacro/ros2_control/external_ee_systems.xacro (robot description, xacro)
@@ -20,7 +20,5 @@
 	<xacro:macro name="external_ee_systems" params="
 		usb_left_port:=/dev/ttyUSB0
-		usb_right_port:=/dev/ttyUSB2
-		usb_left_ft_port:=/dev/ttyUSB1
-		usb_right_ft_port:=/dev/ttyUSB3">
+		usb_right_port:=/dev/ttyUSB2">
 		<xacro:if value="${left_drive_type == 'usb' and (left_hand_type == 'linkerhand_o6' or left_hand_type == 'linkerhand_l6' or left_hand_type == 'linkerhand_o7')}">
 			<xacro:side_usb_hand_system side="left" hand_type="${left_hand_type}" serial_port="${usb_left_port}"/>
@@ -78,6 +76,7 @@
 		</xacro:if>
 		<xacro:ft_sensor_systems
-			usb_left_ft_port="${usb_left_ft_port}"
-			usb_right_ft_port="${usb_right_ft_port}"/>
+			kwr75_ft_mode="$(arg kwr75_ft_mode)"
+			usb_left_ft_port="$(arg usb_left_ft_port)"
+			usb_right_ft_port="$(arg usb_right_ft_port)"/>
 	</xacro:macro>
 </robot>

File: m6_ccs_description/xacro/ros2_control/ft_sensor_systems.xacro (robot description, xacro)
@@ -4,7 +4,9 @@
 		<xacro:if value="${side == 'left'}">
 			<xacro:property name="wrench_topic" value="/left_arm_external_wrench"/>
+			<xacro:property name="ee_frame_id" value="left_eef"/>
 		</xacro:if>
 		<xacro:unless value="${side == 'left'}">
 			<xacro:property name="wrench_topic" value="/right_arm_external_wrench"/>
+			<xacro:property name="ee_frame_id" value="right_eef"/>
 		</xacro:unless>
 		<ros2_control name="kwr75_${side}_ft_system" type="sensor">
@@ -13,4 +15,5 @@
 				<param name="serial_port">${serial_port}</param>
 				<param name="wrench_topic">${wrench_topic}</param>
+				<param name="frame_id">${ee_frame_id}</param>
 			</hardware>
 			<sensor name="kwr75_${side}_ft">
@@ -25,11 +28,14 @@
 	</xacro:macro>
 	<xacro:macro name="ft_sensor_systems" params="
+		kwr75_ft_mode:=none
 		usb_left_ft_port:=/dev/ttyUSB1
 		usb_right_ft_port:=/dev/ttyUSB3">
-		<xacro:if value="${selected_arm_config == 'dual' or selected_arm_config == 'left'}">
-			<xacro:side_kwr75_ft_sensor side="left" serial_port="${usb_left_ft_port}"/>
-		</xacro:if>
-		<xacro:if value="${selected_arm_config == 'dual' or selected_arm_config == 'right'}">
-			<xacro:side_kwr75_ft_sensor side="right" serial_port="${usb_right_ft_port}"/>
+		<xacro:if value="${kwr75_ft_mode == 'usb'}">
+			<xacro:if value="${selected_arm_config == 'dual' or selected_arm_config == 'left'}">
+				<xacro:side_kwr75_ft_sensor side="left" serial_port="${usb_left_ft_port}"/>
+			</xacro:if>
+			<xacro:if value="${selected_arm_config == 'dual' or selected_arm_config == 'right'}">
+				<xacro:side_kwr75_ft_sensor side="right" serial_port="${usb_right_ft_port}"/>
+			</xacro:if>
 		</xacro:if>
 	</xacro:macro>

File: m6_ccs_description/xacro/ros2_control/marvin_hardware.xacro (robot description, xacro)
@@ -2,4 +2,10 @@
 <robot xmlns:xacro="http://www.ros.org/wiki/xacro">
 	<xacro:include filename="$(find m6_ccs_description)/xacro/eefs.xacro"/>
+	<!-- KWR75: launch profile hardware.* maps here; shared by m6_ccs and fa-w2 -->
+	<xacro:arg name="kwr75_ft_mode" default="none"/>
+	<xacro:arg name="left_ft_channel" default="3"/>
+	<xacro:arg name="right_ft_channel" default="3"/>
+	<xacro:arg name="usb_left_ft_port" default="/dev/ttyUSB1"/>
+	<xacro:arg name="usb_right_ft_port" default="/dev/ttyUSB3"/>
 	<!-- arm_type: dual | left | right -->
 	<xacro:macro name="marvin_hardware_block" params="
@@ -14,4 +20,12 @@
 		<plugin>marvin_ros2_control/MarvinHardware</plugin>
 		<param name="arm_type">${arm_type}</param>
+		<xacro:if value="${'$(arg kwr75_ft_mode)' == '485'}">
+			<param name="kwr75_ft_enabled">true</param>
+			<param name="left_ft_channel">$(arg left_ft_channel)</param>
+			<param name="right_ft_channel">$(arg right_ft_channel)</param>
+			<param name="left_ft_frame_id">left_eef</param>
+			<param name="right_ft_frame_id">right_eef</param>
+			<param name="use_async_tool_comm">true</param>
+		</xacro:if>
 		<xacro:if value="${arm_type == 'dual'}">
 			<xacro:property name="left_ee_type" value="${left_hand_type if left_hand_type != '' else left_gripper_type}"/>

File: m6_ccs_description/xacro/ros2_control/robot.xacro (robot description, xacro)
@@ -17,6 +17,4 @@
 	<xacro:arg name="usb_left_port" default="/dev/ttyUSB0"/>
 	<xacro:arg name="usb_right_port" default="/dev/ttyUSB2"/>
-	<xacro:arg name="usb_left_ft_port" default="/dev/ttyUSB1"/>
-	<xacro:arg name="usb_right_ft_port" default="/dev/ttyUSB3"/>
 	<link name="world"/>
 	<joint name="world_fixed" type="fixed">
@@ -63,10 +61,9 @@
 		<xacro:external_ee_systems
 			usb_left_port="$(arg usb_left_port)"
-			usb_right_port="$(arg usb_right_port)"
-			usb_left_ft_port="$(arg usb_left_ft_port)"
-			usb_right_ft_port="$(arg usb_right_ft_port)"/>
+			usb_right_port="$(arg usb_right_port)"/>
 	</xacro:if>
 	<xacro:if value="${is_real_hardware and selected_arm_config != 'dual'}">
 		<xacro:ft_sensor_systems
+			kwr75_ft_mode="$(arg kwr75_ft_mode)"
 			usb_left_ft_port="$(arg usb_left_ft_port)"
 			usb_right_ft_port="$(arg usb_right_ft_port)"/>

Commit message: 不再hardware_interface继续发布力矩传感器topic,改由ft_sensor_broadcaster在上层读取发布 (#13)

File: m6_ccs_description/xacro/ros2_control/external_ee_systems.xacro (robot description, xacro)
@@ -39,6 +39,5 @@
 		right_ft:=$(arg right_ft)
 		usb_left_ft_port:=$(arg usb_left_ft_port)
-		usb_right_ft_port:=$(arg usb_right_ft_port)
-		arm_config:=dual">
+		usb_right_ft_port:=$(arg usb_right_ft_port)">
 		<xacro:if value="${left_drive_type == 'usb' and (left_hand_type == 'linkerhand_o6' or left_hand_type == 'linkerhand_l6' or left_hand_type == 'linkerhand_o7')}">
 			<xacro:side_usb_hand_system side="left" hand_type="${left_hand_type}" serial_port="${usb_left_port}"/>
@@ -105,6 +104,5 @@
 			right_ft="${right_ft}"
 			usb_left_ft_port="${usb_left_ft_port}"
-			usb_right_ft_port="${usb_right_ft_port}"
-			arm_config="${arm_config}"/>
+			usb_right_ft_port="${usb_right_ft_port}"/>
 	</xacro:macro>
 </robot>

File: m6_ccs_description/xacro/ros2_control/ft_sensor_systems.xacro (robot description, xacro)
@@ -1,21 +1,18 @@
 <?xml version="1.0"?>
 <robot xmlns:xacro="http://www.ros.org/wiki/xacro">
-	<xacro:macro name="side_kwr75_ft_sensor" params="side serial_port">
-		<xacro:if value="${side == 'left'}">
-			<xacro:property name="wrench_topic" value="/left_arm_external_wrench"/>
-			<xacro:property name="ee_frame_id" value="left_eef"/>
-		</xacro:if>
-		<xacro:unless value="${side == 'left'}">
-			<xacro:property name="wrench_topic" value="/right_arm_external_wrench"/>
-			<xacro:property name="ee_frame_id" value="right_eef"/>
-		</xacro:unless>
-		<ros2_control name="kwr75_${side}_ft_system" type="sensor">
+	<!--
+		Generic FT sensor system (type=sensor, independent of Marvin).
+		robot.local.yaml left_ft/right_ft value selects the transport:
+		  kwr75_usb → this block,  kwr75_485 → Marvin built-in.
+		Exports left_ft_sensor / right_ft_sensor — same names regardless
+		of transport, so controllers/broadcasters only need one config.
+	-->
+	<xacro:macro name="side_ft_sensor_system" params="side serial_port">
+		<ros2_control name="${side}_ft_system" type="sensor">
 			<hardware>
 				<plugin>modbus_ros2_control/Kwr75ForceTorqueSensor</plugin>
 				<param name="serial_port">${serial_port}</param>
-				<param name="wrench_topic">${wrench_topic}</param>
-				<param name="frame_id">${ee_frame_id}</param>
 			</hardware>
-			<sensor name="kwr75_${side}_ft">
+			<sensor name="${side}_ft_sensor">
 				<state_interface name="force.x"/>
 				<state_interface name="force.y"/>
@@ -31,11 +28,10 @@
 		right_ft:=$(arg right_ft)
 		usb_left_ft_port:=$(arg usb_left_ft_port)
-		usb_right_ft_port:=$(arg usb_right_ft_port)
-		arm_config:=dual">
-		<xacro:if value="${(arm_config == 'dual' or arm_config == 'left') and left_ft == 'kwr75_usb'}">
-			<xacro:side_kwr75_ft_sensor side="left" serial_port="${usb_left_ft_port}"/>
+		usb_right_ft_port:=$(arg usb_right_ft_port)">
+		<xacro:if value="${left_ft == 'kwr75_usb'}">
+			<xacro:side_ft_sensor_system side="left" serial_port="${usb_left_ft_port}"/>
 		</xacro:if>
-		<xacro:if value="${(arm_config == 'dual' or arm_config == 'right') and right_ft == 'kwr75_usb'}">
-			<xacro:side_kwr75_ft_sensor side="right" serial_port="${usb_right_ft_port}"/>
+		<xacro:if value="${right_ft == 'kwr75_usb'}">
+			<xacro:side_ft_sensor_system side="right" serial_port="${usb_right_ft_port}"/>
 		</xacro:if>
 	</xacro:macro>

File: m6_ccs_description/xacro/ros2_control/marvin_hardware.xacro (robot description, xacro)
@@ -73,3 +73,31 @@
 		</xacro:if>
 	</xacro:macro>
+	<!--
+		KWR75 FT state interfaces within the Marvin ros2_control block.
+		Only declared for kwr75_485 (COM2 RS485); kwr75_usb uses a separate
+		SensorInterface that exports the same names (see ft_sensor_systems.xacro).
+		Only dual-arm supported on this platform.
+	-->
+	<xacro:macro name="marvin_ft_sensor_interfaces" params="">
+		<xacro:if value="${'$(arg left_ft)' == 'kwr75_485'}">
+			<sensor name="left_ft_sensor">
+				<state_interface name="force.x"/>
+				<state_interface name="force.y"/>
+				<state_interface name="force.z"/>
+				<state_interface name="torque.x"/>
+				<state_interface name="torque.y"/>
+				<state_interface name="torque.z"/>
+			</sensor>
+		</xacro:if>
+		<xacro:if value="${'$(arg right_ft)' == 'kwr75_485'}">
+			<sensor name="right_ft_sensor">
+				<state_interface name="force.x"/>
+				<state_interface name="force.y"/>
+				<state_interface name="force.z"/>
+				<state_interface name="torque.x"/>
+				<state_interface name="torque.y"/>
+				<state_interface name="torque.z"/>
+			</sensor>
+		</xacro:if>
+	</xacro:macro>
 </robot>

File: m6_ccs_description/xacro/ros2_control/robot.xacro (robot description, xacro)
@@ -58,14 +58,10 @@
 			</xacro:if>
 		</xacro:unless>
+		<xacro:marvin_ft_sensor_interfaces/>
 	</ros2_control>
 	<xacro:if value="${is_real_hardware and selected_arm_config == 'dual'}">
 		<xacro:external_ee_systems
 			usb_left_port="$(arg usb_left_port)"
-			usb_right_port="$(arg usb_right_port)"
-			arm_config="${selected_arm_config}"/>
-	</xacro:if>
-	<xacro:if value="${is_real_hardware and selected_arm_config != 'dual'}">
-		<xacro:ft_sensor_systems
-			arm_config="${selected_arm_config}"/>
+			usb_right_port="$(arg usb_right_port)"/>
 	</xacro:if>
 	<xacro:arg name="gazebo" default="false"/>

Commit message: Add support for LinkerHand O6 in USB CAN configuration

File: m6_ccs_description/xacro/ros2_control/external_ee_systems.xacro (robot description, xacro)
@@ -31,4 +31,17 @@
 		</ros2_control>
 	</xacro:macro>
+	<xacro:macro name="o6_usb_can_side_system" params="side can_interface">
+		<ros2_control name="linkerhand_o6_${side}_can_system" type="system">
+			<hardware>
+				<plugin>can_ros2_control/O6CanHardware</plugin>
+				<param name="can_interface">${can_interface}</param>
+				<param name="hand_side">${side}</param>
+				<param name="hand_type">linkerhand_o6</param>
+				<param name="${side}_tool_torque">1.0</param>
+				<param name="${side}_tool_velocity">1.0</param>
+			</hardware>
+			<xacro:side_hand_interfaces side="${side}" hand_type="linkerhand_o6"/>
+		</ros2_control>
+	</xacro:macro>
 	<!-- left_ft / right_ft / usb_*_ft_port: declared in marvin_hardware.xacro; defaults read $(arg ...) here. -->
 	<xacro:macro name="external_ee_systems" params="
@@ -40,4 +53,10 @@
 		usb_left_ft_port:=$(arg usb_left_ft_port)
 		usb_right_ft_port:=$(arg usb_right_ft_port)">
+		<xacro:if value="${left_drive_type == 'usb_can' and left_hand_type == 'linkerhand_o6'}">
+			<xacro:o6_usb_can_side_system side="left" can_interface="can0"/>
+		</xacro:if>
+		<xacro:if value="${right_drive_type == 'usb_can' and right_hand_type == 'linkerhand_o6'}">
+			<xacro:o6_usb_can_side_system side="right" can_interface="can1"/>
+		</xacro:if>
 		<xacro:if value="${left_drive_type == 'usb' and (left_hand_type == 'linkerhand_o6' or left_hand_type == 'linkerhand_l6' or left_hand_type == 'linkerhand_o7')}">
 			<xacro:side_usb_hand_system side="left" hand_type="${left_hand_type}" serial_port="${usb_left_port}"/>

Commit message: Enhance LinkerHand support in USB CAN configuration and external systems integration

File: m6_ccs_description/xacro/ros2_control/external_ee_systems.xacro (robot description, xacro)
@@ -31,15 +31,24 @@
 		</ros2_control>
 	</xacro:macro>
-	<xacro:macro name="o6_usb_can_side_system" params="side can_interface">
-		<ros2_control name="linkerhand_o6_${side}_can_system" type="system">
+	<xacro:macro name="linkerhand_usb_can_side_system" params="side hand_type can_interface read_tactile:=false">
+		<ros2_control name="${hand_type}_${side}_can_system" type="system">
 			<hardware>
-				<plugin>can_ros2_control/O6CanHardware</plugin>
+				<xacro:if value="${hand_type == 'linkerhand_o6'}">
+					<plugin>can_ros2_control/O6CanHardware</plugin>
+				</xacro:if>
+				<xacro:if value="${hand_type == 'linkerhand_l6'}">
+					<plugin>can_ros2_control/L6CanHardware</plugin>
+				</xacro:if>
+				<xacro:if value="${hand_type == 'linkerhand_o7'}">
+					<plugin>can_ros2_control/O7CanHardware</plugin>
+				</xacro:if>
 				<param name="can_interface">${can_interface}</param>
 				<param name="hand_side">${side}</param>
-				<param name="hand_type">linkerhand_o6</param>
+				<param name="read_feedback">true</param>
+				<param name="read_tactile">${read_tactile}</param>
 				<param name="${side}_tool_torque">1.0</param>
 				<param name="${side}_tool_velocity">1.0</param>
 			</hardware>
-			<xacro:side_hand_interfaces side="${side}" hand_type="linkerhand_o6"/>
+			<xacro:side_hand_interfaces side="${side}" hand_type="${hand_type}"/>
 		</ros2_control>
 	</xacro:macro>
@@ -48,4 +57,8 @@
 		usb_left_port:=/dev/ttyUSB0
 		usb_right_port:=/dev/ttyUSB2
+		left_ee_can_interface:=can0
+		right_ee_can_interface:=can1
+		left_read_tactile:=false
+		right_read_tactile:=false
 		usb_baudrate:=115200
 		left_ft:=$(arg left_ft)
@@ -53,9 +66,9 @@
 		usb_left_ft_port:=$(arg usb_left_ft_port)
 		usb_right_ft_port:=$(arg usb_right_ft_port)">
-		<xacro:if value="${left_drive_type == 'usb_can' and left_hand_type == 'linkerhand_o6'}">
-			<xacro:o6_usb_can_side_system side="left" can_interface="can0"/>
+		<xacro:if value="${left_drive_type == 'usb_can' and (left_hand_type == 'linkerhand_o6' or left_hand_type == 'linkerhand_l6' or left_hand_type == 'linkerhand_o7')}">
+			<xacro:linkerhand_usb_can_side_system side="left" hand_type="${left_hand_type}" can_interface="${left_ee_can_interface}" read_tactile="${left_read_tactile}"/>
 		</xacro:if>
-		<xacro:if value="${right_drive_type == 'usb_can' and right_hand_type == 'linkerhand_o6'}">
-			<xacro:o6_usb_can_side_system side="right" can_interface="can1"/>
+		<xacro:if value="${right_drive_type == 'usb_can' and (right_hand_type == 'linkerhand_o6' or right_hand_type == 'linkerhand_l6' or right_hand_type == 'linkerhand_o7')}">
+			<xacro:linkerhand_usb_can_side_system side="right" hand_type="${right_hand_type}" can_interface="${right_ee_can_interface}" read_tactile="${right_read_tactile}"/>
 		</xacro:if>
 		<xacro:if value="${left_drive_type == 'usb' and (left_hand_type == 'linkerhand_o6' or left_hand_type == 'linkerhand_l6' or left_hand_type == 'linkerhand_o7')}">
@@ -102,20 +115,20 @@
 		</xacro:if>
 		<xacro:if value="${left_drive_type == 'usb_can' and left_hand_type == 'freedom_v1'}">
-			<xacro:freedom_can_side_system side="left" can_interface="can0" device_id="0"/>
+			<xacro:freedom_can_side_system side="left" can_interface="${left_ee_can_interface}" device_id="0"/>
 		</xacro:if>
 		<xacro:if value="${right_drive_type == 'usb_can' and right_hand_type == 'freedom_v1'}">
-			<xacro:freedom_can_side_system side="right" can_interface="can1" device_id="1"/>
+			<xacro:freedom_can_side_system side="right" can_interface="${right_ee_can_interface}" device_id="1"/>
 		</xacro:if>
 		<xacro:if value="${left_drive_type == 'usb_can' and left_hand_type == 'inspire_e2'}">
-			<xacro:inspire_canfd_side_system side="left" can_interface="can0"/>
+			<xacro:inspire_canfd_side_system side="left" can_interface="${left_ee_can_interface}"/>
 		</xacro:if>
 		<xacro:if value="${right_drive_type == 'usb_can' and right_hand_type == 'inspire_e2'}">
-			<xacro:inspire_canfd_side_system side="right" can_interface="can1"/>
+			<xacro:inspire_canfd_side_system side="right" can_interface="${right_ee_can_interface}"/>
 		</xacro:if>
 		<xacro:if value="${left_drive_type == 'usb_can' and left_hand_type == 'inspire_f2'}">
-			<xacro:inspire_canfd_side_system side="left" can_interface="can0" hand_type="inspire_f2"/>
+			<xacro:inspire_canfd_side_system side="left" can_interface="${left_ee_can_interface}" hand_type="inspire_f2"/>
 		</xacro:if>
 		<xacro:if value="${right_drive_type == 'usb_can' and right_hand_type == 'inspire_f2'}">
-			<xacro:inspire_canfd_side_system side="right" can_interface="can1" hand_type="inspire_f2"/>
+			<xacro:inspire_canfd_side_system side="right" can_interface="${right_ee_can_interface}" hand_type="inspire_f2"/>
 		</xacro:if>
 		<xacro:ft_sensor_systems

File: m6_ccs_description/xacro/ros2_control/robot.xacro (robot description, xacro)
@@ -17,4 +17,8 @@
 	<xacro:arg name="usb_left_port" default="/dev/ttyUSB0"/>
 	<xacro:arg name="usb_right_port" default="/dev/ttyUSB2"/>
+	<xacro:arg name="left_ee_can_interface" default="can0"/>
+	<xacro:arg name="right_ee_can_interface" default="can1"/>
+	<xacro:arg name="left_read_tactile" default="false"/>
+	<xacro:arg name="right_read_tactile" default="false"/>
 	<!-- left_ft / right_ft / usb_*_ft_port: see marvin_hardware.xacro -->
 	<link name="world"/>
@@ -63,5 +67,9 @@
 		<xacro:external_ee_systems
 			usb_left_port="$(arg usb_left_port)"
-			usb_right_port="$(arg usb_right_port)"/>
+			usb_right_port="$(arg usb_right_port)"
+			left_ee_can_interface="$(arg left_ee_can_interface)"
+			right_ee_can_interface="$(arg right_ee_can_interface)"
+			left_read_tactile="$(arg left_read_tactile)"
+			right_read_tactile="$(arg right_read_tactile)"/>
 	</xacro:if>
 	<xacro:arg name="gazebo" default="false"/>

Commit message: Feature/add o6 can support (#15)
* Add support for LinkerHand O6 in USB CAN configuration

* Enhance LinkerHand support in USB CAN configuration and external systems integration

* Add rw_rate parameter to linkerhand USB CAN system for O6 support

File: m6_ccs_description/xacro/ros2_control/external_ee_systems.xacro (robot description, xacro)
@@ -31,8 +31,34 @@
 		</ros2_control>
 	</xacro:macro>
+	<xacro:macro name="linkerhand_usb_can_side_system" params="side hand_type can_interface read_tactile:=false">
+		<ros2_control name="${hand_type}_${side}_can_system" type="system" rw_rate="50">
+			<hardware>
+				<xacro:if value="${hand_type == 'linkerhand_o6'}">
+					<plugin>can_ros2_control/O6CanHardware</plugin>
+				</xacro:if>
+				<xacro:if value="${hand_type == 'linkerhand_l6'}">
+					<plugin>can_ros2_control/L6CanHardware</plugin>
+				</xacro:if>
+				<xacro:if value="${hand_type == 'linkerhand_o7'}">
+					<plugin>can_ros2_control/O7CanHardware</plugin>
+				</xacro:if>
+				<param name="can_interface">${can_interface}</param>
+				<param name="hand_side">${side}</param>
+				<param name="read_feedback">true</param>
+				<param name="read_tactile">${read_tactile}</param>
+				<param name="${side}_tool_torque">1.0</param>
+				<param name="${side}_tool_velocity">1.0</param>
+			</hardware>
+			<xacro:side_hand_interfaces side="${side}" hand_type="${hand_type}"/>
+		</ros2_control>
+	</xacro:macro>
 	<!-- left_ft / right_ft / usb_*_ft_port: declared in marvin_hardware.xacro; defaults read $(arg ...) here. -->
 	<xacro:macro name="external_ee_systems" params="
 		usb_left_port:=/dev/ttyUSB0
 		usb_right_port:=/dev/ttyUSB2
+		left_ee_can_interface:=can0
+		right_ee_can_interface:=can1
+		left_read_tactile:=false
+		right_read_tactile:=false
 		usb_baudrate:=115200
 		left_ft:=$(arg left_ft)
@@ -40,4 +66,10 @@
 		usb_left_ft_port:=$(arg usb_left_ft_port)
 		usb_right_ft_port:=$(arg usb_right_ft_port)">
+		<xacro:if value="${left_drive_type == 'usb_can' and (left_hand_type == 'linkerhand_o6' or left_hand_type == 'linkerhand_l6' or left_hand_type == 'linkerhand_o7')}">
+			<xacro:linkerhand_usb_can_side_system side="left" hand_type="${left_hand_type}" can_interface="${left_ee_can_interface}" read_tactile="${left_read_tactile}"/>
+		</xacro:if>
+		<xacro:if value="${right_drive_type == 'usb_can' and (right_hand_type == 'linkerhand_o6' or right_hand_type == 'linkerhand_l6' or right_hand_type == 'linkerhand_o7')}">
+			<xacro:linkerhand_usb_can_side_system side="right" hand_type="${right_hand_type}" can_interface="${right_ee_can_interface}" read_tactile="${right_read_tactile}"/>
+		</xacro:if>
 		<xacro:if value="${left_drive_type == 'usb' and (left_hand_type == 'linkerhand_o6' or left_hand_type == 'linkerhand_l6' or left_hand_type == 'linkerhand_o7')}">
 			<xacro:side_usb_hand_system side="left" hand_type="${left_hand_type}" serial_port="${usb_left_port}"/>
@@ -83,20 +115,20 @@
 		</xacro:if>
 		<xacro:if value="${left_drive_type == 'usb_can' and left_hand_type == 'freedom_v1'}">
-			<xacro:freedom_can_side_system side="left" can_interface="can0" device_id="0"/>
+			<xacro:freedom_can_side_system side="left" can_interface="${left_ee_can_interface}" device_id="0"/>
 		</xacro:if>
 		<xacro:if value="${right_drive_type == 'usb_can' and right_hand_type == 'freedom_v1'}">
-			<xacro:freedom_can_side_system side="right" can_interface="can1" device_id="1"/>
+			<xacro:freedom_can_side_system side="right" can_interface="${right_ee_can_interface}" device_id="1"/>
 		</xacro:if>
 		<xacro:if value="${left_drive_type == 'usb_can' and left_hand_type == 'inspire_e2'}">
-			<xacro:inspire_canfd_side_system side="left" can_interface="can0"/>
+			<xacro:inspire_canfd_side_system side="left" can_interface="${left_ee_can_interface}"/>
 		</xacro:if>
 		<xacro:if value="${right_drive_type == 'usb_can' and right_hand_type == 'inspire_e2'}">
-			<xacro:inspire_canfd_side_system side="right" can_interface="can1"/>
+			<xacro:inspire_canfd_side_system side="right" can_interface="${right_ee_can_interface}"/>
 		</xacro:if>
 		<xacro:if value="${left_drive_type == 'usb_can' and left_hand_type == 'inspire_f2'}">
-			<xacro:inspire_canfd_side_system side="left" can_interface="can0" hand_type="inspire_f2"/>
+			<xacro:inspire_canfd_side_system side="left" can_interface="${left_ee_can_interface}" hand_type="inspire_f2"/>
 		</xacro:if>
 		<xacro:if value="${right_drive_type == 'usb_can' and right_hand_type == 'inspire_f2'}">
-			<xacro:inspire_canfd_side_system side="right" can_interface="can1" hand_type="inspire_f2"/>
+			<xacro:inspire_canfd_side_system side="right" can_interface="${right_ee_can_interface}" hand_type="inspire_f2"/>
 		</xacro:if>
 		<xacro:ft_sensor_systems
