Commit message: update tianji

File: m6_ccs_description/xacro/ros2_control/end_effector_interfaces.xacro (robot description, xacro)
@@ -99,8 +99,8 @@
 				<xacro:side_gripper_joint side="right"/>
 			</xacro:if>
-			<xacro:if value="${(left_drive_type == 'marvin' or left_drive_type == 'tianji_can') and left_hand_type != '' and left_hand_type != 'xhand1' and left_hand_type != 'inspire_e2'}">
+			<xacro:if value="${(left_drive_type == 'marvin' or left_drive_type == 'tianji_can') and left_hand_type != '' and left_hand_type != 'xhand1' and left_hand_type != 'inspire_e2' and left_hand_type != 'wuji_hand2'}">
 				<xacro:side_hand_interfaces side="left" hand_type="${left_hand_type}"/>
 			</xacro:if>
-			<xacro:if value="${(right_drive_type == 'marvin' or right_drive_type == 'tianji_can') and right_hand_type != '' and right_hand_type != 'xhand1' and right_hand_type != 'inspire_e2'}">
+			<xacro:if value="${(right_drive_type == 'marvin' or right_drive_type == 'tianji_can') and right_hand_type != '' and right_hand_type != 'xhand1' and right_hand_type != 'inspire_e2' and right_hand_type != 'wuji_hand2'}">
 				<xacro:side_hand_interfaces side="right" hand_type="${right_hand_type}"/>
 			</xacro:if>

File: m6_ccs_description/xacro/ros2_control/external_ee_systems.xacro (robot description, xacro)
@@ -5,4 +5,37 @@
 	<xacro:include filename="$(find freedom_description)/xacro/ros2_control/side_systems.xacro"/>
 	<xacro:include filename="$(find inspire_description)/xacro/ros2_control/side_systems.xacro"/>
+	<xacro:macro name="wuji_hand2_ethernet_side_system" params="
+		side
+		hand_side
+		device_address
+		serial_number
+		mit_kp:=3.0
+		mit_kd:=0.05
+		effort_limit:=1.5
+		read_feedback:=true
+		require_initial_feedback:=true
+		command_deadband:=0.0
+		connect_timeout_ms:=5000
+		enable_timeout_s:=5.0">
+		<ros2_control name="wuji_hand2_${side}_system" type="system">
+			<hardware>
+				<plugin>wujihand2_ros2_control/WujiHand2Hardware</plugin>
+				<param name="hand_side">${hand_side}</param>
+				<param name="device_address">${device_address}</param>
+				<xacro:if value="${serial_number != ''}">
+					<param name="serial_number">${serial_number}</param>
+				</xacro:if>
+				<param name="mit_kp">${mit_kp}</param>
+				<param name="mit_kd">${mit_kd}</param>
+				<param name="effort_limit">${effort_limit}</param>
+				<param name="read_feedback">${read_feedback}</param>
+				<param name="require_initial_feedback">${require_initial_feedback}</param>
+				<param name="command_deadband">${command_deadband}</param>
+				<param name="connect_timeout_ms">${connect_timeout_ms}</param>
+				<param name="enable_timeout_s">${enable_timeout_s}</param>
+			</hardware>
+			<xacro:wuji_hand2_interfaces name="${side}_hand"/>
+		</ros2_control>
+	</xacro:macro>
 	<xacro:macro name="side_usb_hand_system" params="side hand_type serial_port">
 		<xacro:property name="usb_hand_system_name" value="${str('linkerhand_7' if hand_type == 'linkerhand_o7' else 'linkerhand_6')}"/>
@@ -62,4 +95,16 @@
 		right_read_tactile:=false
 		usb_baudrate:=115200
+		device_address_left:=$(arg device_address_left)
+		device_address_right:=$(arg device_address_right)
+		serial_number_left:=$(arg serial_number_left)
+		serial_number_right:=$(arg serial_number_right)
+		mit_kp:=$(arg mit_kp)
+		mit_kd:=$(arg mit_kd)
+		effort_limit:=$(arg effort_limit)
+		read_feedback:=$(arg read_feedback)
+		require_initial_feedback:=$(arg require_initial_feedback)
+		command_deadband:=$(arg command_deadband)
+		connect_timeout_ms:=$(arg connect_timeout_ms)
+		enable_timeout_s:=$(arg enable_timeout_s)
 		left_ft:=$(arg left_ft)
 		right_ft:=$(arg right_ft)
@@ -132,4 +177,34 @@
 			<xacro:inspire_canfd_side_system side="right" can_interface="${right_ee_can_interface}" hand_type="inspire_f2"/>
 		</xacro:if>
+		<xacro:if value="${left_drive_type == 'ethernet' and left_hand_type == 'wuji_hand2'}">
+			<xacro:wuji_hand2_ethernet_side_system
+				side="left"
+				hand_side="left"
+				device_address="${device_address_left}"
+				serial_number="${serial_number_left}"
+				mit_kp="${mit_kp}"
+				mit_kd="${mit_kd}"
+				effort_limit="${effort_limit}"
+				read_feedback="${read_feedback}"
+				require_initial_feedback="${require_initial_feedback}"
+				command_deadband="${command_deadband}"
+				connect_timeout_ms="${connect_timeout_ms}"
+				enable_timeout_s="${enable_timeout_s}"/>
+		</xacro:if>
+		<xacro:if value="${right_drive_type == 'ethernet' and right_hand_type == 'wuji_hand2'}">
+			<xacro:wuji_hand2_ethernet_side_system
+				side="right"
+				hand_side="right"
+				device_address="${device_address_right}"
+				serial_number="${serial_number_right}"
+				mit_kp="${mit_kp}"
+				mit_kd="${mit_kd}"
+				effort_limit="${effort_limit}"
+				read_feedback="${read_feedback}"
+				require_initial_feedback="${require_initial_feedback}"
+				command_deadband="${command_deadband}"
+				connect_timeout_ms="${connect_timeout_ms}"
+				enable_timeout_s="${enable_timeout_s}"/>
+		</xacro:if>
 		<xacro:ft_sensor_systems
 			left_ft="${left_ft}"

File: m6_ccs_description/xacro/ros2_control/marvin_hardware.xacro (robot description, xacro)
@@ -40,5 +40,5 @@
 			<xacro:property name="left_ee_type" value="${left_hand_type if left_hand_type != '' else left_gripper_type}"/>
 			<xacro:property name="right_ee_type" value="${right_hand_type if right_hand_type != '' else right_gripper_type}"/>
-			<xacro:if value="${(left_drive_type == 'marvin' or left_drive_type == 'tianji_can') and left_ee_type != '' and left_ee_type != 'xhand1' and left_ee_type != 'inspire_e2'}">
+			<xacro:if value="${(left_drive_type == 'marvin' or left_drive_type == 'tianji_can') and left_ee_type != '' and left_ee_type != 'xhand1' and left_ee_type != 'inspire_e2' and left_ee_type != 'wuji_hand2'}">
 				<param name="left_ee_type">${left_ee_type}</param>
 				<xacro:if value="${left_drive_type == 'tianji_can'}">
@@ -46,5 +46,5 @@
 				</xacro:if>
 			</xacro:if>
-			<xacro:if value="${(right_drive_type == 'marvin' or right_drive_type == 'tianji_can') and right_ee_type != '' and right_ee_type != 'xhand1' and right_ee_type != 'inspire_e2'}">
+			<xacro:if value="${(right_drive_type == 'marvin' or right_drive_type == 'tianji_can') and right_ee_type != '' and right_ee_type != 'xhand1' and right_ee_type != 'inspire_e2' and right_ee_type != 'wuji_hand2'}">
 				<param name="right_ee_type">${right_ee_type}</param>
 				<xacro:if value="${right_drive_type == 'tianji_can'}">

File: m6_ccs_description/xacro/ros2_control/robot.xacro (robot description, xacro)
@@ -21,4 +21,16 @@
 	<xacro:arg name="left_read_tactile" default="false"/>
 	<xacro:arg name="right_read_tactile" default="false"/>
+	<xacro:arg name="device_address_left" default=""/>
+	<xacro:arg name="device_address_right" default=""/>
+	<xacro:arg name="serial_number_left" default=""/>
+	<xacro:arg name="serial_number_right" default=""/>
+	<xacro:arg name="mit_kp" default="3.0"/>
+	<xacro:arg name="mit_kd" default="0.05"/>
+	<xacro:arg name="effort_limit" default="1.5"/>
+	<xacro:arg name="read_feedback" default="true"/>
+	<xacro:arg name="require_initial_feedback" default="true"/>
+	<xacro:arg name="command_deadband" default="0.0"/>
+	<xacro:arg name="connect_timeout_ms" default="5000"/>
+	<xacro:arg name="enable_timeout_s" default="5.0"/>
 	<!-- left_ft / right_ft / usb_*_ft_port: see marvin_hardware.xacro -->
 	<link name="world"/>

Commit message: update tianji

File: m6_ccs_description/xacro/ros2_control/end_effector_interfaces.xacro (robot description, xacro)
@@ -100,8 +100,8 @@
 				<xacro:side_gripper_joint side="right"/>
 			</xacro:if>
-			<xacro:if value="${(left_drive_type == 'marvin' or left_drive_type == 'tianji_can') and left_hand_type != '' and left_hand_type != 'xhand1' and left_hand_type != 'inspire_e2'}">
+			<xacro:if value="${(left_drive_type == 'marvin' or left_drive_type == 'tianji_can') and left_hand_type != '' and left_hand_type != 'xhand1' and left_hand_type != 'inspire_e2' and left_hand_type != 'wuji_hand2'}">
 				<xacro:side_hand_interfaces side="left" hand_type="${left_hand_type}"/>
 			</xacro:if>
-			<xacro:if value="${(right_drive_type == 'marvin' or right_drive_type == 'tianji_can') and right_hand_type != '' and right_hand_type != 'xhand1' and right_hand_type != 'inspire_e2'}">
+			<xacro:if value="${(right_drive_type == 'marvin' or right_drive_type == 'tianji_can') and right_hand_type != '' and right_hand_type != 'xhand1' and right_hand_type != 'inspire_e2' and right_hand_type != 'wuji_hand2'}">
 				<xacro:side_hand_interfaces side="right" hand_type="${right_hand_type}"/>
 			</xacro:if>

File: m6_ccs_description/xacro/ros2_control/external_ee_systems.xacro (robot description, xacro)
@@ -9,4 +9,40 @@
 	<xacro:include filename="$(find jodell_description)/xacro/ros2_control/side_systems.xacro"/>
 	<xacro:include filename="$(find changingtek_description)/xacro/ros2_control/side_systems.xacro"/>
+	<!-- rw_rate: empty → default 200 Hz (same idea as LinkerHand USB-CAN empty → 50). -->
+	<xacro:macro name="wuji_hand2_ethernet_side_system" params="
+		side
+		hand_side
+		device_address
+		serial_number
+		mit_kp:=3.0
+		mit_kd:=0.05
+		effort_limit:=1.5
+		read_feedback:=true
+		require_initial_feedback:=true
+		command_deadband:=0.0
+		connect_timeout_ms:=5000
+		enable_timeout_s:=5.0
+		rw_rate:=''">
+		<xacro:property name="wuji_effective_rw_rate" value="${rw_rate if rw_rate != '' else 200}"/>
+		<ros2_control name="wuji_hand2_${side}_system" type="system" rw_rate="${wuji_effective_rw_rate}">
+			<hardware>
+				<plugin>wujihand2_ros2_control/WujiHand2Hardware</plugin>
+				<param name="hand_side">${hand_side}</param>
+				<param name="device_address">${device_address}</param>
+				<xacro:if value="${serial_number != ''}">
+					<param name="serial_number">${serial_number}</param>
+				</xacro:if>
+				<param name="mit_kp">${mit_kp}</param>
+				<param name="mit_kd">${mit_kd}</param>
+				<param name="effort_limit">${effort_limit}</param>
+				<param name="read_feedback">${read_feedback}</param>
+				<param name="require_initial_feedback">${require_initial_feedback}</param>
+				<param name="command_deadband">${command_deadband}</param>
+				<param name="connect_timeout_ms">${connect_timeout_ms}</param>
+				<param name="enable_timeout_s">${enable_timeout_s}</param>
+			</hardware>
+			<xacro:wuji_hand2_interfaces name="${side}_hand"/>
+		</ros2_control>
+	</xacro:macro>
 	<!-- left_ft / right_ft / usb_*_ft_port: declared in marvin_hardware.xacro; defaults read $(arg ...) here. -->
 	<xacro:macro name="external_ee_systems" params="
@@ -20,4 +56,16 @@
 		right_ee_rw_rate:=''
 		usb_baudrate:=115200
+		device_address_left:=$(arg device_address_left)
+		device_address_right:=$(arg device_address_right)
+		serial_number_left:=$(arg serial_number_left)
+		serial_number_right:=$(arg serial_number_right)
+		mit_kp:=$(arg mit_kp)
+		mit_kd:=$(arg mit_kd)
+		effort_limit:=$(arg effort_limit)
+		read_feedback:=$(arg read_feedback)
+		require_initial_feedback:=$(arg require_initial_feedback)
+		command_deadband:=$(arg command_deadband)
+		connect_timeout_ms:=$(arg connect_timeout_ms)
+		enable_timeout_s:=$(arg enable_timeout_s)
 		left_ft:=$(arg left_ft)
 		right_ft:=$(arg right_ft)
@@ -103,4 +151,36 @@
 			<xacro:jodell_usb_side_system side="right" serial_port="${usb_right_port}" rw_rate="${right_ee_rw_rate}"/>
 		</xacro:if>
+		<xacro:if value="${left_drive_type == 'ethernet' and left_hand_type == 'wuji_hand2'}">
+			<xacro:wuji_hand2_ethernet_side_system
+				side="left"
+				hand_side="left"
+				device_address="${device_address_left}"
+				serial_number="${serial_number_left}"
+				mit_kp="${mit_kp}"
+				mit_kd="${mit_kd}"
+				effort_limit="${effort_limit}"
+				read_feedback="${read_feedback}"
+				require_initial_feedback="${require_initial_feedback}"
+				command_deadband="${command_deadband}"
+				connect_timeout_ms="${connect_timeout_ms}"
+				enable_timeout_s="${enable_timeout_s}"
+				rw_rate="${left_ee_rw_rate}"/>
+		</xacro:if>
+		<xacro:if value="${right_drive_type == 'ethernet' and right_hand_type == 'wuji_hand2'}">
+			<xacro:wuji_hand2_ethernet_side_system
+				side="right"
+				hand_side="right"
+				device_address="${device_address_right}"
+				serial_number="${serial_number_right}"
+				mit_kp="${mit_kp}"
+				mit_kd="${mit_kd}"
+				effort_limit="${effort_limit}"
+				read_feedback="${read_feedback}"
+				require_initial_feedback="${require_initial_feedback}"
+				command_deadband="${command_deadband}"
+				connect_timeout_ms="${connect_timeout_ms}"
+				enable_timeout_s="${enable_timeout_s}"
+				rw_rate="${right_ee_rw_rate}"/>
+		</xacro:if>
 		<xacro:ft_sensor_systems
 			left_ft="${left_ft}"

File: m6_ccs_description/xacro/ros2_control/robot.xacro (robot description, xacro)
@@ -23,4 +23,16 @@
 	<xacro:arg name="left_ee_rw_rate" default=""/>
 	<xacro:arg name="right_ee_rw_rate" default=""/>
+	<xacro:arg name="device_address_left" default=""/>
+	<xacro:arg name="device_address_right" default=""/>
+	<xacro:arg name="serial_number_left" default=""/>
+	<xacro:arg name="serial_number_right" default=""/>
+	<xacro:arg name="mit_kp" default="3.0"/>
+	<xacro:arg name="mit_kd" default="0.05"/>
+	<xacro:arg name="effort_limit" default="1.5"/>
+	<xacro:arg name="read_feedback" default="true"/>
+	<xacro:arg name="require_initial_feedback" default="true"/>
+	<xacro:arg name="command_deadband" default="0.0"/>
+	<xacro:arg name="connect_timeout_ms" default="5000"/>
+	<xacro:arg name="enable_timeout_s" default="5.0"/>
 	<!-- left_ft / right_ft / usb_*_ft_port: see marvin_hardware.xacro -->
 	<link name="world"/>

Commit message: 增加rg75 usb 485 模式

File: m6_ccs_description/xacro/ros2_control/end_effector_interfaces.xacro (robot description, xacro)
@@ -89,8 +89,9 @@
 		</xacro:if>
 		<xacro:if value="${mode == 'real'}">
-			<xacro:if value="${left_gripper_type != ''}">
+			<!-- 夹爪关节接口由实际驱动它的硬件块声明：marvin/tianji_can → M6_CCS_System；usb (USB-485) → external modbus system -->
+			<xacro:if value="${left_gripper_type != '' and (left_drive_type == 'marvin' or left_drive_type == 'tianji_can')}">
 				<xacro:side_gripper_joint side="left"/>
 			</xacro:if>
-			<xacro:if value="${right_gripper_type != ''}">
+			<xacro:if value="${right_gripper_type != '' and (right_drive_type == 'marvin' or right_drive_type == 'tianji_can')}">
 				<xacro:side_gripper_joint side="right"/>
 			</xacro:if>

File: m6_ccs_description/xacro/ros2_control/external_ee_systems.xacro (robot description, xacro)
@@ -29,4 +29,26 @@
 			</hardware>
 			<xacro:side_hand_interfaces side="${side}" hand_type="theohand_std16a"/>
+		</ros2_control>
+	</xacro:macro>
+	<!-- USB-485 夹爪（modbus_ros2_control/ModbusHardware）：rg75 (Jodell) / ag2f90_d (Changingtek 90D) -->
+	<xacro:macro name="changingtek_usb_side_system" params="side variant serial_port">
+		<ros2_control name="changingtek_${side}_system" type="system">
+			<hardware>
+				<plugin>modbus_ros2_control/ModbusHardware</plugin>
+				<param name="gripper_type">changingtek</param>
+				<param name="variant">${variant}</param>
+				<param name="serial_port">${serial_port}</param>
+			</hardware>
+			<xacro:side_gripper_joint side="${side}"/>
+		</ros2_control>
+	</xacro:macro>
+	<xacro:macro name="jodell_usb_side_system" params="side serial_port">
+		<ros2_control name="jodell_${side}_system" type="system">
+			<hardware>
+				<plugin>modbus_ros2_control/ModbusHardware</plugin>
+				<param name="gripper_type">jodell</param>
+				<param name="serial_port">${serial_port}</param>
+			</hardware>
+			<xacro:side_gripper_joint side="${side}"/>
 		</ros2_control>
 	</xacro:macro>
@@ -132,4 +154,17 @@
 			<xacro:inspire_canfd_side_system side="right" can_interface="${right_ee_can_interface}" hand_type="inspire_f2"/>
 		</xacro:if>
+		<!-- USB-485 夹爪（rg75 / ag2f90_d） -->
+		<xacro:if value="${left_drive_type == 'usb' and left_gripper_type == 'ag2f90_d'}">
+			<xacro:changingtek_usb_side_system side="left" variant="90d" serial_port="${usb_left_port}"/>
+		</xacro:if>
+		<xacro:if value="${right_drive_type == 'usb' and right_gripper_type == 'ag2f90_d'}">
+			<xacro:changingtek_usb_side_system side="right" variant="90d" serial_port="${usb_right_port}"/>
+		</xacro:if>
+		<xacro:if value="${left_drive_type == 'usb' and left_gripper_type == 'rg75'}">
+			<xacro:jodell_usb_side_system side="left" serial_port="${usb_left_port}"/>
+		</xacro:if>
+		<xacro:if value="${right_drive_type == 'usb' and right_gripper_type == 'rg75'}">
+			<xacro:jodell_usb_side_system side="right" serial_port="${usb_right_port}"/>
+		</xacro:if>
 		<xacro:ft_sensor_systems
 			left_ft="${left_ft}"

Commit message: Drop the local side_ros2_control_system copy.
Standalone side systems now include the shared helper from robot_common_launch.

File: m6_ccs_description/xacro/ros2_control/end_effector_interfaces.xacro (robot description, xacro)
@@ -16,17 +16,4 @@
 	<xacro:include filename="$(find theohand_description)/xacro/ros2_control/std16a.xacro"/>
 	<xacro:include filename="$(find marvin_gripper_description)/xacro/ros2_control/marvin_gripper.xacro"/>
-	<!-- Optional ros2_control rw_rate: omit the attribute when empty so CM rate is used. -->
-	<xacro:macro name="side_ros2_control_system" params="name rw_rate:='' *contents">
-		<xacro:if value="${rw_rate != ''}">
-			<ros2_control name="${name}" type="system" rw_rate="${rw_rate}">
-				<xacro:insert_block name="contents"/>
-			</ros2_control>
-		</xacro:if>
-		<xacro:unless value="${rw_rate != ''}">
-			<ros2_control name="${name}" type="system">
-				<xacro:insert_block name="contents"/>
-			</ros2_control>
-		</xacro:unless>
-	</xacro:macro>
 	<xacro:macro name="side_gripper_joint" params="side">
 		<joint name="${side}_gripper_joint">
