Commit message: update xacro

File: m6_ccs_description/xacro/ros2_control/end_effector_interfaces.xacro (robot description, xacro)
@@ -100,8 +100,8 @@
 				<xacro:side_gripper_joint side="right"/>
 			</xacro:if>
-			<xacro:if value="${(left_drive_type == 'marvin' or left_drive_type == 'tianji_can') and left_hand_type != '' and left_hand_type != 'xhand1' and left_hand_type != 'inspire_e2' and left_hand_type != 'wuji_hand2'}">
+			<xacro:if value="${(left_drive_type == 'marvin' or left_drive_type == 'tianji_can') and left_hand_type != '' and left_hand_type != 'xhand1' and left_hand_type != 'inspire_e2'}">
 				<xacro:side_hand_interfaces side="left" hand_type="${left_hand_type}"/>
 			</xacro:if>
-			<xacro:if value="${(right_drive_type == 'marvin' or right_drive_type == 'tianji_can') and right_hand_type != '' and right_hand_type != 'xhand1' and right_hand_type != 'inspire_e2' and right_hand_type != 'wuji_hand2'}">
+			<xacro:if value="${(right_drive_type == 'marvin' or right_drive_type == 'tianji_can') and right_hand_type != '' and right_hand_type != 'xhand1' and right_hand_type != 'inspire_e2'}">
 				<xacro:side_hand_interfaces side="right" hand_type="${right_hand_type}"/>
 			</xacro:if>

File: m6_ccs_description/xacro/ros2_control/external_ee_systems.xacro (robot description, xacro)
@@ -9,40 +9,5 @@
 	<xacro:include filename="$(find jodell_description)/xacro/ros2_control/side_systems.xacro"/>
 	<xacro:include filename="$(find changingtek_description)/xacro/ros2_control/side_systems.xacro"/>
-	<!-- rw_rate: empty → default 200 Hz (same idea as LinkerHand USB-CAN empty → 50). -->
-	<xacro:macro name="wuji_hand2_ethernet_side_system" params="
-		side
-		hand_side
-		device_address
-		serial_number
-		mit_kp:=3.0
-		mit_kd:=0.05
-		effort_limit:=1.5
-		read_feedback:=true
-		require_initial_feedback:=true
-		command_deadband:=0.0
-		connect_timeout_ms:=5000
-		enable_timeout_s:=5.0
-		rw_rate:=''">
-		<xacro:property name="wuji_effective_rw_rate" value="${rw_rate if rw_rate != '' else 200}"/>
-		<ros2_control name="wuji_hand2_${side}_system" type="system" rw_rate="${wuji_effective_rw_rate}">
-			<hardware>
-				<plugin>wujihand2_ros2_control/WujiHand2Hardware</plugin>
-				<param name="hand_side">${hand_side}</param>
-				<param name="device_address">${device_address}</param>
-				<xacro:if value="${serial_number != ''}">
-					<param name="serial_number">${serial_number}</param>
-				</xacro:if>
-				<param name="mit_kp">${mit_kp}</param>
-				<param name="mit_kd">${mit_kd}</param>
-				<param name="effort_limit">${effort_limit}</param>
-				<param name="read_feedback">${read_feedback}</param>
-				<param name="require_initial_feedback">${require_initial_feedback}</param>
-				<param name="command_deadband">${command_deadband}</param>
-				<param name="connect_timeout_ms">${connect_timeout_ms}</param>
-				<param name="enable_timeout_s">${enable_timeout_s}</param>
-			</hardware>
-			<xacro:wuji_hand2_interfaces name="${side}_hand"/>
-		</ros2_control>
-	</xacro:macro>
+	<xacro:include filename="$(find wuji_description)/xacro/ros2_control/side_systems.xacro"/>
 	<!-- left_ft / right_ft / usb_*_ft_port: declared in marvin_hardware.xacro; defaults read $(arg ...) here. -->
 	<xacro:macro name="external_ee_systems" params="
@@ -56,16 +21,4 @@
 		right_ee_rw_rate:=''
 		usb_baudrate:=115200
-		device_address_left:=$(arg device_address_left)
-		device_address_right:=$(arg device_address_right)
-		serial_number_left:=$(arg serial_number_left)
-		serial_number_right:=$(arg serial_number_right)
-		mit_kp:=$(arg mit_kp)
-		mit_kd:=$(arg mit_kd)
-		effort_limit:=$(arg effort_limit)
-		read_feedback:=$(arg read_feedback)
-		require_initial_feedback:=$(arg require_initial_feedback)
-		command_deadband:=$(arg command_deadband)
-		connect_timeout_ms:=$(arg connect_timeout_ms)
-		enable_timeout_s:=$(arg enable_timeout_s)
 		left_ft:=$(arg left_ft)
 		right_ft:=$(arg right_ft)
@@ -152,34 +105,8 @@
 		</xacro:if>
 		<xacro:if value="${left_drive_type == 'ethernet' and left_hand_type == 'wuji_hand2'}">
-			<xacro:wuji_hand2_ethernet_side_system
-				side="left"
-				hand_side="left"
-				device_address="${device_address_left}"
-				serial_number="${serial_number_left}"
-				mit_kp="${mit_kp}"
-				mit_kd="${mit_kd}"
-				effort_limit="${effort_limit}"
-				read_feedback="${read_feedback}"
-				require_initial_feedback="${require_initial_feedback}"
-				command_deadband="${command_deadband}"
-				connect_timeout_ms="${connect_timeout_ms}"
-				enable_timeout_s="${enable_timeout_s}"
-				rw_rate="${left_ee_rw_rate}"/>
+			<xacro:wuji_hand2_ethernet_side_system side="left" rw_rate="${left_ee_rw_rate}"/>
 		</xacro:if>
 		<xacro:if value="${right_drive_type == 'ethernet' and right_hand_type == 'wuji_hand2'}">
-			<xacro:wuji_hand2_ethernet_side_system
-				side="right"
-				hand_side="right"
-				device_address="${device_address_right}"
-				serial_number="${serial_number_right}"
-				mit_kp="${mit_kp}"
-				mit_kd="${mit_kd}"
-				effort_limit="${effort_limit}"
-				read_feedback="${read_feedback}"
-				require_initial_feedback="${require_initial_feedback}"
-				command_deadband="${command_deadband}"
-				connect_timeout_ms="${connect_timeout_ms}"
-				enable_timeout_s="${enable_timeout_s}"
-				rw_rate="${right_ee_rw_rate}"/>
+			<xacro:wuji_hand2_ethernet_side_system side="right" rw_rate="${right_ee_rw_rate}"/>
 		</xacro:if>
 		<xacro:ft_sensor_systems

File: m6_ccs_description/xacro/ros2_control/marvin_hardware.xacro (robot description, xacro)
@@ -40,5 +40,5 @@
 			<xacro:property name="left_ee_type" value="${left_hand_type if left_hand_type != '' else left_gripper_type}"/>
 			<xacro:property name="right_ee_type" value="${right_hand_type if right_hand_type != '' else right_gripper_type}"/>
-			<xacro:if value="${(left_drive_type == 'marvin' or left_drive_type == 'tianji_can') and left_ee_type != '' and left_ee_type != 'xhand1' and left_ee_type != 'inspire_e2' and left_ee_type != 'wuji_hand2'}">
+			<xacro:if value="${(left_drive_type == 'marvin' or left_drive_type == 'tianji_can') and left_ee_type != '' and left_ee_type != 'xhand1' and left_ee_type != 'inspire_e2'}">
 				<param name="left_ee_type">${left_ee_type}</param>
 				<xacro:if value="${left_drive_type == 'tianji_can'}">
@@ -46,5 +46,5 @@
 				</xacro:if>
 			</xacro:if>
-			<xacro:if value="${(right_drive_type == 'marvin' or right_drive_type == 'tianji_can') and right_ee_type != '' and right_ee_type != 'xhand1' and right_ee_type != 'inspire_e2' and right_ee_type != 'wuji_hand2'}">
+			<xacro:if value="${(right_drive_type == 'marvin' or right_drive_type == 'tianji_can') and right_ee_type != '' and right_ee_type != 'xhand1' and right_ee_type != 'inspire_e2'}">
 				<param name="right_ee_type">${right_ee_type}</param>
 				<xacro:if value="${right_drive_type == 'tianji_can'}">

File: m6_ccs_description/xacro/ros2_control/robot.xacro (robot description, xacro)
@@ -23,16 +23,4 @@
 	<xacro:arg name="left_ee_rw_rate" default=""/>
 	<xacro:arg name="right_ee_rw_rate" default=""/>
-	<xacro:arg name="device_address_left" default=""/>
-	<xacro:arg name="device_address_right" default=""/>
-	<xacro:arg name="serial_number_left" default=""/>
-	<xacro:arg name="serial_number_right" default=""/>
-	<xacro:arg name="mit_kp" default="3.0"/>
-	<xacro:arg name="mit_kd" default="0.05"/>
-	<xacro:arg name="effort_limit" default="1.5"/>
-	<xacro:arg name="read_feedback" default="true"/>
-	<xacro:arg name="require_initial_feedback" default="true"/>
-	<xacro:arg name="command_deadband" default="0.0"/>
-	<xacro:arg name="connect_timeout_ms" default="5000"/>
-	<xacro:arg name="enable_timeout_s" default="5.0"/>
 	<!-- left_ft / right_ft / usb_*_ft_port: see marvin_hardware.xacro -->
 	<link name="world"/>
