Commit message: using high precision pi

File: m6_ccs_description/xacro/arm.xacro (robot description, xacro)
@@ -57,5 +57,5 @@
 			<xacro:if value="${collider == 'simple'}">
 				<collision>
-					<origin rpy="1.5708 0 0"/>
+					<origin rpy="${PI/2} 0 0"/>
 					<geometry>
 						<cylinder length="0.125958" radius="0.057588"/>
@@ -70,5 +70,5 @@
 			<child link="${prefix}link1"/>
 			<axis xyz="0 0 1"/>
-			<limit lower="-3.1067" upper="3.1067" effort="108" velocity="3.1416"/>
+			<limit lower="-3.1067" upper="3.1067" effort="108" velocity="${PI}"/>
 		</joint>
 		<!-- Link 2 -->
@@ -95,5 +95,5 @@
 			<xacro:if value="${collider == 'simple'}">
 				<collision>
-					<origin xyz="0 0.099087 0" rpy="1.5708 0 0"/>
+					<origin xyz="0 0.099087 0" rpy="${PI/2} 0 0"/>
 					<geometry>
 						<cylinder length="0.078386" radius="0.046717"/>
@@ -104,9 +104,9 @@
 		<!-- Joint 2 -->
 		<joint name="${prefix}joint2" type="revolute">
-			<origin rpy="1.5708 0 0"/>
+			<origin rpy="${PI/2} 0 0"/>
 			<parent link="${prefix}link1"/>
 			<child link="${prefix}link2"/>
 			<axis xyz="0 0 1"/>
-			<limit lower="-2.0944" upper="2.0944" effort="108" velocity="3.1416"/>
+			<limit lower="-2.0944" upper="2.0944" effort="108" velocity="${PI}"/>
 		</joint>
 		<!-- Link 3 -->
@@ -139,5 +139,5 @@
 				</collision>
 				<collision>
-					<origin xyz="0.018119 0 0" rpy="1.5708 0 0"/>
+					<origin xyz="0.018119 0 0" rpy="${PI/2} 0 0"/>
 					<geometry>
 						<cylinder length="0.117016" radius="0.049964"/>
@@ -148,9 +148,9 @@
 		<!-- Joint 3 -->
 		<joint name="${prefix}joint3" type="revolute">
-			<origin xyz="0 0.287 0" rpy="-1.5708 0 0"/>
+			<origin xyz="0 0.287 0" rpy="-${PI/2} 0 0"/>
 			<parent link="${prefix}link2"/>
 			<child link="${prefix}link3"/>
 			<axis xyz="0 0 1"/>
-			<limit lower="-3.1067" upper="3.1067" effort="66" velocity="3.1416"/>
+			<limit lower="-3.1067" upper="3.1067" effort="66" velocity="${PI}"/>
 		</joint>
 		<!-- Link 4 -->
@@ -177,5 +177,5 @@
 			<xacro:if value="${collider == 'simple'}">
 				<collision>
-					<origin xyz="0.017721 -0.079733 0" rpy="1.5708 0 0"/>
+					<origin xyz="0.017721 -0.079733 0" rpy="${PI/2} 0 0"/>
 					<geometry>
 						<cylinder length="0.080203" radius="0.041759"/>
@@ -186,9 +186,9 @@
 		<!-- Joint 4 -->
 		<joint name="${prefix}joint4" type="revolute">
-			<origin xyz="0.018 0 0" rpy="-1.5708 0 3.1416"/>
+			<origin xyz="0.018 0 0" rpy="-${PI/2} 0 ${PI}"/>
 			<parent link="${prefix}link3"/>
 			<child link="${prefix}link4"/>
 			<axis xyz="0 0 1"/>
-			<limit lower="-2.5307" upper="1.0472" effort="66" velocity="3.1416"/>
+			<limit lower="-2.5307" upper="1.0472" effort="66" velocity="${PI}"/>
 		</joint>
 		<!-- Link 5 - Mirrored COM and partial inertia -->
@@ -224,9 +224,9 @@
 		<!-- Joint 5 -->
 		<joint name="${prefix}joint5" type="revolute">
-			<origin xyz="0.018 -0.314 0" rpy="-1.5708 0 3.1416"/>
+			<origin xyz="0.018 -0.314 0" rpy="-${PI/2} 0 ${PI}"/>
 			<parent link="${prefix}link4"/>
 			<child link="${prefix}link5"/>
 			<axis xyz="0 0 1"/>
-			<limit lower="-3.1067" upper="3.1067" effort="18" velocity="3.1416"/>
+			<limit lower="-3.1067" upper="3.1067" effort="18" velocity="${PI}"/>
 		</joint>
 		<!-- Link 6 - Partially mirrored COM and inertia -->
@@ -253,5 +253,5 @@
 			<xacro:if value="${collider == 'simple'}">
 				<collision>
-					<origin xyz="0 0 0" rpy="1.5708 0 0"/>
+					<origin xyz="0 0 0" rpy="${PI/2} 0 0"/>
 					<geometry>
 						<cylinder length="0.108046" radius="0.038348"/>
@@ -262,9 +262,9 @@
 		<!-- Joint 6 -->
 		<joint name="${prefix}joint6" type="revolute">
-			<origin rpy="1.5708 -1.5708 0"/>
+			<origin rpy="${PI/2} -${PI/2} 0"/>
 			<parent link="${prefix}link5"/>
 			<child link="${prefix}link6"/>
 			<axis xyz="0 0 1"/>
-			<limit lower="-1.0472" upper="1.0472" effort="18" velocity="3.1416"/>
+			<limit lower="-1.0472" upper="1.0472" effort="18" velocity="${PI}"/>
 		</joint>
 		<!-- Link 7 -->
@@ -296,5 +296,5 @@
 			<xacro:if value="${collider == 'simple'}">
 				<collision>
-					<origin xyz="0 -0.075732 0" rpy="1.5708 0 0"/>
+					<origin xyz="0 -0.075732 0" rpy="${PI/2} 0 0"/>
 					<geometry>
 						<cylinder length="0.038392" radius="0.041707"/>
@@ -305,9 +305,9 @@
 		<!-- Joint 7 -->
 		<joint name="${prefix}joint7" type="revolute">
-			<origin rpy="1.5708 -1.5708 0"/>
+			<origin rpy="${PI/2} -${PI/2} 0"/>
 			<parent link="${prefix}link6"/>
 			<child link="${prefix}link7"/>
 			<axis xyz="0 0 1"/>
-			<limit lower="-1.5708" upper="1.5708" effort="18" velocity="3.1416"/>
+			<limit lower="-${PI/2}" upper="${PI/2}" effort="18" velocity="${PI}"/>
 		</joint>
 		<link name="${prefix}eef"/>

File: m6_ccs_description/xacro/robot.xacro (robot description, xacro)
@@ -28,5 +28,5 @@
 			<parent link="arm_base"/>
 			<child link="left_base_link"/>
-			<origin rpy="-1.5708 0 0" xyz="0.0 0.062 0"/>
+			<origin rpy="-${PI/2} 0 0" xyz="0.0 0.062 0"/>
 		</joint>
 		<!-- Right Arm -->
@@ -34,5 +34,5 @@
 			<parent link="arm_base"/>
 			<child link="right_base_link"/>
-			<origin rpy="1.5708 0 0" xyz="0 -0.062 0"/>
+			<origin rpy="${PI/2} 0 0" xyz="0 -0.062 0"/>
 		</joint>
 		<xacro:M6_CCS name="left" collider="$(arg collider)"/>
@@ -57,5 +57,5 @@
 			<parent link="base_link"/>
 			<child link="left_base_link"/>
-			<origin rpy="-1.5708 0 0" xyz="0.0 0.12 0.701"/>
+			<origin rpy="-${PI/2} 0 0" xyz="0.0 0.12 0.701"/>
 		</joint>
 		<!-- Right Arm -->
@@ -63,5 +63,5 @@
 			<parent link="base_link"/>
 			<child link="right_base_link"/>
-			<origin rpy="1.5708 0 0" xyz="0.0 -0.12 0.701"/>
+			<origin rpy="${PI/2} 0 0" xyz="0.0 -0.12 0.701"/>
 		</joint>
 		<xacro:M6_CCS name="left" collider="$(arg collider)"/>

Commit message: add visual support for agibot g2

File: m6_ccs_description/xacro/arm.xacro (robot description, xacro)
@@ -4,6 +4,19 @@
 	<xacro:property name="PI" value="3.1415926535897931"/>
 	<xacro:property name="collider_type" value="$(arg collider)"/>
-	<xacro:macro name="M6_CCS" params="name:='' direction:=1">
+	<xacro:macro name="M6_CCS" params="name:='' direction:=1 style:=default">
 		<xacro:property name="prefix" value="${name + '_' if name else ''}"/>
+		<!-- Set visual and collision package/path based on style -->
+		<xacro:property name="visual_package" value="m6_ccs_description"/>
+		<xacro:property name="visual_path" value=""/>
+		<xacro:property name="collision_package" value="m6_ccs_description"/>
+		<xacro:property name="collision_path" value=""/>
+		<xacro:if value="${style == 'fiveages_w2'}">
+			<xacro:property name="visual_package" value="fiveages_w2_description"/>
+			<xacro:property name="visual_path" value="arm/"/>
+		</xacro:if>
+		<xacro:if value="${style == 'agibot_g2'}">
+			<xacro:property name="visual_package" value="agibot_g2_description"/>
+			<xacro:property name="visual_path" value="arm/"/>
+		</xacro:if>
 		<!-- Base Link -->
 		<link name="${prefix}base_link">
@@ -47,11 +60,11 @@
 			<visual>
 				<geometry>
-					<mesh filename="file://$(find m6_ccs_description)/meshes/link1.glb"/>
-				</geometry>
-			</visual>
-			<xacro:if value="${collider_type == 'convex'}">
-				<collision>
-					<geometry>
-						<mesh filename="file://$(find m6_ccs_description)/meshes/link1.glb"/>
+					<mesh filename="file://$(find ${visual_package})/meshes/${visual_path}link1.glb"/>
+				</geometry>
+			</visual>
+			<xacro:if value="${collider_type == 'convex'}">
+				<collision>
+					<geometry>
+						<mesh filename="file://$(find ${collision_package})/meshes/${collision_path}link1.glb"/>
 					</geometry>
 				</collision>
@@ -85,11 +98,11 @@
 			<visual>
 				<geometry>
-					<mesh filename="file://$(find m6_ccs_description)/meshes/link2.glb"/>
-				</geometry>
-			</visual>
-			<xacro:if value="${collider_type == 'convex'}">
-				<collision>
-					<geometry>
-						<mesh filename="file://$(find m6_ccs_description)/meshes/link2.glb"/>
+					<mesh filename="file://$(find ${visual_package})/meshes/${visual_path}link2.glb" scale="1 1 ${direction}"/>
+				</geometry>
+			</visual>
+			<xacro:if value="${collider_type == 'convex'}">
+				<collision>
+					<geometry>
+						<mesh filename="file://$(find ${collision_package})/meshes/${collision_path}link2.glb"/>
 					</geometry>
 				</collision>
@@ -123,11 +136,11 @@
 			<visual>
 				<geometry>
-					<mesh filename="file://$(find m6_ccs_description)/meshes/link3.glb"/>
-				</geometry>
-			</visual>
-			<xacro:if value="${collider_type == 'convex'}">
-				<collision>
-					<geometry>
-						<mesh filename="file://$(find m6_ccs_description)/meshes/link3.glb"/>
+					<mesh filename="file://$(find ${visual_package})/meshes/${visual_path}link3.glb"/>
+				</geometry>
+			</visual>
+			<xacro:if value="${collider_type == 'convex'}">
+				<collision>
+					<geometry>
+						<mesh filename="file://$(find ${collision_package})/meshes/${collision_path}link3.glb"/>
 					</geometry>
 				</collision>
@@ -167,11 +180,11 @@
 			<visual>
 				<geometry>
-					<mesh filename="file://$(find m6_ccs_description)/meshes/link4.glb"/>
-				</geometry>
-			</visual>
-			<xacro:if value="${collider_type == 'convex'}">
-				<collision>
-					<geometry>
-						<mesh filename="file://$(find m6_ccs_description)/meshes/link4.glb"/>
+					<mesh filename="file://$(find ${visual_package})/meshes/${visual_path}link4.glb"/>
+				</geometry>
+			</visual>
+			<xacro:if value="${collider_type == 'convex'}">
+				<collision>
+					<geometry>
+						<mesh filename="file://$(find ${collision_package})/meshes/${collision_path}link4.glb"/>
 					</geometry>
 				</collision>
@@ -205,11 +218,11 @@
 			<visual>
 				<geometry>
-					<mesh filename="file://$(find m6_ccs_description)/meshes/link5.glb" scale="1 ${direction} 1"/>
-				</geometry>
-			</visual>
-			<xacro:if value="${collider_type == 'convex'}">
-				<collision>
-					<geometry>
-						<mesh filename="file://$(find m6_ccs_description)/meshes/link5.glb"/>
+					<mesh filename="file://$(find ${visual_package})/meshes/${visual_path}link5.glb" scale="1 ${direction} 1"/>
+				</geometry>
+			</visual>
+			<xacro:if value="${collider_type == 'convex'}">
+				<collision>
+					<geometry>
+						<mesh filename="file://$(find ${collision_package})/meshes/${collision_path}link5.glb"/>
 					</geometry>
 				</collision>
@@ -243,11 +256,11 @@
 			<visual>
 				<geometry>
-					<mesh filename="file://$(find m6_ccs_description)/meshes/link6.glb"/>
-				</geometry>
-			</visual>
-			<xacro:if value="${collider_type == 'convex'}">
-				<collision>
-					<geometry>
-						<mesh filename="file://$(find m6_ccs_description)/meshes/link6.glb"/>
+					<mesh filename="file://$(find ${visual_package})/meshes/${visual_path}link6.glb"/>
+				</geometry>
+			</visual>
+			<xacro:if value="${collider_type == 'convex'}">
+				<collision>
+					<geometry>
+						<mesh filename="file://$(find ${collision_package})/meshes/${collision_path}link6.glb"/>
 					</geometry>
 				</collision>
@@ -282,8 +295,8 @@
 				<geometry>
 					<xacro:if value="${direction == 1}">
-						<mesh filename="file://$(find m6_ccs_description)/meshes/link7.glb"/>
+						<mesh filename="file://$(find ${visual_package})/meshes/${visual_path}link7.glb"/>
 					</xacro:if>
 					<xacro:if value="${direction == -1}">
-						<mesh filename="file://$(find m6_ccs_description)/meshes/link7_r.glb"/>
+						<mesh filename="file://$(find ${visual_package})/meshes/${visual_path}link7_r.glb"/>
 					</xacro:if>
 				</geometry>
@@ -292,5 +305,5 @@
 				<collision>
 					<geometry>
-						<mesh filename="file://$(find m6_ccs_description)/meshes/link7.glb"/>
+						<mesh filename="file://$(find ${collision_package})/meshes/${collision_path}link7.glb"/>
 					</geometry>
 				</collision>

Commit message: add rg75 heavy config

File: m6_ccs_description/xacro/arm.xacro (robot description, xacro)
@@ -323,10 +323,20 @@
 						</geometry>
 					</collision>
-					<collision>
-						<origin xyz="0 -0.28 0" rpy="${PI/2} 0 0"/>
-						<geometry>
-							<cylinder length="0.08" radius="0.021707"/>
-						</geometry>
-					</collision>
+					<xacro:if value="${selected_gripper_pad == 'heavy_carry'}">
+						<collision>
+							<origin xyz="${-direction*0.02} -0.26 -0.05" rpy="${PI/2} 0 0"/>
+							<geometry>
+								<box size="0.1 0.1 0.08"/>
+							</geometry>
+						</collision>
+					</xacro:if>
+					<xacro:if value="${selected_gripper_pad == 'default'}">
+						<collision>
+							<origin xyz="0 -0.28 0" rpy="${PI/2} 0 0"/>
+							<geometry>
+								<cylinder length="0.08" radius="0.021707"/>
+							</geometry>
+						</collision>
+					</xacro:if>
 				</xacro:if>
 				<xacro:if value="${selected_gripper_type == 'ag2f90_c' or selected_gripper_type == 'ag2f90_d'}">

File: m6_ccs_description/xacro/robot.xacro (robot description, xacro)
@@ -37,4 +37,8 @@
 	<xacro:if value="${type_arg == 'rg75'}">
 		<xacro:property name="selected_gripper_type" value="rg75"/>
+	</xacro:if>
+	<xacro:if value="${type_arg == 'rg75_heavy'}">
+		<xacro:property name="selected_gripper_type" value="rg75"/>
+		<xacro:property name="selected_gripper_pad" value="heavy_carry"/>
 	</xacro:if>
 	<!-- 适用纯双臂演示场景的配置 -->
@@ -160,13 +164,19 @@
 		<xacro:if value="${selected_gripper_type == 'rg75'}">
 			<xacro:include filename="$(find jodell_description)/xacro/RG75-300.xacro"/>
-			<xacro:RG75-300 name="left" use_flange="true"/>
-			<xacro:RG75-300 name="right" use_flange="true"/>
+			<xacro:RG75-300 name="left" use_flange="true" pad="${selected_gripper_pad}"/>
+			<xacro:RG75-300 name="right" use_flange="true" pad="${selected_gripper_pad}"/>
 			<joint name="left_gripper_base_joint" type="fixed">
 				<parent link="left_tcp"/>
 				<child link="left_flange"/>
+				<xacro:if value="${selected_gripper_pad == 'heavy_carry'}">
+					<origin rpy="0 0 ${PI/2}"/>
+				</xacro:if>
 			</joint>
 			<joint name="right_gripper_base_joint" type="fixed">
 				<parent link="right_tcp"/>
 				<child link="right_flange"/>
+				<xacro:if value="${selected_gripper_pad == 'heavy_carry'}">
+					<origin rpy="0 0 ${PI/2}"/>
+				</xacro:if>
 			</joint>
 		</xacro:if>
