Commit message: feat(m6_ccs): arm visual skins (fiveages_w2, agibot_g2, sinopec) in-package
Co-authored-by: Cursor <cursoragent@cursor.com>

File: m6_ccs_description/xacro/arm.xacro (robot description, xacro)
@@ -4,19 +4,20 @@
 	<xacro:property name="PI" value="3.1415926535897931"/>
 	<xacro:property name="collider_type" value="$(arg collider)"/>
-	<xacro:macro name="M6_CCS" params="name:='' direction:=1 style:=default">
+	<xacro:macro name="M6_CCS" params="name:='' direction:=1 skin:='default' variant:=''">
 		<xacro:property name="prefix" value="${name + '_' if name else ''}"/>
-		<!-- Set visual and collision package/path based on style -->
+		<!-- Visual skins live under m6_ccs_description/meshes/{skin}/[sinopec]/ -->
 		<xacro:property name="visual_package" value="m6_ccs_description"/>
 		<xacro:property name="visual_path" value=""/>
+		<xacro:if value="${skin == 'fiveages_w2' and variant == 'sinopec'}">
+			<xacro:property name="visual_path" value="fiveages_w2/sinopec/"/>
+		</xacro:if>
+		<xacro:if value="${skin == 'fiveages_w2' and variant != 'sinopec'}">
+			<xacro:property name="visual_path" value="fiveages_w2/"/>
+		</xacro:if>
+		<xacro:if value="${skin == 'agibot_g2'}">
+			<xacro:property name="visual_path" value="agibot_g2/"/>
+		</xacro:if>
 		<xacro:property name="collision_package" value="m6_ccs_description"/>
 		<xacro:property name="collision_path" value=""/>
-		<xacro:if value="${style == 'fiveages_w2'}">
-			<xacro:property name="visual_package" value="fiveages_w2_description"/>
-			<xacro:property name="visual_path" value="arm/"/>
-		</xacro:if>
-		<xacro:if value="${style == 'agibot_g2'}">
-			<xacro:property name="visual_package" value="agibot_g2_description"/>
-			<xacro:property name="visual_path" value="arm/"/>
-		</xacro:if>
 		<!-- Base Link -->
 		<link name="${prefix}base_link">

File: m6_ccs_description/xacro/robot.xacro (robot description, xacro)
@@ -2,4 +2,6 @@
 <robot name="M6_CCS" xmlns:xacro="http://www.ros.org/wiki/xacro">
 	<xacro:arg name="collider" default="convex"/>
+	<xacro:arg name="skin" default="default"/>
+	<xacro:arg name="variant" default=""/>
 	<xacro:arg name="type" default="dual"/>
 	<xacro:arg name="scene" default=""/>
@@ -76,5 +78,5 @@
 	<!-- 单左臂（不包括 usb-90c 场景） -->
 	<xacro:if value="${selected_arm_config == 'left' and selected_scene != 'usb-90c'}">
-		<xacro:M6_CCS/>
+		<xacro:M6_CCS skin="$(arg skin)" variant="$(arg variant)"/>
 		<xacro:if value="${selected_gripper_type == 'rg75'}">
 			<xacro:include filename="$(find jodell_description)/xacro/RG75-300.xacro"/>
@@ -88,5 +90,5 @@
 	<!-- 单右臂 -->
 	<xacro:if value="${selected_arm_config == 'right'}">
-		<xacro:M6_CCS direction="-1"/>
+		<xacro:M6_CCS direction="-1" skin="$(arg skin)" variant="$(arg variant)"/>
 	</xacro:if>
 	<!-- 双臂配置 -->
@@ -144,6 +146,6 @@
 		</xacro:unless>
 		<!-- 双臂和末端执行器（两种场景共用） -->
-		<xacro:M6_CCS name="left"/>
-		<xacro:M6_CCS name="right" direction="-1"/>
+		<xacro:M6_CCS name="left" skin="$(arg skin)" variant="$(arg variant)"/>
+		<xacro:M6_CCS name="right" direction="-1" skin="$(arg skin)" variant="$(arg variant)"/>
 		<xacro:include filename="$(find m6_ccs_description)/xacro/eef_type_resolver.xacro"/>
 		<xacro:set_side_eef_types side="left" type_key="${effective_left_type}"/>
@@ -181,5 +183,5 @@
 		</link>
 		<xacro:LeftArmMount parent="base"/>
-		<xacro:M6_CCS name="left"/>
+		<xacro:M6_CCS name="left" skin="$(arg skin)" variant="$(arg variant)"/>
 		<xacro:include filename="$(find changingtek_description)/xacro/AG2F90-C.xacro"/>
 		<xacro:AG2F90-C name="" use_flange="true"/>
