Commit message: update default task info param; default speed change to 100

File: m6_ccs_description/xacro/arm.xacro (robot description, xacro)
@@ -2,8 +2,12 @@
 <robot xmlns:xacro="http://www.ros.org/wiki/xacro">
 	<xacro:arg name="collider" default="convex"/>
+	<!-- Shared with eefs.xacro / parent robot.xacro; planning URDF injects true via robot_common_launch -->
+	<xacro:arg name="eef_fixed_joints" default="false"/>
 	<xacro:property name="PI" value="3.1415926535897931"/>
 	<xacro:property name="collider_type" value="$(arg collider)"/>
 	<xacro:macro name="M6_CCS" params="name:='' direction:=1 skin:='default' variant:=''">
 		<xacro:property name="prefix" value="${name + '_' if name else ''}"/>
+		<!-- OCS2 planning URDF (eef_fixed_joints): tighten joint4 upper; viz / ros2_control keep hardware limits -->
+		<xacro:property name="joint4_upper" value="${0 if '$(arg eef_fixed_joints)' == 'true' else PI*58/180}"/>
 		<!-- Visual skins live under m6_ccs_description/meshes/{skin}/[sinopec]/ -->
 		<xacro:property name="visual_package" value="m6_ccs_description"/>
@@ -206,5 +210,5 @@
 			<child link="${prefix}link4"/>
 			<axis xyz="0 0 1"/>
-			<limit lower="-${PI*143/180}" upper="${PI*58/180}" effort="66" velocity="${PI}"/>
+			<limit lower="-${PI*143/180}" upper="${joint4_upper}" effort="66" velocity="${PI}"/>
 		</joint>
 		<!-- Link 5 - Mirrored COM and partial inertia -->

File: m6_ccs_description/xacro/robot.xacro (robot description, xacro)
@@ -7,5 +7,5 @@
 	<xacro:arg name="left_type" default=""/>
 	<xacro:arg name="right_type" default=""/>
-	<xacro:arg name="eef_fixed_joints" default="false"/>
+	<!-- eef_fixed_joints: declared in arm.xacro (included below); used by EndEffectors -->
 	<!-- 从 type 参数解析 arm_config / 对称末端 -->
 	<xacro:property name="type_arg" value="$(arg type)"/>

File: m6_ccs_description/xacro/ros2_control/robot.xacro (robot description, xacro)
@@ -13,6 +13,6 @@
 	<xacro:arg name="left_dyn_param" default=""/>
 	<xacro:arg name="right_dyn_param" default=""/>
-	<xacro:arg name="max_joint_speed" default="50"/>
-	<xacro:arg name="max_joint_acceleration" default="30"/>
+	<xacro:arg name="max_joint_speed" default="100"/>
+	<xacro:arg name="max_joint_acceleration" default="100"/>
 	<xacro:arg name="usb_left_port" default="/dev/ttyUSB0"/>
 	<xacro:arg name="usb_right_port" default="/dev/ttyUSB2"/>

Commit message: Add TCP offset parameters for left and right arms in robot.xacro and update M6_CCS macro

File: m6_ccs_description/xacro/arm.xacro (robot description, xacro)
@@ -6,5 +6,5 @@
 	<xacro:property name="PI" value="3.1415926535897931"/>
 	<xacro:property name="collider_type" value="$(arg collider)"/>
-	<xacro:macro name="M6_CCS" params="name:='' direction:=1 skin:='default' variant:=''">
+	<xacro:macro name="M6_CCS" params="name:='' direction:=1 skin:='default' variant:='' tcp_offset_xyz:='0 0 0' tcp_offset_rpy:='0 0 0'">
 		<xacro:property name="prefix" value="${name + '_' if name else ''}"/>
 		<!-- OCS2 planning URDF (eef_fixed_joints): tighten joint4 upper; viz / ros2_control keep hardware limits -->
@@ -337,4 +337,12 @@
 			<child link="${prefix}tcp"/>
 		</joint>
+		<!-- Virtual tool frame for planning/control. It is a sibling of the physical
+		     end-effector subtree, so changing the offset never moves hand/gripper geometry. -->
+		<link name="${prefix}tcp_offset"/>
+		<joint name="${prefix}tcp_offset_joint" type="fixed">
+			<origin xyz="${tcp_offset_xyz}" rpy="${tcp_offset_rpy}"/>
+			<parent link="${prefix}tcp"/>
+			<child link="${prefix}tcp_offset"/>
+		</joint>
 	</xacro:macro>
 </robot>

File: m6_ccs_description/xacro/robot.xacro (robot description, xacro)
@@ -7,4 +7,8 @@
 	<xacro:arg name="left_type" default=""/>
 	<xacro:arg name="right_type" default=""/>
+	<xacro:arg name="left_tcp_offset_xyz" default="0 0 0"/>
+	<xacro:arg name="left_tcp_offset_rpy" default="0 0 0"/>
+	<xacro:arg name="right_tcp_offset_xyz" default="0 0 0"/>
+	<xacro:arg name="right_tcp_offset_rpy" default="0 0 0"/>
 	<!-- eef_fixed_joints: declared in arm.xacro (included below); used by EndEffectors -->
 	<!-- 从 type 参数解析 arm_config / 对称末端 -->
@@ -55,5 +59,7 @@
 	<!-- 单左臂 -->
 	<xacro:if value="${selected_arm_config == 'left'}">
-		<xacro:M6_CCS skin="$(arg skin)" variant="$(arg variant)"/>
+		<xacro:M6_CCS skin="$(arg skin)" variant="$(arg variant)"
+			tcp_offset_xyz="$(arg left_tcp_offset_xyz)"
+			tcp_offset_rpy="$(arg left_tcp_offset_rpy)"/>
 		<xacro:if value="${selected_gripper_type == 'rg75'}">
 			<xacro:include filename="$(find jodell_description)/xacro/RG75-300.xacro"/>
@@ -67,5 +73,7 @@
 	<!-- 单右臂 -->
 	<xacro:if value="${selected_arm_config == 'right'}">
-		<xacro:M6_CCS direction="-1" skin="$(arg skin)" variant="$(arg variant)"/>
+		<xacro:M6_CCS direction="-1" skin="$(arg skin)" variant="$(arg variant)"
+			tcp_offset_xyz="$(arg right_tcp_offset_xyz)"
+			tcp_offset_rpy="$(arg right_tcp_offset_rpy)"/>
 	</xacro:if>
 	<!-- 双臂配置 -->
@@ -108,6 +116,10 @@
 			<xacro:DualArmMount parent="arm_base"/>
 		</xacro:unless>
-		<xacro:M6_CCS name="left" skin="$(arg skin)" variant="$(arg variant)"/>
-		<xacro:M6_CCS name="right" direction="-1" skin="$(arg skin)" variant="$(arg variant)"/>
+		<xacro:M6_CCS name="left" skin="$(arg skin)" variant="$(arg variant)"
+			tcp_offset_xyz="$(arg left_tcp_offset_xyz)"
+			tcp_offset_rpy="$(arg left_tcp_offset_rpy)"/>
+		<xacro:M6_CCS name="right" direction="-1" skin="$(arg skin)" variant="$(arg variant)"
+			tcp_offset_xyz="$(arg right_tcp_offset_xyz)"
+			tcp_offset_rpy="$(arg right_tcp_offset_rpy)"/>
 		<xacro:include filename="$(find m6_ccs_description)/xacro/eef_type_resolver.xacro"/>
 		<xacro:set_side_eef_types side="left" type_key="${effective_left_type}"/>
