Commit message: add template support

File: m6_ccs_description/xacro/arm_mount.xacro (robot description, xacro)
@@ -2,30 +2,46 @@
 <robot xmlns:xacro="http://www.ros.org/wiki/xacro">
 	<xacro:property name="PI" value="3.1415926535897931"/>
+	<!-- Empty arm_base + dual mounts (standalone arms viz / component URDF). -->
+	<xacro:macro name="DualArmBase" params="
+		left_xyz:='0 0.062 0'
+		right_xyz:='0 -0.062 0'
+		left_rpy:=''
+		right_rpy:=''
+	">
+		<link name="arm_base"/>
+		<xacro:DualArmMount parent="arm_base"
+			left_xyz="${left_xyz}" right_xyz="${right_xyz}"
+			left_rpy="${left_rpy}" right_rpy="${right_rpy}"/>
+	</xacro:macro>
 	<!--
-	  Dual-arm mount joints on arm_base (mechanism only).
-	  Spacing must be supplied via xacro args (from host config/xacro/mount.yaml
-	  through robot_common_launch). No built-in product presets here.
+	  Dual-arm fixed mounts on an existing parent (e.g. W2 / G2 arm_base).
+	  Defaults: M6/W2 style (±Y, roll ±90°). Override xyz/rpy at call site when needed.
 	-->
-	<xacro:macro name="set_arm_mount_properties" params="arm_half_spacing arm_mount_z">
-		<xacro:property name="effective_arm_half_spacing" value="${arm_half_spacing}" scope="parent"/>
-		<xacro:property name="effective_arm_mount_z" value="${arm_mount_z}" scope="parent"/>
-	</xacro:macro>
-	<xacro:macro name="DualArmMountJoints" params="parent">
+	<xacro:macro name="DualArmMount" params="
+		parent
+		left_xyz:='0 0.062 0'
+		right_xyz:='0 -0.062 0'
+		left_rpy:=''
+		right_rpy:=''
+	">
+		<xacro:property name="_left_rpy" value="${left_rpy if left_rpy != '' else '-'+str(PI/2)+' 0 0'}"/>
+		<xacro:property name="_right_rpy" value="${right_rpy if right_rpy != '' else str(PI/2)+' 0 0'}"/>
 		<joint name="left_arm_base_joint" type="fixed">
 			<parent link="${parent}"/>
 			<child link="left_base_link"/>
-			<origin rpy="-${PI/2} 0 0" xyz="0.0 ${effective_arm_half_spacing} ${effective_arm_mount_z}"/>
+			<origin xyz="${left_xyz}" rpy="${_left_rpy}"/>
 		</joint>
 		<joint name="right_arm_base_joint" type="fixed">
 			<parent link="${parent}"/>
 			<child link="right_base_link"/>
-			<origin rpy="${PI/2} 0 0" xyz="0.0 ${-effective_arm_half_spacing} ${effective_arm_mount_z}"/>
+			<origin xyz="${right_xyz}" rpy="${_right_rpy}"/>
 		</joint>
 	</xacro:macro>
-	<xacro:macro name="LeftArmMountJoint" params="parent">
+	<xacro:macro name="LeftArmMount" params="parent left_xyz:='0 0.062 0' left_rpy:=''">
+		<xacro:property name="_left_rpy" value="${left_rpy if left_rpy != '' else '-'+str(PI/2)+' 0 0'}"/>
 		<joint name="left_arm_base_joint" type="fixed">
 			<parent link="${parent}"/>
 			<child link="left_base_link"/>
-			<origin rpy="-${PI/2} 0 0" xyz="0.0 ${effective_arm_half_spacing} ${effective_arm_mount_z}"/>
+			<origin xyz="${left_xyz}" rpy="${_left_rpy}"/>
 		</joint>
 	</xacro:macro>

File: m6_ccs_description/xacro/robot.xacro (robot description, xacro)
@@ -7,13 +7,8 @@
 	<xacro:arg name="right_type" default=""/>
 	<xacro:arg name="eef_fixed_joints" default="false"/>
-	<!-- Arm mount: values from config/xacro/mount.yaml via launch (see arm_mount.xacro) -->
-	<xacro:arg name="arm_half_spacing" default=""/>
-	<xacro:arg name="arm_mount_z" default=""/>
 	<!-- 从 type 参数解析出 arm_config、gripper_type 和 scene -->
 	<xacro:property name="type_arg" value="$(arg type)"/>
 	<xacro:property name="left_type_arg" value="$(arg left_type)"/>
 	<xacro:property name="right_type_arg" value="$(arg right_type)"/>
-	<xacro:property name="arm_half_spacing_arg" value="$(arg arm_half_spacing)"/>
-	<xacro:property name="arm_mount_z_arg" value="$(arg arm_mount_z)"/>
 	<xacro:property name="effective_left_type" value="${left_type_arg if left_type_arg != '' else type_arg}"/>
 	<xacro:property name="effective_right_type" value="${right_type_arg if right_type_arg != '' else type_arg}"/>
@@ -79,7 +74,4 @@
 	<xacro:include filename="$(find m6_ccs_description)/xacro/arm.xacro"/>
 	<xacro:include filename="$(find m6_ccs_description)/xacro/arm_mount.xacro"/>
-	<xacro:set_arm_mount_properties
-		arm_half_spacing="${arm_half_spacing_arg}"
-		arm_mount_z="${arm_mount_z_arg}"/>
 	<!-- 单左臂（不包括 usb-90c 场景） -->
 	<xacro:if value="${selected_arm_config == 'left' and selected_scene != 'usb-90c'}">
@@ -120,6 +112,5 @@
 				<child link="arm_base"/>
 			</joint>
-			<!-- Left / Right Arm mounts (desktop preset: wider spacing + raised z) -->
-			<xacro:DualArmMountJoints parent="arm_base"/>
+			<xacro:DualArmMount parent="arm_base" left_xyz="0 0.12 0.701" right_xyz="0 -0.12 0.701"/>
 			<xacro:if value="${selected_gripper_type == 'none'}">
 				<link name="right_eef"/>
@@ -150,5 +141,5 @@
 				<child link="arm_base"/>
 			</joint>
-			<xacro:DualArmMountJoints parent="arm_base"/>
+			<xacro:DualArmMount parent="arm_base"/>
 		</xacro:unless>
 		<!-- 双臂和末端执行器（两种场景共用） -->
@@ -189,5 +180,5 @@
 			</collision>
 		</link>
-		<xacro:LeftArmMountJoint parent="base"/>
+		<xacro:LeftArmMount parent="base"/>
 		<xacro:M6_CCS name="left"/>
 		<xacro:include filename="$(find changingtek_description)/xacro/AG2F90-C.xacro"/>
