Commit message: add dual configuration for m6 ccs

File: m6_ccs_description/xacro/robot.xacro (robot description, xacro)
@@ -10,3 +10,20 @@
 		<xacro:M6_CCS direction="-1"/>
 	</xacro:if>
+	<xacro:if value="${'$(arg type)' == 'dual'}">
+		<link name="base_link"/>
+		<!-- Left Arm -->
+		<joint name="left_arm_base_joint" type="fixed">
+			<parent link="base_link"/>
+			<child link="left_base_link"/>
+			<origin rpy="-1.5708 1.5708 0" xyz="0.0 0.05 0"/>
+		</joint>
+		<!-- Right Arm -->
+		<joint name="right_arm_base_joint" type="fixed">
+			<parent link="base_link"/>
+			<child link="right_base_link"/>
+			<origin rpy="1.5708 1.5708 0" xyz="0.0 -0.05 0"/>
+		</joint>
+		<xacro:M6_CCS name="left"/>
+		<xacro:M6_CCS name="right" direction="-1"/>
+	</xacro:if>
 </robot>

File: m6_ccs_description/xacro/ros2_control/robot.xacro (robot description, xacro)
@@ -26,5 +26,11 @@
       </xacro:if>
     </hardware>
-    <xacro:m6_interfaces name=""/>
+    <xacro:if value="${'$(arg type)' == 'dual'}">
+      <xacro:m6_interfaces name="left"/>
+      <xacro:m6_interfaces name="right"/>
+    </xacro:if>
+    <xacro:unless value="${'$(arg type)' == 'dual'}">
+      <xacro:m6_interfaces name=""/>
+    </xacro:unless>
   </ros2_control>
   <xacro:arg name="gazebo" default="false"/>

Commit message: add tianji dual base

File: m6_ccs_description/xacro/robot.xacro (robot description, xacro)
@@ -11,10 +11,16 @@
 	</xacro:if>
 	<xacro:if value="${'$(arg type)' == 'dual'}">
-		<link name="base_link"/>
+		<link name="base_link">
+			<visual>
+				<geometry>
+					<mesh filename="file://$(find m6_ccs_description)/meshes/dual_base.obj"/>
+				</geometry>
+			</visual>
+		</link>
 		<!-- Left Arm -->
 		<joint name="left_arm_base_joint" type="fixed">
 			<parent link="base_link"/>
 			<child link="left_base_link"/>
-			<origin rpy="-1.5708 1.5708 0" xyz="0.0 0.05 0"/>
+			<origin rpy="-1.5708 1.5708 0" xyz="0.0 0.12 0.701"/>
 		</joint>
 		<!-- Right Arm -->
@@ -22,5 +28,5 @@
 			<parent link="base_link"/>
 			<child link="right_base_link"/>
-			<origin rpy="1.5708 1.5708 0" xyz="0.0 -0.05 0"/>
+			<origin rpy="1.5708 1.5708 0" xyz="0.0 -0.12 0.701"/>
 		</joint>
 		<xacro:M6_CCS name="left"/>

Commit message: add tianji test

File: m6_ccs_description/xacro/robot.xacro (robot description, xacro)
@@ -33,3 +33,33 @@
 		<xacro:M6_CCS name="right" direction="-1"/>
 	</xacro:if>
+	<xacro:if value="${'$(arg type)' == 'usb-90c'}">
+		<link name="base_link"/>
+		<!-- Left Arm -->
+		<joint name="base_joint" type="fixed">
+			<parent link="base_link"/>
+			<child link="base"/>
+			<origin rpy="0 0 -${PI/2}"/>
+		</joint>
+		<link name="base">
+			<visual>
+				<geometry>
+					<mesh filename="file://$(find m6_ccs_description)/meshes/dual_base.obj"/>
+				</geometry>
+			</visual>
+		</link>
+		<!-- Left Arm -->
+		<joint name="left_arm_base_joint" type="fixed">
+			<parent link="base"/>
+			<child link="left_base_link"/>
+			<origin rpy="-${PI/2} 0 0" xyz="0.0 0.12 0.701"/>
+		</joint>
+		<xacro:M6_CCS name="left"/>
+		<xacro:include filename="$(find changingtek_description)/xacro/AG2F90-C.xacro"/>
+		<xacro:AG2F90-C name="" use_flange="true"/>
+		<joint name="gripper_fix" type="fixed">
+			<parent link="left_link7"/>
+			<child link="flange"/>
+			<origin xyz="0 -0.0995 0" rpy=" ${PI/2} 0 0"/>
+		</joint>
+	</xacro:if>
 </robot>

File: m6_ccs_description/xacro/ros2_control/robot.xacro (robot description, xacro)
@@ -1,68 +1,70 @@
 <?xml version="1.0"?>
 <robot xmlns:xacro="http://www.ros.org/wiki/xacro" name="AR5">
-  <xacro:arg name="ros2_control_hardware_type" default="mock_components"/>
-  <link name="world"/>
-  <joint name="world_fixed" type="fixed">
-    <parent link="world"/>
-    <child link="base_link"/>
-    <origin/>
-  </joint>
-  <xacro:include filename="$(find m6_ccs_description)/xacro/robot.xacro"/>
-  <xacro:include filename="$(find m6_ccs_description)/xacro/ros2_control/interfaces.xacro"/>
-  <ros2_control name="M6_CCS_System" type="system">
-    <hardware>
-      <xacro:if value="${'$(arg ros2_control_hardware_type)' == 'gz'}">
-        <plugin>gz_ros2_control/GazeboSimSystem</plugin>
-      </xacro:if>
-      <xacro:if value="${'$(arg ros2_control_hardware_type)' == 'mock_components'}">
-        <plugin>mock_components/GenericSystem</plugin>
-      </xacro:if>
-      <xacro:if value="${'$(arg ros2_control_hardware_type)' == 'isaac'}">
-        <plugin>topic_based_ros2_control/TopicBasedSystem</plugin>
-        <param name="joint_commands_topic">/isaac/joint_command</param>
-        <param name="joint_states_topic">/isaac/joint_states</param>
-        <param name="sum_wrapped_joint_states">false</param>
-        <param name="initialize_commands_from_state">true</param>
-      </xacro:if>
-       <xacro:if value="${'$(arg ros2_control_hardware_type)' == 'real'}">
-        <plugin>tj2_ros2_control/TJ2Hardware</plugin>
-        <xacro:if value="${'$(arg type)' == 'dual'}">
-          <param name="left_right_arm">2</param>
-        </xacro:if>
-         <xacro:unless value="${'$(arg type)' == 'dual'}">
-          <xacro:if value="${'$(arg type)' == 'left'}">
-            <param name="left_right_arm">0</param>
-          </xacro:if>
-          <xacro:unless value="${'$(arg type)' == 'left'}">
-            <param name="left_right_arm">1</param>
-        </xacro:unless>
-    </xacro:unless>
-      </xacro:if>
-    </hardware>
-    <xacro:if value="${'$(arg type)' == 'dual'}">
-      <xacro:m6_interfaces name="left"/>
-      <xacro:m6_interfaces name="right"/>
-    </xacro:if>
-    <xacro:unless value="${'$(arg type)' == 'dual'}">
-       <xacro:if value="${'$(arg type)' == 'left'}">
-        <xacro:m6_interfaces name=""/>
-       </xacro:if>
-       <xacro:unless value="${'$(arg type)' == 'left'}">
-        <xacro:m6_interfaces name=""/>
-       </xacro:unless>
-    </xacro:unless>
-  </ros2_control>
-  <xacro:arg name="gazebo" default="false"/>
-  <xacro:if value="$(arg gazebo)">
-    <gazebo>
-      <plugin filename="gz_ros2_control-system" name="gz_ros2_control::GazeboSimROS2ControlPlugin">
-        <xacro:if value="${'$(arg type)' == 'left'}">
-          <parameters>$(find rokae_ar5_description)/config/ros2_control/ros2_controllers.yaml</parameters>
-        </xacro:if>
-        <xacro:if value="${'$(arg type)' == 'right'}">
-          <parameters>$(find rokae_ar5_description)/config/ros2_control/right.yaml</parameters>
-        </xacro:if>
-      </plugin>
-    </gazebo>
-  </xacro:if>
+	<xacro:arg name="ros2_control_hardware_type" default="mock_components"/>
+	<link name="world"/>
+	<joint name="world_fixed" type="fixed">
+		<parent link="world"/>
+		<child link="base_link"/>
+		<origin/>
+	</joint>
+	<xacro:include filename="$(find m6_ccs_description)/xacro/robot.xacro"/>
+	<xacro:include filename="$(find m6_ccs_description)/xacro/ros2_control/interfaces.xacro"/>
+	<ros2_control name="M6_CCS_System" type="system">
+		<hardware>
+			<xacro:if value="${'$(arg ros2_control_hardware_type)' == 'gz'}">
+				<plugin>gz_ros2_control/GazeboSimSystem</plugin>
+			</xacro:if>
+			<xacro:if value="${'$(arg ros2_control_hardware_type)' == 'mock_components'}">
+				<plugin>mock_components/GenericSystem</plugin>
+			</xacro:if>
+			<xacro:if value="${'$(arg ros2_control_hardware_type)' == 'isaac'}">
+				<plugin>topic_based_ros2_control/TopicBasedSystem</plugin>
+				<param name="joint_commands_topic">/isaac/joint_command</param>
+				<param name="joint_states_topic">/isaac/joint_states</param>
+				<param name="sum_wrapped_joint_states">false</param>
+				<param name="initialize_commands_from_state">true</param>
+			</xacro:if>
+			<xacro:if value="${'$(arg ros2_control_hardware_type)' == 'real'}">
+				<plugin>tj2_ros2_control/TJ2Hardware</plugin>
+				<xacro:if value="${'$(arg type)' == 'dual'}">
+					<param name="left_right_arm">2</param>
+				</xacro:if>
+				<xacro:unless value="${'$(arg type)' == 'dual'}">
+					<xacro:if value="${'$(arg type)' == 'left'}">
+						<param name="left_right_arm">0</param>
+					</xacro:if>
+					<xacro:unless value="${'$(arg type)' == 'left'}">
+						<param name="left_right_arm">1</param>
+					</xacro:unless>
+				</xacro:unless>
+			</xacro:if>
+		</hardware>
+		<xacro:if value="${'$(arg type)' == 'dual'}">
+			<xacro:m6_interfaces name="left"/>
+			<xacro:m6_interfaces name="right"/>
+		</xacro:if>
+		<xacro:unless value="${'$(arg type)' == 'dual'}">
+			<xacro:if value="${'$(arg type)' == 'usb-90c'}">
+				<xacro:m6_interfaces name="left"/>
+				<xacro:include filename="$(find changingtek_description)/xacro/ros2_control/AG2F90-C.xacro"/>
+				<xacro:ag2f90c_interfaces name=""/>
+			</xacro:if>
+			<xacro:unless value="${'$(arg type)' == 'usb-90c'}">
+				<xacro:m6_interfaces name=""/>
+			</xacro:unless>
+		</xacro:unless>
+	</ros2_control>
+	<xacro:arg name="gazebo" default="false"/>
+	<xacro:if value="$(arg gazebo)">
+		<gazebo>
+			<plugin filename="gz_ros2_control-system" name="gz_ros2_control::GazeboSimROS2ControlPlugin">
+				<xacro:if value="${'$(arg type)' == 'left'}">
+					<parameters>$(find rokae_ar5_description)/config/ros2_control/ros2_controllers.yaml</parameters>
+				</xacro:if>
+				<xacro:if value="${'$(arg type)' == 'right'}">
+					<parameters>$(find rokae_ar5_description)/config/ros2_control/right.yaml</parameters>
+				</xacro:if>
+			</plugin>
+		</gazebo>
+	</xacro:if>
 </robot>

Commit message: add dual config

File: m6_ccs_description/xacro/robot.xacro (robot description, xacro)
@@ -11,4 +11,33 @@
 	</xacro:if>
 	<xacro:if value="${'$(arg type)' == 'dual'}">
+		<link name="base_link"/>
+		<link name="arm_base">
+			<collision>
+				<origin xyz="0.0091 0 -0.086"/>
+				<geometry>
+					<box size="0.2509 0.35 0.5029"/>
+				</geometry>
+			</collision>
+		</link>
+		<joint name="arm_base_joint" type="fixed">
+			<parent link="base_link"/>
+			<child link="arm_base"/>
+		</joint>
+		<!-- Left Arm -->
+		<joint name="left_arm_base_joint" type="fixed">
+			<parent link="arm_base"/>
+			<child link="left_base_link"/>
+			<origin rpy="-1.5708 0 0" xyz="0.0 0.062 0"/>
+		</joint>
+		<!-- Right Arm -->
+		<joint name="right_arm_base_joint" type="fixed">
+			<parent link="arm_base"/>
+			<child link="right_base_link"/>
+			<origin rpy="1.5708 0 0" xyz="0 -0.062 0"/>
+		</joint>
+		<xacro:M6_CCS name="left" collider="$(arg collider)"/>
+		<xacro:M6_CCS name="right" direction="-1" collider="$(arg collider)"/>
+	</xacro:if>
+	<xacro:if value="${'$(arg type)' == 'dual_desktop'}">
 		<link name="base_link">
 			<visual>

Commit message: 修改碰撞体 配置split body control

File: m6_ccs_description/xacro/robot.xacro (robot description, xacro)
@@ -14,7 +14,7 @@
 		<link name="arm_base">
 			<collision>
-				<origin xyz="0.0091 0 -0.086"/>
+				<origin xyz="0.0091 0 -0.2"/>
 				<geometry>
-					<box size="0.2509 0.35 0.5029"/>
+					<box size="0.2000 0.32 0.5029"/>
 				</geometry>
 			</collision>

Commit message: dual arm config with jodell gripper

File: m6_ccs_description/xacro/robot.xacro (robot description, xacro)
@@ -51,4 +51,19 @@
 				<child link="right_flange"/>
 				<origin xyz="0 -0.0995 0" rpy=" ${PI/2} 0 0"/>
+			</joint>
+		</xacro:if>
+		<xacro:if value="${'$(arg type)' == 'dual_rg75'}">
+			<xacro:include filename="$(find jodell_description)/xacro/RG75-300.xacro"/>
+			<xacro:RG75-300 name="left" use_flange="true"/>
+			<xacro:RG75-300 name="right" use_flange="true"/>
+			<joint name="left_gripper_base_joint" type="fixed">
+				<origin xyz="0 0 -0.0045" rpy="${PI/2} 0 0"/>
+				<parent link="left_tcp"/>
+				<child link="left_flange"/>
+			</joint>
+			<joint name="right_gripper_base_joint" type="fixed">
+				<origin xyz="0 0 -0.0045" rpy="${PI/2} 0 0"/>
+				<parent link="right_tcp"/>
+				<child link="right_flange"/>
 			</joint>
 		</xacro:if>

File: m6_ccs_description/xacro/ros2_control/robot.xacro (robot description, xacro)
@@ -28,5 +28,5 @@
 			<xacro:if value="${'$(arg ros2_control_hardware_type)' == 'real'}">
 				<plugin>marvin_ros2_control/MarvinHardware</plugin>
-				<xacro:if value="${'$(arg type)' == 'dual' or '$(arg type)' == 'dual_ag2f90'}">
+				<xacro:if value="${'$(arg type)' == 'dual' or '$(arg type)' == 'dual_ag2f90' or '$(arg type)' == 'dual_rg75'}">
 					<param name="left_right_arm">2</param>
 				</xacro:if>
@@ -55,5 +55,5 @@
 			</xacro:unless>
 		</hardware>
-		<xacro:if value="${'$(arg type)' == 'dual' or '$(arg type)' == 'dual_ag2f90'}">
+		<xacro:if value="${'$(arg type)' == 'dual' or '$(arg type)' == 'dual_ag2f90'  or '$(arg type)' == 'dual_rg75'}">
 			<xacro:m6_interfaces name="left"/>
 			<xacro:m6_interfaces name="right"/>
@@ -63,6 +63,11 @@
 				<xacro:ag2f90c_interfaces name="right"/>
 			</xacro:if>
+			<xacro:if value="${'$(arg type)' == 'dual_rg75'}">
+				<xacro:include filename="$(find jodell_description)/xacro/ros2_control/RG75-300.xacro"/>
+				<xacro:rg75_interfaces name="left"/>
+				<xacro:rg75_interfaces name="right"/>
+			</xacro:if>
 		</xacro:if>
-		<xacro:unless value="${'$(arg type)' == 'dual' or '$(arg type)' == 'dual_ag2f90'}">
+		<xacro:unless value="${'$(arg type)' == 'dual' or '$(arg type)' == 'dual_ag2f90'  or '$(arg type)' == 'dual_rg75'}">
 			<xacro:if value="${'$(arg type)' == 'usb-90c'}">
 				<xacro:m6_interfaces name="left"/>
