Commit message: Add Gripper Hardware Common

File: m6_ccs_description/xacro/robot.xacro (robot description, xacro)
@@ -3,40 +3,107 @@
 	<xacro:arg name="collider" default="convex"/>
 	<xacro:arg name="type" default="left"/>
+	<xacro:arg name="scene" default=""/>
+	<!-- 从 type 参数解析出 arm_config、gripper_type 和 scene -->
+	<xacro:property name="type_arg" value="$(arg type)"/>
+	<!-- 默认值 -->
+	<xacro:property name="selected_arm_config" value="dual"/>
+	<xacro:property name="selected_gripper_type" value="none"/>
+	<xacro:property name="selected_scene" value=""/>
+	<!-- 从 type 解析 arm_config 和 gripper_type -->
+	<!-- 单臂配置 -->
+	<xacro:if value="${type_arg == 'left'}">
+		<xacro:property name="selected_arm_config" value="left"/>
+	</xacro:if>
+	<xacro:if value="${type_arg == 'right'}">
+		<xacro:property name="selected_arm_config" value="right"/>
+	</xacro:if>
+	<xacro:if value="${type_arg == 'usb-90c'}">
+		<xacro:property name="selected_arm_config" value="left"/>
+		<xacro:property name="selected_gripper_type" value="ag2f90"/>
+		<xacro:property name="selected_scene" value="usb-90c"/>
+	</xacro:if>
+	<!-- 双臂配置 -->
+	<xacro:if value="${type_arg == 'dual_ag2f90'}">
+		<xacro:property name="selected_gripper_type" value="ag2f90"/>
+	</xacro:if>
+	<xacro:if value="${type_arg == 'dual_rg75'}">
+		<xacro:property name="selected_gripper_type" value="rg75"/>
+	</xacro:if>
+	<xacro:if value="${type_arg == 'dual_desktop'}">
+		<xacro:property name="selected_scene" value="desktop"/>
+	</xacro:if>
 	<xacro:include filename="$(find m6_ccs_description)/xacro/arm.xacro"/>
-	<xacro:if value="${'$(arg type)' == 'left'}">
+	<!-- 单左臂（不包括 usb-90c 场景） -->
+	<xacro:if value="${selected_arm_config == 'left' and selected_scene != 'usb-90c'}">
 		<xacro:M6_CCS collider="$(arg collider)"/>
 	</xacro:if>
-	<xacro:if value="${'$(arg type)' == 'right'}">
+	<!-- 单右臂 -->
+	<xacro:if value="${selected_arm_config == 'right'}">
 		<xacro:M6_CCS direction="-1" collider="$(arg collider)"/>
 	</xacro:if>
-	<xacro:if value="${'$(arg type)' == 'dual' or '$(arg type)' == 'dual_ag2f90' or '$(arg type)' == 'dual_rg75'}">
-		<link name="base_link"/>
-		<link name="arm_base">
-			<collision>
-				<origin xyz="0.0091 0 -0.2"/>
-				<geometry>
-					<box size="0.2000 0.32 0.5029"/>
-				</geometry>
-			</collision>
-		</link>
-		<joint name="arm_base_joint" type="fixed">
-			<parent link="base_link"/>
-			<child link="arm_base"/>
-		</joint>
-		<!-- Left Arm -->
-		<joint name="left_arm_base_joint" type="fixed">
-			<parent link="arm_base"/>
-			<child link="left_base_link"/>
-			<origin rpy="-${PI/2} 0 0" xyz="0.0 0.062 0"/>
-		</joint>
-		<!-- Right Arm -->
-		<joint name="right_arm_base_joint" type="fixed">
-			<parent link="arm_base"/>
-			<child link="right_base_link"/>
-			<origin rpy="${PI/2} 0 0" xyz="0 -0.062 0"/>
-		</joint>
+	<!-- 双臂配置 -->
+	<xacro:if value="${selected_arm_config == 'dual'}">
+		<!-- Base link 和 arm_base 根据 scene 设置 -->
+		<xacro:if value="${selected_scene == 'desktop'}">
+			<!-- Desktop 场景：base_link 有视觉和碰撞，没有 arm_base -->
+			<link name="base_link">
+				<visual>
+					<geometry>
+						<mesh filename="file://$(find m6_ccs_description)/meshes/dual_base.obj"/>
+					</geometry>
+				</visual>
+				<collision>
+					<origin xyz="0 0 0.324331"/>
+					<geometry>
+						<box size="0.10045 0.100398 0.648662"/>
+					</geometry>
+				</collision>
+			</link>
+			<!-- Left Arm -->
+			<joint name="left_arm_base_joint" type="fixed">
+				<parent link="base_link"/>
+				<child link="left_base_link"/>
+				<origin rpy="-${PI/2} 0 0" xyz="0.0 0.12 0.701"/>
+			</joint>
+			<!-- Right Arm -->
+			<joint name="right_arm_base_joint" type="fixed">
+				<parent link="base_link"/>
+				<child link="right_base_link"/>
+				<origin rpy="${PI/2} 0 0" xyz="0.0 -0.12 0.701"/>
+			</joint>
+		</xacro:if>
+		<xacro:unless value="${selected_scene == 'desktop'}">
+			<!-- 非 Desktop 场景：base_link 为空，有 arm_base -->
+			<link name="base_link"/>
+			<link name="arm_base">
+				<collision>
+					<origin xyz="0.0091 0 -0.2"/>
+					<geometry>
+						<box size="0.2000 0.32 0.5029"/>
+					</geometry>
+				</collision>
+			</link>
+			<joint name="arm_base_joint" type="fixed">
+				<parent link="base_link"/>
+				<child link="arm_base"/>
+			</joint>
+			<!-- Left Arm -->
+			<joint name="left_arm_base_joint" type="fixed">
+				<parent link="arm_base"/>
+				<child link="left_base_link"/>
+				<origin rpy="-${PI/2} 0 0" xyz="0.0 0.062 0"/>
+			</joint>
+			<!-- Right Arm -->
+			<joint name="right_arm_base_joint" type="fixed">
+				<parent link="arm_base"/>
+				<child link="right_base_link"/>
+				<origin rpy="${PI/2} 0 0" xyz="0 -0.062 0"/>
+			</joint>
+		</xacro:unless>
+		<!-- 双臂和末端执行器（两种场景共用） -->
 		<xacro:M6_CCS name="left" collider="$(arg collider)"/>
 		<xacro:M6_CCS name="right" direction="-1" collider="$(arg collider)"/>
-		<xacro:if value="${'$(arg type)' == 'dual_ag2f90'}">
+		<!-- 双臂末端执行器 -->
+		<xacro:if value="${selected_gripper_type == 'ag2f90'}">
 			<xacro:include filename="$(find changingtek_description)/xacro/AG2F90-C.xacro"/>
 			<xacro:AG2F90-C name="left" use_flange="true"/>
@@ -53,5 +120,5 @@
 			</joint>
 		</xacro:if>
-		<xacro:if value="${'$(arg type)' == 'dual_rg75'}">
+		<xacro:if value="${selected_gripper_type == 'rg75'}">
 			<xacro:include filename="$(find jodell_description)/xacro/RG75-300.xacro"/>
 			<xacro:RG75-300 name="left" use_flange="true"/>
@@ -67,34 +134,6 @@
 		</xacro:if>
 	</xacro:if>
-	<xacro:if value="${'$(arg type)' == 'dual_desktop'}">
-		<link name="base_link">
-			<visual>
-				<geometry>
-					<mesh filename="file://$(find m6_ccs_description)/meshes/dual_base.obj"/>
-				</geometry>
-			</visual>
-			<collision>
-				<origin xyz="0 0 0.324331"/>
-				<geometry>
-					<box size="0.10045 0.100398 0.648662"/>
-				</geometry>
-			</collision>
-		</link>
-		<!-- Left Arm -->
-		<joint name="left_arm_base_joint" type="fixed">
-			<parent link="base_link"/>
-			<child link="left_base_link"/>
-			<origin rpy="-${PI/2} 0 0" xyz="0.0 0.12 0.701"/>
-		</joint>
-		<!-- Right Arm -->
-		<joint name="right_arm_base_joint" type="fixed">
-			<parent link="base_link"/>
-			<child link="right_base_link"/>
-			<origin rpy="${PI/2} 0 0" xyz="0.0 -0.12 0.701"/>
-		</joint>
-		<xacro:M6_CCS name="left" collider="$(arg collider)"/>
-		<xacro:M6_CCS name="right" direction="-1" collider="$(arg collider)"/>
-	</xacro:if>
-	<xacro:if value="${'$(arg type)' == 'usb-90c'}">
+	<!-- USB-90C 配置 -->
+	<xacro:if value="${selected_arm_config == 'left' and selected_scene == 'usb-90c'}">
 		<link name="base_link"/>
 		<!-- Left Arm -->
@@ -124,11 +163,14 @@
 		</joint>
 		<xacro:M6_CCS name="left" collider="$(arg collider)"/>
-		<xacro:include filename="$(find changingtek_description)/xacro/AG2F90-C.xacro"/>
-		<xacro:AG2F90-C name="" use_flange="true"/>
-		<joint name="gripper_fix" type="fixed">
-			<parent link="left_link7"/>
-			<child link="flange"/>
-			<origin xyz="0 -0.0995 0" rpy=" ${PI/2} 0 0"/>
-		</joint>
+		<!-- USB-90C 默认使用 AG2F90 末端 -->
+		<xacro:if value="${selected_gripper_type == 'ag2f90' or selected_gripper_type == 'none'}">
+			<xacro:include filename="$(find changingtek_description)/xacro/AG2F90-C.xacro"/>
+			<xacro:AG2F90-C name="" use_flange="true"/>
+			<joint name="gripper_fix" type="fixed">
+				<parent link="left_link7"/>
+				<child link="flange"/>
+				<origin xyz="0 -0.0995 0" rpy=" ${PI/2} 0 0"/>
+			</joint>
+		</xacro:if>
 	</xacro:if>
 </robot>

File: m6_ccs_description/xacro/ros2_control/robot.xacro (robot description, xacro)
@@ -3,4 +3,5 @@
 	<xacro:arg name="ros2_control_hardware_type" default="mock_components"/>
 	<xacro:arg name="ctrl_mode" default="position"/>
+	<xacro:arg name="type" default="left"/>
 	<link name="world"/>
 	<joint name="world_fixed" type="fixed">
@@ -9,4 +10,5 @@
 		<origin/>
 	</joint>
+	<!-- Include robot.xacro，它会解析 type 并设置 selected_arm_config 和 selected_gripper_type -->
 	<xacro:include filename="$(find m6_ccs_description)/xacro/robot.xacro"/>
 	<xacro:include filename="$(find m6_ccs_description)/xacro/ros2_control/interfaces.xacro"/>
@@ -28,40 +30,22 @@
 			<xacro:if value="${'$(arg ros2_control_hardware_type)' == 'real'}">
 				<plugin>marvin_ros2_control/MarvinHardware</plugin>
-				<xacro:if value="${'$(arg type)' == 'dual' or '$(arg type)' == 'dual_ag2f90' or '$(arg type)' == 'dual_rg75'}">
-					<param name="left_right_arm">2</param>
-				</xacro:if>
-				<xacro:unless value="${'$(arg type)' == 'dual'}">
-					<xacro:if value="${'$(arg type)' == 'left'}">
-						<param name="left_right_arm">0</param>
-					</xacro:if>
-					<xacro:if value="${'$(arg type)' == 'usb-90c'}">
-						<param name="left_right_arm">0</param>
-					</xacro:if>
-					<xacro:if value="${'$(arg type)' == 'right'}">
-						<param name="left_right_arm">1</param>
-					</xacro:if>
-				</xacro:unless>
+				<param name="arm_type">${selected_arm_config}</param>
+				<param name="ctrl_mode">position</param>
+				<param name="gripper_type">${selected_gripper_type}</param>
+				<param name="max_velocity">40</param>
+				<param name="max_acceleration">10</param>
 			</xacro:if>
-			<xacro:if value="${'$(arg ctrl_mode)' == 'position'}">
-				<param name="ctrl_mode">2</param>
-			</xacro:if>
-			<xacro:unless value="${'$(arg ctrl_mode)' == 'position'}">
-				<xacro:if value="${'$(arg ctrl_mode)' == 'joint_imp'}">
-					<param name="ctrl_mode">3</param>
-				</xacro:if>
-				<xacro:unless value="${'$(arg ctrl_mode)' == 'joint_imp'}">
-					<param name="ctrl_mode">4</param>
-				</xacro:unless>
-			</xacro:unless>
 		</hardware>
-		<xacro:if value="${'$(arg type)' == 'dual' or '$(arg type)' == 'dual_ag2f90'  or '$(arg type)' == 'dual_rg75'}">
+		<!-- 使用 robot.xacro 中已解析的属性 -->
+		<!-- 双臂配置 -->
+		<xacro:if value="${selected_arm_config == 'dual'}">
 			<xacro:m6_interfaces name="left"/>
 			<xacro:m6_interfaces name="right"/>
-			<xacro:if value="${'$(arg type)' == 'dual_ag2f90'}">
+			<xacro:if value="${selected_gripper_type == 'ag2f90'}">
 				<xacro:include filename="$(find changingtek_description)/xacro/ros2_control/AG2F90-C.xacro"/>
 				<xacro:ag2f90c_interfaces name="left"/>
 				<xacro:ag2f90c_interfaces name="right"/>
 			</xacro:if>
-			<xacro:if value="${'$(arg type)' == 'dual_rg75'}">
+			<xacro:if value="${selected_gripper_type == 'rg75'}">
 				<xacro:include filename="$(find jodell_description)/xacro/ros2_control/RG75-300.xacro"/>
 				<xacro:rg75_interfaces name="left"/>
@@ -69,13 +53,16 @@
 			</xacro:if>
 		</xacro:if>
-		<xacro:unless value="${'$(arg type)' == 'dual' or '$(arg type)' == 'dual_ag2f90'  or '$(arg type)' == 'dual_rg75'}">
-			<xacro:if value="${'$(arg type)' == 'usb-90c'}">
-				<xacro:m6_interfaces name="left"/>
-				<xacro:include filename="$(find changingtek_description)/xacro/ros2_control/AG2F90-C.xacro"/>
-				<xacro:ag2f90c_interfaces name=""/>
+		<!-- 单臂配置 -->
+		<xacro:unless value="${selected_arm_config == 'dual'}">
+			<xacro:if value="${selected_arm_config == 'left'}">
+				<xacro:m6_interfaces name=""/>
+				<xacro:if value="${selected_gripper_type == 'ag2f90'}">
+					<xacro:include filename="$(find changingtek_description)/xacro/ros2_control/AG2F90-C.xacro"/>
+					<xacro:ag2f90c_interfaces name=""/>
+				</xacro:if>
 			</xacro:if>
-			<xacro:unless value="${'$(arg type)' == 'usb-90c'}">
+			<xacro:if value="${selected_arm_config == 'right'}">
 				<xacro:m6_interfaces name=""/>
-			</xacro:unless>
+			</xacro:if>
 		</xacro:unless>
 	</ros2_control>
@@ -84,8 +71,8 @@
 		<gazebo>
 			<plugin filename="gz_ros2_control-system" name="gz_ros2_control::GazeboSimROS2ControlPlugin">
-				<xacro:if value="${'$(arg type)' == 'left'}">
+				<xacro:if value="${selected_arm_config == 'left'}">
 					<parameters>$(find rokae_ar5_description)/config/ros2_control/ros2_controllers.yaml</parameters>
 				</xacro:if>
-				<xacro:if value="${'$(arg type)' == 'right'}">
+				<xacro:if value="${selected_arm_config == 'right'}">
 					<parameters>$(find rokae_ar5_description)/config/ros2_control/right.yaml</parameters>
 				</xacro:if>

Commit message: add single left rg75

File: m6_ccs_description/xacro/robot.xacro (robot description, xacro)
@@ -14,4 +14,8 @@
 	<xacro:if value="${type_arg == 'left'}">
 		<xacro:property name="selected_arm_config" value="left"/>
+	</xacro:if>
+	<xacro:if value="${type_arg == 'rg75'}">
+		<xacro:property name="selected_arm_config" value="left"/>
+		<xacro:property name="selected_gripper_type" value="rg75"/>
 	</xacro:if>
 	<xacro:if value="${type_arg == 'right'}">
@@ -37,4 +41,12 @@
 	<xacro:if value="${selected_arm_config == 'left' and selected_scene != 'usb-90c'}">
 		<xacro:M6_CCS collider="$(arg collider)"/>
+		<xacro:if value="${selected_gripper_type == 'rg75'}">
+			<xacro:include filename="$(find jodell_description)/xacro/RG75-300.xacro"/>
+			<xacro:RG75-300 name="" use_flange="true"/>
+			<joint name="gripper_base_joint" type="fixed">
+				<parent link="tcp"/>
+				<child link="flange"/>
+			</joint>
+		</xacro:if>
 	</xacro:if>
 	<!-- 单右臂 -->

File: m6_ccs_description/xacro/ros2_control/robot.xacro (robot description, xacro)
@@ -61,4 +61,8 @@
 					<xacro:ag2f90c_interfaces name=""/>
 				</xacro:if>
+				<xacro:if value="${selected_gripper_type == 'rg75'}">
+					<xacro:include filename="$(find jodell_description)/xacro/ros2_control/RG75-300.xacro"/>
+					<xacro:rg75_interfaces name=""/>
+				</xacro:if>
 			</xacro:if>
 			<xacro:if value="${selected_arm_config == 'right'}">
