Commit message: Updated hand ctrl for tool parameter and IP

File: m6_ccs_description/xacro/robot.xacro (robot description, xacro)
@@ -4,4 +4,19 @@
 	<xacro:arg name="type" default="left"/>
 	<xacro:arg name="scene" default=""/>
+	<!-- 质量中心偏移参数 (单位: 米) - 用于 LinkerHand 的 dyn_param 计算 -->
+	<!-- 这些参数可以通过 launch 文件传递，用于调整手部的质量中心位置 -->
+	<xacro:arg name="com_offset_left_x" default="0"/>
+	<xacro:arg name="com_offset_left_y" default="0"/>
+	<xacro:arg name="com_offset_left_z" default="0"/>
+	<xacro:arg name="com_offset_right_x" default="0"/>
+	<xacro:arg name="com_offset_right_y" default="0"/>
+	<xacro:arg name="com_offset_right_z" default="0"/>
+	<!-- 将参数值设置为 property，以便在 ros2_control/robot.xacro 中读取 -->
+	<xacro:property name="com_offset_left_x" value="$(arg com_offset_left_x)"/>
+	<xacro:property name="com_offset_left_y" value="$(arg com_offset_left_y)"/>
+	<xacro:property name="com_offset_left_z" value="$(arg com_offset_left_z)"/>
+	<xacro:property name="com_offset_right_x" value="$(arg com_offset_right_x)"/>
+	<xacro:property name="com_offset_right_y" value="$(arg com_offset_right_y)"/>
+	<xacro:property name="com_offset_right_z" value="$(arg com_offset_right_z)"/>
 	<!-- 从 type 参数解析出 arm_config、gripper_type 和 scene -->
 	<xacro:property name="type_arg" value="$(arg type)"/>
@@ -51,11 +66,21 @@
 	<!-- LinkerHand dexterous hand configurations -->
 	<xacro:if value="${type_arg == 'dual_o6'}">
-		<xacro:property name="selected_gripper_type" value="linkerhand_o6"/>
+		<xacro:property name="selected_gripper_type" value="o6"/>
 	</xacro:if>
 	<xacro:if value="${type_arg == 'dual_l6'}">
-		<xacro:property name="selected_gripper_type" value="linkerhand_l6"/>
+		<xacro:property name="selected_gripper_type" value="l6"/>
 	</xacro:if>
 	<xacro:if value="${type_arg == 'dual_o7'}">
-		<xacro:property name="selected_gripper_type" value="linkerhand_o7"/>
+		<xacro:property name="selected_gripper_type" value="o7"/>
+	</xacro:if>
+	<!-- Support for linkerhand_o6, linkerhand_l6, linkerhand_o7 (from fiveages_w2_description) -->
+	<xacro:if value="${type_arg == 'linkerhand_o6'}">
+		<xacro:property name="selected_gripper_type" value="o6"/>
+	</xacro:if>
+	<xacro:if value="${type_arg == 'linkerhand_l6'}">
+		<xacro:property name="selected_gripper_type" value="l6"/>
+	</xacro:if>
+	<xacro:if value="${type_arg == 'linkerhand_o7'}">
+		<xacro:property name="selected_gripper_type" value="o7"/>
 	</xacro:if>
 	<xacro:include filename="$(find m6_ccs_description)/xacro/arm.xacro"/>
@@ -105,5 +130,5 @@
 			</joint>
 			<!-- Right Arm -->
-			<joint name="right_arm_base_joint" type="fixed">
+			<joint name="right_arm_base_joint" type="fixed">left
 				<parent link="arm_base"/>
 				<child link="right_base_link"/>

File: m6_ccs_description/xacro/ros2_control/robot.xacro (robot description, xacro)
@@ -4,4 +4,14 @@
 	<xacro:arg name="ctrl_mode" default="position"/>
 	<xacro:arg name="type" default="left"/>
+	<!-- LinkerHand 质量中心偏移参数 (单位: 米) - 从 hand.xacro 中获取，默认为 0 -->
+	<xacro:arg name="com_offset_o6_x" default="0"/>
+	<xacro:arg name="com_offset_o6_y" default="0"/>
+	<xacro:arg name="com_offset_o6_z" default="0"/>
+	<xacro:arg name="com_offset_l6_x" default="0"/>
+	<xacro:arg name="com_offset_l6_y" default="0"/>
+	<xacro:arg name="com_offset_l6_z" default="0"/>
+	<xacro:arg name="com_offset_o7_x" default="0"/>
+	<xacro:arg name="com_offset_o7_y" default="0"/>
+	<xacro:arg name="com_offset_o7_z" default="0"/>
 	<link name="world"/>
 	<joint name="world_fixed" type="fixed">
@@ -34,9 +44,36 @@
 				<param name="max_joint_speed">50</param>
 				<param name="max_joint_acceleration">30</param>
+				<!-- Device IP address for network communication (default: 192.168.1.190) -->
+				<xacro:arg name="device_ip" default="192.168.1.190"/>
+				<param name="device_ip">$(arg device_ip)</param>
+				<!-- 如果是手（o6/l6/o7），设置手的质量参数 -->
+				<xacro:if value="${selected_hand_type == 'linkerhand_o6'}">
+					<xacro:include filename="$(find linkerhand_description)/xacro/o6.xacro"/>
+					<param name="left_dyn_param"><xacro:LinkerHandO6_DynParams direction="1" com_offset_x="$(arg com_offset_o6_x)" com_offset_y="$(arg com_offset_o6_y)" com_offset_z="$(arg com_offset_o6_z)"/></param>
+					<param name="right_dyn_param"><xacro:LinkerHandO6_DynParams direction="-1" com_offset_x="$(arg com_offset_o6_x)" com_offset_y="$(arg com_offset_o6_y)" com_offset_z="$(arg com_offset_o6_z)"/></param>
+				</xacro:if>
+				<xacro:if value="${selected_hand_type == 'linkerhand_l6'}">
+					<xacro:include filename="$(find linkerhand_description)/xacro/l6.xacro"/>
+					<param name="left_dyn_param"><xacro:LinkerHandL6_DynParams direction="1" com_offset_x="$(arg com_offset_l6_x)" com_offset_y="$(arg com_offset_l6_y)" com_offset_z="$(arg com_offset_l6_z)"/></param>
+					<param name="right_dyn_param"><xacro:LinkerHandL6_DynParams direction="-1" com_offset_x="$(arg com_offset_l6_x)" com_offset_y="$(arg com_offset_l6_y)" com_offset_z="$(arg com_offset_l6_z)"/></param>
+				</xacro:if>
+				<xacro:if value="${selected_hand_type == 'linkerhand_o7'}">
+					<xacro:include filename="$(find linkerhand_description)/xacro/o7.xacro"/>
+					<param name="left_dyn_param"><xacro:LinkerHandO7_DynParams direction="1" com_offset_x="$(arg com_offset_o7_x)" com_offset_y="$(arg com_offset_o7_y)" com_offset_z="$(arg com_offset_o7_z)"/></param>
+					<param name="right_dyn_param"><xacro:LinkerHandO7_DynParams direction="-1" com_offset_x="$(arg com_offset_o7_x)" com_offset_y="$(arg com_offset_o7_y)" com_offset_z="$(arg com_offset_o7_z)"/></param>
+				</xacro:if>
+				<!-- desktop 场景的 dyn_param（只在不是手的情况下设置） -->
+				<xacro:if value="${selected_scene == 'desktop' and selected_hand_type != 'linkerhand_o6' and selected_hand_type != 'linkerhand_l6' and selected_hand_type != 'linkerhand_o7'}">
+					<param name="left_dyn_param">1.2874,-10.145,30,114.65,0,0,0,0,0,0</param>
+					<param name="right_dyn_param">1.2874,-30.145,-10,147.85,0,0,0,0,0,0</param>
+				</xacro:if>
+				<!-- 如果没有 tool（既不是手也不是 desktop 场景），设置 dyn_param 为 0 -->
+				<xacro:if value="${selected_hand_type != 'linkerhand_o6' and selected_hand_type != 'linkerhand_l6' and selected_hand_type != 'linkerhand_o7' and (selected_gripper_type == 'none' or selected_gripper_type == '') and selected_scene != 'desktop'}">
+					<param name="left_dyn_param">0,0,0,0,0,0,0,0,0,0</param>
+					<param name="right_dyn_param">0,0,0,0,0,0,0,0,0,0</param>
+				</xacro:if>
 				<xacro:if value="${selected_scene == 'desktop'}">
 					<param name="device_ip">192.168.10.190</param>
 					<param name="ctrl_mode">CART_IMPEDANCE</param>
-					<param name="left_dyn_param">1.2874,-10.145,30,114.65,0,0,0,0,0,0</param>
-					<param name="right_dyn_param">1.2874,-30.145,-10,147.85,0,0,0,0,0,0</param>
 				</xacro:if>
 				<xacro:if value="${selected_scene == 'usb-90c'}">
@@ -61,37 +98,4 @@
 				<xacro:rg75_interfaces name="right"/>
 			</xacro:if>
-			<!-- LinkerHand dexterous hand interfaces -->
-			<!-- Note: LinkerHand requires separate hardware interface (Modbus), so interfaces are included here -->
-			<!-- but the actual hardware will be handled by separate DexterousHandHardware instances -->
-			<xacro:if value="${selected_gripper_type == 'linkerhand_o6' or selected_gripper_type == 'linkerhand_l6'}">
-				<xacro:include filename="$(find linkerhand_description)/xacro/ros2_control/o6.xacro"/>
-				<!-- Left hand -->
-				<xacro:linkerhand_o6_interfaces name="left"/>
-				<!-- Right hand -->
-				<xacro:linkerhand_o6_interfaces name="right"/>
-			</xacro:if>
-			<xacro:if value="${selected_gripper_type == 'linkerhand_o7'}">
-				<xacro:include filename="$(find linkerhand_description)/xacro/ros2_control/o7.xacro"/>
-				<!-- Left hand -->
-				<xacro:linkerhand_o7_interfaces name="left"/>
-				<!-- Right hand -->
-				<xacro:linkerhand_o7_interfaces name="right"/>
-			</xacro:if>
-		</xacro:if>
-		<!-- LinkerHand separate ros2_control systems (for real hardware with Modbus) -->
-		<!-- These are separate systems because LinkerHand uses DexterousHandHardware, not MarvinHardware -->
-		<xacro:if value="${selected_gripper_type == 'linkerhand_o6' or selected_gripper_type == 'linkerhand_l6' or selected_gripper_type == 'linkerhand_o7'}">
-			<!-- Left hand system -->
-			<xacro:include filename="$(find linkerhand_description)/xacro/ros2_control/hand.xacro">
-				<xacro:arg name="type" value="${selected_gripper_type == 'linkerhand_o6' ? 'o6' : (selected_gripper_type == 'linkerhand_l6' ? 'l6' : 'o7')}"/>
-				<xacro:arg name="direction" value="1"/>
-				<xacro:arg name="ros2_control_hardware_type" value="$(arg ros2_control_hardware_type)"/>
-			</xacro:include>
-			<!-- Right hand system -->
-			<xacro:include filename="$(find linkerhand_description)/xacro/ros2_control/hand.xacro">
-				<xacro:arg name="type" value="${selected_gripper_type == 'linkerhand_o6' ? 'o6' : (selected_gripper_type == 'linkerhand_l6' ? 'l6' : 'o7')}"/>
-				<xacro:arg name="direction" value="-1"/>
-				<xacro:arg name="ros2_control_hardware_type" value="$(arg ros2_control_hardware_type)"/>
-			</xacro:include>
 		</xacro:if>
 		<!-- 单臂配置 -->
@@ -120,6 +124,7 @@
 	<!-- LinkerHand separate ros2_control systems (for real hardware with Modbus) -->
 	<!-- These are separate systems because LinkerHand uses DexterousHandHardware, not MarvinHardware -->
-	<!-- Left hand system -->
-	<xacro:if value="${selected_gripper_type == 'linkerhand_o6'}">
+	<!-- 如果是手（o6/l6/o7），创建手的 ros2_control 系统 -->
+	<xacro:if value="${selected_hand_type == 'linkerhand_o6'}">
+		<!-- Left hand system -->
 		<xacro:include filename="$(find linkerhand_description)/xacro/ros2_control/hand.xacro">
 			<xacro:arg name="type" value="o6"/>
@@ -127,21 +132,5 @@
 			<xacro:arg name="ros2_control_hardware_type" value="$(arg ros2_control_hardware_type)"/>
 		</xacro:include>
-	</xacro:if>
-	<xacro:if value="${selected_gripper_type == 'linkerhand_l6'}">
-		<xacro:include filename="$(find linkerhand_description)/xacro/ros2_control/hand.xacro">
-			<xacro:arg name="type" value="l6"/>
-			<xacro:arg name="direction" value="1"/>
-			<xacro:arg name="ros2_control_hardware_type" value="$(arg ros2_control_hardware_type)"/>
-		</xacro:include>
-	</xacro:if>
-	<xacro:if value="${selected_gripper_type == 'linkerhand_o7'}">
-		<xacro:include filename="$(find linkerhand_description)/xacro/ros2_control/hand.xacro">
-			<xacro:arg name="type" value="o7"/>
-			<xacro:arg name="direction" value="1"/>
-			<xacro:arg name="ros2_control_hardware_type" value="$(arg ros2_control_hardware_type)"/>
-		</xacro:include>
-	</xacro:if>
-	<!-- Right hand system -->
-	<xacro:if value="${selected_gripper_type == 'linkerhand_o6'}">
+		<!-- Right hand system -->
 		<xacro:include filename="$(find linkerhand_description)/xacro/ros2_control/hand.xacro">
 			<xacro:arg name="type" value="o6"/>
@@ -150,5 +139,12 @@
 		</xacro:include>
 	</xacro:if>
-	<xacro:if value="${selected_gripper_type == 'linkerhand_l6'}">
+	<xacro:if value="${selected_hand_type == 'linkerhand_l6'}">
+		<!-- Left hand system -->
+		<xacro:include filename="$(find linkerhand_description)/xacro/ros2_control/hand.xacro">
+			<xacro:arg name="type" value="l6"/>
+			<xacro:arg name="direction" value="1"/>
+			<xacro:arg name="ros2_control_hardware_type" value="$(arg ros2_control_hardware_type)"/>
+		</xacro:include>
+		<!-- Right hand system -->
 		<xacro:include filename="$(find linkerhand_description)/xacro/ros2_control/hand.xacro">
 			<xacro:arg name="type" value="l6"/>
@@ -157,5 +153,12 @@
 		</xacro:include>
 	</xacro:if>
-	<xacro:if value="${selected_gripper_type == 'linkerhand_o7'}">
+	<xacro:if value="${selected_hand_type == 'linkerhand_o7'}">
+		<!-- Left hand system -->
+		<xacro:include filename="$(find linkerhand_description)/xacro/ros2_control/hand.xacro">
+			<xacro:arg name="type" value="o7"/>
+			<xacro:arg name="direction" value="1"/>
+			<xacro:arg name="ros2_control_hardware_type" value="$(arg ros2_control_hardware_type)"/>
+		</xacro:include>
+		<!-- Right hand system -->
 		<xacro:include filename="$(find linkerhand_description)/xacro/ros2_control/hand.xacro">
 			<xacro:arg name="type" value="o7"/>

Commit message: add ag2f90c_soft

File: m6_ccs_description/xacro/robot.xacro (robot description, xacro)
@@ -9,4 +9,5 @@
 	<xacro:property name="selected_arm_config" value="dual"/>
 	<xacro:property name="selected_gripper_type" value="none"/>
+	<xacro:property name="selected_gripper_pad" value="default"/>
 	<xacro:property name="selected_scene" value=""/>
 	<!-- 从 type 解析 arm_config 和 gripper_type -->
@@ -48,4 +49,9 @@
 		<xacro:property name="selected_scene" value="desktop"/>
 		<xacro:property name="selected_gripper_type" value="ag2f90_c"/>
+	</xacro:if>
+	<xacro:if value="${type_arg == 'dual_desktop_90c_soft'}">
+		<xacro:property name="selected_scene" value="desktop"/>
+		<xacro:property name="selected_gripper_type" value="ag2f90_c"/>
+		<xacro:property name="selected_gripper_pad" value="soft"/>
 	</xacro:if>
 	<xacro:include filename="$(find m6_ccs_description)/xacro/arm.xacro"/>
@@ -147,5 +153,6 @@
 		<xacro:if value="${selected_gripper_type == 'ag2f90_c' or selected_gripper_type == 'ag2f90_d'}">
 			<xacro:include filename="$(find changingtek_description)/xacro/AG2F90-C.xacro"/>
-			<xacro:AG2F90-C name="left" use_flange="true"/>
+			<xacro:AG2F90-C name="left" use_flange="true" pad="${selected_gripper_pad}"/>
+			<xacro:AG2F90-C name="right" use_flange="true" pad="${selected_gripper_pad}"/>
 			<joint name="left_gripper_fix" type="fixed">
 				<parent link="left_tcp"/>
@@ -153,5 +160,4 @@
 				<origin xyz="0 0 0.0045"/>
 			</joint>
-			<xacro:AG2F90-C name="right" use_flange="true"/>
 			<joint name="right_gripper_fix" type="fixed">
 				<parent link="right_tcp"/>

Commit message: Update with new task info weight for manipulation

File: m6_ccs_description/xacro/robot.xacro (robot description, xacro)
@@ -33,4 +33,10 @@
 	</xacro:if>
 	<xacro:if value="${type_arg == 'ag2f90_d'}">
+		<xacro:property name="selected_gripper_type" value="ag2f90_d"/>
+	</xacro:if>
+	<xacro:if value="${type_arg == 'dual_ag2f90_c'}">
+		<xacro:property name="selected_gripper_type" value="ag2f90_c"/>
+	</xacro:if>
+	<xacro:if value="${type_arg == 'dual_ag2f90_d'}">
 		<xacro:property name="selected_gripper_type" value="ag2f90_d"/>
 	</xacro:if>

Commit message: add marvin robot config

File: m6_ccs_description/xacro/robot.xacro (robot description, xacro)
@@ -9,4 +9,5 @@
 	<xacro:property name="selected_arm_config" value="dual"/>
 	<xacro:property name="selected_gripper_type" value="none"/>
+	<xacro:property name="selected_hand_type" value="none"/>
 	<xacro:property name="selected_gripper_pad" value="default"/>
 	<xacro:property name="selected_scene" value=""/>
@@ -41,4 +42,13 @@
 		<xacro:property name="selected_gripper_type" value="rg75"/>
 		<xacro:property name="selected_gripper_pad" value="heavy_carry"/>
+	</xacro:if>
+	<xacro:if value="${type_arg == 'linkerhand_o6'}">
+		<xacro:property name="selected_hand_type" value="linkerhand_o6"/>
+	</xacro:if>
+	<xacro:if value="${type_arg == 'linkerhand_l6'}">
+		<xacro:property name="selected_hand_type" value="linkerhand_l6"/>
+	</xacro:if>
+	<xacro:if value="${type_arg == 'linkerhand_o7'}">
+		<xacro:property name="selected_hand_type" value="linkerhand_o7"/>
 	</xacro:if>
 	<!-- 适用纯双臂演示场景的配置 -->
@@ -179,4 +189,49 @@
 					<origin rpy="0 0 ${PI/2}"/>
 				</xacro:if>
+			</joint>
+		</xacro:if>
+		<xacro:if value="${selected_hand_type == 'linkerhand_o6'}">
+			<xacro:include filename="$(find linkerhand_description)/xacro/o6.xacro"/>
+			<xacro:LinkerHandO6 name="left_hand" direction="1" use_flange="true" fixed_joints="false"/>
+			<joint name="left_hand_base_joint" type="fixed">
+				<origin xyz="0 0 0.0045" rpy="0 0 ${PI}"/>
+				<parent link="left_tcp"/>
+				<child link="left_hand_flange"/>
+			</joint>
+			<xacro:LinkerHandO6 name="right_hand" direction="-1" use_flange="true" fixed_joints="false"/>
+			<joint name="right_hand_base_joint" type="fixed">
+				<parent link="right_tcp"/>
+				<child link="right_hand_flange"/>
+				<origin xyz="0 0 0.0045"/>
+			</joint>
+		</xacro:if>
+		<xacro:if value="${selected_hand_type == 'linkerhand_o7'}">
+			<xacro:include filename="$(find linkerhand_description)/xacro/o7.xacro"/>
+			<xacro:LinkerHandO7 name="left_hand" direction="1" use_flange="true" fixed_joints="false"/>
+			<joint name="left_hand_base_joint" type="fixed">
+				<origin rpy="0 0 ${PI/2}"/>
+				<parent link="left_tcp"/>
+				<child link="left_hand_flange"/>
+			</joint>
+			<xacro:LinkerHandO7 name="right_hand" direction="-1" use_flange="true" fixed_joints="false"/>
+			<joint name="right_hand_base_joint" type="fixed">
+				<origin rpy="0 0 ${-PI/2}"/>
+				<parent link="right_tcp"/>
+				<child link="right_hand_flange"/>
+			</joint>
+		</xacro:if>
+		<xacro:if value="${selected_hand_type == 'linkerhand_l6'}">
+			<xacro:include filename="$(find linkerhand_description)/xacro/l6.xacro"/>
+			<xacro:LinkerHandL6 name="left_hand" direction="1" use_flange="true" fixed_joints="false"/>
+			<joint name="left_hand_base_joint" type="fixed">
+				<origin xyz="0 0 0.0045" rpy="0 0 ${PI}"/>
+				<parent link="left_tcp"/>
+				<child link="left_hand_flange"/>
+			</joint>
+			<xacro:LinkerHandL6 name="right_hand" direction="-1" use_flange="true" fixed_joints="false"/>
+			<joint name="right_hand_base_joint" type="fixed">
+				<parent link="right_tcp"/>
+				<child link="right_hand_flange"/>
+				<origin xyz="0 0 0.0045"/>
 			</joint>
 		</xacro:if>

File: m6_ccs_description/xacro/ros2_control/robot.xacro (robot description, xacro)
@@ -31,5 +31,10 @@
 				<plugin>marvin_ros2_control/MarvinHardware</plugin>
 				<param name="arm_type">${selected_arm_config}</param>
-				<param name="gripper_type">${selected_gripper_type}</param>
+				<xacro:if value="${selected_hand_type != 'none'}">
+					<param name="gripper_type">${selected_hand_type}</param>
+				</xacro:if>
+				<xacro:unless value="${selected_hand_type != 'none'}">
+					<param name="gripper_type">${selected_gripper_type}</param>
+				</xacro:unless>
 				<param name="max_joint_speed">50</param>
 				<param name="max_joint_acceleration">30</param>
@@ -60,4 +65,14 @@
 				<xacro:rg75_interfaces name="left"/>
 				<xacro:rg75_interfaces name="right"/>
+			</xacro:if>
+			<xacro:if value="${selected_hand_type == 'linkerhand_o6' or selected_hand_type == 'linkerhand_l6'}">
+				<xacro:include filename="$(find linkerhand_description)/xacro/ros2_control/o6.xacro"/>
+				<xacro:linkerhand_o6_interfaces name="left_hand"/>
+				<xacro:linkerhand_o6_interfaces name="right_hand"/>
+			</xacro:if>
+			<xacro:if value="${selected_hand_type == 'linkerhand_o7'}">
+				<xacro:include filename="$(find linkerhand_description)/xacro/ros2_control/o7.xacro"/>
+				<xacro:linkerhand_o7_interfaces name="left_hand"/>
+				<xacro:linkerhand_o7_interfaces name="right_hand"/>
 			</xacro:if>
 		</xacro:if>

Commit message: 增加90c-soft

File: m6_ccs_description/xacro/robot.xacro (robot description, xacro)
@@ -32,4 +32,8 @@
 	<xacro:if value="${type_arg == 'ag2f90_c'}">
 		<xacro:property name="selected_gripper_type" value="ag2f90_c"/>
+	</xacro:if>
+	<xacro:if value="${type_arg == 'ag2f90_c_soft'}">
+		<xacro:property name="selected_gripper_type" value="ag2f90_c"/>
+		<xacro:property name="selected_gripper_pad" value="soft"/>
 	</xacro:if>
 	<xacro:if value="${type_arg == 'ag2f90_d'}">
