Commit message: Feature/diff eef (#4)
* add diff eef support

* add diff eef support

* add template support

* add diff eef

* add diff eef

* add hand eef

File: m6_ccs_description/xacro/robot.xacro (robot description, xacro)
@@ -4,6 +4,13 @@
 	<xacro:arg name="type" default="dual"/>
 	<xacro:arg name="scene" default=""/>
+	<xacro:arg name="left_type" default=""/>
+	<xacro:arg name="right_type" default=""/>
+	<xacro:arg name="eef_fixed_joints" default="false"/>
 	<!-- 从 type 参数解析出 arm_config、gripper_type 和 scene -->
 	<xacro:property name="type_arg" value="$(arg type)"/>
+	<xacro:property name="left_type_arg" value="$(arg left_type)"/>
+	<xacro:property name="right_type_arg" value="$(arg right_type)"/>
+	<xacro:property name="effective_left_type" value="${left_type_arg if left_type_arg != '' else type_arg}"/>
+	<xacro:property name="effective_right_type" value="${right_type_arg if right_type_arg != '' else type_arg}"/>
 	<!-- 默认值 -->
 	<xacro:property name="selected_arm_config" value="dual"/>
@@ -66,4 +73,5 @@
 	</xacro:if>
 	<xacro:include filename="$(find m6_ccs_description)/xacro/arm.xacro"/>
+	<xacro:include filename="$(find m6_ccs_description)/xacro/arm_mount.xacro"/>
 	<!-- 单左臂（不包括 usb-90c 场景） -->
 	<xacro:if value="${selected_arm_config == 'left' and selected_scene != 'usb-90c'}">
@@ -104,16 +112,5 @@
 				<child link="arm_base"/>
 			</joint>
-			<!-- Left Arm -->
-			<joint name="left_arm_base_joint" type="fixed">
-				<parent link="arm_base"/>
-				<child link="left_base_link"/>
-				<origin rpy="-${PI/2} 0 0" xyz="0.0 0.12 0.701"/>
-			</joint>
-			<!-- Right Arm -->
-			<joint name="right_arm_base_joint" type="fixed">
-				<parent link="arm_base"/>
-				<child link="right_base_link"/>
-				<origin rpy="${PI/2} 0 0" xyz="0.0 -0.12 0.701"/>
-			</joint>
+			<xacro:DualArmMount parent="arm_base" left_xyz="0 0.12 0.701" right_xyz="0 -0.12 0.701"/>
 			<xacro:if value="${selected_gripper_type == 'none'}">
 				<link name="right_eef"/>
@@ -144,100 +141,21 @@
 				<child link="arm_base"/>
 			</joint>
-			<!-- Left Arm -->
-			<joint name="left_arm_base_joint" type="fixed">
-				<parent link="arm_base"/>
-				<child link="left_base_link"/>
-				<origin rpy="-${PI/2} 0 0" xyz="0.0 0.062 0"/>
-			</joint>
-			<!-- Right Arm -->
-			<joint name="right_arm_base_joint" type="fixed">
-				<parent link="arm_base"/>
-				<child link="right_base_link"/>
-				<origin rpy="${PI/2} 0 0" xyz="0 -0.062 0"/>
-			</joint>
+			<xacro:DualArmMount parent="arm_base"/>
 		</xacro:unless>
 		<!-- 双臂和末端执行器（两种场景共用） -->
 		<xacro:M6_CCS name="left"/>
 		<xacro:M6_CCS name="right" direction="-1"/>
-		<!-- 双臂末端执行器 -->
-		<xacro:if value="${selected_gripper_type == 'ag2f90_c' or selected_gripper_type == 'ag2f90_d'}">
-			<xacro:include filename="$(find changingtek_description)/xacro/AG2F90-C.xacro"/>
-			<xacro:AG2F90-C name="left" use_flange="true" pad="${selected_gripper_pad}"/>
-			<xacro:AG2F90-C name="right" use_flange="true" pad="${selected_gripper_pad}"/>
-			<joint name="left_gripper_fix" type="fixed">
-				<parent link="left_tcp"/>
-				<child link="left_flange"/>
-				<origin xyz="0 0 0.0045"/>
-			</joint>
-			<joint name="right_gripper_fix" type="fixed">
-				<parent link="right_tcp"/>
-				<child link="right_flange"/>
-				<origin xyz="0 0 0.0045"/>
-			</joint>
-		</xacro:if>
-		<xacro:if value="${selected_gripper_type == 'rg75'}">
-			<xacro:include filename="$(find jodell_description)/xacro/RG75-300.xacro"/>
-			<xacro:RG75-300 name="left" use_flange="true" pad="${selected_gripper_pad}"/>
-			<xacro:RG75-300 name="right" use_flange="true" pad="${selected_gripper_pad}"/>
-			<joint name="left_gripper_base_joint" type="fixed">
-				<parent link="left_tcp"/>
-				<child link="left_flange"/>
-				<xacro:if value="${selected_gripper_pad == 'heavy_carry'}">
-					<origin rpy="0 0 ${PI/2}"/>
-				</xacro:if>
-			</joint>
-			<joint name="right_gripper_base_joint" type="fixed">
-				<parent link="right_tcp"/>
-				<child link="right_flange"/>
-				<xacro:if value="${selected_gripper_pad == 'heavy_carry'}">
-					<origin rpy="0 0 ${PI/2}"/>
-				</xacro:if>
-			</joint>
-		</xacro:if>
-		<xacro:if value="${selected_hand_type == 'linkerhand_o6'}">
-			<xacro:include filename="$(find linkerhand_description)/xacro/o6.xacro"/>
-			<xacro:LinkerHandO6 name="left_hand" direction="1" use_flange="true" fixed_joints="false"/>
-			<joint name="left_hand_base_joint" type="fixed">
-				<origin xyz="0 0 0.0045" rpy="0 0 ${PI}"/>
-				<parent link="left_tcp"/>
-				<child link="left_hand_flange"/>
-			</joint>
-			<xacro:LinkerHandO6 name="right_hand" direction="-1" use_flange="true" fixed_joints="false"/>
-			<joint name="right_hand_base_joint" type="fixed">
-				<parent link="right_tcp"/>
-				<child link="right_hand_flange"/>
-				<origin xyz="0 0 0.0045"/>
-			</joint>
-		</xacro:if>
-		<xacro:if value="${selected_hand_type == 'linkerhand_o7'}">
-			<xacro:include filename="$(find linkerhand_description)/xacro/o7.xacro"/>
-			<xacro:LinkerHandO7 name="left_hand" direction="1" use_flange="true" fixed_joints="false"/>
-			<joint name="left_hand_base_joint" type="fixed">
-				<origin rpy="0 0 ${PI/2}"/>
-				<parent link="left_tcp"/>
-				<child link="left_hand_flange"/>
-			</joint>
-			<xacro:LinkerHandO7 name="right_hand" direction="-1" use_flange="true" fixed_joints="false"/>
-			<joint name="right_hand_base_joint" type="fixed">
-				<origin rpy="0 0 ${-PI/2}"/>
-				<parent link="right_tcp"/>
-				<child link="right_hand_flange"/>
-			</joint>
-		</xacro:if>
-		<xacro:if value="${selected_hand_type == 'linkerhand_l6'}">
-			<xacro:include filename="$(find linkerhand_description)/xacro/l6.xacro"/>
-			<xacro:LinkerHandL6 name="left_hand" direction="1" use_flange="true" fixed_joints="false"/>
-			<joint name="left_hand_base_joint" type="fixed">
-				<origin xyz="0 0 0.0045" rpy="0 0 ${PI}"/>
-				<parent link="left_tcp"/>
-				<child link="left_hand_flange"/>
-			</joint>
-			<xacro:LinkerHandL6 name="right_hand" direction="-1" use_flange="true" fixed_joints="false"/>
-			<joint name="right_hand_base_joint" type="fixed">
-				<parent link="right_tcp"/>
-				<child link="right_hand_flange"/>
-				<origin xyz="0 0 0.0045"/>
-			</joint>
-		</xacro:if>
+		<xacro:include filename="$(find m6_ccs_description)/xacro/eef_type_resolver.xacro"/>
+		<xacro:set_side_eef_types side="left" type_key="${effective_left_type}"/>
+		<xacro:set_side_eef_types side="right" type_key="${effective_right_type}"/>
+		<xacro:include filename="$(find m6_ccs_description)/xacro/eefs.xacro"/>
+		<xacro:EndEffectors
+			eef_fixed_joints="$(arg eef_fixed_joints)"
+			left_hand_type="${left_hand_type}"
+			left_gripper_type="${left_gripper_type}"
+			left_gripper_pad="${left_gripper_pad}"
+			right_hand_type="${right_hand_type}"
+			right_gripper_type="${right_gripper_type}"
+			right_gripper_pad="${right_gripper_pad}"/>
 	</xacro:if>
 	<!-- USB-90C 配置 -->
@@ -262,10 +180,5 @@
 			</collision>
 		</link>
-		<!-- Left Arm -->
-		<joint name="left_arm_base_joint" type="fixed">
-			<parent link="base"/>
-			<child link="left_base_link"/>
-			<origin rpy="-${PI/2} 0 0" xyz="0.0 0.12 0.701"/>
-		</joint>
+		<xacro:LeftArmMount parent="base"/>
 		<xacro:M6_CCS name="left"/>
 		<xacro:include filename="$(find changingtek_description)/xacro/AG2F90-C.xacro"/>

File: m6_ccs_description/xacro/ros2_control/robot.xacro (robot description, xacro)
@@ -31,10 +31,6 @@
 				<plugin>marvin_ros2_control/MarvinHardware</plugin>
 				<param name="arm_type">${selected_arm_config}</param>
-				<xacro:if value="${selected_hand_type != 'none'}">
-					<param name="gripper_type">${selected_hand_type}</param>
-				</xacro:if>
-				<xacro:unless value="${selected_hand_type != 'none'}">
-					<param name="gripper_type">${selected_gripper_type}</param>
-				</xacro:unless>
+				<param name="left_ee_type">${left_hand_type if left_hand_type != '' else left_gripper_type}</param>
+				<param name="right_ee_type">${right_hand_type if right_hand_type != '' else right_gripper_type}</param>
 				<param name="max_joint_speed">50</param>
 				<param name="max_joint_acceleration">30</param>
@@ -51,27 +47,34 @@
 			</xacro:if>
 		</hardware>
-		<!-- 使用 robot.xacro 中已解析的属性 -->
-		<!-- 双臂配置 -->
+		<!-- 双臂配置：按侧末端（left_type/right_type 或对称 type） -->
 		<xacro:if value="${selected_arm_config == 'dual'}">
 			<xacro:m6_interfaces name="left"/>
 			<xacro:m6_interfaces name="right"/>
-			<xacro:if value="${selected_gripper_type == 'ag2f90_c' or selected_gripper_type == 'ag2f90_d'}">
-				<xacro:include filename="$(find changingtek_description)/xacro/ros2_control/AG2F90-C.xacro"/>
+			<xacro:include filename="$(find jodell_description)/xacro/ros2_control/RG75-300.xacro"/>
+			<xacro:include filename="$(find changingtek_description)/xacro/ros2_control/AG2F90-C.xacro"/>
+			<xacro:include filename="$(find linkerhand_description)/xacro/ros2_control/o6.xacro"/>
+			<xacro:include filename="$(find linkerhand_description)/xacro/ros2_control/o7.xacro"/>
+			<xacro:if value="${left_gripper_type == 'rg75'}">
+				<xacro:rg75_interfaces name="left"/>
+			</xacro:if>
+			<xacro:if value="${right_gripper_type == 'rg75'}">
+				<xacro:rg75_interfaces name="right"/>
+			</xacro:if>
+			<xacro:if value="${left_gripper_type == 'ag2f90_c' or left_gripper_type == 'ag2f90_d'}">
 				<xacro:ag2f90c_interfaces name="left"/>
+			</xacro:if>
+			<xacro:if value="${right_gripper_type == 'ag2f90_c' or right_gripper_type == 'ag2f90_d'}">
 				<xacro:ag2f90c_interfaces name="right"/>
 			</xacro:if>
-			<xacro:if value="${selected_gripper_type == 'rg75'}">
-				<xacro:include filename="$(find jodell_description)/xacro/ros2_control/RG75-300.xacro"/>
-				<xacro:rg75_interfaces name="left"/>
-				<xacro:rg75_interfaces name="right"/>
+			<xacro:if value="${left_hand_type == 'linkerhand_o6' or left_hand_type == 'linkerhand_l6'}">
+				<xacro:linkerhand_o6_interfaces name="left_hand"/>
 			</xacro:if>
-			<xacro:if value="${selected_hand_type == 'linkerhand_o6' or selected_hand_type == 'linkerhand_l6'}">
-				<xacro:include filename="$(find linkerhand_description)/xacro/ros2_control/o6.xacro"/>
-				<xacro:linkerhand_o6_interfaces name="left_hand"/>
+			<xacro:if value="${right_hand_type == 'linkerhand_o6' or right_hand_type == 'linkerhand_l6'}">
 				<xacro:linkerhand_o6_interfaces name="right_hand"/>
 			</xacro:if>
-			<xacro:if value="${selected_hand_type == 'linkerhand_o7'}">
-				<xacro:include filename="$(find linkerhand_description)/xacro/ros2_control/o7.xacro"/>
+			<xacro:if value="${left_hand_type == 'linkerhand_o7'}">
 				<xacro:linkerhand_o7_interfaces name="left_hand"/>
+			</xacro:if>
+			<xacro:if value="${right_hand_type == 'linkerhand_o7'}">
 				<xacro:linkerhand_o7_interfaces name="right_hand"/>
 			</xacro:if>

Commit message: simplified xacro

File: m6_ccs_description/xacro/robot.xacro (robot description, xacro)
@@ -5,10 +5,10 @@
 	<xacro:arg name="variant" default=""/>
 	<xacro:arg name="type" default="dual"/>
-	<xacro:arg name="scene" default=""/>
 	<xacro:arg name="left_type" default=""/>
 	<xacro:arg name="right_type" default=""/>
 	<xacro:arg name="eef_fixed_joints" default="false"/>
-	<!-- 从 type 参数解析出 arm_config、gripper_type 和 scene -->
+	<!-- 从 type 参数解析 arm_config / 对称末端 -->
 	<xacro:property name="type_arg" value="$(arg type)"/>
+	<xacro:property name="variant_arg" value="$(arg variant)"/>
 	<xacro:property name="left_type_arg" value="$(arg left_type)"/>
 	<xacro:property name="right_type_arg" value="$(arg right_type)"/>
@@ -20,5 +20,4 @@
 	<xacro:property name="selected_hand_type" value="none"/>
 	<xacro:property name="selected_gripper_pad" value="default"/>
-	<xacro:property name="selected_scene" value=""/>
 	<!-- 从 type 解析 arm_config 和 gripper_type -->
 	<!-- 单臂配置 -->
@@ -28,9 +27,4 @@
 	<xacro:if value="${type_arg == 'right'}">
 		<xacro:property name="selected_arm_config" value="right"/>
-	</xacro:if>
-	<xacro:if value="${type_arg == 'usb-90c'}">
-		<xacro:property name="selected_arm_config" value="left"/>
-		<xacro:property name="selected_gripper_type" value="ag2f90_c"/>
-		<xacro:property name="selected_scene" value="usb-90c"/>
 	</xacro:if>
 	<!-- 双臂配置 -->
@@ -71,17 +65,8 @@
 		<xacro:property name="selected_hand_type" value="linkerhand_o7"/>
 	</xacro:if>
-	<!-- 适用纯双臂演示场景的配置 -->
-	<xacro:if value="${type_arg == 'desktop'}">
-		<xacro:property name="selected_scene" value="desktop"/>
-	</xacro:if>
-	<xacro:if value="${type_arg == 'desktop_90c'}">
-		<xacro:property name="selected_scene" value="desktop"/>
-		<xacro:property name="selected_gripper_type" value="ag2f90_c"/>
-		<xacro:property name="selected_gripper_pad" value="soft"/>
-	</xacro:if>
 	<xacro:include filename="$(find m6_ccs_description)/xacro/arm.xacro"/>
 	<xacro:include filename="$(find m6_ccs_description)/xacro/arm_mount.xacro"/>
-	<!-- 单左臂（不包括 usb-90c 场景） -->
-	<xacro:if value="${selected_arm_config == 'left' and selected_scene != 'usb-90c'}">
+	<!-- 单左臂 -->
+	<xacro:if value="${selected_arm_config == 'left'}">
 		<xacro:M6_CCS skin="$(arg skin)" variant="$(arg variant)"/>
 		<xacro:if value="${selected_gripper_type == 'rg75'}">
@@ -100,6 +85,5 @@
 	<!-- 双臂配置 -->
 	<xacro:if value="${selected_arm_config == 'dual'}">
-		<!-- Base link 和 arm_base 根据 scene 设置 -->
-		<xacro:if value="${selected_scene == 'desktop'}">
+		<xacro:if value="${variant_arg == 'desktop'}">
 			<link name="base_link"/>
 			<link name="arm_base">
@@ -121,19 +105,6 @@
 			</joint>
 			<xacro:DualArmMount parent="arm_base" left_xyz="0 0.12 0.701" right_xyz="0 -0.12 0.701"/>
-			<xacro:if value="${selected_gripper_type == 'none'}">
-				<link name="right_eef"/>
-				<joint name="right_eef_joint" type="fixed">
-					<parent link="right_tcp"/>
-					<child link="right_eef"/>
-				</joint>
-				<link name="left_eef"/>
-				<joint name="left_eef_joint" type="fixed">
-					<parent link="left_tcp"/>
-					<child link="left_eef"/>
-				</joint>
-			</xacro:if>
 		</xacro:if>
-		<xacro:unless value="${selected_scene == 'desktop'}">
-			<!-- 非 Desktop 场景：base_link 为空，有 arm_base -->
+		<xacro:unless value="${variant_arg == 'desktop'}">
 			<link name="base_link"/>
 			<link name="arm_base">
@@ -151,5 +122,4 @@
 			<xacro:DualArmMount parent="arm_base"/>
 		</xacro:unless>
-		<!-- 双臂和末端执行器（两种场景共用） -->
 		<xacro:M6_CCS name="left" skin="$(arg skin)" variant="$(arg variant)"/>
 		<xacro:M6_CCS name="right" direction="-1" skin="$(arg skin)" variant="$(arg variant)"/>
@@ -167,34 +137,3 @@
 			right_gripper_pad="${right_gripper_pad}"/>
 	</xacro:if>
-	<!-- USB-90C 配置 -->
-	<xacro:if value="${selected_arm_config == 'left' and selected_scene == 'usb-90c'}">
-		<link name="base_link"/>
-		<!-- Left Arm -->
-		<joint name="base_joint" type="fixed">
-			<parent link="base_link"/>
-			<child link="base"/>
-		</joint>
-		<link name="base">
-			<visual>
-				<geometry>
-					<mesh filename="file://$(find m6_ccs_description)/meshes/desktop_base.glb"/>
-				</geometry>
-			</visual>
-			<collision>
-				<origin xyz="0 0 0.324331"/>
-				<geometry>
-					<box size="0.10045 0.100398 0.648662"/>
-				</geometry>
-			</collision>
-		</link>
-		<xacro:LeftArmMount parent="base"/>
-		<xacro:M6_CCS name="left" skin="$(arg skin)" variant="$(arg variant)"/>
-		<xacro:include filename="$(find changingtek_description)/xacro/AG2F90-C.xacro"/>
-		<xacro:AG2F90-C name="" use_flange="true"/>
-		<joint name="gripper_fix" type="fixed">
-			<parent link="left_link7"/>
-			<child link="flange"/>
-			<origin xyz="0 -0.0995 0" rpy=" ${PI/2} 0 0"/>
-		</joint>
-	</xacro:if>
 </robot>

File: m6_ccs_description/xacro/ros2_control/robot.xacro (robot description, xacro)
@@ -2,7 +2,7 @@
 <robot xmlns:xacro="http://www.ros.org/wiki/xacro" name="AR5">
 	<xacro:arg name="ros2_control_hardware_type" default="mock_components"/>
-	<xacro:arg name="ctrl_mode" default="position"/>
+	<xacro:arg name="arm_ctrl_mode" default="position"/>
+	<xacro:arg name="device_ip" default=""/>
 	<xacro:arg name="type" default="dual"/>
-	<!-- Non-desktop only: from robot.local.yaml via launch (robot_profile) -->
 	<xacro:arg name="left_dyn_param" default=""/>
 	<xacro:arg name="right_dyn_param" default=""/>
@@ -16,6 +16,7 @@
 		<origin/>
 	</joint>
-	<!-- Include robot.xacro，它会解析 type 并设置 selected_arm_config 和 selected_gripper_type -->
+	<!-- Include robot.xacro（解析 type / selected_arm_config） -->
 	<xacro:include filename="$(find m6_ccs_description)/xacro/robot.xacro"/>
+	<xacro:include filename="$(find m6_ccs_description)/xacro/eefs.xacro"/>
 	<xacro:include filename="$(find m6_ccs_description)/xacro/ros2_control/interfaces.xacro"/>
 	<ros2_control name="M6_CCS_System" type="system">
@@ -41,22 +42,14 @@
 				<param name="max_joint_speed">$(arg max_joint_speed)</param>
 				<param name="max_joint_acceleration">$(arg max_joint_acceleration)</param>
-				<xacro:if value="${selected_scene == 'desktop'}">
-					<param name="device_ip">192.168.10.190</param>
-					<param name="ctrl_mode">JOINT_IMPEDANCE</param>
-					<param name="left_dyn_param">1.2874,-10.145,30,114.65,0,0,0,0,0,0</param>
-					<param name="right_dyn_param">1.2874,-30.145,-10,147.85,0,0,0,0,0,0</param>
+				<param name="ctrl_mode">$(arg arm_ctrl_mode)</param>
+				<xacro:if value="${'$(arg device_ip)' != ''}">
+					<param name="device_ip">$(arg device_ip)</param>
 				</xacro:if>
-				<xacro:if value="${selected_scene != 'desktop'}">
-					<xacro:ee_dyn_param side="left"
-						ee_key="${left_hand_type if left_hand_type != '' else left_gripper_type}"
-						arg_val="$(arg left_dyn_param)"/>
-					<xacro:ee_dyn_param side="right"
-						ee_key="${right_hand_type if right_hand_type != '' else right_gripper_type}"
-						arg_val="$(arg right_dyn_param)"/>
-				</xacro:if>
-				<xacro:if value="${selected_scene == 'usb-90c'}">
-					<param name="device_ip">192.168.10.190</param>
-					<param name="ctrl_mode">CART_IMPEDANCE</param>
-				</xacro:if>
+				<xacro:ee_dyn_param side="left"
+					ee_key="${left_hand_type if left_hand_type != '' else left_gripper_type}"
+					arg_val="$(arg left_dyn_param)"/>
+				<xacro:ee_dyn_param side="right"
+					ee_key="${right_hand_type if right_hand_type != '' else right_gripper_type}"
+					arg_val="$(arg right_dyn_param)"/>
 			</xacro:if>
 		</hardware>
@@ -104,10 +97,5 @@
 		<xacro:unless value="${selected_arm_config == 'dual'}">
 			<xacro:if value="${selected_arm_config == 'left'}">
-				<xacro:if value="${selected_scene == 'usb-90c'}">
-					<xacro:m6_interfaces name="left"/>
-				</xacro:if>
-				<xacro:unless value="${selected_scene == 'usb-90c'}">
-					<xacro:m6_interfaces name=""/>
-				</xacro:unless>
+				<xacro:m6_interfaces name=""/>
 				<xacro:if value="${selected_gripper_type == 'ag2f90_c' or selected_gripper_type == 'ag2f90_d'}">
 					<xacro:include filename="$(find changingtek_description)/xacro/ros2_control/AG2F90-C.xacro"/>
