Commit message: Fix collision geometry and adjust origin for arm base in robot.xacro

File: m6_ccs_description/xacro/robot.xacro (robot description, xacro)
@@ -104,7 +104,13 @@
 			<link name="arm_base">
 				<collision>
-					<origin xyz="0.0091 0 -0.25"/>
+					<origin xyz="0.0091 0 -0.05"/>
 					<geometry>
-						<box size="0.2000 0.3 0.4029"/>
+						<box size="0.20 0.32 0.20"/>
+					</geometry>
+				</collision>
+				<collision>
+					<origin xyz="0.0091 0 -0.30"/>
+					<geometry>
+						<box size="0.16 0.26 0.30"/>
 					</geometry>
 				</collision>

Commit message: Comment out collision geometry for arm base in robot.xacro

File: m6_ccs_description/xacro/robot.xacro (robot description, xacro)
@@ -103,10 +103,10 @@
 			<link name="base_link"/>
 			<link name="arm_base">
-				<collision>
+				<!-- <collision>
 					<origin xyz="0.0091 0 -0.05"/>
 					<geometry>
 						<box size="0.20 0.32 0.20"/>
 					</geometry>
-				</collision>
+				</collision> -->
 				<collision>
 					<origin xyz="0.0091 0 -0.30"/>
