Commit message: add freedom and inspire hand configurations and dependencies

File: m6_ccs_description/xacro/eef_type_resolver.xacro (robot description, xacro)
@@ -32,4 +32,10 @@
             <xacro:property name="${side}_hand_type" value="linkerhand_o7" scope="parent"/>
         </xacro:if>
+        <xacro:if value="${type_key == 'freedom_v1' or type_key == 'freedom-v1'}">
+            <xacro:property name="${side}_hand_type" value="freedom_v1" scope="parent"/>
+        </xacro:if>
+        <xacro:if value="${type_key == 'inspire_e2' or type_key == 'inspire-e2'}">
+            <xacro:property name="${side}_hand_type" value="inspire_e2" scope="parent"/>
+        </xacro:if>
     </xacro:macro>
 </robot>

File: m6_ccs_description/xacro/eefs.xacro (robot description, xacro)
@@ -5,4 +5,6 @@
     <xacro:include filename="$(find jodell_description)/xacro/RG75-300.xacro"/>
     <xacro:include filename="$(find changingtek_description)/xacro/AG2F90-C.xacro"/>
+    <xacro:include filename="$(find freedom_description)/xacro/freedom.xacro"/>
+    <xacro:include filename="$(find inspire_description)/xacro/hands/RH56E2.xacro"/>
     <xacro:macro name="Ocs2SideEefFrame" params="side parent_link">
         <link name="${side}_eef"/>
@@ -55,4 +57,30 @@
             </joint>
         </xacro:if>
+        <xacro:if value="${hand_type == 'freedom_v1'}">
+            <xacro:FreedomHand name="${side}_hand" direction="${1 if side == 'left' else -1}" fixed_joints="${eef_fixed_joints}"/>
+            <joint name="${side}_hand_base_joint" type="fixed">
+                <xacro:if value="${side == 'left'}">
+                    <origin xyz="0 0 0.0045" rpy="${PI/2} 0 ${PI}"/>
+                </xacro:if>
+                <xacro:if value="${side == 'right'}">
+                    <origin xyz="0 0 0.0045" rpy="${PI/2} 0 0"/>
+                </xacro:if>
+                <parent link="${side}_tcp"/>
+                <child link="${side}_hand_hand_base"/>
+            </joint>
+        </xacro:if>
+        <xacro:if value="${hand_type == 'inspire_e2'}">
+            <xacro:InspireHandRH56E2 name="${side}_hand" direction="${1 if side == 'left' else -1}" use_flange="true"/>
+            <joint name="${side}_hand_base_joint" type="fixed">
+                <xacro:if value="${side == 'left'}">
+                    <origin xyz="0 0 0.0045" rpy="0 0 ${PI/2}"/>
+                </xacro:if>
+                <xacro:if value="${side == 'right'}">
+                    <origin xyz="0 0 0.0045" rpy="0 0 ${-PI/2}"/>
+                </xacro:if>
+                <parent link="${side}_tcp"/>
+                <child link="${side}_hand_flange"/>
+            </joint>
+        </xacro:if>
         <!-- LinkerHand O6/L6/O7: built-in ${side}_hand_eef; alias ${side}_eef for OCS2 / task.info -->
         <xacro:if value="${hand_type == 'linkerhand_o6' or hand_type == 'linkerhand_l6' or hand_type == 'linkerhand_o7'}">
@@ -63,12 +91,19 @@
             </joint>
         </xacro:if>
+        <xacro:if value="${hand_type == 'freedom_v1' or hand_type == 'inspire_e2'}">
+            <link name="${side}_eef"/>
+            <joint name="${side}_eef_joint" type="fixed">
+                <parent link="${side}_hand_hand_base"/>
+                <child link="${side}_eef"/>
+            </joint>
+        </xacro:if>
     </xacro:macro>
     <xacro:macro name="SideEndEffector" params="side hand_type gripper_type gripper_pad eef_fixed_joints:=false">
         <!-- OCS2 planning URDF: no actuated EEF DOF (avoids per-tool removeJoints in .info) -->
         <xacro:if value="${eef_fixed_joints}">
-            <xacro:if value="${hand_type == 'linkerhand_o6' or hand_type == 'linkerhand_o7' or hand_type == 'linkerhand_l6'}">
+            <xacro:if value="${hand_type == 'linkerhand_o6' or hand_type == 'linkerhand_o7' or hand_type == 'linkerhand_l6' or hand_type == 'freedom_v1' or hand_type == 'inspire_e2'}">
                 <xacro:SideEndEffectorLinkerHand side="${side}" hand_type="${hand_type}" eef_fixed_joints="true"/>
             </xacro:if>
-            <xacro:unless value="${hand_type == 'linkerhand_o6' or hand_type == 'linkerhand_o7' or hand_type == 'linkerhand_l6'}">
+            <xacro:unless value="${hand_type == 'linkerhand_o6' or hand_type == 'linkerhand_o7' or hand_type == 'linkerhand_l6' or hand_type == 'freedom_v1' or hand_type == 'inspire_e2'}">
                 <xacro:if value="${gripper_type == 'ag2f90_c' or gripper_type == 'ag2f90_d'}">
                     <xacro:AG2F90-C name="${side}" use_flange="true" pad="${gripper_pad}" kinematic_only="true"/>

File: m6_ccs_description/xacro/ros2_control/robot.xacro (robot description, xacro)
@@ -55,4 +55,6 @@
 			<xacro:include filename="$(find linkerhand_description)/xacro/ros2_control/o6.xacro"/>
 			<xacro:include filename="$(find linkerhand_description)/xacro/ros2_control/o7.xacro"/>
+			<xacro:include filename="$(find freedom_description)/xacro/ros2_control/freedom.xacro"/>
+			<xacro:include filename="$(find inspire_description)/xacro/ros2_control/RH56E2.xacro"/>
 			<xacro:if value="${left_gripper_type == 'rg75'}">
 				<xacro:rg75_interfaces name="left"/>
@@ -78,4 +80,16 @@
 			<xacro:if value="${right_hand_type == 'linkerhand_o7'}">
 				<xacro:linkerhand_o7_interfaces name="right_hand"/>
+			</xacro:if>
+			<xacro:if value="${left_hand_type == 'freedom_v1'}">
+				<xacro:freedom_interfaces name="left_hand"/>
+			</xacro:if>
+			<xacro:if value="${right_hand_type == 'freedom_v1'}">
+				<xacro:freedom_interfaces name="right_hand"/>
+			</xacro:if>
+			<xacro:if value="${left_hand_type == 'inspire_e2'}">
+				<xacro:inspire_rh56e2_interfaces name="left_hand"/>
+			</xacro:if>
+			<xacro:if value="${right_hand_type == 'inspire_e2'}">
+				<xacro:inspire_rh56e2_interfaces name="right_hand"/>
 			</xacro:if>
 		</xacro:if>

Commit message: 规范freedom xacro

File: m6_ccs_description/xacro/eef_type_resolver.xacro (robot description, xacro)
@@ -32,8 +32,8 @@
             <xacro:property name="${side}_hand_type" value="linkerhand_o7" scope="parent"/>
         </xacro:if>
-        <xacro:if value="${type_key == 'freedom_v1' or type_key == 'freedom-v1'}">
+        <xacro:if value="${type_key == 'freedom_v1'}">
             <xacro:property name="${side}_hand_type" value="freedom_v1" scope="parent"/>
         </xacro:if>
-        <xacro:if value="${type_key == 'inspire_e2' or type_key == 'inspire-e2'}">
+        <xacro:if value="${type_key == 'inspire_e2'}">
             <xacro:property name="${side}_hand_type" value="inspire_e2" scope="parent"/>
         </xacro:if>

File: m6_ccs_description/xacro/ros2_control/robot.xacro (robot description, xacro)
@@ -19,26 +19,26 @@
 	<xacro:include filename="$(find m6_ccs_description)/xacro/robot.xacro"/>
 	<xacro:include filename="$(find m6_ccs_description)/xacro/ros2_control/interfaces.xacro"/>
-	<xacro:include filename="$(find jodell_description)/xacro/ros2_control/RG75-300.xacro"/>
-	<xacro:include filename="$(find changingtek_description)/xacro/ros2_control/AG2F90-C.xacro"/>
-	<xacro:include filename="$(find linkerhand_description)/xacro/ros2_control/o6.xacro"/>
-	<xacro:include filename="$(find linkerhand_description)/xacro/ros2_control/o7.xacro"/>
-	<xacro:include filename="$(find freedom_description)/xacro/ros2_control/freedom.xacro"/>
-	<xacro:include filename="$(find inspire_description)/xacro/ros2_control/RH56E2.xacro"/>
+	<xacro:include filename="$(find freedom_description)/xacro/ros2_control/side_systems.xacro"/>
+	<xacro:include filename="$(find inspire_description)/xacro/ros2_control/side_systems.xacro"/>
 	<xacro:macro name="side_hand_interfaces" params="side hand_type">
 		<xacro:if value="${hand_type == 'linkerhand_o6' or hand_type == 'linkerhand_l6'}">
+			<xacro:include filename="$(find linkerhand_description)/xacro/ros2_control/o6.xacro"/>
 			<xacro:linkerhand_o6_interfaces name="${side}_hand"/>
 		</xacro:if>
 		<xacro:if value="${hand_type == 'linkerhand_o7'}">
+			<xacro:include filename="$(find linkerhand_description)/xacro/ros2_control/o7.xacro"/>
 			<xacro:linkerhand_o7_interfaces name="${side}_hand"/>
 		</xacro:if>
-		<xacro:if value="${hand_type == 'freedom_v1' or hand_type == 'freedom-v1'}">
+		<xacro:if value="${hand_type == 'freedom_v1'}">
+			<xacro:include filename="$(find freedom_description)/xacro/ros2_control/freedom.xacro"/>
 			<xacro:freedom_interfaces name="${side}_hand"/>
 		</xacro:if>
-		<xacro:if value="${hand_type == 'inspire_e2' or hand_type == 'inspire-e2'}">
+		<xacro:if value="${hand_type == 'inspire_e2'}">
+			<xacro:include filename="$(find inspire_description)/xacro/ros2_control/RH56E2.xacro"/>
 			<xacro:inspire_rh56e2_interfaces name="${side}_hand"/>
 		</xacro:if>
 	</xacro:macro>
 	<xacro:macro name="side_usb_hand_system" params="side hand_type serial_port">
-		<xacro:property name="usb_hand_system_name" value="${str('linkerhand_7' if hand_type == 'linkerhand_o7' else ('inspire_e2' if hand_type == 'inspire_e2' or hand_type == 'inspire-e2' else 'linkerhand_6'))}"/>
+		<xacro:property name="usb_hand_system_name" value="${str('linkerhand_7' if hand_type == 'linkerhand_o7' else 'linkerhand_6')}"/>
 		<ros2_control name="${usb_hand_system_name}_${side}_system" type="system">
 			<hardware>
@@ -50,30 +50,4 @@
 			</hardware>
 			<xacro:side_hand_interfaces side="${side}" hand_type="${hand_type}"/>
-		</ros2_control>
-	</xacro:macro>
-	<xacro:macro name="side_freedom_usb_hand_system" params="side serial_port">
-		<ros2_control name="freedom_v1_${side}_system" type="system">
-			<hardware>
-				<plugin>modbus_ros2_control/FreedomRS485Hardware</plugin>
-				<param name="serial_port">${serial_port}</param>
-				<param name="hand_side">${side}</param>
-				<param name="slave_id">auto</param>
-				<param name="baudrate">115200</param>
-				<param name="read_feedback">true</param>
-				<param name="feedback_timeout_ms">20</param>
-			</hardware>
-			<xacro:freedom_interfaces name="${side}_hand"/>
-		</ros2_control>
-	</xacro:macro>
-	<xacro:macro name="side_freedom_usb_can_hand_system" params="side can_interface device_id">
-		<ros2_control name="freedom_v1_${side}_can_system" type="system">
-			<hardware>
-				<plugin>can_ros2_control/FreedomCanHardware</plugin>
-				<param name="can_interface">${can_interface}</param>
-				<param name="device_id">${device_id}</param>
-				<param name="read_feedback">true</param>
-				<param name="feedback_timeout_ms">1</param>
-			</hardware>
-			<xacro:freedom_interfaces name="${side}_hand"/>
 		</ros2_control>
 	</xacro:macro>
@@ -135,24 +109,26 @@
 			<xacro:m6_interfaces name="left"/>
 			<xacro:m6_interfaces name="right"/>
-			<xacro:include filename="$(find jodell_description)/xacro/ros2_control/RG75-300.xacro"/>
-			<xacro:include filename="$(find changingtek_description)/xacro/ros2_control/AG2F90-C.xacro"/>
-			<xacro:include filename="$(find linkerhand_description)/xacro/ros2_control/o6.xacro"/>
-			<xacro:include filename="$(find linkerhand_description)/xacro/ros2_control/o7.xacro"/>
 			<xacro:if value="${left_gripper_type == 'rg75'}">
+				<xacro:include filename="$(find jodell_description)/xacro/ros2_control/RG75-300.xacro"/>
 				<xacro:rg75_interfaces name="left"/>
 			</xacro:if>
 			<xacro:if value="${right_gripper_type == 'rg75'}">
+				<xacro:include filename="$(find jodell_description)/xacro/ros2_control/RG75-300.xacro"/>
 				<xacro:rg75_interfaces name="right"/>
 			</xacro:if>
 			<xacro:if value="${left_gripper_type == 'ag2f90_c' or left_gripper_type == 'ag2f90_d'}">
+				<xacro:include filename="$(find changingtek_description)/xacro/ros2_control/AG2F90-C.xacro"/>
 				<xacro:ag2f90c_interfaces name="left"/>
 			</xacro:if>
 			<xacro:if value="${right_gripper_type == 'ag2f90_c' or right_gripper_type == 'ag2f90_d'}">
+				<xacro:include filename="$(find changingtek_description)/xacro/ros2_control/AG2F90-C.xacro"/>
 				<xacro:ag2f90c_interfaces name="right"/>
 			</xacro:if>
 			<xacro:if value="${left_hand_type == 'linkerhand_o6' or left_hand_type == 'linkerhand_l6'}">
+				<xacro:include filename="$(find linkerhand_description)/xacro/ros2_control/o6.xacro"/>
 				<xacro:linkerhand_o6_interfaces name="left_hand"/>
 			</xacro:if>
 			<xacro:if value="${right_hand_type == 'linkerhand_o6' or right_hand_type == 'linkerhand_l6'}">
+				<xacro:include filename="$(find linkerhand_description)/xacro/ros2_control/o6.xacro"/>
 				<xacro:linkerhand_o6_interfaces name="right_hand"/>
 			</xacro:if>
@@ -163,7 +139,9 @@
 			</xacro:if>
 			<xacro:if value="${left_hand_type == 'linkerhand_o7'}">
+				<xacro:include filename="$(find linkerhand_description)/xacro/ros2_control/o7.xacro"/>
 				<xacro:linkerhand_o7_interfaces name="left_hand"/>
 			</xacro:if>
 			<xacro:if value="${right_hand_type == 'linkerhand_o7'}">
+				<xacro:include filename="$(find linkerhand_description)/xacro/ros2_control/o7.xacro"/>
 				<xacro:linkerhand_o7_interfaces name="right_hand"/>
 			</xacro:if>
@@ -198,21 +176,27 @@
 	</ros2_control>
 	<xacro:if value="${is_real_hardware and selected_arm_config == 'dual'}">
-		<xacro:if value="${left_drive_type == 'usb' and (left_hand_type == 'linkerhand_o6' or left_hand_type == 'linkerhand_l6' or left_hand_type == 'linkerhand_o7' or left_hand_type == 'inspire_e2' or left_hand_type == 'inspire-e2')}">
+		<xacro:if value="${left_drive_type == 'usb' and (left_hand_type == 'linkerhand_o6' or left_hand_type == 'linkerhand_l6' or left_hand_type == 'linkerhand_o7')}">
 			<xacro:side_usb_hand_system side="left" hand_type="${left_hand_type}" serial_port="/dev/ttyUSB0"/>
 		</xacro:if>
-		<xacro:if value="${right_drive_type == 'usb' and (right_hand_type == 'linkerhand_o6' or right_hand_type == 'linkerhand_l6' or right_hand_type == 'linkerhand_o7' or right_hand_type == 'inspire_e2' or right_hand_type == 'inspire-e2')}">
+		<xacro:if value="${right_drive_type == 'usb' and (right_hand_type == 'linkerhand_o6' or right_hand_type == 'linkerhand_l6' or right_hand_type == 'linkerhand_o7')}">
 			<xacro:side_usb_hand_system side="right" hand_type="${right_hand_type}" serial_port="/dev/ttyUSB2"/>
 		</xacro:if>
-		<xacro:if value="${left_drive_type == 'usb' and (left_hand_type == 'freedom_v1' or left_hand_type == 'freedom-v1')}">
-			<xacro:side_freedom_usb_hand_system side="left" serial_port="/dev/ttyUSB0"/>
-		</xacro:if>
-		<xacro:if value="${right_drive_type == 'usb' and (right_hand_type == 'freedom_v1' or right_hand_type == 'freedom-v1')}">
-			<xacro:side_freedom_usb_hand_system side="right" serial_port="/dev/ttyUSB2"/>
-		</xacro:if>
-		<xacro:if value="${left_drive_type == 'usb_can' and (left_hand_type == 'freedom_v1' or left_hand_type == 'freedom-v1')}">
-			<xacro:side_freedom_usb_can_hand_system side="left" can_interface="can0" device_id="0"/>
-		</xacro:if>
-		<xacro:if value="${right_drive_type == 'usb_can' and (right_hand_type == 'freedom_v1' or right_hand_type == 'freedom-v1')}">
-			<xacro:side_freedom_usb_can_hand_system side="right" can_interface="can1" device_id="1"/>
+		<xacro:if value="${left_drive_type == 'usb' and left_hand_type == 'inspire_e2'}">
+			<xacro:inspire_rs485_side_system side="left" serial_port="/dev/ttyUSB0"/>
+		</xacro:if>
+		<xacro:if value="${right_drive_type == 'usb' and right_hand_type == 'inspire_e2'}">
+			<xacro:inspire_rs485_side_system side="right" serial_port="/dev/ttyUSB2"/>
+		</xacro:if>
+		<xacro:if value="${left_drive_type == 'usb' and left_hand_type == 'freedom_v1'}">
+			<xacro:freedom_rs485_side_system side="left" serial_port="/dev/ttyUSB0"/>
+		</xacro:if>
+		<xacro:if value="${right_drive_type == 'usb' and right_hand_type == 'freedom_v1'}">
+			<xacro:freedom_rs485_side_system side="right" serial_port="/dev/ttyUSB2"/>
+		</xacro:if>
+		<xacro:if value="${left_drive_type == 'usb_can' and left_hand_type == 'freedom_v1'}">
+			<xacro:freedom_can_side_system side="left" can_interface="can0" device_id="0"/>
+		</xacro:if>
+		<xacro:if value="${right_drive_type == 'usb_can' and right_hand_type == 'freedom_v1'}">
+			<xacro:freedom_can_side_system side="right" can_interface="can1" device_id="1"/>
 		</xacro:if>
 	</xacro:if>

Commit message: 添加freedomv2

File: m6_ccs_description/xacro/eef_type_resolver.xacro (robot description, xacro)
@@ -35,4 +35,7 @@
             <xacro:property name="${side}_hand_type" value="freedom_v1" scope="parent"/>
         </xacro:if>
+        <xacro:if value="${type_key == 'freedom_v2'}">
+            <xacro:property name="${side}_hand_type" value="freedom_v2" scope="parent"/>
+        </xacro:if>
         <xacro:if value="${type_key == 'inspire_e2'}">
             <xacro:property name="${side}_hand_type" value="inspire_e2" scope="parent"/>

File: m6_ccs_description/xacro/eefs.xacro (robot description, xacro)
@@ -5,5 +5,6 @@
     <xacro:include filename="$(find jodell_description)/xacro/RG75-300.xacro"/>
     <xacro:include filename="$(find changingtek_description)/xacro/AG2F90-C.xacro"/>
-    <xacro:include filename="$(find freedom_description)/xacro/freedom.xacro"/>
+    <xacro:include filename="$(find freedom_description)/xacro/freedomv1.xacro"/>
+    <xacro:include filename="$(find freedom_description)/xacro/freedomv2.xacro"/>
     <xacro:include filename="$(find inspire_description)/xacro/hands/RH56E2.xacro"/>
     <xacro:macro name="Ocs2SideEefFrame" params="side parent_link">
@@ -70,4 +71,17 @@
             </joint>
         </xacro:if>
+        <xacro:if value="${hand_type == 'freedom_v2'}">
+            <xacro:FreedomHandV2 name="${side}_hand" direction="${1 if side == 'left' else -1}" fixed_joints="${eef_fixed_joints}"/>
+            <joint name="${side}_hand_base_joint" type="fixed">
+                <xacro:if value="${side == 'left'}">
+                    <origin xyz="0 0 0" rpy="0 0 ${PI/2}"/>
+                </xacro:if>
+                <xacro:if value="${side == 'right'}">
+                    <origin xyz="0 0 0" rpy="0 0 ${-PI/2}"/>
+                </xacro:if>
+                <parent link="${side}_tcp"/>
+                <child link="${side}_hand_hand_base"/>
+            </joint>
+        </xacro:if>
         <xacro:if value="${hand_type == 'inspire_e2'}">
             <xacro:InspireHandRH56E2 name="${side}_hand" direction="${1 if side == 'left' else -1}" use_flange="true"/>
@@ -91,5 +105,5 @@
             </joint>
         </xacro:if>
-        <xacro:if value="${hand_type == 'freedom_v1' or hand_type == 'inspire_e2'}">
+        <xacro:if value="${hand_type == 'freedom_v1' or hand_type == 'freedom_v2' or hand_type == 'inspire_e2'}">
             <link name="${side}_eef"/>
             <joint name="${side}_eef_joint" type="fixed">
@@ -102,8 +116,8 @@
         <!-- OCS2 planning URDF: no actuated EEF DOF (avoids per-tool removeJoints in .info) -->
         <xacro:if value="${eef_fixed_joints}">
-            <xacro:if value="${hand_type == 'linkerhand_o6' or hand_type == 'linkerhand_o7' or hand_type == 'linkerhand_l6' or hand_type == 'freedom_v1' or hand_type == 'inspire_e2'}">
+            <xacro:if value="${hand_type == 'linkerhand_o6' or hand_type == 'linkerhand_o7' or hand_type == 'linkerhand_l6' or hand_type == 'freedom_v1' or hand_type == 'freedom_v2' or hand_type == 'inspire_e2'}">
                 <xacro:SideEndEffectorLinkerHand side="${side}" hand_type="${hand_type}" eef_fixed_joints="true"/>
             </xacro:if>
-            <xacro:unless value="${hand_type == 'linkerhand_o6' or hand_type == 'linkerhand_o7' or hand_type == 'linkerhand_l6' or hand_type == 'freedom_v1' or hand_type == 'inspire_e2'}">
+            <xacro:unless value="${hand_type == 'linkerhand_o6' or hand_type == 'linkerhand_o7' or hand_type == 'linkerhand_l6' or hand_type == 'freedom_v1' or hand_type == 'freedom_v2' or hand_type == 'inspire_e2'}">
                 <xacro:if value="${gripper_type == 'ag2f90_c' or gripper_type == 'ag2f90_d'}">
                     <xacro:AG2F90-C name="${side}" use_flange="true" pad="${gripper_pad}" kinematic_only="true"/>

File: m6_ccs_description/xacro/ros2_control/robot.xacro (robot description, xacro)
@@ -31,6 +31,10 @@
 		</xacro:if>
 		<xacro:if value="${hand_type == 'freedom_v1'}">
-			<xacro:include filename="$(find freedom_description)/xacro/ros2_control/freedom.xacro"/>
+			<xacro:include filename="$(find freedom_description)/xacro/ros2_control/freedomv1.xacro"/>
 			<xacro:freedom_interfaces name="${side}_hand"/>
+		</xacro:if>
+		<xacro:if value="${hand_type == 'freedom_v2'}">
+			<xacro:include filename="$(find freedom_description)/xacro/ros2_control/freedomv2.xacro"/>
+			<xacro:freedomv2_interfaces name="${side}_hand"/>
 		</xacro:if>
 		<xacro:if value="${hand_type == 'inspire_e2'}">
@@ -194,4 +198,10 @@
 			<xacro:freedom_rs485_side_system side="right" serial_port="/dev/ttyUSB2"/>
 		</xacro:if>
+		<xacro:if value="${left_drive_type == 'usb' and left_hand_type == 'freedom_v2'}">
+			<xacro:freedom_rs485_side_system side="left" serial_port="/dev/ttyUSB0" type="freedomv2"/>
+		</xacro:if>
+		<xacro:if value="${right_drive_type == 'usb' and right_hand_type == 'freedom_v2'}">
+			<xacro:freedom_rs485_side_system side="right" serial_port="/dev/ttyUSB2" type="freedomv2"/>
+		</xacro:if>
 		<xacro:if value="${left_drive_type == 'usb_can' and left_hand_type == 'freedom_v1'}">
 			<xacro:freedom_can_side_system side="left" can_interface="can0" device_id="0"/>
