Commit message: 增加120s夹爪

File: m6_ccs_description/xacro/eef_type_resolver.xacro (robot description, xacro)
@@ -23,4 +23,7 @@
             <xacro:property name="${side}_gripper_pad" value="soft" scope="parent"/>
         </xacro:if>
+        <xacro:if value="${type_key == 'ctag2f120s'}">
+            <xacro:property name="${side}_gripper_type" value="ctag2f120s" scope="parent"/>
+        </xacro:if>
         <xacro:if value="${type_key == 'linkerhand_o6'}">
             <xacro:property name="${side}_hand_type" value="linkerhand_o6" scope="parent"/>

File: m6_ccs_description/xacro/eefs.xacro (robot description, xacro)
@@ -5,4 +5,5 @@
     <xacro:include filename="$(find jodell_description)/xacro/RG75-300.xacro"/>
     <xacro:include filename="$(find changingtek_description)/xacro/AG2F90-C.xacro"/>
+    <xacro:include filename="$(find changingtek_description)/xacro/AG2F120S.xacro"/>
     <!-- Per-side default load (dyn_param) for MarvinHardware; 10 values: m, mx, my, mz, ixx, ixy, ixz, iyy, iyz, izz.
          Override via launch left_dyn_param/right_dyn_param (robot.local.yaml).
@@ -21,5 +22,5 @@
                     <param name="${side}_dyn_param">1.6200799541791235, 1.4285009257202586, -0.5789585762443014, 104.39051192831192, 0.004873874899366342, 0.0, 0.0, 0.001, 0.0, 0.0019355638096347936</param>
                 </xacro:if>
-                <xacro:if value="${ee_key == 'ag2f90_c' or ee_key == 'ag2f90_d' or ee_key == 'ag2f90_c_soft'}">
+                <xacro:if value="${ee_key == 'ag2f90_c' or ee_key == 'ag2f90_d' or ee_key == 'ag2f90_c_soft' or ee_key == 'ctag2f120s'}">
                     <param name="${side}_dyn_param">0.9464750422461978, -8.366166030270293, -9.50810456883501, 71.59365292895114, 0.02313627009490121, 0.0, 0.0, 0.017136701127687514, 0.0, 0.008640226166892327</param>
                 </xacro:if>
@@ -38,5 +39,5 @@
                     <param name="${side}_dyn_param">1.6200799541791235, 1.4285009257202586, -0.5789585762443014, 104.39051192831192, 0.004873874899366342, 0.0, 0.0, 0.001, 0.0, 0.0019355638096347936</param>
                 </xacro:if>
-                <xacro:if value="${ee_key == 'ag2f90_c' or ee_key == 'ag2f90_d' or ee_key == 'ag2f90_c_soft'}">
+                <xacro:if value="${ee_key == 'ag2f90_c' or ee_key == 'ag2f90_d' or ee_key == 'ag2f90_c_soft' or ee_key == 'ctag2f120s'}">
                     <param name="${side}_dyn_param">0.9464750422461978, -8.366166030270293, -9.50810456883501, 71.59365292895114, 0.02313627009490121, 0.0, 0.0, 0.017136701127687514, 0.0, 0.008640226166892327</param>
                 </xacro:if>
@@ -125,4 +126,12 @@
                         <parent link="${side}_tcp"/>
                         <child link="${side}_flange"/>
+                        <origin xyz="0 0 0.0045"/>
+                    </joint>
+                </xacro:if>
+                <xacro:if value="${gripper_type == 'ctag2f120s'}">
+                    <xacro:AG2F120S name="${side}" kinematic_only="true"/>
+                    <joint name="${side}_gripper_fix" type="fixed">
+                        <parent link="${side}_tcp"/>
+                        <child link="${side}_gripper_base"/>
                         <origin xyz="0 0 0.0045"/>
                     </joint>
@@ -156,4 +165,12 @@
                     <parent link="${side}_tcp"/>
                     <child link="${side}_flange"/>
+                    <origin xyz="0 0 0.0045"/>
+                </joint>
+            </xacro:if>
+            <xacro:if value="${gripper_type == 'ctag2f120s'}">
+                <xacro:AG2F120S name="${side}"/>
+                <joint name="${side}_gripper_fix" type="fixed">
+                    <parent link="${side}_tcp"/>
+                    <child link="${side}_gripper_base"/>
                     <origin xyz="0 0 0.0045"/>
                 </joint>

File: m6_ccs_description/xacro/robot.xacro (robot description, xacro)
@@ -48,4 +48,7 @@
 	<xacro:if value="${type_arg == 'ag2f90_d'}">
 		<xacro:property name="selected_gripper_type" value="ag2f90_d"/>
+	</xacro:if>
+	<xacro:if value="${type_arg == 'ctag2f120s'}">
+		<xacro:property name="selected_gripper_type" value="ctag2f120s"/>
 	</xacro:if>
 	<xacro:if value="${type_arg == 'rg75'}">

File: m6_ccs_description/xacro/ros2_control/robot.xacro (robot description, xacro)
@@ -64,4 +64,5 @@
 			<xacro:include filename="$(find jodell_description)/xacro/ros2_control/RG75-300.xacro"/>
 			<xacro:include filename="$(find changingtek_description)/xacro/ros2_control/AG2F90-C.xacro"/>
+			<xacro:include filename="$(find changingtek_description)/xacro/ros2_control/AG2F120S.xacro"/>
 			<xacro:include filename="$(find linkerhand_description)/xacro/ros2_control/o6.xacro"/>
 			<xacro:include filename="$(find linkerhand_description)/xacro/ros2_control/o7.xacro"/>
@@ -77,4 +78,10 @@
 			<xacro:if value="${right_gripper_type == 'ag2f90_c' or right_gripper_type == 'ag2f90_d'}">
 				<xacro:ag2f90c_interfaces name="right"/>
+			</xacro:if>
+			<xacro:if value="${left_gripper_type == 'ctag2f120s'}">
+				<xacro:ag2f120s_interfaces name="left"/>
+			</xacro:if>
+			<xacro:if value="${right_gripper_type == 'ctag2f120s'}">
+				<xacro:ag2f120s_interfaces name="right"/>
 			</xacro:if>
 			<xacro:if value="${left_hand_type == 'linkerhand_o6' or left_hand_type == 'linkerhand_l6'}">
@@ -103,4 +110,8 @@
 					<xacro:include filename="$(find changingtek_description)/xacro/ros2_control/AG2F90-C.xacro"/>
 					<xacro:ag2f90c_interfaces name=""/>
+				</xacro:if>
+				<xacro:if value="${selected_gripper_type == 'ctag2f120s'}">
+					<xacro:include filename="$(find changingtek_description)/xacro/ros2_control/AG2F120S.xacro"/>
+					<xacro:ag2f120s_interfaces name=""/>
 				</xacro:if>
 				<xacro:if value="${selected_gripper_type == 'rg75'}">

Commit message: add xhand1 support

File: m6_ccs_description/xacro/eef_type_resolver.xacro (robot description, xacro)
@@ -41,4 +41,7 @@
             <xacro:property name="${side}_hand_type" value="inspire_e2" scope="parent"/>
         </xacro:if>
+        <xacro:if value="${type_key == 'xhand1'}">
+            <xacro:property name="${side}_hand_type" value="xhand1" scope="parent"/>
+        </xacro:if>
     </xacro:macro>
 </robot>

File: m6_ccs_description/xacro/eefs.xacro (robot description, xacro)
@@ -8,4 +8,5 @@
     <xacro:include filename="$(find freedom_description)/xacro/freedomv2.xacro"/>
     <xacro:include filename="$(find inspire_description)/xacro/hands/RH56E2.xacro"/>
+    <xacro:include filename="$(find xhand1_description)/xacro/xhand1.xacro"/>
     <!-- Per-side default load (dyn_param) for MarvinHardware; 10 values: m, mx, my, mz, ixx, ixy, ixz, iyy, iyz, izz.
          Override via launch left_dyn_param/right_dyn_param (robot.local.yaml).
@@ -146,5 +147,25 @@
             </joint>
         </xacro:if>
+        <xacro:if value="${hand_type == 'xhand1'}">
+            <xacro:XHand1 name="${side}_hand" direction="${1 if side == 'left' else -1}"/>
+            <joint name="${side}_hand_base_joint" type="fixed">
+                <xacro:if value="${side == 'left'}">
+                    <origin xyz="0 0 0" rpy="0 0 ${PI}"/>
+                </xacro:if>
+                <xacro:if value="${side == 'right'}">
+                    <origin xyz="0 0 0" rpy="0 0 ${PI}"/>
+                </xacro:if>
+                <parent link="${side}_tcp"/>
+                <child link="${side}_hand_hand_base"/>
+            </joint>
+        </xacro:if>
         <!-- Hands with built-in ${side}_hand_eef; alias ${side}_eef for OCS2 / task.info -->
+        <xacro:if value="${hand_type == 'xhand1'}">
+            <link name="${side}_eef"/>
+            <joint name="${side}_eef_joint" type="fixed">
+                <parent link="${side}_hand_hand_ee_link"/>
+                <child link="${side}_eef"/>
+            </joint>
+        </xacro:if>
         <xacro:if value="${hand_type == 'linkerhand_o6' or hand_type == 'linkerhand_l6' or hand_type == 'linkerhand_o7' or hand_type == 'freedom_v1' or hand_type == 'freedom_v2' or hand_type == 'inspire_e2'}">
             <link name="${side}_eef"/>
@@ -158,8 +179,8 @@
         <!-- OCS2 planning URDF: no actuated EEF DOF (avoids per-tool removeJoints in .info) -->
         <xacro:if value="${eef_fixed_joints}">
-            <xacro:if value="${hand_type == 'linkerhand_o6' or hand_type == 'linkerhand_o7' or hand_type == 'linkerhand_l6' or hand_type == 'freedom_v1' or hand_type == 'freedom_v2' or hand_type == 'inspire_e2'}">
+            <xacro:if value="${hand_type == 'linkerhand_o6' or hand_type == 'linkerhand_o7' or hand_type == 'linkerhand_l6' or hand_type == 'freedom_v1' or hand_type == 'freedom_v2' or hand_type == 'inspire_e2' or hand_type == 'xhand1'}">
                 <xacro:SideEndEffectorLinkerHand side="${side}" hand_type="${hand_type}" eef_fixed_joints="true"/>
             </xacro:if>
-            <xacro:unless value="${hand_type == 'linkerhand_o6' or hand_type == 'linkerhand_o7' or hand_type == 'linkerhand_l6' or hand_type == 'freedom_v1' or hand_type == 'freedom_v2' or hand_type == 'inspire_e2'}">
+            <xacro:unless value="${hand_type == 'linkerhand_o6' or hand_type == 'linkerhand_o7' or hand_type == 'linkerhand_l6' or hand_type == 'freedom_v1' or hand_type == 'freedom_v2' or hand_type == 'inspire_e2' or hand_type == 'xhand1'}">
                 <xacro:if value="${gripper_type == 'ag2f90_c' or gripper_type == 'ag2f90_d'}">
                     <xacro:AG2F90-C name="${side}" use_flange="true" pad="${gripper_pad}" kinematic_only="true"/>

File: m6_ccs_description/xacro/robot.xacro (robot description, xacro)
@@ -64,4 +64,7 @@
 	<xacro:if value="${type_arg == 'linkerhand_o7'}">
 		<xacro:property name="selected_hand_type" value="linkerhand_o7"/>
+	</xacro:if>
+	<xacro:if value="${type_arg == 'xhand1'}">
+		<xacro:property name="selected_hand_type" value="xhand1"/>
 	</xacro:if>
 	<!-- 适用纯双臂演示场景的配置 -->

File: m6_ccs_description/xacro/ros2_control/robot.xacro (robot description, xacro)
@@ -24,4 +24,5 @@
 	<xacro:include filename="$(find freedom_description)/xacro/ros2_control/side_systems.xacro"/>
 	<xacro:include filename="$(find inspire_description)/xacro/ros2_control/side_systems.xacro"/>
+	<xacro:include filename="$(find xhand1_description)/xacro/ros2_control/side_systems.xacro"/>
 	<xacro:macro name="side_hand_interfaces" params="side hand_type">
 		<xacro:if value="${hand_type == 'linkerhand_o6' or hand_type == 'linkerhand_l6'}">
@@ -44,4 +45,7 @@
 			<xacro:include filename="$(find inspire_description)/xacro/ros2_control/RH56E2.xacro"/>
 			<xacro:inspire_rh56e2_interfaces name="${side}_hand"/>
+		</xacro:if>
+		<xacro:if value="${hand_type == 'xhand1'}">
+			<xacro:xhand1_interfaces name="${side}_hand"/>
 		</xacro:if>
 	</xacro:macro>
@@ -80,5 +84,5 @@
 					<xacro:property name="left_ee_type" value="${left_hand_type if left_hand_type != '' else left_gripper_type}"/>
 					<xacro:property name="right_ee_type" value="${right_hand_type if right_hand_type != '' else right_gripper_type}"/>
-					<xacro:if value="${(left_drive_type == 'marvin' or left_drive_type == 'tianji_can') and left_ee_type != ''}">
+					<xacro:if value="${(left_drive_type == 'marvin' or left_drive_type == 'tianji_can') and left_ee_type != '' and left_ee_type != 'xhand1'}">
 						<param name="left_ee_type">${left_ee_type}</param>
 						<xacro:if value="${left_drive_type == 'tianji_can'}">
@@ -86,5 +90,5 @@
 						</xacro:if>
 					</xacro:if>
-					<xacro:if value="${(right_drive_type == 'marvin' or right_drive_type == 'tianji_can') and right_ee_type != ''}">
+					<xacro:if value="${(right_drive_type == 'marvin' or right_drive_type == 'tianji_can') and right_ee_type != '' and right_ee_type != 'xhand1'}">
 						<param name="right_ee_type">${right_ee_type}</param>
 						<xacro:if value="${right_drive_type == 'tianji_can'}">
@@ -144,10 +148,10 @@
 				<xacro:ag2f90c_interfaces name="right"/>
 			</xacro:if>
-			<xacro:if value="${not is_real_hardware or left_drive_type == 'marvin' or left_drive_type == 'tianji_can'}">
+			<xacro:if value="${(not is_real_hardware) or ((left_drive_type == 'marvin' or left_drive_type == 'tianji_can') and left_hand_type != 'xhand1')}">
 				<xacro:if value="${left_hand_type != ''}">
 					<xacro:side_hand_interfaces side="left" hand_type="${left_hand_type}"/>
 				</xacro:if>
 			</xacro:if>
-			<xacro:if value="${not is_real_hardware or right_drive_type == 'marvin' or right_drive_type == 'tianji_can'}">
+			<xacro:if value="${(not is_real_hardware) or ((right_drive_type == 'marvin' or right_drive_type == 'tianji_can') and right_hand_type != 'xhand1')}">
 				<xacro:if value="${right_hand_type != ''}">
 					<xacro:side_hand_interfaces side="right" hand_type="${right_hand_type}"/>
@@ -202,4 +206,10 @@
 		<xacro:if value="${right_drive_type == 'usb' and right_hand_type == 'freedom_v2'}">
 			<xacro:freedom_rs485_side_system side="right" serial_port="/dev/ttyUSB2" type="freedomv2"/>
+		</xacro:if>
+		<xacro:if value="${left_drive_type == 'usb' and left_hand_type == 'xhand1'}">
+			<xacro:xhand1_rs485_side_system side="left" serial_port="/dev/ttyUSB1"/>
+		</xacro:if>
+		<xacro:if value="${right_drive_type == 'usb' and right_hand_type == 'xhand1'}">
+			<xacro:xhand1_rs485_side_system side="right" serial_port="/dev/ttyUSB0"/>
 		</xacro:if>
 		<xacro:if value="${left_drive_type == 'usb_can' and left_hand_type == 'freedom_v1'}">

Commit message: add 120s

File: m6_ccs_description/xacro/eef_type_resolver.xacro (robot description, xacro)
@@ -23,6 +23,9 @@
             <xacro:property name="${side}_gripper_pad" value="soft" scope="parent"/>
         </xacro:if>
-        <xacro:if value="${type_key == 'ctag2f120s'}">
-            <xacro:property name="${side}_gripper_type" value="ctag2f120s" scope="parent"/>
+        <xacro:if value="${type_key == 'ag2f120s'}">
+            <xacro:property name="${side}_gripper_type" value="ag2f120s" scope="parent"/>
+        </xacro:if>
+        <xacro:if value="${type_key == 'ag2f120s_d'}">
+            <xacro:property name="${side}_gripper_type" value="ag2f120s_d" scope="parent"/>
         </xacro:if>
         <xacro:if value="${type_key == 'linkerhand_o6'}">

File: m6_ccs_description/xacro/eefs.xacro (robot description, xacro)
@@ -22,5 +22,9 @@
                     <param name="${side}_dyn_param">1.6200799541791235, 1.4285009257202586, -0.5789585762443014, 104.39051192831192, 0.004873874899366342, 0.0, 0.0, 0.001, 0.0, 0.0019355638096347936</param>
                 </xacro:if>
-                <xacro:if value="${ee_key == 'ag2f90_c' or ee_key == 'ag2f90_d' or ee_key == 'ag2f90_c_soft' or ee_key == 'ctag2f120s'}">
+                <xacro:if value="${ee_key == 'ag2f90_c' or ee_key == 'ag2f90_d' or ee_key == 'ag2f90_c_soft'}">
+                    <param name="${side}_dyn_param">0.9464750422461978, -8.366166030270293, -9.50810456883501, 71.59365292895114, 0.02313627009490121, 0.0, 0.0, 0.017136701127687514, 0.0, 0.008640226166892327</param>
+                </xacro:if>
+                <xacro:if value="${ee_key == 'ag2f120s' or ee_key == 'ag2f120s_d'}">
+                    <!-- TODO: replace with measured values; temporarily reuse ag2f90 series -->
                     <param name="${side}_dyn_param">0.9464750422461978, -8.366166030270293, -9.50810456883501, 71.59365292895114, 0.02313627009490121, 0.0, 0.0, 0.017136701127687514, 0.0, 0.008640226166892327</param>
                 </xacro:if>
@@ -39,5 +43,9 @@
                     <param name="${side}_dyn_param">1.6200799541791235, 1.4285009257202586, -0.5789585762443014, 104.39051192831192, 0.004873874899366342, 0.0, 0.0, 0.001, 0.0, 0.0019355638096347936</param>
                 </xacro:if>
-                <xacro:if value="${ee_key == 'ag2f90_c' or ee_key == 'ag2f90_d' or ee_key == 'ag2f90_c_soft' or ee_key == 'ctag2f120s'}">
+                <xacro:if value="${ee_key == 'ag2f90_c' or ee_key == 'ag2f90_d' or ee_key == 'ag2f90_c_soft'}">
+                    <param name="${side}_dyn_param">0.9464750422461978, -8.366166030270293, -9.50810456883501, 71.59365292895114, 0.02313627009490121, 0.0, 0.0, 0.017136701127687514, 0.0, 0.008640226166892327</param>
+                </xacro:if>
+                <xacro:if value="${ee_key == 'ag2f120s' or ee_key == 'ag2f120s_d'}">
+                    <!-- TODO: replace with measured values; temporarily reuse ag2f90 series -->
                     <param name="${side}_dyn_param">0.9464750422461978, -8.366166030270293, -9.50810456883501, 71.59365292895114, 0.02313627009490121, 0.0, 0.0, 0.017136701127687514, 0.0, 0.008640226166892327</param>
                 </xacro:if>
@@ -129,9 +137,9 @@
                     </joint>
                 </xacro:if>
-                <xacro:if value="${gripper_type == 'ctag2f120s'}">
-                    <xacro:AG2F120S name="${side}" kinematic_only="true"/>
+                <xacro:if value="${gripper_type == 'ag2f120s' or gripper_type == 'ag2f120s_d'}">
+                    <xacro:AG2F120S name="${side}" use_flange="true" kinematic_only="true"/>
                     <joint name="${side}_gripper_fix" type="fixed">
                         <parent link="${side}_tcp"/>
-                        <child link="${side}_gripper_base"/>
+                        <child link="${side}_flange"/>
                         <origin xyz="0 0 0.0045"/>
                     </joint>
@@ -168,9 +176,9 @@
                 </joint>
             </xacro:if>
-            <xacro:if value="${gripper_type == 'ctag2f120s'}">
-                <xacro:AG2F120S name="${side}"/>
+            <xacro:if value="${gripper_type == 'ag2f120s' or gripper_type == 'ag2f120s_d'}">
+                <xacro:AG2F120S name="${side}" use_flange="true"/>
                 <joint name="${side}_gripper_fix" type="fixed">
                     <parent link="${side}_tcp"/>
-                    <child link="${side}_gripper_base"/>
+                    <child link="${side}_flange"/>
                     <origin xyz="0 0 0.0045"/>
                 </joint>

File: m6_ccs_description/xacro/robot.xacro (robot description, xacro)
@@ -49,6 +49,9 @@
 		<xacro:property name="selected_gripper_type" value="ag2f90_d"/>
 	</xacro:if>
-	<xacro:if value="${type_arg == 'ctag2f120s'}">
-		<xacro:property name="selected_gripper_type" value="ctag2f120s"/>
+	<xacro:if value="${type_arg == 'ag2f120s'}">
+		<xacro:property name="selected_gripper_type" value="ag2f120s"/>
+	</xacro:if>
+	<xacro:if value="${type_arg == 'ag2f120s_d'}">
+		<xacro:property name="selected_gripper_type" value="ag2f120s_d"/>
 	</xacro:if>
 	<xacro:if value="${type_arg == 'rg75'}">

File: m6_ccs_description/xacro/ros2_control/robot.xacro (robot description, xacro)
@@ -82,8 +82,8 @@
 				<xacro:ag2f90c_interfaces name="right"/>
 			</xacro:if>
-			<xacro:if value="${left_gripper_type == 'ctag2f120s'}">
+			<xacro:if value="${left_gripper_type == 'ag2f120s' or left_gripper_type == 'ag2f120s_d'}">
 				<xacro:ag2f120s_interfaces name="left"/>
 			</xacro:if>
-			<xacro:if value="${right_gripper_type == 'ctag2f120s'}">
+			<xacro:if value="${right_gripper_type == 'ag2f120s' or right_gripper_type == 'ag2f120s_d'}">
 				<xacro:ag2f120s_interfaces name="right"/>
 			</xacro:if>
@@ -114,5 +114,5 @@
 					<xacro:ag2f90c_interfaces name=""/>
 				</xacro:if>
-				<xacro:if value="${selected_gripper_type == 'ctag2f120s'}">
+				<xacro:if value="${selected_gripper_type == 'ag2f120s' or selected_gripper_type == 'ag2f120s_d'}">
 					<xacro:include filename="$(find changingtek_description)/xacro/ros2_control/AG2F120S.xacro"/>
 					<xacro:ag2f120s_interfaces name=""/>
