Commit message: Feature/add 120s gripper (#7)
* 增加120s夹爪

* add 120s

* 更新120s负载

* simplified xacro

---------

Co-authored-by: hja <2486401522@qq.com>

File: m6_ccs_description/xacro/eef_type_resolver.xacro (robot description, xacro)
@@ -23,4 +23,10 @@
             <xacro:property name="${side}_gripper_pad" value="soft" scope="parent"/>
         </xacro:if>
+        <xacro:if value="${type_key == 'ag2f120s'}">
+            <xacro:property name="${side}_gripper_type" value="ag2f120s" scope="parent"/>
+        </xacro:if>
+        <xacro:if value="${type_key == 'ag2f120s_d'}">
+            <xacro:property name="${side}_gripper_type" value="ag2f120s_d" scope="parent"/>
+        </xacro:if>
         <xacro:if value="${type_key == 'linkerhand_o6'}">
             <xacro:property name="${side}_hand_type" value="linkerhand_o6" scope="parent"/>

File: m6_ccs_description/xacro/eefs.xacro (robot description, xacro)
@@ -5,4 +5,5 @@
     <xacro:include filename="$(find jodell_description)/xacro/RG75-300.xacro"/>
     <xacro:include filename="$(find changingtek_description)/xacro/AG2F90-C.xacro"/>
+    <xacro:include filename="$(find changingtek_description)/xacro/AG2F120S.xacro"/>
     <!-- Per-side default load (dyn_param) for MarvinHardware; 10 values: m, mx, my, mz, ixx, ixy, ixz, iyy, iyz, izz.
          Override via launch left_dyn_param/right_dyn_param (robot.local.yaml).
@@ -24,4 +25,8 @@
                     <param name="${side}_dyn_param">0.9464750422461978, -8.366166030270293, -9.50810456883501, 71.59365292895114, 0.02313627009490121, 0.0, 0.0, 0.017136701127687514, 0.0, 0.008640226166892327</param>
                 </xacro:if>
+                <xacro:if value="${ee_key == 'ag2f120s' or ee_key == 'ag2f120s_d'}">
+                    <!-- TODO: replace with measured values; temporarily reuse ag2f90 series -->
+                    <param name="${side}_dyn_param">1.3944348661120496, -7.913087934362548, 10.50004773179898, 72.44110460800299, 0.014948849408945898, 0.0, 0.0, 0.005470384569170036, 0.0, 0.002567996881581655</param>
+                </xacro:if>
                 <xacro:if value="${ee_key == 'linkerhand_o6'}">
                     <param name="${side}_dyn_param">0.6,0,0,70.0,0,0,0,0,0,0</param>
@@ -40,4 +45,8 @@
                 <xacro:if value="${ee_key == 'ag2f90_c' or ee_key == 'ag2f90_d' or ee_key == 'ag2f90_c_soft'}">
                     <param name="${side}_dyn_param">0.9464750422461978, -8.366166030270293, -9.50810456883501, 71.59365292895114, 0.02313627009490121, 0.0, 0.0, 0.017136701127687514, 0.0, 0.008640226166892327</param>
+                </xacro:if>
+                <xacro:if value="${ee_key == 'ag2f120s' or ee_key == 'ag2f120s_d'}">
+                    <!-- TODO: replace with measured values; temporarily reuse ag2f90 series -->
+                    <param name="${side}_dyn_param">1.4038028109970075, 3.8873998644204817, -10.865529763155825, 73.06884012186562, 0.001, 0.0, 0.0, 0.001, 0.0, 0.0057238484709952525</param>
                 </xacro:if>
                 <xacro:if value="${ee_key == 'linkerhand_o6'}">
@@ -122,4 +131,12 @@
                 <xacro:if value="${gripper_type == 'ag2f90_c' or gripper_type == 'ag2f90_d'}">
                     <xacro:AG2F90-C name="${side}" use_flange="true" pad="${gripper_pad}" kinematic_only="true"/>
+                    <joint name="${side}_gripper_fix" type="fixed">
+                        <parent link="${side}_tcp"/>
+                        <child link="${side}_flange"/>
+                        <origin xyz="0 0 0.0045"/>
+                    </joint>
+                </xacro:if>
+                <xacro:if value="${gripper_type == 'ag2f120s' or gripper_type == 'ag2f120s_d'}">
+                    <xacro:AG2F120S name="${side}" use_flange="true" kinematic_only="true"/>
                     <joint name="${side}_gripper_fix" type="fixed">
                         <parent link="${side}_tcp"/>
@@ -153,4 +170,12 @@
             <xacro:if value="${gripper_type == 'ag2f90_c' or gripper_type == 'ag2f90_d'}">
                 <xacro:AG2F90-C name="${side}" use_flange="true" pad="${gripper_pad}"/>
+                <joint name="${side}_gripper_fix" type="fixed">
+                    <parent link="${side}_tcp"/>
+                    <child link="${side}_flange"/>
+                    <origin xyz="0 0 0.0045"/>
+                </joint>
+            </xacro:if>
+            <xacro:if value="${gripper_type == 'ag2f120s' or gripper_type == 'ag2f120s_d'}">
+                <xacro:AG2F120S name="${side}" use_flange="true"/>
                 <joint name="${side}_gripper_fix" type="fixed">
                     <parent link="${side}_tcp"/>

File: m6_ccs_description/xacro/robot.xacro (robot description, xacro)
@@ -5,10 +5,10 @@
 	<xacro:arg name="variant" default=""/>
 	<xacro:arg name="type" default="dual"/>
-	<xacro:arg name="scene" default=""/>
 	<xacro:arg name="left_type" default=""/>
 	<xacro:arg name="right_type" default=""/>
 	<xacro:arg name="eef_fixed_joints" default="false"/>
-	<!-- 从 type 参数解析出 arm_config、gripper_type 和 scene -->
+	<!-- 从 type 参数解析 arm_config / 对称末端 -->
 	<xacro:property name="type_arg" value="$(arg type)"/>
+	<xacro:property name="variant_arg" value="$(arg variant)"/>
 	<xacro:property name="left_type_arg" value="$(arg left_type)"/>
 	<xacro:property name="right_type_arg" value="$(arg right_type)"/>
@@ -20,5 +20,4 @@
 	<xacro:property name="selected_hand_type" value="none"/>
 	<xacro:property name="selected_gripper_pad" value="default"/>
-	<xacro:property name="selected_scene" value=""/>
 	<!-- 从 type 解析 arm_config 和 gripper_type -->
 	<!-- 单臂配置 -->
@@ -28,9 +27,4 @@
 	<xacro:if value="${type_arg == 'right'}">
 		<xacro:property name="selected_arm_config" value="right"/>
-	</xacro:if>
-	<xacro:if value="${type_arg == 'usb-90c'}">
-		<xacro:property name="selected_arm_config" value="left"/>
-		<xacro:property name="selected_gripper_type" value="ag2f90_c"/>
-		<xacro:property name="selected_scene" value="usb-90c"/>
 	</xacro:if>
 	<!-- 双臂配置 -->
@@ -48,4 +42,10 @@
 	<xacro:if value="${type_arg == 'ag2f90_d'}">
 		<xacro:property name="selected_gripper_type" value="ag2f90_d"/>
+	</xacro:if>
+	<xacro:if value="${type_arg == 'ag2f120s'}">
+		<xacro:property name="selected_gripper_type" value="ag2f120s"/>
+	</xacro:if>
+	<xacro:if value="${type_arg == 'ag2f120s_d'}">
+		<xacro:property name="selected_gripper_type" value="ag2f120s_d"/>
 	</xacro:if>
 	<xacro:if value="${type_arg == 'rg75'}">
@@ -65,17 +65,8 @@
 		<xacro:property name="selected_hand_type" value="linkerhand_o7"/>
 	</xacro:if>
-	<!-- 适用纯双臂演示场景的配置 -->
-	<xacro:if value="${type_arg == 'desktop'}">
-		<xacro:property name="selected_scene" value="desktop"/>
-	</xacro:if>
-	<xacro:if value="${type_arg == 'desktop_90c'}">
-		<xacro:property name="selected_scene" value="desktop"/>
-		<xacro:property name="selected_gripper_type" value="ag2f90_c"/>
-		<xacro:property name="selected_gripper_pad" value="soft"/>
-	</xacro:if>
 	<xacro:include filename="$(find m6_ccs_description)/xacro/arm.xacro"/>
 	<xacro:include filename="$(find m6_ccs_description)/xacro/arm_mount.xacro"/>
-	<!-- 单左臂（不包括 usb-90c 场景） -->
-	<xacro:if value="${selected_arm_config == 'left' and selected_scene != 'usb-90c'}">
+	<!-- 单左臂 -->
+	<xacro:if value="${selected_arm_config == 'left'}">
 		<xacro:M6_CCS skin="$(arg skin)" variant="$(arg variant)"/>
 		<xacro:if value="${selected_gripper_type == 'rg75'}">
@@ -94,6 +85,5 @@
 	<!-- 双臂配置 -->
 	<xacro:if value="${selected_arm_config == 'dual'}">
-		<!-- Base link 和 arm_base 根据 scene 设置 -->
-		<xacro:if value="${selected_scene == 'desktop'}">
+		<xacro:if value="${variant_arg == 'desktop'}">
 			<link name="base_link"/>
 			<link name="arm_base">
@@ -115,19 +105,6 @@
 			</joint>
 			<xacro:DualArmMount parent="arm_base" left_xyz="0 0.12 0.701" right_xyz="0 -0.12 0.701"/>
-			<xacro:if value="${selected_gripper_type == 'none'}">
-				<link name="right_eef"/>
-				<joint name="right_eef_joint" type="fixed">
-					<parent link="right_tcp"/>
-					<child link="right_eef"/>
-				</joint>
-				<link name="left_eef"/>
-				<joint name="left_eef_joint" type="fixed">
-					<parent link="left_tcp"/>
-					<child link="left_eef"/>
-				</joint>
-			</xacro:if>
 		</xacro:if>
-		<xacro:unless value="${selected_scene == 'desktop'}">
-			<!-- 非 Desktop 场景：base_link 为空，有 arm_base -->
+		<xacro:unless value="${variant_arg == 'desktop'}">
 			<link name="base_link"/>
 			<link name="arm_base">
@@ -145,5 +122,4 @@
 			<xacro:DualArmMount parent="arm_base"/>
 		</xacro:unless>
-		<!-- 双臂和末端执行器（两种场景共用） -->
 		<xacro:M6_CCS name="left" skin="$(arg skin)" variant="$(arg variant)"/>
 		<xacro:M6_CCS name="right" direction="-1" skin="$(arg skin)" variant="$(arg variant)"/>
@@ -161,34 +137,3 @@
 			right_gripper_pad="${right_gripper_pad}"/>
 	</xacro:if>
-	<!-- USB-90C 配置 -->
-	<xacro:if value="${selected_arm_config == 'left' and selected_scene == 'usb-90c'}">
-		<link name="base_link"/>
-		<!-- Left Arm -->
-		<joint name="base_joint" type="fixed">
-			<parent link="base_link"/>
-			<child link="base"/>
-		</joint>
-		<link name="base">
-			<visual>
-				<geometry>
-					<mesh filename="file://$(find m6_ccs_description)/meshes/desktop_base.glb"/>
-				</geometry>
-			</visual>
-			<collision>
-				<origin xyz="0 0 0.324331"/>
-				<geometry>
-					<box size="0.10045 0.100398 0.648662"/>
-				</geometry>
-			</collision>
-		</link>
-		<xacro:LeftArmMount parent="base"/>
-		<xacro:M6_CCS name="left" skin="$(arg skin)" variant="$(arg variant)"/>
-		<xacro:include filename="$(find changingtek_description)/xacro/AG2F90-C.xacro"/>
-		<xacro:AG2F90-C name="" use_flange="true"/>
-		<joint name="gripper_fix" type="fixed">
-			<parent link="left_link7"/>
-			<child link="flange"/>
-			<origin xyz="0 -0.0995 0" rpy=" ${PI/2} 0 0"/>
-		</joint>
-	</xacro:if>
 </robot>

File: m6_ccs_description/xacro/ros2_control/robot.xacro (robot description, xacro)
@@ -2,7 +2,7 @@
 <robot xmlns:xacro="http://www.ros.org/wiki/xacro" name="AR5">
 	<xacro:arg name="ros2_control_hardware_type" default="mock_components"/>
-	<xacro:arg name="ctrl_mode" default="position"/>
+	<xacro:arg name="arm_ctrl_mode" default="position"/>
+	<xacro:arg name="device_ip" default=""/>
 	<xacro:arg name="type" default="dual"/>
-	<!-- Non-desktop only: from robot.local.yaml via launch (robot_profile) -->
 	<xacro:arg name="left_dyn_param" default=""/>
 	<xacro:arg name="right_dyn_param" default=""/>
@@ -16,6 +16,7 @@
 		<origin/>
 	</joint>
-	<!-- Include robot.xacro，它会解析 type 并设置 selected_arm_config 和 selected_gripper_type -->
+	<!-- Include robot.xacro（解析 type / selected_arm_config） -->
 	<xacro:include filename="$(find m6_ccs_description)/xacro/robot.xacro"/>
+	<xacro:include filename="$(find m6_ccs_description)/xacro/eefs.xacro"/>
 	<xacro:include filename="$(find m6_ccs_description)/xacro/ros2_control/interfaces.xacro"/>
 	<ros2_control name="M6_CCS_System" type="system">
@@ -41,22 +42,14 @@
 				<param name="max_joint_speed">$(arg max_joint_speed)</param>
 				<param name="max_joint_acceleration">$(arg max_joint_acceleration)</param>
-				<xacro:if value="${selected_scene == 'desktop'}">
-					<param name="device_ip">192.168.10.190</param>
-					<param name="ctrl_mode">JOINT_IMPEDANCE</param>
-					<param name="left_dyn_param">1.2874,-10.145,30,114.65,0,0,0,0,0,0</param>
-					<param name="right_dyn_param">1.2874,-30.145,-10,147.85,0,0,0,0,0,0</param>
+				<param name="ctrl_mode">$(arg arm_ctrl_mode)</param>
+				<xacro:if value="${'$(arg device_ip)' != ''}">
+					<param name="device_ip">$(arg device_ip)</param>
 				</xacro:if>
-				<xacro:if value="${selected_scene != 'desktop'}">
-					<xacro:ee_dyn_param side="left"
-						ee_key="${left_hand_type if left_hand_type != '' else left_gripper_type}"
-						arg_val="$(arg left_dyn_param)"/>
-					<xacro:ee_dyn_param side="right"
-						ee_key="${right_hand_type if right_hand_type != '' else right_gripper_type}"
-						arg_val="$(arg right_dyn_param)"/>
-				</xacro:if>
-				<xacro:if value="${selected_scene == 'usb-90c'}">
-					<param name="device_ip">192.168.10.190</param>
-					<param name="ctrl_mode">CART_IMPEDANCE</param>
-				</xacro:if>
+				<xacro:ee_dyn_param side="left"
+					ee_key="${left_hand_type if left_hand_type != '' else left_gripper_type}"
+					arg_val="$(arg left_dyn_param)"/>
+				<xacro:ee_dyn_param side="right"
+					ee_key="${right_hand_type if right_hand_type != '' else right_gripper_type}"
+					arg_val="$(arg right_dyn_param)"/>
 			</xacro:if>
 		</hardware>
@@ -67,4 +60,5 @@
 			<xacro:include filename="$(find jodell_description)/xacro/ros2_control/RG75-300.xacro"/>
 			<xacro:include filename="$(find changingtek_description)/xacro/ros2_control/AG2F90-C.xacro"/>
+			<xacro:include filename="$(find changingtek_description)/xacro/ros2_control/AG2F120S.xacro"/>
 			<xacro:include filename="$(find linkerhand_description)/xacro/ros2_control/o6.xacro"/>
 			<xacro:include filename="$(find linkerhand_description)/xacro/ros2_control/o7.xacro"/>
@@ -80,4 +74,10 @@
 			<xacro:if value="${right_gripper_type == 'ag2f90_c' or right_gripper_type == 'ag2f90_d'}">
 				<xacro:ag2f90c_interfaces name="right"/>
+			</xacro:if>
+			<xacro:if value="${left_gripper_type == 'ag2f120s' or left_gripper_type == 'ag2f120s_d'}">
+				<xacro:ag2f120s_interfaces name="left"/>
+			</xacro:if>
+			<xacro:if value="${right_gripper_type == 'ag2f120s' or right_gripper_type == 'ag2f120s_d'}">
+				<xacro:ag2f120s_interfaces name="right"/>
 			</xacro:if>
 			<xacro:if value="${left_hand_type == 'linkerhand_o6' or left_hand_type == 'linkerhand_l6'}">
@@ -97,13 +97,12 @@
 		<xacro:unless value="${selected_arm_config == 'dual'}">
 			<xacro:if value="${selected_arm_config == 'left'}">
-				<xacro:if value="${selected_scene == 'usb-90c'}">
-					<xacro:m6_interfaces name="left"/>
-				</xacro:if>
-				<xacro:unless value="${selected_scene == 'usb-90c'}">
-					<xacro:m6_interfaces name=""/>
-				</xacro:unless>
+				<xacro:m6_interfaces name=""/>
 				<xacro:if value="${selected_gripper_type == 'ag2f90_c' or selected_gripper_type == 'ag2f90_d'}">
 					<xacro:include filename="$(find changingtek_description)/xacro/ros2_control/AG2F90-C.xacro"/>
 					<xacro:ag2f90c_interfaces name=""/>
+				</xacro:if>
+				<xacro:if value="${selected_gripper_type == 'ag2f120s' or selected_gripper_type == 'ag2f120s_d'}">
+					<xacro:include filename="$(find changingtek_description)/xacro/ros2_control/AG2F120S.xacro"/>
+					<xacro:ag2f120s_interfaces name=""/>
 				</xacro:if>
 				<xacro:if value="${selected_gripper_type == 'rg75'}">

Commit message: add erg32 support

File: m6_ccs_description/xacro/eef_type_resolver.xacro (robot description, xacro)
@@ -8,4 +8,7 @@
         <xacro:if value="${type_key == 'rg75'}">
             <xacro:property name="${side}_gripper_type" value="rg75" scope="parent"/>
+        </xacro:if>
+        <xacro:if value="${type_key == 'erg32'}">
+            <xacro:property name="${side}_hand_type" value="erg32" scope="parent"/>
         </xacro:if>
         <xacro:if value="${type_key == 'ag2f90' or type_key == 'ag2f90_d'}">

File: m6_ccs_description/xacro/eefs.xacro (robot description, xacro)
@@ -4,4 +4,5 @@
     <!-- Eager includes so collider is configured once at file scope. -->
     <xacro:include filename="$(find jodell_description)/xacro/RG75-300.xacro"/>
+    <xacro:include filename="$(find jodell_description)/xacro/ERG32.xacro"/>
     <xacro:include filename="$(find changingtek_description)/xacro/AG2F90-C.xacro"/>
     <xacro:include filename="$(find changingtek_description)/xacro/AG2F120S.xacro"/>
@@ -27,4 +28,8 @@
                     <param name="${side}_dyn_param">1.6200799541791235, 1.4285009257202586, -0.5789585762443014, 104.39051192831192, 0.004873874899366342, 0.0, 0.0, 0.001, 0.0, 0.0019355638096347936</param>
                 </xacro:if>
+                <xacro:if value="${ee_key == 'erg32'}">
+                    <!-- TODO: replace with measured ERG32 values -->
+                    <param name="${side}_dyn_param">1.6200799541791235, 1.4285009257202586, -0.5789585762443014, 104.39051192831192, 0.004873874899366342, 0.0, 0.0, 0.001, 0.0, 0.0019355638096347936</param>
+                </xacro:if>
                 <xacro:if value="${ee_key == 'ag2f90_c' or ee_key == 'ag2f90_d' or ee_key == 'ag2f90_c_soft'}">
                     <param name="${side}_dyn_param">0.9464750422461978, -8.366166030270293, -9.50810456883501, 71.59365292895114, 0.02313627009490121, 0.0, 0.0, 0.017136701127687514, 0.0, 0.008640226166892327</param>
@@ -46,4 +51,8 @@
             <xacro:if value="${side == 'right'}">
                 <xacro:if value="${ee_key == 'rg75'}">
+                    <param name="${side}_dyn_param">1.6200799541791235, 1.4285009257202586, -0.5789585762443014, 104.39051192831192, 0.004873874899366342, 0.0, 0.0, 0.001, 0.0, 0.0019355638096347936</param>
+                </xacro:if>
+                <xacro:if value="${ee_key == 'erg32'}">
+                    <!-- TODO: replace with measured ERG32 values -->
                     <param name="${side}_dyn_param">1.6200799541791235, 1.4285009257202586, -0.5789585762443014, 104.39051192831192, 0.004873874899366342, 0.0, 0.0, 0.001, 0.0, 0.0019355638096347936</param>
                 </xacro:if>
@@ -199,4 +208,22 @@
         </xacro:if>
     </xacro:macro>
+    <xacro:macro name="SideEndEffectorERG32" params="side eef_fixed_joints:=false">
+        <xacro:ERG32 name="${side}_hand" use_flange="true"
+                     kinematic_only="${eef_fixed_joints}"
+                     eef_flip="${side == 'right'}"/>
+        <joint name="${side}_hand_base_joint" type="fixed">
+            <parent link="${side}_tcp"/>
+            <child link="${side}_hand_flange"/>
+            <xacro:if value="${side == 'right'}">
+                <origin rpy="0 0 ${PI}"/>
+            </xacro:if>
+        </joint>
+        <!-- ERG32 built-in ${side}_hand_eef; alias ${side}_eef for OCS2 / task.info -->
+        <link name="${side}_eef"/>
+        <joint name="${side}_eef_joint" type="fixed">
+            <parent link="${side}_hand_eef"/>
+            <child link="${side}_eef"/>
+        </joint>
+    </xacro:macro>
     <xacro:macro name="SideEndEffector" params="side hand_type gripper_type gripper_pad eef_fixed_joints:=false">
         <!-- OCS2 planning URDF: no actuated EEF DOF (avoids per-tool removeJoints in .info) -->
@@ -205,5 +232,8 @@
                 <xacro:SideEndEffectorLinkerHand side="${side}" hand_type="${hand_type}" eef_fixed_joints="true"/>
             </xacro:if>
-            <xacro:unless value="${hand_type == 'linkerhand_o6' or hand_type == 'linkerhand_o7' or hand_type == 'linkerhand_l6' or hand_type == 'freedom_v1' or hand_type == 'freedom_v2' or hand_type == 'inspire_e2' or hand_type == 'inspire_f2' or hand_type == 'xhand1'}">
+            <xacro:if value="${hand_type == 'erg32'}">
+                <xacro:SideEndEffectorERG32 side="${side}" eef_fixed_joints="true"/>
+            </xacro:if>
+            <xacro:unless value="${hand_type == 'linkerhand_o6' or hand_type == 'linkerhand_o7' or hand_type == 'linkerhand_l6' or hand_type == 'freedom_v1' or hand_type == 'freedom_v2' or hand_type == 'inspire_e2' or hand_type == 'inspire_f2' or hand_type == 'xhand1' or hand_type == 'erg32'}">
                 <xacro:if value="${gripper_type == 'ag2f90_c' or gripper_type == 'ag2f90_d'}">
                     <xacro:AG2F90-C name="${side}" use_flange="true" pad="${gripper_pad}" kinematic_only="true"/>
@@ -264,4 +294,7 @@
                     <child link="${side}_flange"/>
                 </joint>
+            </xacro:if>
+            <xacro:if value="${hand_type == 'erg32'}">
+                <xacro:SideEndEffectorERG32 side="${side}" eef_fixed_joints="false"/>
             </xacro:if>
             <xacro:SideEndEffectorLinkerHand side="${side}" hand_type="${hand_type}" eef_fixed_joints="false"/>

File: m6_ccs_description/xacro/ros2_control/end_effector_interfaces.xacro (robot description, xacro)
@@ -3,4 +3,5 @@
 	<xacro:include filename="$(find m6_ccs_description)/xacro/ros2_control/interfaces.xacro"/>
 	<xacro:include filename="$(find jodell_description)/xacro/ros2_control/RG75-300.xacro"/>
+	<xacro:include filename="$(find jodell_description)/xacro/ros2_control/ERG32.xacro"/>
 	<xacro:include filename="$(find changingtek_description)/xacro/ros2_control/AG2F90-C.xacro"/>
 	<xacro:include filename="$(find changingtek_description)/xacro/ros2_control/AG2F120S.xacro"/>
@@ -41,4 +42,7 @@
 		<xacro:if value="${hand_type == 'xhand1'}">
 			<xacro:xhand1_interfaces name="${side}_hand"/>
+		</xacro:if>
+		<xacro:if value="${hand_type == 'erg32'}">
+			<xacro:erg32_interfaces name="${side}_hand"/>
 		</xacro:if>
 	</xacro:macro>
