Commit message: update m6 ccs readme

File: m6_ccs_description/xacro/eef_type_resolver.xacro (robot description, xacro)
@@ -8,8 +8,4 @@
         <xacro:if value="${type_key == 'rg75'}">
             <xacro:property name="${side}_gripper_type" value="rg75" scope="parent"/>
-        </xacro:if>
-        <xacro:if value="${type_key == 'rg75_heavy'}">
-            <xacro:property name="${side}_gripper_type" value="rg75" scope="parent"/>
-            <xacro:property name="${side}_gripper_pad" value="heavy_carry" scope="parent"/>
         </xacro:if>
         <xacro:if value="${type_key == 'ag2f90' or type_key == 'ag2f90_d'}">
@@ -47,4 +43,7 @@
             <xacro:property name="${side}_hand_type" value="inspire_e2" scope="parent"/>
         </xacro:if>
+        <xacro:if value="${type_key == 'inspire_f2'}">
+            <xacro:property name="${side}_hand_type" value="inspire_f2" scope="parent"/>
+        </xacro:if>
         <xacro:if value="${type_key == 'xhand1'}">
             <xacro:property name="${side}_hand_type" value="xhand1" scope="parent"/>

File: m6_ccs_description/xacro/eefs.xacro (robot description, xacro)
@@ -9,4 +9,5 @@
     <xacro:include filename="$(find freedom_description)/xacro/freedomv2.xacro"/>
     <xacro:include filename="$(find inspire_description)/xacro/hands/RH56E2.xacro"/>
+    <xacro:include filename="$(find inspire_description)/xacro/hands/RH56F2.xacro"/>
     <xacro:include filename="$(find xhand1_description)/xacro/xhand1.xacro"/>
     <!-- Per-side default load (dyn_param) for MarvinHardware; 10 values: m, mx, my, mz, ixx, ixy, ixz, iyy, iyz, izz.
@@ -156,4 +157,17 @@
             </joint>
         </xacro:if>
+        <xacro:if value="${hand_type == 'inspire_f2'}">
+            <xacro:InspireHandRH56F2 name="${side}_hand" direction="${1 if side == 'left' else -1}" use_flange="true" fixed_joints="${eef_fixed_joints}"/>
+            <joint name="${side}_hand_base_joint" type="fixed">
+                <xacro:if value="${side == 'left'}">
+                    <origin xyz="0 0 0.0045" rpy="0 0 ${PI}"/>
+                </xacro:if>
+                <xacro:if value="${side == 'right'}">
+                    <origin xyz="0 0 0.0045" rpy="0 0 ${-PI}"/>
+                </xacro:if>
+                <parent link="${side}_tcp"/>
+                <child link="${side}_hand_flange"/>
+            </joint>
+        </xacro:if>
         <xacro:if value="${hand_type == 'xhand1'}">
             <xacro:XHand1 name="${side}_hand" direction="${1 if side == 'left' else -1}" fixed_joints="${eef_fixed_joints}"/>
@@ -177,5 +191,5 @@
             </joint>
         </xacro:if>
-        <xacro:if value="${hand_type == 'linkerhand_o6' or hand_type == 'linkerhand_l6' or hand_type == 'linkerhand_o7' or hand_type == 'freedom_v1' or hand_type == 'freedom_v2' or hand_type == 'inspire_e2'}">
+        <xacro:if value="${hand_type == 'linkerhand_o6' or hand_type == 'linkerhand_l6' or hand_type == 'linkerhand_o7' or hand_type == 'freedom_v1' or hand_type == 'freedom_v2' or hand_type == 'inspire_e2' or hand_type == 'inspire_f2'}">
             <link name="${side}_eef"/>
             <joint name="${side}_eef_joint" type="fixed">
@@ -188,8 +202,8 @@
         <!-- OCS2 planning URDF: no actuated EEF DOF (avoids per-tool removeJoints in .info) -->
         <xacro:if value="${eef_fixed_joints}">
-            <xacro:if value="${hand_type == 'linkerhand_o6' or hand_type == 'linkerhand_o7' or hand_type == 'linkerhand_l6' or hand_type == 'freedom_v1' or hand_type == 'freedom_v2' or hand_type == 'inspire_e2' or hand_type == 'xhand1'}">
+            <xacro:if value="${hand_type == 'linkerhand_o6' or hand_type == 'linkerhand_o7' or hand_type == 'linkerhand_l6' or hand_type == 'freedom_v1' or hand_type == 'freedom_v2' or hand_type == 'inspire_e2' or hand_type == 'inspire_f2' or hand_type == 'xhand1'}">
                 <xacro:SideEndEffectorLinkerHand side="${side}" hand_type="${hand_type}" eef_fixed_joints="true"/>
             </xacro:if>
-            <xacro:unless value="${hand_type == 'linkerhand_o6' or hand_type == 'linkerhand_o7' or hand_type == 'linkerhand_l6' or hand_type == 'freedom_v1' or hand_type == 'freedom_v2' or hand_type == 'inspire_e2' or hand_type == 'xhand1'}">
+            <xacro:unless value="${hand_type == 'linkerhand_o6' or hand_type == 'linkerhand_o7' or hand_type == 'linkerhand_l6' or hand_type == 'freedom_v1' or hand_type == 'freedom_v2' or hand_type == 'inspire_e2' or hand_type == 'inspire_f2' or hand_type == 'xhand1'}">
                 <xacro:if value="${gripper_type == 'ag2f90_c' or gripper_type == 'ag2f90_d'}">
                     <xacro:AG2F90-C name="${side}" use_flange="true" pad="${gripper_pad}" kinematic_only="true"/>
@@ -213,7 +227,4 @@
                         <parent link="${side}_tcp"/>
                         <child link="${side}_flange"/>
-                        <xacro:if value="${gripper_pad == 'heavy_carry'}">
-                            <origin rpy="0 0 ${PI/2}"/>
-                        </xacro:if>
                     </joint>
                 </xacro:if>
@@ -252,7 +263,4 @@
                     <parent link="${side}_tcp"/>
                     <child link="${side}_flange"/>
-                    <xacro:if value="${gripper_pad == 'heavy_carry'}">
-                        <origin rpy="0 0 ${PI/2}"/>
-                    </xacro:if>
                 </joint>
             </xacro:if>

File: m6_ccs_description/xacro/robot.xacro (robot description, xacro)
@@ -50,8 +50,4 @@
 	<xacro:if value="${type_arg == 'rg75'}">
 		<xacro:property name="selected_gripper_type" value="rg75"/>
-	</xacro:if>
-	<xacro:if value="${type_arg == 'rg75_heavy'}">
-		<xacro:property name="selected_gripper_type" value="rg75"/>
-		<xacro:property name="selected_gripper_pad" value="heavy_carry"/>
 	</xacro:if>
 	<xacro:include filename="$(find m6_ccs_description)/xacro/arm.xacro"/>

File: m6_ccs_description/xacro/ros2_control/robot.xacro (robot description, xacro)
@@ -51,4 +51,8 @@
 			<xacro:inspire_rh56e2_interfaces name="${side}_hand"/>
 		</xacro:if>
+		<xacro:if value="${hand_type == 'inspire_f2'}">
+			<xacro:include filename="$(find inspire_description)/xacro/ros2_control/RH56F2.xacro"/>
+			<xacro:inspire_rh56f2_interfaces name="${side}_hand"/>
+		</xacro:if>
 		<xacro:if value="${hand_type == 'xhand1'}">
 			<xacro:xhand1_interfaces name="${side}_hand"/>
@@ -89,5 +93,5 @@
 					<xacro:property name="left_ee_type" value="${left_hand_type if left_hand_type != '' else left_gripper_type}"/>
 					<xacro:property name="right_ee_type" value="${right_hand_type if right_hand_type != '' else right_gripper_type}"/>
-					<xacro:if value="${(left_drive_type == 'marvin' or left_drive_type == 'tianji_can') and left_ee_type != '' and left_ee_type != 'xhand1'}">
+					<xacro:if value="${(left_drive_type == 'marvin' or left_drive_type == 'tianji_can') and left_ee_type != '' and left_ee_type != 'xhand1' and left_ee_type != 'inspire_e2'}">
 						<param name="left_ee_type">${left_ee_type}</param>
 						<xacro:if value="${left_drive_type == 'tianji_can'}">
@@ -95,5 +99,5 @@
 						</xacro:if>
 					</xacro:if>
-					<xacro:if value="${(right_drive_type == 'marvin' or right_drive_type == 'tianji_can') and right_ee_type != '' and right_ee_type != 'xhand1'}">
+					<xacro:if value="${(right_drive_type == 'marvin' or right_drive_type == 'tianji_can') and right_ee_type != '' and right_ee_type != 'xhand1' and right_ee_type != 'inspire_e2'}">
 						<param name="right_ee_type">${right_ee_type}</param>
 						<xacro:if value="${right_drive_type == 'tianji_can'}">
@@ -152,10 +156,10 @@
 				<xacro:ag2f120s_interfaces name="right"/>
 			</xacro:if>
-			<xacro:if value="${(not is_real_hardware) or ((left_drive_type == 'marvin' or left_drive_type == 'tianji_can') and left_hand_type != 'xhand1')}">
+			<xacro:if value="${(not is_real_hardware) or ((left_drive_type == 'marvin' or left_drive_type == 'tianji_can') and left_hand_type != 'xhand1' and left_hand_type != 'inspire_e2')}">
 				<xacro:if value="${left_hand_type != ''}">
 					<xacro:side_hand_interfaces side="left" hand_type="${left_hand_type}"/>
 				</xacro:if>
 			</xacro:if>
-			<xacro:if value="${(not is_real_hardware) or ((right_drive_type == 'marvin' or right_drive_type == 'tianji_can') and right_hand_type != 'xhand1')}">
+			<xacro:if value="${(not is_real_hardware) or ((right_drive_type == 'marvin' or right_drive_type == 'tianji_can') and right_hand_type != 'xhand1' and right_hand_type != 'inspire_e2')}">
 				<xacro:if value="${right_hand_type != ''}">
 					<xacro:side_hand_interfaces side="right" hand_type="${right_hand_type}"/>
@@ -198,4 +202,10 @@
 			<xacro:inspire_rs485_side_system side="right" serial_port="/dev/ttyUSB2"/>
 		</xacro:if>
+		<xacro:if value="${left_drive_type == 'usb' and left_hand_type == 'inspire_f2'}">
+			<xacro:inspire_rs485_side_system side="left" serial_port="/dev/ttyUSB0" hand_type="inspire_f2"/>
+		</xacro:if>
+		<xacro:if value="${right_drive_type == 'usb' and right_hand_type == 'inspire_f2'}">
+			<xacro:inspire_rs485_side_system side="right" serial_port="/dev/ttyUSB2" hand_type="inspire_f2"/>
+		</xacro:if>
 		<xacro:if value="${left_drive_type == 'usb' and left_hand_type == 'freedom_v1'}">
 			<xacro:freedom_rs485_side_system side="left" serial_port="/dev/ttyUSB0"/>
@@ -227,4 +237,10 @@
 		<xacro:if value="${right_drive_type == 'usb_can' and right_hand_type == 'inspire_e2'}">
 			<xacro:inspire_canfd_side_system side="right" can_interface="can1"/>
+		</xacro:if>
+		<xacro:if value="${left_drive_type == 'usb_can' and left_hand_type == 'inspire_f2'}">
+			<xacro:inspire_canfd_side_system side="left" can_interface="can0" hand_type="inspire_f2"/>
+		</xacro:if>
+		<xacro:if value="${right_drive_type == 'usb_can' and right_hand_type == 'inspire_f2'}">
+			<xacro:inspire_canfd_side_system side="right" can_interface="can1" hand_type="inspire_f2"/>
 		</xacro:if>
 	</xacro:if>
