Commit message: Feature/add more hand (#8)
* add diff eef support

* add diff eef support

* add template support

* add diff eef

* add diff eef

* add hand eef

* add freedom and inspire hand configurations and dependencies

* add additional hand configurations and update dependencies for ROS2 control

* merge main后调整

* 规范freedom xacro

* 添加freedomv2

* 更新freedomv2

* 修正marker

* 添加inspireCANFD

* 添加inspireCANFD，修掉频率过低的问题

* 添加inspireCANFD，修掉频率过低的问题

* 添加xhand1 485   hardware 速度 力控参数

* 增加120s夹爪

* add xhand1 support

* 修改home位置以及参数

* add 120s

* 更新120s负载

* simplified xacro

* Add fixed_joints parameter to xhand1 definition in eefs.xacro

* Remove xhand1.yaml configuration file for dual-arm XHAND1 variant

* update m6 ccs readme

* add macro for m6 ccs

---------

Co-authored-by: Huang Zhenbiao <biao876990970@hotmail.com>
Co-authored-by: ldh9299 <929908985@qq.com>
Co-authored-by: xsnan24 <k2571675874@163.com>
Co-authored-by: hja <2486401522@qq.com>

File: m6_ccs_description/xacro/eef_type_resolver.xacro (robot description, xacro)
@@ -8,8 +8,4 @@
         <xacro:if value="${type_key == 'rg75'}">
             <xacro:property name="${side}_gripper_type" value="rg75" scope="parent"/>
-        </xacro:if>
-        <xacro:if value="${type_key == 'rg75_heavy'}">
-            <xacro:property name="${side}_gripper_type" value="rg75" scope="parent"/>
-            <xacro:property name="${side}_gripper_pad" value="heavy_carry" scope="parent"/>
         </xacro:if>
         <xacro:if value="${type_key == 'ag2f90' or type_key == 'ag2f90_d'}">
@@ -38,4 +34,19 @@
             <xacro:property name="${side}_hand_type" value="linkerhand_o7" scope="parent"/>
         </xacro:if>
+        <xacro:if value="${type_key == 'freedom_v1'}">
+            <xacro:property name="${side}_hand_type" value="freedom_v1" scope="parent"/>
+        </xacro:if>
+        <xacro:if value="${type_key == 'freedom_v2'}">
+            <xacro:property name="${side}_hand_type" value="freedom_v2" scope="parent"/>
+        </xacro:if>
+        <xacro:if value="${type_key == 'inspire_e2'}">
+            <xacro:property name="${side}_hand_type" value="inspire_e2" scope="parent"/>
+        </xacro:if>
+        <xacro:if value="${type_key == 'inspire_f2'}">
+            <xacro:property name="${side}_hand_type" value="inspire_f2" scope="parent"/>
+        </xacro:if>
+        <xacro:if value="${type_key == 'xhand1'}">
+            <xacro:property name="${side}_hand_type" value="xhand1" scope="parent"/>
+        </xacro:if>
     </xacro:macro>
 </robot>

File: m6_ccs_description/xacro/eefs.xacro (robot description, xacro)
@@ -6,4 +6,9 @@
     <xacro:include filename="$(find changingtek_description)/xacro/AG2F90-C.xacro"/>
     <xacro:include filename="$(find changingtek_description)/xacro/AG2F120S.xacro"/>
+    <xacro:include filename="$(find freedom_description)/xacro/freedomv1.xacro"/>
+    <xacro:include filename="$(find freedom_description)/xacro/freedomv2.xacro"/>
+    <xacro:include filename="$(find inspire_description)/xacro/hands/RH56E2.xacro"/>
+    <xacro:include filename="$(find inspire_description)/xacro/hands/RH56F2.xacro"/>
+    <xacro:include filename="$(find xhand1_description)/xacro/xhand1.xacro"/>
     <!-- Per-side default load (dyn_param) for MarvinHardware; 10 values: m, mx, my, mz, ixx, ixy, ixz, iyy, iyz, izz.
          Override via launch left_dyn_param/right_dyn_param (robot.local.yaml).
@@ -113,6 +118,78 @@
             </joint>
         </xacro:if>
-        <!-- LinkerHand O6/L6/O7: built-in ${side}_hand_eef; alias ${side}_eef for OCS2 / task.info -->
-        <xacro:if value="${hand_type == 'linkerhand_o6' or hand_type == 'linkerhand_l6' or hand_type == 'linkerhand_o7'}">
+        <xacro:if value="${hand_type == 'freedom_v1'}">
+            <xacro:FreedomHand name="${side}_hand" direction="${1 if side == 'left' else -1}" fixed_joints="${eef_fixed_joints}"/>
+            <joint name="${side}_hand_base_joint" type="fixed">
+                <xacro:if value="${side == 'left'}">
+                    <origin xyz="0 0 0.0045" rpy="${PI/2} 0 ${PI}"/>
+                </xacro:if>
+                <xacro:if value="${side == 'right'}">
+                    <origin xyz="0 0 0.0045" rpy="${PI/2} 0 0"/>
+                </xacro:if>
+                <parent link="${side}_tcp"/>
+                <child link="${side}_hand_hand_base"/>
+            </joint>
+        </xacro:if>
+        <xacro:if value="${hand_type == 'freedom_v2'}">
+            <xacro:FreedomHandV2 name="${side}_hand" direction="${1 if side == 'left' else -1}" fixed_joints="${eef_fixed_joints}" enable_dip_joints="false"/>
+            <joint name="${side}_hand_base_joint" type="fixed">
+                <xacro:if value="${side == 'left'}">
+                    <origin xyz="0 0 0" rpy="0 0 ${PI}"/>
+                </xacro:if>
+                <xacro:if value="${side == 'right'}">
+                    <origin xyz="0 0 0" rpy="0 0 ${PI}"/>
+                </xacro:if>
+                <parent link="${side}_tcp"/>
+                <child link="${side}_hand_hand_base"/>
+            </joint>
+        </xacro:if>
+        <xacro:if value="${hand_type == 'inspire_e2'}">
+            <xacro:InspireHandRH56E2 name="${side}_hand" direction="${1 if side == 'left' else -1}" use_flange="true" fixed_joints="${eef_fixed_joints}"/>
+            <joint name="${side}_hand_base_joint" type="fixed">
+                <xacro:if value="${side == 'left'}">
+                    <origin xyz="0 0 0.0045" rpy="0 0 ${PI}"/>
+                </xacro:if>
+                <xacro:if value="${side == 'right'}">
+                    <origin xyz="0 0 0.0045" rpy="0 0 ${-PI}"/>
+                </xacro:if>
+                <parent link="${side}_tcp"/>
+                <child link="${side}_hand_flange"/>
+            </joint>
+        </xacro:if>
+        <xacro:if value="${hand_type == 'inspire_f2'}">
+            <xacro:InspireHandRH56F2 name="${side}_hand" direction="${1 if side == 'left' else -1}" use_flange="true" fixed_joints="${eef_fixed_joints}"/>
+            <joint name="${side}_hand_base_joint" type="fixed">
+                <xacro:if value="${side == 'left'}">
+                    <origin xyz="0 0 0.0045" rpy="0 0 ${PI}"/>
+                </xacro:if>
+                <xacro:if value="${side == 'right'}">
+                    <origin xyz="0 0 0.0045" rpy="0 0 ${-PI}"/>
+                </xacro:if>
+                <parent link="${side}_tcp"/>
+                <child link="${side}_hand_flange"/>
+            </joint>
+        </xacro:if>
+        <xacro:if value="${hand_type == 'xhand1'}">
+            <xacro:XHand1 name="${side}_hand" direction="${1 if side == 'left' else -1}" fixed_joints="${eef_fixed_joints}"/>
+            <joint name="${side}_hand_base_joint" type="fixed">
+                <xacro:if value="${side == 'left'}">
+                    <origin xyz="0 0 0" rpy="0 0 ${PI}"/>
+                </xacro:if>
+                <xacro:if value="${side == 'right'}">
+                    <origin xyz="0 0 0" rpy="0 0 ${PI}"/>
+                </xacro:if>
+                <parent link="${side}_tcp"/>
+                <child link="${side}_hand_hand_base"/>
+            </joint>
+        </xacro:if>
+        <!-- Hands with built-in ${side}_hand_eef; alias ${side}_eef for OCS2 / task.info -->
+        <xacro:if value="${hand_type == 'xhand1'}">
+            <link name="${side}_eef"/>
+            <joint name="${side}_eef_joint" type="fixed">
+                <parent link="${side}_hand_hand_ee_link"/>
+                <child link="${side}_eef"/>
+            </joint>
+        </xacro:if>
+        <xacro:if value="${hand_type == 'linkerhand_o6' or hand_type == 'linkerhand_l6' or hand_type == 'linkerhand_o7' or hand_type == 'freedom_v1' or hand_type == 'freedom_v2' or hand_type == 'inspire_e2' or hand_type == 'inspire_f2'}">
             <link name="${side}_eef"/>
             <joint name="${side}_eef_joint" type="fixed">
@@ -125,8 +202,8 @@
         <!-- OCS2 planning URDF: no actuated EEF DOF (avoids per-tool removeJoints in .info) -->
         <xacro:if value="${eef_fixed_joints}">
-            <xacro:if value="${hand_type == 'linkerhand_o6' or hand_type == 'linkerhand_o7' or hand_type == 'linkerhand_l6'}">
+            <xacro:if value="${hand_type == 'linkerhand_o6' or hand_type == 'linkerhand_o7' or hand_type == 'linkerhand_l6' or hand_type == 'freedom_v1' or hand_type == 'freedom_v2' or hand_type == 'inspire_e2' or hand_type == 'inspire_f2' or hand_type == 'xhand1'}">
                 <xacro:SideEndEffectorLinkerHand side="${side}" hand_type="${hand_type}" eef_fixed_joints="true"/>
             </xacro:if>
-            <xacro:unless value="${hand_type == 'linkerhand_o6' or hand_type == 'linkerhand_o7' or hand_type == 'linkerhand_l6'}">
+            <xacro:unless value="${hand_type == 'linkerhand_o6' or hand_type == 'linkerhand_o7' or hand_type == 'linkerhand_l6' or hand_type == 'freedom_v1' or hand_type == 'freedom_v2' or hand_type == 'inspire_e2' or hand_type == 'inspire_f2' or hand_type == 'xhand1'}">
                 <xacro:if value="${gripper_type == 'ag2f90_c' or gripper_type == 'ag2f90_d'}">
                     <xacro:AG2F90-C name="${side}" use_flange="true" pad="${gripper_pad}" kinematic_only="true"/>
@@ -150,7 +227,4 @@
                         <parent link="${side}_tcp"/>
                         <child link="${side}_flange"/>
-                        <xacro:if value="${gripper_pad == 'heavy_carry'}">
-                            <origin rpy="0 0 ${PI/2}"/>
-                        </xacro:if>
                     </joint>
                 </xacro:if>
@@ -189,7 +263,4 @@
                     <parent link="${side}_tcp"/>
                     <child link="${side}_flange"/>
-                    <xacro:if value="${gripper_pad == 'heavy_carry'}">
-                        <origin rpy="0 0 ${PI/2}"/>
-                    </xacro:if>
                 </joint>
             </xacro:if>

File: m6_ccs_description/xacro/robot.xacro (robot description, xacro)
@@ -18,5 +18,4 @@
 	<xacro:property name="selected_arm_config" value="dual"/>
 	<xacro:property name="selected_gripper_type" value="none"/>
-	<xacro:property name="selected_hand_type" value="none"/>
 	<xacro:property name="selected_gripper_pad" value="default"/>
 	<!-- 从 type 解析 arm_config 和 gripper_type -->
@@ -51,17 +50,4 @@
 	<xacro:if value="${type_arg == 'rg75'}">
 		<xacro:property name="selected_gripper_type" value="rg75"/>
-	</xacro:if>
-	<xacro:if value="${type_arg == 'rg75_heavy'}">
-		<xacro:property name="selected_gripper_type" value="rg75"/>
-		<xacro:property name="selected_gripper_pad" value="heavy_carry"/>
-	</xacro:if>
-	<xacro:if value="${type_arg == 'linkerhand_o6'}">
-		<xacro:property name="selected_hand_type" value="linkerhand_o6"/>
-	</xacro:if>
-	<xacro:if value="${type_arg == 'linkerhand_l6'}">
-		<xacro:property name="selected_hand_type" value="linkerhand_l6"/>
-	</xacro:if>
-	<xacro:if value="${type_arg == 'linkerhand_o7'}">
-		<xacro:property name="selected_hand_type" value="linkerhand_o7"/>
 	</xacro:if>
 	<xacro:include filename="$(find m6_ccs_description)/xacro/arm.xacro"/>

File: m6_ccs_description/xacro/ros2_control/robot.xacro (robot description, xacro)
@@ -5,9 +5,16 @@
 	<xacro:arg name="device_ip" default=""/>
 	<xacro:arg name="type" default="dual"/>
+	<xacro:arg name="left_ee_drive_type" default=""/>
+	<xacro:arg name="right_ee_drive_type" default=""/>
+	<xacro:property name="is_real_hardware" value="${'$(arg ros2_control_hardware_type)' == 'real' or '$(arg ros2_control_hardware_type)' == 'real_usb'}"/>
+	<xacro:property name="ee_drive_type" value="${'usb' if '$(arg ros2_control_hardware_type)' == 'real_usb' else ('marvin' if '$(arg ros2_control_hardware_type)' == 'real' else '')}"/>
+	<xacro:property name="left_drive_type" value="${'$(arg left_ee_drive_type)' if '$(arg left_ee_drive_type)' != '' else ee_drive_type}"/>
+	<xacro:property name="right_drive_type" value="${'$(arg right_ee_drive_type)' if '$(arg right_ee_drive_type)' != '' else ee_drive_type}"/>
 	<xacro:arg name="left_dyn_param" default=""/>
 	<xacro:arg name="right_dyn_param" default=""/>
-	<!-- Marvin joint limits; override via robot.local.yaml hardware: or hardware_max_joint_*:= launch args -->
 	<xacro:arg name="max_joint_speed" default="50"/>
 	<xacro:arg name="max_joint_acceleration" default="30"/>
+	<xacro:arg name="usb_left_port" default="/dev/ttyUSB0"/>
+	<xacro:arg name="usb_right_port" default="/dev/ttyUSB2"/>
 	<link name="world"/>
 	<joint name="world_fixed" type="fixed">
@@ -16,98 +23,33 @@
 		<origin/>
 	</joint>
-	<!-- Include robot.xacro（解析 type / selected_arm_config） -->
 	<xacro:include filename="$(find m6_ccs_description)/xacro/robot.xacro"/>
-	<xacro:include filename="$(find m6_ccs_description)/xacro/eefs.xacro"/>
-	<xacro:include filename="$(find m6_ccs_description)/xacro/ros2_control/interfaces.xacro"/>
+	<xacro:include filename="$(find robot_common_launch)/xacro/ros2_control/simulation_hardware.xacro"/>
+	<xacro:include filename="$(find m6_ccs_description)/xacro/ros2_control/marvin_hardware.xacro"/>
+	<xacro:include filename="$(find m6_ccs_description)/xacro/ros2_control/end_effector_interfaces.xacro"/>
+	<xacro:include filename="$(find m6_ccs_description)/xacro/ros2_control/external_ee_systems.xacro"/>
+	<xacro:property name="ee_block_mode" value="${'real' if is_real_hardware else 'sim'}"/>
 	<ros2_control name="M6_CCS_System" type="system">
 		<hardware>
-			<xacro:if value="${'$(arg ros2_control_hardware_type)' == 'gz'}">
-				<plugin>gz_ros2_control/GazeboSimSystem</plugin>
-			</xacro:if>
-			<xacro:if value="${'$(arg ros2_control_hardware_type)' == 'mock_components'}">
-				<plugin>mock_components/GenericSystem</plugin>
-			</xacro:if>
-			<xacro:if value="${'$(arg ros2_control_hardware_type)' == 'isaac'}">
-				<plugin>topic_based_ros2_control/TopicBasedSystem</plugin>
-				<param name="joint_commands_topic">/isaac/joint_command</param>
-				<param name="joint_states_topic">/isaac/joint_states</param>
-				<param name="sum_wrapped_joint_states">false</param>
-				<param name="initialize_commands_from_state">true</param>
-			</xacro:if>
-			<xacro:if value="${'$(arg ros2_control_hardware_type)' == 'real'}">
-				<plugin>marvin_ros2_control/MarvinHardware</plugin>
-				<param name="arm_type">${selected_arm_config}</param>
-				<param name="left_ee_type">${left_hand_type if left_hand_type != '' else left_gripper_type}</param>
-				<param name="right_ee_type">${right_hand_type if right_hand_type != '' else right_gripper_type}</param>
-				<param name="max_joint_speed">$(arg max_joint_speed)</param>
-				<param name="max_joint_acceleration">$(arg max_joint_acceleration)</param>
-				<param name="ctrl_mode">$(arg arm_ctrl_mode)</param>
-				<xacro:if value="${'$(arg device_ip)' != ''}">
-					<param name="device_ip">$(arg device_ip)</param>
-				</xacro:if>
-				<xacro:ee_dyn_param side="left"
-					ee_key="${left_hand_type if left_hand_type != '' else left_gripper_type}"
-					arg_val="$(arg left_dyn_param)"/>
-				<xacro:ee_dyn_param side="right"
-					ee_key="${right_hand_type if right_hand_type != '' else right_gripper_type}"
-					arg_val="$(arg right_dyn_param)"/>
+			<xacro:unless value="${is_real_hardware}">
+				<xacro:simulation_hardware_plugin hardware_type="$(arg ros2_control_hardware_type)"/>
+			</xacro:unless>
+			<xacro:if value="${is_real_hardware}">
+				<xacro:marvin_hardware_block
+					arm_type="${selected_arm_config}"
+					arm_ctrl_mode="$(arg arm_ctrl_mode)"
+					max_joint_speed="$(arg max_joint_speed)"
+					max_joint_acceleration="$(arg max_joint_acceleration)"
+					device_ip="$(arg device_ip)"
+					left_dyn_param="$(arg left_dyn_param)"
+					right_dyn_param="$(arg right_dyn_param)"
+					selected_gripper_type="${selected_gripper_type}"/>
 			</xacro:if>
 		</hardware>
-		<!-- 双臂配置：按侧末端（left_type/right_type 或对称 type） -->
 		<xacro:if value="${selected_arm_config == 'dual'}">
-			<xacro:m6_interfaces name="left"/>
-			<xacro:m6_interfaces name="right"/>
-			<xacro:include filename="$(find jodell_description)/xacro/ros2_control/RG75-300.xacro"/>
-			<xacro:include filename="$(find changingtek_description)/xacro/ros2_control/AG2F90-C.xacro"/>
-			<xacro:include filename="$(find changingtek_description)/xacro/ros2_control/AG2F120S.xacro"/>
-			<xacro:include filename="$(find linkerhand_description)/xacro/ros2_control/o6.xacro"/>
-			<xacro:include filename="$(find linkerhand_description)/xacro/ros2_control/o7.xacro"/>
-			<xacro:if value="${left_gripper_type == 'rg75'}">
-				<xacro:rg75_interfaces name="left"/>
-			</xacro:if>
-			<xacro:if value="${right_gripper_type == 'rg75'}">
-				<xacro:rg75_interfaces name="right"/>
-			</xacro:if>
-			<xacro:if value="${left_gripper_type == 'ag2f90_c' or left_gripper_type == 'ag2f90_d'}">
-				<xacro:ag2f90c_interfaces name="left"/>
-			</xacro:if>
-			<xacro:if value="${right_gripper_type == 'ag2f90_c' or right_gripper_type == 'ag2f90_d'}">
-				<xacro:ag2f90c_interfaces name="right"/>
-			</xacro:if>
-			<xacro:if value="${left_gripper_type == 'ag2f120s' or left_gripper_type == 'ag2f120s_d'}">
-				<xacro:ag2f120s_interfaces name="left"/>
-			</xacro:if>
-			<xacro:if value="${right_gripper_type == 'ag2f120s' or right_gripper_type == 'ag2f120s_d'}">
-				<xacro:ag2f120s_interfaces name="right"/>
-			</xacro:if>
-			<xacro:if value="${left_hand_type == 'linkerhand_o6' or left_hand_type == 'linkerhand_l6'}">
-				<xacro:linkerhand_o6_interfaces name="left_hand"/>
-			</xacro:if>
-			<xacro:if value="${right_hand_type == 'linkerhand_o6' or right_hand_type == 'linkerhand_l6'}">
-				<xacro:linkerhand_o6_interfaces name="right_hand"/>
-			</xacro:if>
-			<xacro:if value="${left_hand_type == 'linkerhand_o7'}">
-				<xacro:linkerhand_o7_interfaces name="left_hand"/>
-			</xacro:if>
-			<xacro:if value="${right_hand_type == 'linkerhand_o7'}">
-				<xacro:linkerhand_o7_interfaces name="right_hand"/>
-			</xacro:if>
+			<xacro:dual_arm_ee_block mode="${ee_block_mode}"/>
 		</xacro:if>
-		<!-- 单臂配置 -->
 		<xacro:unless value="${selected_arm_config == 'dual'}">
 			<xacro:if value="${selected_arm_config == 'left'}">
-				<xacro:m6_interfaces name=""/>
-				<xacro:if value="${selected_gripper_type == 'ag2f90_c' or selected_gripper_type == 'ag2f90_d'}">
-					<xacro:include filename="$(find changingtek_description)/xacro/ros2_control/AG2F90-C.xacro"/>
-					<xacro:ag2f90c_interfaces name=""/>
-				</xacro:if>
-				<xacro:if value="${selected_gripper_type == 'ag2f120s' or selected_gripper_type == 'ag2f120s_d'}">
-					<xacro:include filename="$(find changingtek_description)/xacro/ros2_control/AG2F120S.xacro"/>
-					<xacro:ag2f120s_interfaces name=""/>
-				</xacro:if>
-				<xacro:if value="${selected_gripper_type == 'rg75'}">
-					<xacro:include filename="$(find jodell_description)/xacro/ros2_control/RG75-300.xacro"/>
-					<xacro:rg75_interfaces name=""/>
-				</xacro:if>
+				<xacro:single_arm_ee_block mode="${ee_block_mode}" gripper_type="${selected_gripper_type}"/>
 			</xacro:if>
 			<xacro:if value="${selected_arm_config == 'right'}">
@@ -116,4 +58,9 @@
 		</xacro:unless>
 	</ros2_control>
+	<xacro:if value="${is_real_hardware and selected_arm_config == 'dual'}">
+		<xacro:external_ee_systems
+			usb_left_port="$(arg usb_left_port)"
+			usb_right_port="$(arg usb_right_port)"/>
+	</xacro:if>
 	<xacro:arg name="gazebo" default="false"/>
 	<xacro:if value="$(arg gazebo)">
