Commit message: Feature/add hand (#12)
* 添加 theo hand std16a

* 添加 theo hand std16a hardware

* 添加 theo hand std16a 负载辨识

* 更新 theo hand std16a 负载辨识

* 更新 theohand 进ocs2 marker问题

* 补充readme

* 修改xacro增加flange

---------

Co-authored-by: Cursor <cursoragent@cursor.com>

File: m6_ccs_description/xacro/eef_type_resolver.xacro (robot description, xacro)
@@ -55,4 +55,7 @@
             <xacro:property name="${side}_hand_type" value="xhand1" scope="parent"/>
         </xacro:if>
+        <xacro:if value="${type_key == 'theohand_std16a' or type_key == 'theohand' or type_key == 'std16a'}">
+            <xacro:property name="${side}_hand_type" value="theohand_std16a" scope="parent"/>
+        </xacro:if>
     </xacro:macro>
 </robot>

File: m6_ccs_description/xacro/eefs.xacro (robot description, xacro)
@@ -13,4 +13,5 @@
     <xacro:include filename="$(find inspire_description)/xacro/hands/RH56F2.xacro"/>
     <xacro:include filename="$(find xhand1_description)/xacro/xhand1.xacro"/>
+    <xacro:include filename="$(find theohand_description)/xacro/std16a.xacro"/>
     <!-- Per-side default load (dyn_param) for MarvinHardware; 10 values: m, mx, my, mz, ixx, ixy, ixz, iyy, iyz, izz.
          Override via launch left_dyn_param/right_dyn_param (robot.local.yaml).
@@ -53,4 +54,7 @@
                     <param name="${side}_dyn_param">0.8,0,0,85.0,0,0,0,0,0,0</param>
                 </xacro:if>
+                <xacro:if value="${ee_key == 'theohand_std16a'}">
+                    <param name="${side}_dyn_param">1.192858777460025,-7.03987422170533,9.818292790393933,137.26999822427345,0.006918520800192261,0.0,0.0,0.001,0.0,7.865109749824159e-05</param>
+                </xacro:if>
             </xacro:if>
             <xacro:if value="${side == 'right'}">
@@ -81,4 +85,7 @@
                 <xacro:if value="${ee_key == 'linkerhand_o7'}">
                     <param name="${side}_dyn_param">0.8,0,0,85.0,0,0,0,0,0,0</param>
+                </xacro:if>
+                <xacro:if value="${ee_key == 'theohand_std16a'}">
+                    <param name="${side}_dyn_param">1.12002894189523,-18.48421622732829,-10.560222740339876,133.50284161880847,0.019335154889632066,0.0,0.0,0.01016838892588266,0.0,0.0034378184491521903</param>
                 </xacro:if>
             </xacro:if>
@@ -201,4 +208,17 @@
             </joint>
         </xacro:if>
+        <xacro:if value="${hand_type == 'theohand_std16a'}">
+            <xacro:TheoHandStd16A name="${side}_hand" direction="${1 if side == 'left' else -1}" use_flange="true" fixed_joints="${eef_fixed_joints}"/>
+            <joint name="${side}_hand_base_joint" type="fixed">
+                <xacro:if value="${side == 'left'}">
+                    <origin xyz="0 0 0.011043" rpy="0 0 ${PI/2}"/>
+                </xacro:if>
+                <xacro:if value="${side == 'right'}">
+                    <origin xyz="0 0 0.011043" rpy="0 0 ${-PI/2}"/>
+                </xacro:if>
+                <parent link="${side}_tcp"/>
+                <child link="${side}_hand_flange"/>
+            </joint>
+        </xacro:if>
         <!-- Hands with built-in ${side}_hand_eef; alias ${side}_eef for OCS2 / task.info -->
         <xacro:if value="${hand_type == 'xhand1'}">
@@ -210,4 +230,11 @@
         </xacro:if>
         <xacro:if value="${hand_type == 'linkerhand_o6' or hand_type == 'linkerhand_l6' or hand_type == 'linkerhand_o7' or hand_type == 'freedom_v1' or hand_type == 'freedom_v2' or hand_type == 'inspire_e2' or hand_type == 'inspire_f2'}">
+            <link name="${side}_eef"/>
+            <joint name="${side}_eef_joint" type="fixed">
+                <parent link="${side}_hand_eef"/>
+                <child link="${side}_eef"/>
+            </joint>
+        </xacro:if>
+        <xacro:if value="${hand_type == 'theohand_std16a'}">
             <link name="${side}_eef"/>
             <joint name="${side}_eef_joint" type="fixed">
@@ -238,5 +265,5 @@
         <!-- OCS2 planning URDF: no actuated EEF DOF (avoids per-tool removeJoints in .info) -->
         <xacro:if value="${eef_fixed_joints}">
-            <xacro:if value="${hand_type == 'linkerhand_o6' or hand_type == 'linkerhand_o7' or hand_type == 'linkerhand_l6' or hand_type == 'freedom_v1' or hand_type == 'freedom_v2' or hand_type == 'inspire_e2' or hand_type == 'inspire_f2' or hand_type == 'xhand1'}">
+            <xacro:if value="${hand_type == 'linkerhand_o6' or hand_type == 'linkerhand_o7' or hand_type == 'linkerhand_l6' or hand_type == 'freedom_v1' or hand_type == 'freedom_v2' or hand_type == 'inspire_e2' or hand_type == 'inspire_f2' or hand_type == 'xhand1' or hand_type == 'theohand_std16a'}">
                 <xacro:SideEndEffectorLinkerHand side="${side}" hand_type="${hand_type}" eef_fixed_joints="true"/>
             </xacro:if>
@@ -244,5 +271,5 @@
                 <xacro:SideEndEffectorERG32 side="${side}" eef_fixed_joints="true"/>
             </xacro:if>
-            <xacro:unless value="${hand_type == 'linkerhand_o6' or hand_type == 'linkerhand_o7' or hand_type == 'linkerhand_l6' or hand_type == 'freedom_v1' or hand_type == 'freedom_v2' or hand_type == 'inspire_e2' or hand_type == 'inspire_f2' or hand_type == 'xhand1' or hand_type == 'erg32'}">
+            <xacro:unless value="${hand_type == 'linkerhand_o6' or hand_type == 'linkerhand_o7' or hand_type == 'linkerhand_l6' or hand_type == 'freedom_v1' or hand_type == 'freedom_v2' or hand_type == 'inspire_e2' or hand_type == 'inspire_f2' or hand_type == 'xhand1' or hand_type == 'theohand_std16a' or hand_type == 'erg32'}">
                 <xacro:if value="${gripper_type == 'ag2f90_c' or gripper_type == 'ag2f90_d'}">
                     <xacro:AG2F90-C name="${side}" use_flange="true" pad="${gripper_pad}" kinematic_only="true"/>

File: m6_ccs_description/xacro/ros2_control/end_effector_interfaces.xacro (robot description, xacro)
@@ -14,4 +14,5 @@
 	<xacro:include filename="$(find inspire_description)/xacro/ros2_control/RH56F2.xacro"/>
 	<xacro:include filename="$(find xhand1_description)/xacro/ros2_control/side_systems.xacro"/>
+	<xacro:include filename="$(find theohand_description)/xacro/ros2_control/std16a.xacro"/>
 	<xacro:macro name="side_gripper_joint" params="side">
 		<joint name="${side}_gripper_joint">
@@ -46,4 +47,7 @@
 		<xacro:if value="${hand_type == 'erg32'}">
 			<xacro:erg32_interfaces name="${side}_hand"/>
+		</xacro:if>
+		<xacro:if value="${hand_type == 'theohand_std16a'}">
+			<xacro:theohand_std16a_interfaces name="${side}_hand"/>
 		</xacro:if>
 	</xacro:macro>

File: m6_ccs_description/xacro/ros2_control/external_ee_systems.xacro (robot description, xacro)
@@ -18,8 +18,22 @@
 		</ros2_control>
 	</xacro:macro>
+	<xacro:macro name="theohand_usb_side_system" params="side serial_port baudrate:=115200 slave_id:=auto">
+		<xacro:property name="theohand_slave_id" value="${2 if side == 'left' and slave_id == 'auto' else 1 if side == 'right' and slave_id == 'auto' else slave_id}"/>
+		<ros2_control name="theohand_${side}_system" type="system">
+			<hardware>
+				<plugin>modbus_ros2_control/TheoHandModbusHardware</plugin>
+				<param name="serial_port">${serial_port}</param>
+				<param name="slave_id">${theohand_slave_id}</param>
+				<param name="baudrate">${baudrate}</param>
+				<param name="read_feedback">true</param>
+			</hardware>
+			<xacro:side_hand_interfaces side="${side}" hand_type="theohand_std16a"/>
+		</ros2_control>
+	</xacro:macro>
 	<!-- left_ft / right_ft / usb_*_ft_port: declared in marvin_hardware.xacro; defaults read $(arg ...) here. -->
 	<xacro:macro name="external_ee_systems" params="
 		usb_left_port:=/dev/ttyUSB0
 		usb_right_port:=/dev/ttyUSB2
+		usb_baudrate:=115200
 		left_ft:=$(arg left_ft)
 		right_ft:=$(arg right_ft)
@@ -32,4 +46,10 @@
 		<xacro:if value="${right_drive_type == 'usb' and (right_hand_type == 'linkerhand_o6' or right_hand_type == 'linkerhand_l6' or right_hand_type == 'linkerhand_o7')}">
 			<xacro:side_usb_hand_system side="right" hand_type="${right_hand_type}" serial_port="${usb_right_port}"/>
+		</xacro:if>
+		<xacro:if value="${left_drive_type == 'usb' and left_hand_type == 'theohand_std16a'}">
+			<xacro:theohand_usb_side_system side="left" serial_port="${usb_left_port}" baudrate="${usb_baudrate}"/>
+		</xacro:if>
+		<xacro:if value="${right_drive_type == 'usb' and right_hand_type == 'theohand_std16a'}">
+			<xacro:theohand_usb_side_system side="right" serial_port="${usb_right_port}" baudrate="${usb_baudrate}"/>
 		</xacro:if>
 		<xacro:if value="${left_drive_type == 'usb' and left_hand_type == 'inspire_e2'}">

Commit message: add marvin pro
Co-authored-by: Cursor <cursoragent@cursor.com>

File: m6_ccs_description/xacro/eef_type_resolver.xacro (robot description, xacro)
@@ -58,4 +58,10 @@
             <xacro:property name="${side}_hand_type" value="theohand_std16a" scope="parent"/>
         </xacro:if>
+        <xacro:if value="${type_key == 'marvin_gripper'}">
+            <xacro:property name="${side}_gripper_type" value="marvin_gripper" scope="parent"/>
+        </xacro:if>
+        <xacro:if value="${type_key == 'marvin_gripper45'}">
+            <xacro:property name="${side}_gripper_type" value="marvin_gripper45" scope="parent"/>
+        </xacro:if>
     </xacro:macro>
 </robot>

File: m6_ccs_description/xacro/eefs.xacro (robot description, xacro)
@@ -14,4 +14,6 @@
     <xacro:include filename="$(find xhand1_description)/xacro/xhand1.xacro"/>
     <xacro:include filename="$(find theohand_description)/xacro/std16a.xacro"/>
+    <xacro:include filename="$(find marvin_gripper_description)/xacro/marvin_gripper.xacro"/>
+    <xacro:include filename="$(find marvin_gripper_description)/xacro/marvin_gripper45.xacro"/>
     <!-- Per-side default load (dyn_param) for MarvinHardware; 10 values: m, mx, my, mz, ixx, ixy, ixz, iyy, iyz, izz.
          Override via launch left_dyn_param/right_dyn_param (robot.local.yaml).
@@ -45,4 +47,8 @@
                     <param name="${side}_dyn_param">0.9464750422461978, -8.366166030270293, -9.50810456883501, 71.59365292895114, 0.02313627009490121, 0.0, 0.0, 0.017136701127687514, 0.0, 0.008640226166892327</param>
                 </xacro:if>
+                <xacro:if value="${ee_key == 'marvin_gripper' or ee_key == 'marvin_gripper45'}">
+                    <!-- TODO: replace with measured Marvin gripper values -->
+                    <param name="${side}_dyn_param">0.5,0,0,50.0,0.001,0,0,0.001,0,0.001</param>
+                </xacro:if>
                 <xacro:if value="${ee_key == 'linkerhand_o6'}">
                     <param name="${side}_dyn_param">0.6,0,0,70.0,0,0,0,0,0,0</param>
@@ -76,4 +82,8 @@
                     <!-- TODO: replace with measured EPGI180 values; temporarily reuse ag2f90 series -->
                     <param name="${side}_dyn_param">0.9464750422461978, -8.366166030270293, -9.50810456883501, 71.59365292895114, 0.02313627009490121, 0.0, 0.0, 0.017136701127687514, 0.0, 0.008640226166892327</param>
+                </xacro:if>
+                <xacro:if value="${ee_key == 'marvin_gripper' or ee_key == 'marvin_gripper45'}">
+                    <!-- TODO: replace with measured Marvin gripper values -->
+                    <param name="${side}_dyn_param">0.5,0,0,50.0,0.001,0,0,0.001,0,0.001</param>
                 </xacro:if>
                 <xacro:if value="${ee_key == 'linkerhand_o6'}">
@@ -303,4 +313,18 @@
                     </joint>
                 </xacro:if>
+                <xacro:if value="${gripper_type == 'marvin_gripper'}">
+                    <xacro:marvin_gripper name="${side}" kinematic_only="true"/>
+                    <joint name="${side}_gripper_base_joint" type="fixed">
+                        <parent link="${side}_tcp"/>
+                        <child link="${side}_flange"/>
+                    </joint>
+                </xacro:if>
+                <xacro:if value="${gripper_type == 'marvin_gripper45'}">
+                    <xacro:marvin_gripper45 name="${side}" kinematic_only="true"/>
+                    <joint name="${side}_gripper_base_joint" type="fixed">
+                        <parent link="${side}_tcp"/>
+                        <child link="${side}_flange"/>
+                    </joint>
+                </xacro:if>
                 <xacro:if value="${gripper_type == '' and hand_type == ''}">
                     <xacro:Ocs2SideEefFrame side="${side}" parent_link="${side}_tcp"/>
@@ -345,4 +369,18 @@
                     <child link="${side}_flange"/>
                     <origin xyz="0 0 0.0045"/>
+                </joint>
+            </xacro:if>
+            <xacro:if value="${gripper_type == 'marvin_gripper'}">
+                <xacro:marvin_gripper name="${side}"/>
+                <joint name="${side}_gripper_base_joint" type="fixed">
+                    <parent link="${side}_tcp"/>
+                    <child link="${side}_flange"/>
+                </joint>
+            </xacro:if>
+            <xacro:if value="${gripper_type == 'marvin_gripper45'}">
+                <xacro:marvin_gripper45 name="${side}"/>
+                <joint name="${side}_gripper_base_joint" type="fixed">
+                    <parent link="${side}_tcp"/>
+                    <child link="${side}_flange"/>
                 </joint>
             </xacro:if>

File: m6_ccs_description/xacro/ros2_control/end_effector_interfaces.xacro (robot description, xacro)
@@ -15,4 +15,5 @@
 	<xacro:include filename="$(find xhand1_description)/xacro/ros2_control/side_systems.xacro"/>
 	<xacro:include filename="$(find theohand_description)/xacro/ros2_control/std16a.xacro"/>
+	<xacro:include filename="$(find marvin_gripper_description)/xacro/ros2_control/marvin_gripper.xacro"/>
 	<xacro:macro name="side_gripper_joint" params="side">
 		<joint name="${side}_gripper_joint">
@@ -65,4 +66,7 @@
 			<xacro:epgi180_v2_interfaces name="${side}"/>
 		</xacro:if>
+		<xacro:if value="${gripper_type == 'marvin_gripper' or gripper_type == 'marvin_gripper45'}">
+			<xacro:marvin_gripper_interfaces name="${side}"/>
+		</xacro:if>
 	</xacro:macro>
 	<!-- mode: sim | real -->
