Commit message: 添加 theo hand std16a

File: m6_ccs_description/xacro/eef_type_resolver.xacro (robot description, xacro)
@@ -52,4 +52,7 @@
             <xacro:property name="${side}_hand_type" value="xhand1" scope="parent"/>
         </xacro:if>
+        <xacro:if value="${type_key == 'theohand_std16a' or type_key == 'theohand' or type_key == 'std16a'}">
+            <xacro:property name="${side}_hand_type" value="theohand_std16a" scope="parent"/>
+        </xacro:if>
     </xacro:macro>
 </robot>

File: m6_ccs_description/xacro/eefs.xacro (robot description, xacro)
@@ -12,4 +12,5 @@
     <xacro:include filename="$(find inspire_description)/xacro/hands/RH56F2.xacro"/>
     <xacro:include filename="$(find xhand1_description)/xacro/xhand1.xacro"/>
+    <xacro:include filename="$(find theohand_description)/xacro/std16a.xacro"/>
     <!-- Per-side default load (dyn_param) for MarvinHardware; 10 values: m, mx, my, mz, ixx, ixy, ixz, iyy, iyz, izz.
          Override via launch left_dyn_param/right_dyn_param (robot.local.yaml).
@@ -48,4 +49,7 @@
                     <param name="${side}_dyn_param">0.8,0,0,85.0,0,0,0,0,0,0</param>
                 </xacro:if>
+                <xacro:if value="${ee_key == 'theohand_std16a'}">
+                    <param name="${side}_dyn_param">0.57109497006203,-3.81424636269485,2.07802750628399,76.2957680404765,0.000373948529416664,-0.00000649325357222745,-0.0000139657450668528,0.000648700813496535,-0.00000047759577399386,0.000385655630526283</param>
+                </xacro:if>
             </xacro:if>
             <xacro:if value="${side == 'right'}">
@@ -72,4 +76,7 @@
                 <xacro:if value="${ee_key == 'linkerhand_o7'}">
                     <param name="${side}_dyn_param">0.8,0,0,85.0,0,0,0,0,0,0</param>
+                </xacro:if>
+                <xacro:if value="${ee_key == 'theohand_std16a'}">
+                    <param name="${side}_dyn_param">0.57109497006203,-3.81424636269485,-2.07802750628399,76.2957680404765,0.000373948529416664,0.00000649325357222745,-0.0000139657450668528,0.000648700813496535,0.00000047759577399386,0.000385655630526283</param>
                 </xacro:if>
             </xacro:if>
@@ -192,4 +199,12 @@
             </joint>
         </xacro:if>
+        <xacro:if value="${hand_type == 'theohand_std16a'}">
+            <xacro:TheoHandStd16A name="${side}_hand" direction="${1 if side == 'left' else -1}" fixed_joints="${eef_fixed_joints}"/>
+            <joint name="${side}_hand_base_joint" type="fixed">
+                <origin xyz="0 0 0" rpy="0 0 ${PI}"/>
+                <parent link="${side}_tcp"/>
+                <child link="${side}_hand_hand_base"/>
+            </joint>
+        </xacro:if>
         <!-- Hands with built-in ${side}_hand_eef; alias ${side}_eef for OCS2 / task.info -->
         <xacro:if value="${hand_type == 'xhand1'}">
@@ -204,4 +219,11 @@
             <joint name="${side}_eef_joint" type="fixed">
                 <parent link="${side}_hand_eef"/>
+                <child link="${side}_eef"/>
+            </joint>
+        </xacro:if>
+        <xacro:if value="${hand_type == 'theohand_std16a'}">
+            <link name="${side}_eef"/>
+            <joint name="${side}_eef_joint" type="fixed">
+                <parent link="${side}_hand_hand_base"/>
                 <child link="${side}_eef"/>
             </joint>
@@ -229,5 +251,5 @@
         <!-- OCS2 planning URDF: no actuated EEF DOF (avoids per-tool removeJoints in .info) -->
         <xacro:if value="${eef_fixed_joints}">
-            <xacro:if value="${hand_type == 'linkerhand_o6' or hand_type == 'linkerhand_o7' or hand_type == 'linkerhand_l6' or hand_type == 'freedom_v1' or hand_type == 'freedom_v2' or hand_type == 'inspire_e2' or hand_type == 'inspire_f2' or hand_type == 'xhand1'}">
+            <xacro:if value="${hand_type == 'linkerhand_o6' or hand_type == 'linkerhand_o7' or hand_type == 'linkerhand_l6' or hand_type == 'freedom_v1' or hand_type == 'freedom_v2' or hand_type == 'inspire_e2' or hand_type == 'inspire_f2' or hand_type == 'xhand1' or hand_type == 'theohand_std16a'}">
                 <xacro:SideEndEffectorLinkerHand side="${side}" hand_type="${hand_type}" eef_fixed_joints="true"/>
             </xacro:if>
@@ -235,5 +257,5 @@
                 <xacro:SideEndEffectorERG32 side="${side}" eef_fixed_joints="true"/>
             </xacro:if>
-            <xacro:unless value="${hand_type == 'linkerhand_o6' or hand_type == 'linkerhand_o7' or hand_type == 'linkerhand_l6' or hand_type == 'freedom_v1' or hand_type == 'freedom_v2' or hand_type == 'inspire_e2' or hand_type == 'inspire_f2' or hand_type == 'xhand1' or hand_type == 'erg32'}">
+            <xacro:unless value="${hand_type == 'linkerhand_o6' or hand_type == 'linkerhand_o7' or hand_type == 'linkerhand_l6' or hand_type == 'freedom_v1' or hand_type == 'freedom_v2' or hand_type == 'inspire_e2' or hand_type == 'inspire_f2' or hand_type == 'xhand1' or hand_type == 'theohand_std16a' or hand_type == 'erg32'}">
                 <xacro:if value="${gripper_type == 'ag2f90_c' or gripper_type == 'ag2f90_d'}">
                     <xacro:AG2F90-C name="${side}" use_flange="true" pad="${gripper_pad}" kinematic_only="true"/>

File: m6_ccs_description/xacro/ros2_control/end_effector_interfaces.xacro (robot description, xacro)
@@ -13,4 +13,5 @@
 	<xacro:include filename="$(find inspire_description)/xacro/ros2_control/RH56F2.xacro"/>
 	<xacro:include filename="$(find xhand1_description)/xacro/ros2_control/side_systems.xacro"/>
+	<xacro:include filename="$(find theohand_description)/xacro/ros2_control/std16a.xacro"/>
 	<xacro:macro name="side_gripper_joint" params="side">
 		<joint name="${side}_gripper_joint">
@@ -45,4 +46,7 @@
 		<xacro:if value="${hand_type == 'erg32'}">
 			<xacro:erg32_interfaces name="${side}_hand"/>
+		</xacro:if>
+		<xacro:if value="${hand_type == 'theohand_std16a'}">
+			<xacro:theohand_std16a_interfaces name="${side}_hand"/>
 		</xacro:if>
 	</xacro:macro>

File: m6_ccs_description/xacro/ros2_control/external_ee_systems.xacro (robot description, xacro)
@@ -17,7 +17,22 @@
 		</ros2_control>
 	</xacro:macro>
+	<xacro:macro name="theohand_usb_side_system" params="side serial_port baudrate:=115200 slave_id:=1">
+		<ros2_control name="theohand_${side}_system" type="system">
+			<hardware>
+				<plugin>modbus_ros2_control/TheoHandModbusHardware</plugin>
+				<param name="serial_port">${serial_port}</param>
+				<param name="slave_id">${slave_id}</param>
+				<param name="baudrate">${baudrate}</param>
+				<param name="read_feedback">true</param>
+				<param name="background_period_ms">200</param>
+				<param name="feedback_quiet_after_write_ms">500</param>
+			</hardware>
+			<xacro:side_hand_interfaces side="${side}" hand_type="theohand_std16a"/>
+		</ros2_control>
+	</xacro:macro>
 	<xacro:macro name="external_ee_systems" params="
 		usb_left_port:=/dev/ttyUSB0
-		usb_right_port:=/dev/ttyUSB2">
+		usb_right_port:=/dev/ttyUSB2
+		usb_baudrate:=115200">
 		<xacro:if value="${left_drive_type == 'usb' and (left_hand_type == 'linkerhand_o6' or left_hand_type == 'linkerhand_l6' or left_hand_type == 'linkerhand_o7')}">
 			<xacro:side_usb_hand_system side="left" hand_type="${left_hand_type}" serial_port="${usb_left_port}"/>
@@ -25,4 +40,10 @@
 		<xacro:if value="${right_drive_type == 'usb' and (right_hand_type == 'linkerhand_o6' or right_hand_type == 'linkerhand_l6' or right_hand_type == 'linkerhand_o7')}">
 			<xacro:side_usb_hand_system side="right" hand_type="${right_hand_type}" serial_port="${usb_right_port}"/>
+		</xacro:if>
+		<xacro:if value="${left_drive_type == 'usb' and left_hand_type == 'theohand_std16a'}">
+			<xacro:theohand_usb_side_system side="left" serial_port="${usb_left_port}" baudrate="${usb_baudrate}"/>
+		</xacro:if>
+		<xacro:if value="${right_drive_type == 'usb' and right_hand_type == 'theohand_std16a'}">
+			<xacro:theohand_usb_side_system side="right" serial_port="${usb_right_port}" baudrate="${usb_baudrate}"/>
 		</xacro:if>
 		<xacro:if value="${left_drive_type == 'usb' and left_hand_type == 'inspire_e2'}">

Commit message: add support for eincinx epgi180

File: m6_ccs_description/xacro/eef_type_resolver.xacro (robot description, xacro)
@@ -8,4 +8,7 @@
         <xacro:if value="${type_key == 'rg75'}">
             <xacro:property name="${side}_gripper_type" value="rg75" scope="parent"/>
+        </xacro:if>
+        <xacro:if value="${type_key == 'epgi180'}">
+            <xacro:property name="${side}_gripper_type" value="epgi180" scope="parent"/>
         </xacro:if>
         <xacro:if value="${type_key == 'erg32'}">

File: m6_ccs_description/xacro/eefs.xacro (robot description, xacro)
@@ -7,4 +7,5 @@
     <xacro:include filename="$(find changingtek_description)/xacro/AG2F90-C.xacro"/>
     <xacro:include filename="$(find changingtek_description)/xacro/AG2F120S.xacro"/>
+    <xacro:include filename="$(find eincinx_description)/xacro/EPGI180-v2.xacro"/>
     <xacro:include filename="$(find freedom_description)/xacro/freedomv1.xacro"/>
     <xacro:include filename="$(find freedom_description)/xacro/freedomv2.xacro"/>
@@ -39,4 +40,8 @@
                     <param name="${side}_dyn_param">1.3944348661120496, -7.913087934362548, 10.50004773179898, 72.44110460800299, 0.014948849408945898, 0.0, 0.0, 0.005470384569170036, 0.0, 0.002567996881581655</param>
                 </xacro:if>
+                <xacro:if value="${ee_key == 'epgi180'}">
+                    <!-- TODO: replace with measured EPGI180 values; temporarily reuse ag2f90 series -->
+                    <param name="${side}_dyn_param">0.9464750422461978, -8.366166030270293, -9.50810456883501, 71.59365292895114, 0.02313627009490121, 0.0, 0.0, 0.017136701127687514, 0.0, 0.008640226166892327</param>
+                </xacro:if>
                 <xacro:if value="${ee_key == 'linkerhand_o6'}">
                     <param name="${side}_dyn_param">0.6,0,0,70.0,0,0,0,0,0,0</param>
@@ -63,4 +68,8 @@
                     <!-- TODO: replace with measured values; temporarily reuse ag2f90 series -->
                     <param name="${side}_dyn_param">1.4038028109970075, 3.8873998644204817, -10.865529763155825, 73.06884012186562, 0.001, 0.0, 0.0, 0.001, 0.0, 0.0057238484709952525</param>
+                </xacro:if>
+                <xacro:if value="${ee_key == 'epgi180'}">
+                    <!-- TODO: replace with measured EPGI180 values; temporarily reuse ag2f90 series -->
+                    <param name="${side}_dyn_param">0.9464750422461978, -8.366166030270293, -9.50810456883501, 71.59365292895114, 0.02313627009490121, 0.0, 0.0, 0.017136701127687514, 0.0, 0.008640226166892327</param>
                 </xacro:if>
                 <xacro:if value="${ee_key == 'linkerhand_o6'}">
@@ -259,4 +268,12 @@
                     </joint>
                 </xacro:if>
+                <xacro:if value="${gripper_type == 'epgi180'}">
+                    <xacro:EPGI180-v2 name="${side}" use_flange="true" pad="${gripper_pad}" kinematic_only="true"/>
+                    <joint name="${side}_gripper_fix" type="fixed">
+                        <parent link="${side}_tcp"/>
+                        <child link="${side}_flange"/>
+                        <origin xyz="0 0 0.0045"/>
+                    </joint>
+                </xacro:if>
                 <xacro:if value="${gripper_type == '' and hand_type == ''}">
                     <xacro:Ocs2SideEefFrame side="${side}" parent_link="${side}_tcp"/>
@@ -293,4 +310,12 @@
                     <parent link="${side}_tcp"/>
                     <child link="${side}_flange"/>
+                </joint>
+            </xacro:if>
+            <xacro:if value="${gripper_type == 'epgi180'}">
+                <xacro:EPGI180-v2 name="${side}" use_flange="true" pad="${gripper_pad}"/>
+                <joint name="${side}_gripper_fix" type="fixed">
+                    <parent link="${side}_tcp"/>
+                    <child link="${side}_flange"/>
+                    <origin xyz="0 0 0.0045"/>
                 </joint>
             </xacro:if>

File: m6_ccs_description/xacro/ros2_control/end_effector_interfaces.xacro (robot description, xacro)
@@ -6,4 +6,5 @@
 	<xacro:include filename="$(find changingtek_description)/xacro/ros2_control/AG2F90-C.xacro"/>
 	<xacro:include filename="$(find changingtek_description)/xacro/ros2_control/AG2F120S.xacro"/>
+	<xacro:include filename="$(find eincinx_description)/xacro/ros2_control/EPGI180-v2.xacro"/>
 	<xacro:include filename="$(find linkerhand_description)/xacro/ros2_control/o6.xacro"/>
 	<xacro:include filename="$(find linkerhand_description)/xacro/ros2_control/o7.xacro"/>
@@ -57,4 +58,7 @@
 			<xacro:ag2f120s_interfaces name="${side}"/>
 		</xacro:if>
+		<xacro:if value="${gripper_type == 'epgi180'}">
+			<xacro:epgi180_v2_interfaces name="${side}"/>
+		</xacro:if>
 	</xacro:macro>
 	<!-- mode: sim | real -->

Commit message: add wuji hand2

File: m6_ccs_description/xacro/eef_type_resolver.xacro (robot description, xacro)
@@ -58,4 +58,7 @@
             <xacro:property name="${side}_hand_type" value="theohand_std16a" scope="parent"/>
         </xacro:if>
+        <xacro:if value="${type_key == 'wuji_hand2'}">
+            <xacro:property name="${side}_hand_type" value="wuji_hand2" scope="parent"/>
+        </xacro:if>
         <xacro:if value="${type_key == 'marvin_gripper'}">
             <xacro:property name="${side}_gripper_type" value="marvin_gripper" scope="parent"/>

File: m6_ccs_description/xacro/eefs.xacro (robot description, xacro)
@@ -14,4 +14,5 @@
     <xacro:include filename="$(find xhand1_description)/xacro/xhand1.xacro"/>
     <xacro:include filename="$(find theohand_description)/xacro/std16a.xacro"/>
+    <xacro:include filename="$(find wuji_description)/xacro/hand2.xacro"/>
     <xacro:include filename="$(find marvin_gripper_description)/xacro/marvin_gripper.xacro"/>
     <xacro:include filename="$(find marvin_gripper_description)/xacro/marvin_gripper45.xacro"/>
@@ -231,4 +232,14 @@
             </joint>
         </xacro:if>
+        <xacro:if value="${hand_type == 'wuji_hand2'}">
+            <xacro:WujiHand2 name="${side}_hand" direction="${1 if side == 'left' else -1}" use_mount="true" fixed_joints="${eef_fixed_joints}"/>
+            <!-- mount→hand_base has R_x(π); tcp→mount needs R_x(π) so hand_base +Z (fingers) = tcp +Z.
+                 L/R mesh mirror is via direction:=±1 — do not add opposite yaw (fights mirroring). -->
+            <joint name="${side}_hand_base_joint" type="fixed">
+                <origin xyz="0 0 0" rpy="${PI} 0 0"/>
+                <parent link="${side}_tcp"/>
+                <child link="${side}_hand_mount"/>
+            </joint>
+        </xacro:if>
         <!-- Hands with built-in ${side}_hand_eef; alias ${side}_eef for OCS2 / task.info -->
         <xacro:if value="${hand_type == 'xhand1'}">
@@ -246,5 +257,5 @@
             </joint>
         </xacro:if>
-        <xacro:if value="${hand_type == 'theohand_std16a'}">
+        <xacro:if value="${hand_type == 'theohand_std16a' or hand_type == 'wuji_hand2'}">
             <link name="${side}_eef"/>
             <joint name="${side}_eef_joint" type="fixed">
@@ -275,5 +286,5 @@
         <!-- OCS2 planning URDF: no actuated EEF DOF (avoids per-tool removeJoints in .info) -->
         <xacro:if value="${eef_fixed_joints}">
-            <xacro:if value="${hand_type == 'linkerhand_o6' or hand_type == 'linkerhand_o7' or hand_type == 'linkerhand_l6' or hand_type == 'freedom_v1' or hand_type == 'freedom_v2' or hand_type == 'inspire_e2' or hand_type == 'inspire_f2' or hand_type == 'xhand1' or hand_type == 'theohand_std16a'}">
+            <xacro:if value="${hand_type == 'linkerhand_o6' or hand_type == 'linkerhand_o7' or hand_type == 'linkerhand_l6' or hand_type == 'freedom_v1' or hand_type == 'freedom_v2' or hand_type == 'inspire_e2' or hand_type == 'inspire_f2' or hand_type == 'xhand1' or hand_type == 'theohand_std16a' or hand_type == 'wuji_hand2'}">
                 <xacro:SideEndEffectorLinkerHand side="${side}" hand_type="${hand_type}" eef_fixed_joints="true"/>
             </xacro:if>
@@ -281,5 +292,5 @@
                 <xacro:SideEndEffectorERG32 side="${side}" eef_fixed_joints="true"/>
             </xacro:if>
-            <xacro:unless value="${hand_type == 'linkerhand_o6' or hand_type == 'linkerhand_o7' or hand_type == 'linkerhand_l6' or hand_type == 'freedom_v1' or hand_type == 'freedom_v2' or hand_type == 'inspire_e2' or hand_type == 'inspire_f2' or hand_type == 'xhand1' or hand_type == 'theohand_std16a' or hand_type == 'erg32'}">
+            <xacro:unless value="${hand_type == 'linkerhand_o6' or hand_type == 'linkerhand_o7' or hand_type == 'linkerhand_l6' or hand_type == 'freedom_v1' or hand_type == 'freedom_v2' or hand_type == 'inspire_e2' or hand_type == 'inspire_f2' or hand_type == 'xhand1' or hand_type == 'theohand_std16a' or hand_type == 'wuji_hand2' or hand_type == 'erg32'}">
                 <xacro:if value="${gripper_type == 'ag2f90_c' or gripper_type == 'ag2f90_d'}">
                     <xacro:AG2F90-C name="${side}" use_flange="true" pad="${gripper_pad}" kinematic_only="true"/>

File: m6_ccs_description/xacro/ros2_control/end_effector_interfaces.xacro (robot description, xacro)
@@ -15,4 +15,5 @@
 	<xacro:include filename="$(find xhand1_description)/xacro/ros2_control/side_systems.xacro"/>
 	<xacro:include filename="$(find theohand_description)/xacro/ros2_control/std16a.xacro"/>
+	<xacro:include filename="$(find wuji_description)/xacro/ros2_control/hand2.xacro"/>
 	<xacro:include filename="$(find marvin_gripper_description)/xacro/ros2_control/marvin_gripper.xacro"/>
 	<xacro:macro name="side_gripper_joint" params="side">
@@ -51,4 +52,7 @@
 		<xacro:if value="${hand_type == 'theohand_std16a'}">
 			<xacro:theohand_std16a_interfaces name="${side}_hand"/>
+		</xacro:if>
+		<xacro:if value="${hand_type == 'wuji_hand2'}">
+			<xacro:wuji_hand2_interfaces name="${side}_hand"/>
 		</xacro:if>
 	</xacro:macro>
