Commit message: add hand eef

File: m6_ccs_description/xacro/eefs.xacro (robot description, xacro)
@@ -55,6 +55,11 @@
             </joint>
         </xacro:if>
-        <xacro:if value="${hand_type == 'linkerhand_o6' or hand_type == 'linkerhand_o7' or hand_type == 'linkerhand_l6'}">
-            <xacro:Ocs2SideEefFrame side="${side}" parent_link="${side}_hand_hand_base"/>
+        <!-- LinkerHand O6/L6/O7: built-in ${side}_hand_eef; alias ${side}_eef for OCS2 / task.info -->
+        <xacro:if value="${hand_type == 'linkerhand_o6' or hand_type == 'linkerhand_l6' or hand_type == 'linkerhand_o7'}">
+            <link name="${side}_eef"/>
+            <joint name="${side}_eef_joint" type="fixed">
+                <parent link="${side}_hand_eef"/>
+                <child link="${side}_eef"/>
+            </joint>
         </xacro:if>
     </xacro:macro>

Commit message: 添加inspireCANFD，修掉频率过低的问题

File: m6_ccs_description/xacro/eefs.xacro (robot description, xacro)
@@ -85,5 +85,5 @@
         </xacro:if>
         <xacro:if value="${hand_type == 'inspire_e2'}">
-            <xacro:InspireHandRH56E2 name="${side}_hand" direction="${1 if side == 'left' else -1}" use_flange="true"/>
+            <xacro:InspireHandRH56E2 name="${side}_hand" direction="${1 if side == 'left' else -1}" use_flange="true" fixed_joints="${eef_fixed_joints}"/>
             <joint name="${side}_hand_base_joint" type="fixed">
                 <xacro:if value="${side == 'left'}">
@@ -98,15 +98,8 @@
         </xacro:if>
         <!-- Hands with built-in ${side}_hand_eef; alias ${side}_eef for OCS2 / task.info -->
-        <xacro:if value="${hand_type == 'linkerhand_o6' or hand_type == 'linkerhand_l6' or hand_type == 'linkerhand_o7' or hand_type == 'freedom_v2'}">
+        <xacro:if value="${hand_type == 'linkerhand_o6' or hand_type == 'linkerhand_l6' or hand_type == 'linkerhand_o7' or hand_type == 'freedom_v1' or hand_type == 'freedom_v2' or hand_type == 'inspire_e2'}">
             <link name="${side}_eef"/>
             <joint name="${side}_eef_joint" type="fixed">
                 <parent link="${side}_hand_eef"/>
-                <child link="${side}_eef"/>
-            </joint>
-        </xacro:if>
-        <xacro:if value="${hand_type == 'freedom_v1' or hand_type == 'inspire_e2'}">
-            <link name="${side}_eef"/>
-            <joint name="${side}_eef_joint" type="fixed">
-                <parent link="${side}_hand_hand_base"/>
                 <child link="${side}_eef"/>
             </joint>

File: m6_ccs_description/xacro/robot.xacro (robot description, xacro)
@@ -115,17 +115,5 @@
 			</joint>
 			<xacro:DualArmMount parent="arm_base" left_xyz="0 0.12 0.701" right_xyz="0 -0.12 0.701"/>
-			<xacro:if value="${selected_gripper_type == 'none'}">
-				<link name="right_eef"/>
-				<joint name="right_eef_joint" type="fixed">
-					<parent link="right_tcp"/>
-					<child link="right_eef"/>
-				</joint>
-				<link name="left_eef"/>
-				<joint name="left_eef_joint" type="fixed">
-					<parent link="left_tcp"/>
-					<child link="left_eef"/>
-				</joint>
 			</xacro:if>
-		</xacro:if>
 		<xacro:unless value="${selected_scene == 'desktop'}">
 			<!-- 非 Desktop 场景：base_link 为空，有 arm_base -->

Commit message: 添加inspireCANFD，修掉频率过低的问题

File: m6_ccs_description/xacro/eefs.xacro (robot description, xacro)
@@ -75,8 +75,8 @@
             <joint name="${side}_hand_base_joint" type="fixed">
                 <xacro:if value="${side == 'left'}">
-                    <origin xyz="0 0 0" rpy="0 0 ${PI/2}"/>
+                    <origin xyz="0 0 0" rpy="0 0 ${PI}"/>
                 </xacro:if>
                 <xacro:if value="${side == 'right'}">
-                    <origin xyz="0 0 0" rpy="0 0 ${-PI/2}"/>
+                    <origin xyz="0 0 0" rpy="0 0 ${PI}"/>
                 </xacro:if>
                 <parent link="${side}_tcp"/>

File: m6_ccs_description/xacro/ros2_control/robot.xacro (robot description, xacro)
@@ -103,4 +103,8 @@
 					<param name="right_dyn_param">1.2874,-30.145,-10,147.85,0,0,0,0,0,0</param>
 				</xacro:if>
+				<xacro:unless value="${selected_scene == 'desktop'}">
+					<param name="left_dyn_param">0,0,0,0,0,0,0,0,0,0</param>
+					<param name="right_dyn_param">0.9299382555569992,-9.36555486674267,-10.515510521015127,99.40658707033754,0.01874979461327618,0.0,0.0,0.010832861672583472,0.0,0.0035832781118723027</param>
+				</xacro:unless>
 				<xacro:if value="${selected_scene == 'usb-90c'}">
 					<param name="device_ip">192.168.10.190</param>

Commit message: 增加自动从yaml中载入负载

File: m6_ccs_description/xacro/eefs.xacro (robot description, xacro)
@@ -5,4 +5,53 @@
     <xacro:include filename="$(find jodell_description)/xacro/RG75-300.xacro"/>
     <xacro:include filename="$(find changingtek_description)/xacro/AG2F90-C.xacro"/>
+    <!-- Per-side default load (dyn_param) for MarvinHardware; 10 values: m, mx, my, mz, ixx, ixy, ixz, iyy, iyz, izz.
+         Override via launch left_dyn_param/right_dyn_param (robot.local.yaml).
+         No end effector (empty ee_key) -> all zeros. -->
+    <xacro:macro name="ee_dyn_param" params="side ee_key arg_val">
+        <xacro:if value="${arg_val != ''}">
+            <param name="${side}_dyn_param">${arg_val}</param>
+        </xacro:if>
+        <xacro:unless value="${arg_val != ''}">
+            <xacro:if value="${ee_key == '' or ee_key == 'none'}">
+                <param name="${side}_dyn_param">0,0,0,0,0,0,0,0,0,0</param>
+            </xacro:if>
+            <xacro:unless value="${ee_key == '' or ee_key == 'none'}">
+            <xacro:if value="${side == 'left'}">
+                <xacro:if value="${ee_key == 'rg75'}">
+                    <param name="${side}_dyn_param">1.6200799541791235, 1.4285009257202586, -0.5789585762443014, 104.39051192831192, 0.004873874899366342, 0.0, 0.0, 0.001, 0.0, 0.0019355638096347936</param>
+                </xacro:if>
+                <xacro:if value="${ee_key == 'ag2f90_c' or ee_key == 'ag2f90_d' or ee_key == 'ag2f90_c_soft'}">
+                    <param name="${side}_dyn_param">0.9464750422461978, -8.366166030270293, -9.50810456883501, 71.59365292895114, 0.02313627009490121, 0.0, 0.0, 0.017136701127687514, 0.0, 0.008640226166892327</param>
+                </xacro:if>
+                <xacro:if value="${ee_key == 'linkerhand_o6'}">
+                    <param name="${side}_dyn_param">0.6,0,0,70.0,0,0,0,0,0,0</param>
+                </xacro:if>
+                <xacro:if value="${ee_key == 'linkerhand_l6'}">
+                    <param name="${side}_dyn_param">0.6929861562459377, -0.02709362955502027, 21.325042427584716, 142.0468769124068, 0.001, 0.0, 0.0, 0.001, 0.0, 0.004408438461135547</param>
+                </xacro:if>
+                <xacro:if value="${ee_key == 'linkerhand_o7'}">
+                    <param name="${side}_dyn_param">0.8,0,0,85.0,0,0,0,0,0,0</param>
+                </xacro:if>
+            </xacro:if>
+            <xacro:if value="${side == 'right'}">
+                <xacro:if value="${ee_key == 'rg75'}">
+                    <param name="${side}_dyn_param">1.6200799541791235, 1.4285009257202586, -0.5789585762443014, 104.39051192831192, 0.004873874899366342, 0.0, 0.0, 0.001, 0.0, 0.0019355638096347936</param>
+                </xacro:if>
+                <xacro:if value="${ee_key == 'ag2f90_c' or ee_key == 'ag2f90_d' or ee_key == 'ag2f90_c_soft'}">
+                    <param name="${side}_dyn_param">0.9464750422461978, -8.366166030270293, -9.50810456883501, 71.59365292895114, 0.02313627009490121, 0.0, 0.0, 0.017136701127687514, 0.0, 0.008640226166892327</param>
+                </xacro:if>
+                <xacro:if value="${ee_key == 'linkerhand_o6'}">
+                    <param name="${side}_dyn_param">1.6200799541791235, 1.4285009257202586, -0.5789585762443014, 104.39051192831192, 0.004873874899366342, 0.0, 0.0, 0.001, 0.0, 0.0019355638096347936</param>
+                </xacro:if>
+                <xacro:if value="${ee_key == 'linkerhand_l6'}">
+                    <param name="${side}_dyn_param">0.757127258546731, -18.86292230512758, -23.37191007763647, 69.11766685323222, 0.02103669807705659, 0.0, 0.0, 0.01131025204380805, 0.0, 0.00955246486803428</param>
+                </xacro:if>
+                <xacro:if value="${ee_key == 'linkerhand_o7'}">
+                    <param name="${side}_dyn_param">0.8,0,0,85.0,0,0,0,0,0,0</param>
+                </xacro:if>
+            </xacro:if>
+            </xacro:unless>
+        </xacro:unless>
+    </xacro:macro>
     <xacro:macro name="Ocs2SideEefFrame" params="side parent_link">
         <link name="${side}_eef"/>

File: m6_ccs_description/xacro/ros2_control/robot.xacro (robot description, xacro)
@@ -4,4 +4,7 @@
 	<xacro:arg name="ctrl_mode" default="position"/>
 	<xacro:arg name="type" default="dual"/>
+	<!-- Non-desktop only: from robot.local.yaml via launch (robot_profile) -->
+	<xacro:arg name="left_dyn_param" default=""/>
+	<xacro:arg name="right_dyn_param" default=""/>
 	<link name="world"/>
 	<joint name="world_fixed" type="fixed">
@@ -40,4 +43,12 @@
 					<param name="left_dyn_param">1.2874,-10.145,30,114.65,0,0,0,0,0,0</param>
 					<param name="right_dyn_param">1.2874,-30.145,-10,147.85,0,0,0,0,0,0</param>
+				</xacro:if>
+				<xacro:if value="${selected_scene != 'desktop'}">
+					<xacro:ee_dyn_param side="left"
+						ee_key="${left_hand_type if left_hand_type != '' else left_gripper_type}"
+						arg_val="$(arg left_dyn_param)"/>
+					<xacro:ee_dyn_param side="right"
+						ee_key="${right_hand_type if right_hand_type != '' else right_gripper_type}"
+						arg_val="$(arg right_dyn_param)"/>
 				</xacro:if>
 				<xacro:if value="${selected_scene == 'usb-90c'}">

Commit message: 修改home位置以及参数

File: m6_ccs_description/xacro/eefs.xacro (robot description, xacro)
@@ -138,8 +138,8 @@
             <joint name="${side}_hand_base_joint" type="fixed">
                 <xacro:if value="${side == 'left'}">
-                    <origin xyz="0 0 0.0045" rpy="0 0 ${PI/2}"/>
-                </xacro:if>
-                <xacro:if value="${side == 'right'}">
-                    <origin xyz="0 0 0.0045" rpy="0 0 ${-PI/2}"/>
+                    <origin xyz="0 0 0.0045" rpy="0 0 ${PI}"/>
+                </xacro:if>
+                <xacro:if value="${side == 'right'}">
+                    <origin xyz="0 0 0.0045" rpy="0 0 ${-PI}"/>
                 </xacro:if>
                 <parent link="${side}_tcp"/>

Commit message: 修改macro名字为SideEndEffectorDexterousHand

File: m6_ccs_description/xacro/eefs.xacro (robot description, xacro)
@@ -84,5 +84,5 @@
         </joint>
     </xacro:macro>
-    <xacro:macro name="SideEndEffectorLinkerHand" params="side hand_type eef_fixed_joints">
+    <xacro:macro name="SideEndEffectorDexterousHand" params="side hand_type eef_fixed_joints">
         <xacro:if value="${hand_type == 'linkerhand_o6'}">
             <xacro:include filename="$(find linkerhand_description)/xacro/o6.xacro"/>
@@ -230,5 +230,5 @@
         <xacro:if value="${eef_fixed_joints}">
             <xacro:if value="${hand_type == 'linkerhand_o6' or hand_type == 'linkerhand_o7' or hand_type == 'linkerhand_l6' or hand_type == 'freedom_v1' or hand_type == 'freedom_v2' or hand_type == 'inspire_e2' or hand_type == 'inspire_f2' or hand_type == 'xhand1'}">
-                <xacro:SideEndEffectorLinkerHand side="${side}" hand_type="${hand_type}" eef_fixed_joints="true"/>
+                <xacro:SideEndEffectorDexterousHand side="${side}" hand_type="${hand_type}" eef_fixed_joints="true"/>
             </xacro:if>
             <xacro:if value="${hand_type == 'erg32'}">
@@ -298,5 +298,5 @@
                 <xacro:SideEndEffectorERG32 side="${side}" eef_fixed_joints="false"/>
             </xacro:if>
-            <xacro:SideEndEffectorLinkerHand side="${side}" hand_type="${hand_type}" eef_fixed_joints="false"/>
+            <xacro:SideEndEffectorDexterousHand side="${side}" hand_type="${hand_type}" eef_fixed_joints="false"/>
         </xacro:unless>
     </xacro:macro>
