Commit message: 添加 theo hand std16a hardware

File: m6_ccs_description/xacro/eefs.xacro (robot description, xacro)
@@ -202,5 +202,5 @@
             <xacro:TheoHandStd16A name="${side}_hand" direction="${1 if side == 'left' else -1}" fixed_joints="${eef_fixed_joints}"/>
             <joint name="${side}_hand_base_joint" type="fixed">
-                <origin xyz="0 0 0" rpy="0 0 ${PI}"/>
+                <origin xyz="0 0 0"/>
                 <parent link="${side}_tcp"/>
                 <child link="${side}_hand_hand_base"/>
@@ -225,5 +225,5 @@
             <link name="${side}_eef"/>
             <joint name="${side}_eef_joint" type="fixed">
-                <parent link="${side}_hand_hand_base"/>
+                <parent link="${side}_hand_eef"/>
                 <child link="${side}_eef"/>
             </joint>

File: m6_ccs_description/xacro/ros2_control/external_ee_systems.xacro (robot description, xacro)
@@ -17,14 +17,13 @@
 		</ros2_control>
 	</xacro:macro>
-	<xacro:macro name="theohand_usb_side_system" params="side serial_port baudrate:=115200 slave_id:=1">
+	<xacro:macro name="theohand_usb_side_system" params="side serial_port baudrate:=115200 slave_id:=auto">
+		<xacro:property name="theohand_slave_id" value="${2 if side == 'left' and slave_id == 'auto' else 1 if side == 'right' and slave_id == 'auto' else slave_id}"/>
 		<ros2_control name="theohand_${side}_system" type="system">
 			<hardware>
 				<plugin>modbus_ros2_control/TheoHandModbusHardware</plugin>
 				<param name="serial_port">${serial_port}</param>
-				<param name="slave_id">${slave_id}</param>
+				<param name="slave_id">${theohand_slave_id}</param>
 				<param name="baudrate">${baudrate}</param>
 				<param name="read_feedback">true</param>
-				<param name="background_period_ms">200</param>
-				<param name="feedback_quiet_after_write_ms">500</param>
 			</hardware>
 			<xacro:side_hand_interfaces side="${side}" hand_type="theohand_std16a"/>

Commit message: 更新 theohand 进ocs2 marker问题

File: m6_ccs_description/xacro/eefs.xacro (robot description, xacro)
@@ -202,5 +202,10 @@
             <xacro:TheoHandStd16A name="${side}_hand" direction="${1 if side == 'left' else -1}" fixed_joints="${eef_fixed_joints}"/>
             <joint name="${side}_hand_base_joint" type="fixed">
-                <origin xyz="0 0 0"/>
+                <xacro:if value="${side == 'left'}">
+                    <origin xyz="0 0 0" rpy="0 0 ${PI/2}"/>
+                </xacro:if>
+                <xacro:if value="${side == 'right'}">
+                    <origin xyz="0 0 0" rpy="0 0 ${-PI/2}"/>
+                </xacro:if>
                 <parent link="${side}_tcp"/>
                 <child link="${side}_hand_hand_base"/>

Commit message: 修改xacro增加flange

File: m6_ccs_description/xacro/eefs.xacro (robot description, xacro)
@@ -209,14 +209,14 @@
         </xacro:if>
         <xacro:if value="${hand_type == 'theohand_std16a'}">
-            <xacro:TheoHandStd16A name="${side}_hand" direction="${1 if side == 'left' else -1}" fixed_joints="${eef_fixed_joints}"/>
-            <joint name="${side}_hand_base_joint" type="fixed">
-                <xacro:if value="${side == 'left'}">
-                    <origin xyz="0 0 0" rpy="0 0 ${PI/2}"/>
-                </xacro:if>
-                <xacro:if value="${side == 'right'}">
-                    <origin xyz="0 0 0" rpy="0 0 ${-PI/2}"/>
-                </xacro:if>
-                <parent link="${side}_tcp"/>
-                <child link="${side}_hand_hand_base"/>
+            <xacro:TheoHandStd16A name="${side}_hand" direction="${1 if side == 'left' else -1}" use_flange="true" fixed_joints="${eef_fixed_joints}"/>
+            <joint name="${side}_hand_base_joint" type="fixed">
+                <xacro:if value="${side == 'left'}">
+                    <origin xyz="0 0 0.011043" rpy="0 0 ${PI/2}"/>
+                </xacro:if>
+                <xacro:if value="${side == 'right'}">
+                    <origin xyz="0 0 0.011043" rpy="0 0 ${-PI/2}"/>
+                </xacro:if>
+                <parent link="${side}_tcp"/>
+                <child link="${side}_hand_flange"/>
             </joint>
         </xacro:if>

Commit message: remove an if in xacro

File: m6_ccs_description/xacro/eefs.xacro (robot description, xacro)
@@ -258,12 +258,5 @@
             </joint>
         </xacro:if>
-        <xacro:if value="${hand_type == 'linkerhand_o6' or hand_type == 'linkerhand_l6' or hand_type == 'linkerhand_o7' or hand_type == 'freedom_v1' or hand_type == 'freedom_v2' or hand_type == 'inspire_e2' or hand_type == 'inspire_f2'}">
-            <link name="${side}_eef"/>
-            <joint name="${side}_eef_joint" type="fixed">
-                <parent link="${side}_hand_eef"/>
-                <child link="${side}_eef"/>
-            </joint>
-        </xacro:if>
-        <xacro:if value="${hand_type == 'theohand_std16a' or hand_type == 'wuji_hand2'}">
+        <xacro:if value="${hand_type == 'linkerhand_o6' or hand_type == 'linkerhand_l6' or hand_type == 'linkerhand_o7' or hand_type == 'freedom_v1' or hand_type == 'freedom_v2' or hand_type == 'inspire_e2' or hand_type == 'inspire_f2' or hand_type == 'theohand_std16a' or hand_type == 'wuji_hand2'}">
             <link name="${side}_eef"/>
             <joint name="${side}_eef_joint" type="fixed">

Commit message: update xhand position

File: m6_ccs_description/xacro/eefs.xacro (robot description, xacro)
@@ -206,14 +206,14 @@
         </xacro:if>
         <xacro:if value="${hand_type == 'xhand1'}">
-            <xacro:XHand1 name="${side}_hand" direction="${1 if side == 'left' else -1}" fixed_joints="${eef_fixed_joints}"/>
-            <joint name="${side}_hand_base_joint" type="fixed">
-                <xacro:if value="${side == 'left'}">
-                    <origin xyz="0 0 0" rpy="0 0 ${PI}"/>
-                </xacro:if>
-                <xacro:if value="${side == 'right'}">
-                    <origin xyz="0 0 0" rpy="0 0 ${PI}"/>
-                </xacro:if>
-                <parent link="${side}_tcp"/>
-                <child link="${side}_hand_hand_base"/>
+            <xacro:XHand1 name="${side}_hand" direction="${1 if side == 'left' else -1}" use_flange="true" fixed_joints="${eef_fixed_joints}"/>
+            <joint name="${side}_hand_base_joint" type="fixed">
+                <xacro:if value="${side == 'left'}">
+                    <origin xyz="0 0 0.0045" rpy="0 0 ${PI}"/>
+                </xacro:if>
+                <xacro:if value="${side == 'right'}">
+                    <origin xyz="0 0 0.0045" rpy="0 0 ${PI}"/>
+                </xacro:if>
+                <parent link="${side}_tcp"/>
+                <child link="${side}_hand_flange"/>
             </joint>
         </xacro:if>
