Commit message: Feature/gento (#23)
* add m6s lite

* add m6s lite

* update xhand position

---------

Co-authored-by: Cursor <cursoragent@cursor.com>

File: m6_ccs_description/xacro/eefs.xacro (robot description, xacro)
@@ -215,14 +215,14 @@
         </xacro:if>
         <xacro:if value="${hand_type == 'xhand1'}">
-            <xacro:XHand1 name="${side}_hand" direction="${1 if side == 'left' else -1}" fixed_joints="${eef_fixed_joints}"/>
-            <joint name="${side}_hand_base_joint" type="fixed">
-                <xacro:if value="${side == 'left'}">
-                    <origin xyz="0 0 0" rpy="0 0 ${PI}"/>
-                </xacro:if>
-                <xacro:if value="${side == 'right'}">
-                    <origin xyz="0 0 0" rpy="0 0 ${PI}"/>
-                </xacro:if>
-                <parent link="${side}_tcp"/>
-                <child link="${side}_hand_hand_base"/>
+            <xacro:XHand1 name="${side}_hand" direction="${1 if side == 'left' else -1}" use_flange="true" fixed_joints="${eef_fixed_joints}"/>
+            <joint name="${side}_hand_base_joint" type="fixed">
+                <xacro:if value="${side == 'left'}">
+                    <origin xyz="0 0 0.0045" rpy="0 0 ${PI}"/>
+                </xacro:if>
+                <xacro:if value="${side == 'right'}">
+                    <origin xyz="0 0 0.0045" rpy="0 0 ${PI}"/>
+                </xacro:if>
+                <parent link="${side}_tcp"/>
+                <child link="${side}_hand_flange"/>
             </joint>
         </xacro:if>
