Commit message: update mesh

File: marvin_pro_description/xacro/components/base.xacro (robot description, xacro)
@@ -81,5 +81,5 @@
       <visual>
         <geometry>
-          <mesh filename="file://$(find sensor_models)/meshes/gsml_camera/Sensing-SHW5G.glb"/>
+          <mesh filename="file://$(find sensor_models)/meshes/sensing/SHW5G.glb"/>
         </geometry>
       </visual>
@@ -93,5 +93,5 @@
       <visual>
         <geometry>
-          <mesh filename="file://$(find sensor_models)/meshes/gsml_camera/Sensing-SHW5G.glb"/>
+          <mesh filename="file://$(find sensor_models)/meshes/sensing/SHW5G.glb"/>
         </geometry>
       </visual>
