Commit message: 新增：添加了 m20s real hardware

File: m20s_ccs_description/xacro/eefs.xacro (robot description, xacro)
@@ -7,4 +7,69 @@
 	<xacro:include filename="$(find changingtek_description)/xacro/AG2F90-C.xacro"/>
 	<xacro:include filename="$(find changingtek_description)/xacro/AG2F120S.xacro"/>
+	<!-- Per-side default load (dyn_param) for MarvinHardware; 10 values: m, mx, my, mz, ixx, ixy, ixz, iyy, iyz, izz.
+	     Override via launch left_dyn_param/right_dyn_param (robot.local.yaml).
+	     No end effector (empty ee_key) -> all zeros. -->
+	<xacro:macro name="ee_dyn_param" params="side ee_key arg_val">
+		<xacro:if value="${arg_val != ''}">
+			<param name="${side}_dyn_param">${arg_val}</param>
+		</xacro:if>
+		<xacro:unless value="${arg_val != ''}">
+			<xacro:if value="${ee_key == '' or ee_key == 'none'}">
+				<param name="${side}_dyn_param">0,0,0,0,0,0,0,0,0,0</param>
+			</xacro:if>
+			<xacro:unless value="${ee_key == '' or ee_key == 'none'}">
+			<xacro:if value="${side == 'left'}">
+				<xacro:if value="${ee_key == 'rg75'}">
+					<param name="${side}_dyn_param">1.6200799541791235, 1.4285009257202586, -0.5789585762443014, 104.39051192831192, 0.004873874899366342, 0.0, 0.0, 0.001, 0.0, 0.0019355638096347936</param>
+				</xacro:if>
+				<xacro:if value="${ee_key == 'erg32'}">
+					<!-- TODO: replace with measured ERG32 values -->
+					<param name="${side}_dyn_param">1.6200799541791235, 1.4285009257202586, -0.5789585762443014, 104.39051192831192, 0.004873874899366342, 0.0, 0.0, 0.001, 0.0, 0.0019355638096347936</param>
+				</xacro:if>
+				<xacro:if value="${ee_key == 'ag2f90_c' or ee_key == 'ag2f90_d' or ee_key == 'ag2f90_c_soft'}">
+					<param name="${side}_dyn_param">0.9464750422461978, -8.366166030270293, -9.50810456883501, 71.59365292895114, 0.02313627009490121, 0.0, 0.0, 0.017136701127687514, 0.0, 0.008640226166892327</param>
+				</xacro:if>
+				<xacro:if value="${ee_key == 'ag2f120s' or ee_key == 'ag2f120s_d'}">
+					<!-- TODO: replace with measured values; temporarily reuse ag2f90 series -->
+					<param name="${side}_dyn_param">1.3944348661120496, -7.913087934362548, 10.50004773179898, 72.44110460800299, 0.014948849408945898, 0.0, 0.0, 0.005470384569170036, 0.0, 0.002567996881581655</param>
+				</xacro:if>
+				<xacro:if value="${ee_key == 'linkerhand_o6'}">
+					<param name="${side}_dyn_param">0.6,0,0,70.0,0,0,0,0,0,0</param>
+				</xacro:if>
+				<xacro:if value="${ee_key == 'linkerhand_l6'}">
+					<param name="${side}_dyn_param">0.6929861562459377, -0.02709362955502027, 21.325042427584716, 142.0468769124068, 0.001, 0.0, 0.0, 0.001, 0.0, 0.004408438461135547</param>
+				</xacro:if>
+				<xacro:if value="${ee_key == 'linkerhand_o7'}">
+					<param name="${side}_dyn_param">0.8,0,0,85.0,0,0,0,0,0,0</param>
+				</xacro:if>
+			</xacro:if>
+			<xacro:if value="${side == 'right'}">
+				<xacro:if value="${ee_key == 'rg75'}">
+					<param name="${side}_dyn_param">1.6200799541791235, 1.4285009257202586, -0.5789585762443014, 104.39051192831192, 0.004873874899366342, 0.0, 0.0, 0.001, 0.0, 0.0019355638096347936</param>
+				</xacro:if>
+				<xacro:if value="${ee_key == 'erg32'}">
+					<!-- TODO: replace with measured ERG32 values -->
+					<param name="${side}_dyn_param">1.6200799541791235, 1.4285009257202586, -0.5789585762443014, 104.39051192831192, 0.004873874899366342, 0.0, 0.0, 0.001, 0.0, 0.0019355638096347936</param>
+				</xacro:if>
+				<xacro:if value="${ee_key == 'ag2f90_c' or ee_key == 'ag2f90_d' or ee_key == 'ag2f90_c_soft'}">
+					<param name="${side}_dyn_param">0.9464750422461978, -8.366166030270293, -9.50810456883501, 71.59365292895114, 0.02313627009490121, 0.0, 0.0, 0.017136701127687514, 0.0, 0.008640226166892327</param>
+				</xacro:if>
+				<xacro:if value="${ee_key == 'ag2f120s' or ee_key == 'ag2f120s_d'}">
+					<!-- TODO: replace with measured values; temporarily reuse ag2f90 series -->
+					<param name="${side}_dyn_param">1.4038028109970075, 3.8873998644204817, -10.865529763155825, 73.06884012186562, 0.001, 0.0, 0.0, 0.001, 0.0, 0.0057238484709952525</param>
+				</xacro:if>
+				<xacro:if value="${ee_key == 'linkerhand_o6'}">
+					<param name="${side}_dyn_param">1.6200799541791235, 1.4285009257202586, -0.5789585762443014, 104.39051192831192, 0.004873874899366342, 0.0, 0.0, 0.001, 0.0, 0.0019355638096347936</param>
+				</xacro:if>
+				<xacro:if value="${ee_key == 'linkerhand_l6'}">
+					<param name="${side}_dyn_param">0.757127258546731, -18.86292230512758, -23.37191007763647, 69.11766685323222, 0.02103669807705659, 0.0, 0.0, 0.01131025204380805, 0.0, 0.00955246486803428</param>
+				</xacro:if>
+				<xacro:if value="${ee_key == 'linkerhand_o7'}">
+					<param name="${side}_dyn_param">0.8,0,0,85.0,0,0,0,0,0,0</param>
+				</xacro:if>
+			</xacro:if>
+			</xacro:unless>
+		</xacro:unless>
+	</xacro:macro>
 	<xacro:macro name="Ocs2SideEefFrame" params="side parent_link">
 		<link name="${side}_eef"/>

File: m20s_ccs_description/xacro/robot.xacro (robot description, xacro)
@@ -9,4 +9,6 @@
 	<xacro:arg name="right_tcp_offset_xyz" default="0 0 0"/>
 	<xacro:arg name="right_tcp_offset_rpy" default="0 0 0"/>
+	<!-- eef_fixed_joints: declared in arm.xacro (included below); used by EndEffectors -->
+	<!-- 从 type 参数解析 arm_config / 对称末端 -->
 	<xacro:property name="type_arg" value="$(arg type)"/>
 	<xacro:property name="left_type_arg" value="$(arg left_type)"/>
@@ -14,7 +16,10 @@
 	<xacro:property name="effective_left_type" value="${left_type_arg if left_type_arg != '' else type_arg}"/>
 	<xacro:property name="effective_right_type" value="${right_type_arg if right_type_arg != '' else type_arg}"/>
+	<!-- 默认值 -->
 	<xacro:property name="selected_arm_config" value="dual"/>
 	<xacro:property name="selected_gripper_type" value="none"/>
 	<xacro:property name="selected_gripper_pad" value="default"/>
+	<!-- 从 type 解析 arm_config 和 gripper_type -->
+	<!-- 单臂配置 -->
 	<xacro:if value="${type_arg == 'left'}">
 		<xacro:property name="selected_arm_config" value="left"/>
@@ -23,4 +28,6 @@
 		<xacro:property name="selected_arm_config" value="right"/>
 	</xacro:if>
+	<!-- 双臂配置 -->
+	<!-- 适用于人形机器人的配置 -->
 	<xacro:if value="${type_arg == 'ag2f90'}">
 		<xacro:property name="selected_gripper_type" value="ag2f90_d"/>
@@ -47,4 +54,5 @@
 	<xacro:include filename="$(find m20s_ccs_description)/xacro/arm.xacro"/>
 	<xacro:include filename="$(find m6_ccs_description)/xacro/arm_mount.xacro"/>
+	<!-- 单左臂 -->
 	<xacro:if value="${selected_arm_config == 'left'}">
 		<xacro:M20S_CCS side="left"
@@ -60,4 +68,5 @@
 		</xacro:if>
 	</xacro:if>
+	<!-- 单右臂 -->
 	<xacro:if value="${selected_arm_config == 'right'}">
 		<xacro:M20S_CCS side="right"
@@ -65,4 +74,5 @@
 			tcp_offset_rpy="$(arg right_tcp_offset_rpy)"/>
 	</xacro:if>
+	<!-- 双臂配置 -->
 	<xacro:if value="${selected_arm_config == 'dual'}">
 		<link name="base_link"/>
@@ -79,5 +89,9 @@
 			<child link="arm_base"/>
 		</joint>
-		<xacro:DualArmMount parent="arm_base"/>
+		<!-- 65度角，98.785mm间距 -->
+		<xacro:DualArmMount parent="arm_base"
+			left_xyz="0 0.0494 0" right_xyz="0 -0.0494 0"
+			left_rpy="-1.1345 0 0" right_rpy="1.1345 0 0"
+		/>
 		<xacro:M20S_CCS name="left"
 			tcp_offset_xyz="$(arg left_tcp_offset_xyz)"

File: m20s_ccs_description/xacro/ros2_control/end_effector_interfaces.xacro (robot description, xacro)
@@ -30,24 +30,69 @@
 		</xacro:if>
 	</xacro:macro>
+	<!--
+		Real (arm body bus) tool interfaces: MarvinHardware drives a gripper through
+		a single position command / position state interface.
+		ERG32 is a 2-DOF tool (rotate + grip) and keeps its full interface set.
+	-->
+	<xacro:macro name="side_gripper_joint" params="side gripper_type:=''">
+		<xacro:if value="${gripper_type == 'erg32'}">
+			<xacro:erg32_interfaces name="${side}_hand"/>
+		</xacro:if>
+		<xacro:unless value="${gripper_type == 'erg32'}">
+			<joint name="${side}_gripper_joint">
+				<command_interface name="position"/>
+				<state_interface name="position">
+					<param name="initial_value">0</param>
+				</state_interface>
+			</joint>
+		</xacro:unless>
+	</xacro:macro>
+	<!-- mode: sim | real -->
 	<xacro:macro name="dual_arm_ee_block" params="mode">
 		<xacro:m20s_interfaces name="left"/>
 		<xacro:m20s_interfaces name="right"/>
-		<xacro:if value="${left_gripper_type != ''}">
-			<xacro:side_gripper_interfaces_sim side="left" gripper_type="${left_gripper_type}"/>
+		<xacro:if value="${mode == 'sim'}">
+			<xacro:if value="${left_gripper_type != ''}">
+				<xacro:side_gripper_interfaces_sim side="left" gripper_type="${left_gripper_type}"/>
+			</xacro:if>
+			<xacro:if value="${right_gripper_type != ''}">
+				<xacro:side_gripper_interfaces_sim side="right" gripper_type="${right_gripper_type}"/>
+			</xacro:if>
+			<xacro:if value="${left_hand_type != ''}">
+				<xacro:side_hand_interfaces side="left" hand_type="${left_hand_type}"/>
+			</xacro:if>
+			<xacro:if value="${right_hand_type != ''}">
+				<xacro:side_hand_interfaces side="right" hand_type="${right_hand_type}"/>
+			</xacro:if>
 		</xacro:if>
-		<xacro:if value="${right_gripper_type != ''}">
-			<xacro:side_gripper_interfaces_sim side="right" gripper_type="${right_gripper_type}"/>
-		</xacro:if>
-		<xacro:if value="${left_hand_type != ''}">
-			<xacro:side_hand_interfaces side="left" hand_type="${left_hand_type}"/>
-		</xacro:if>
-		<xacro:if value="${right_hand_type != ''}">
-			<xacro:side_hand_interfaces side="right" hand_type="${right_hand_type}"/>
+		<xacro:if value="${mode == 'real'}">
+			<!-- 臂体总线（marvin / tianji_can）的末端接口由 M20S_CCS_System 声明；
+			     usb / usb_can 由 external_ee_systems.xacro 的独立 side system 声明。 -->
+			<xacro:if value="${left_gripper_type != '' and (left_drive_type == 'marvin' or left_drive_type == 'tianji_can')}">
+				<xacro:side_gripper_joint side="left" gripper_type="${left_gripper_type}"/>
+			</xacro:if>
+			<xacro:if value="${right_gripper_type != '' and (right_drive_type == 'marvin' or right_drive_type == 'tianji_can')}">
+				<xacro:side_gripper_joint side="right" gripper_type="${right_gripper_type}"/>
+			</xacro:if>
+			<xacro:if value="${(left_drive_type == 'marvin' or left_drive_type == 'tianji_can') and left_hand_type != ''}">
+				<xacro:side_hand_interfaces side="left" hand_type="${left_hand_type}"/>
+			</xacro:if>
+			<xacro:if value="${(right_drive_type == 'marvin' or right_drive_type == 'tianji_can') and right_hand_type != ''}">
+				<xacro:side_hand_interfaces side="right" hand_type="${right_hand_type}"/>
+			</xacro:if>
 		</xacro:if>
 	</xacro:macro>
-	<xacro:macro name="single_arm_ee_block" params="mode gripper_type:=''">
+	<!-- Single left arm with optional gripper (m20s_ccs type:=left) -->
+	<xacro:macro name="single_arm_ee_block" params="mode gripper_type:=none">
 		<xacro:m20s_interfaces name=""/>
-		<xacro:if value="${gripper_type != ''}">
-			<xacro:side_gripper_interfaces_sim side="" gripper_type="${gripper_type}"/>
+		<xacro:if value="${mode == 'sim'}">
+			<xacro:if value="${gripper_type != 'none'}">
+				<xacro:side_gripper_interfaces_sim side="" gripper_type="${gripper_type}"/>
+			</xacro:if>
+		</xacro:if>
+		<xacro:if value="${mode == 'real'}">
+			<xacro:if value="${gripper_type != 'none'}">
+				<xacro:side_gripper_joint side="" gripper_type="${gripper_type}"/>
+			</xacro:if>
 		</xacro:if>
 	</xacro:macro>

File: m20s_ccs_description/xacro/ros2_control/interfaces.xacro (robot description, xacro)
@@ -5,7 +5,5 @@
 		<joint name="${prefix}joint1">
 			<command_interface name="position"/>
-			<state_interface name="position">
-				<param name="initial_value">0</param>
-			</state_interface>
+			<state_interface name="position"/>
 			<state_interface name="velocity"/>
 			<state_interface name="effort"/>
@@ -13,7 +11,5 @@
 		<joint name="${prefix}joint2">
 			<command_interface name="position"/>
-			<state_interface name="position">
-				<param name="initial_value">0</param>
-			</state_interface>
+			<state_interface name="position"/>
 			<state_interface name="velocity"/>
 			<state_interface name="effort"/>
@@ -21,7 +17,5 @@
 		<joint name="${prefix}joint3">
 			<command_interface name="position"/>
-			<state_interface name="position">
-				<param name="initial_value">0</param>
-			</state_interface>
+			<state_interface name="position"/>
 			<state_interface name="velocity"/>
 			<state_interface name="effort"/>
@@ -29,7 +23,5 @@
 		<joint name="${prefix}joint4">
 			<command_interface name="position"/>
-			<state_interface name="position">
-				<param name="initial_value">0</param>
-			</state_interface>
+			<state_interface name="position"/>
 			<state_interface name="velocity"/>
 			<state_interface name="effort"/>
@@ -37,7 +29,5 @@
 		<joint name="${prefix}joint5">
 			<command_interface name="position"/>
-			<state_interface name="position">
-				<param name="initial_value">0</param>
-			</state_interface>
+			<state_interface name="position"/>
 			<state_interface name="velocity"/>
 			<state_interface name="effort"/>
@@ -45,7 +35,5 @@
 		<joint name="${prefix}joint6">
 			<command_interface name="position"/>
-			<state_interface name="position">
-				<param name="initial_value">0</param>
-			</state_interface>
+			<state_interface name="position"/>
 			<state_interface name="velocity"/>
 			<state_interface name="effort"/>
@@ -53,7 +41,5 @@
 		<joint name="${prefix}joint7">
 			<command_interface name="position"/>
-			<state_interface name="position">
-				<param name="initial_value">0</param>
-			</state_interface>
+			<state_interface name="position"/>
 			<state_interface name="velocity"/>
 			<state_interface name="effort"/>

File: m20s_ccs_description/xacro/ros2_control/robot.xacro (robot description, xacro)
@@ -2,5 +2,26 @@
 <robot xmlns:xacro="http://www.ros.org/wiki/xacro" name="M20S_CCS">
 	<xacro:arg name="ros2_control_hardware_type" default="mock_components"/>
+	<xacro:arg name="arm_ctrl_mode" default="position"/>
+	<xacro:arg name="device_ip" default=""/>
 	<xacro:arg name="type" default="dual"/>
+	<xacro:arg name="left_ee_drive_type" default=""/>
+	<xacro:arg name="right_ee_drive_type" default=""/>
+	<xacro:property name="is_real_hardware" value="${'$(arg ros2_control_hardware_type)' == 'real'}"/>
+	<xacro:property name="ee_drive_type" value="${'marvin' if is_real_hardware else ''}"/>
+	<xacro:property name="left_drive_type" value="${'$(arg left_ee_drive_type)' if '$(arg left_ee_drive_type)' != '' else ee_drive_type}"/>
+	<xacro:property name="right_drive_type" value="${'$(arg right_ee_drive_type)' if '$(arg right_ee_drive_type)' != '' else ee_drive_type}"/>
+	<xacro:arg name="left_dyn_param" default=""/>
+	<xacro:arg name="right_dyn_param" default=""/>
+	<xacro:arg name="max_joint_speed" default="100"/>
+	<xacro:arg name="max_joint_acceleration" default="100"/>
+	<xacro:arg name="usb_left_port" default="/dev/ttyUSB0"/>
+	<xacro:arg name="usb_right_port" default="/dev/ttyUSB2"/>
+	<xacro:arg name="left_ee_can_interface" default="can0"/>
+	<xacro:arg name="right_ee_can_interface" default="can1"/>
+	<xacro:arg name="left_read_tactile" default="false"/>
+	<xacro:arg name="right_read_tactile" default="false"/>
+	<xacro:arg name="left_ee_rw_rate" default=""/>
+	<xacro:arg name="right_ee_rw_rate" default=""/>
+	<!-- left_ft / right_ft / usb_*_ft_port: see marvin_hardware.xacro -->
 	<link name="world"/>
 	<joint name="world_fixed" type="fixed">
@@ -11,15 +32,96 @@
 	<xacro:include filename="$(find m20s_ccs_description)/xacro/robot.xacro"/>
 	<xacro:include filename="$(find robot_common_launch)/xacro/ros2_control/simulation_hardware.xacro"/>
+	<!-- ===== 复用 m6_ccs 的硬件 / 力传感器 / 外接末端宏（不改动 m6 包） =====
+	     m6 侧有两个会干扰本包的 eager include，因此顺序与条件受约束：
+	       1. marvin_hardware.xacro 会 include m6 的 eefs.xacro → 同名宏覆盖本包；
+	       2. external_ee_systems.xacro 会 include m6 的 end_effector_interfaces.xacro
+	          → side_gripper_joint / dual_arm_ee_block 同名覆盖本包；且它无条件
+	          include 各 side_systems.xacro，而这些文件在 linkerhand / jodell /
+	          changingtek / theohand 中尚不存在，故只能按外接驱动条件加载
+	          （加载后 external_ee_systems 宏才存在，调用点也须同样加条件）。
+	     ft_sensor_systems.xacro 自带宏、无 include，可安全直接引入。
+	     结论：m6 文件之后必须重新引入本包 eefs / end_effector_interfaces 夺回宏定义。 -->
+	<xacro:property name="has_external_ee"
+		value="${left_drive_type == 'usb' or right_drive_type == 'usb' or left_drive_type == 'usb_can' or right_drive_type == 'usb_can'}"/>
+	<xacro:include filename="$(find m6_ccs_description)/xacro/ros2_control/marvin_hardware.xacro"/>
+	<xacro:include filename="$(find m6_ccs_description)/xacro/ros2_control/ft_sensor_systems.xacro"/>
+	<xacro:if value="${has_external_ee}">
+		<xacro:include filename="$(find m6_ccs_description)/xacro/ros2_control/external_ee_systems.xacro"/>
+	</xacro:if>
+	<!-- 以下两个 include 必须在上面 m6 的 include 之后，职责不同：
+	    - xacro/eefs.xacro：夺回被 m6 覆盖的同名宏，主要是 ee_dyn_param（负载参数表）。
+	       另需注意单臂时 xacro/robot.xacro 走的是非 dual 分支、不会引入 eefs，故此处必须显式 include。
+	    - ros2_control/end_effector_interfaces.xacro：双重职责
+	        a) 非外接驱动（marvin / tianji_can / mock）时，m6 的 external_ee_systems 未被引入，
+	            本行是 dual_arm_ee_block / single_arm_ee_block / side_gripper_joint 的唯一来源；
+	        b) 外接驱动（usb / usb_can）时，m6 的 external_ee_systems 会引入 m6 版同名宏并覆盖，
+	            本行负责夺回。m6 版 side_gripper_joint 没有 gripper_type 形参，被覆盖会直接报
+	            "Invalid parameter gripper_type"。
+	     综上：这两个 include 不可删除，也不可上移到 m6 include 之前。 -->
+	<xacro:include filename="$(find m20s_ccs_description)/xacro/eefs.xacro"/>
 	<xacro:include filename="$(find m20s_ccs_description)/xacro/ros2_control/end_effector_interfaces.xacro"/>
+	<xacro:property name="ee_block_mode" value="${'real' if is_real_hardware else 'sim'}"/>
 	<ros2_control name="M20S_CCS_System" type="system">
 		<hardware>
-			<xacro:simulation_hardware_plugin hardware_type="$(arg ros2_control_hardware_type)"/>
+			<xacro:unless value="${is_real_hardware}">
+				<xacro:simulation_hardware_plugin hardware_type="$(arg ros2_control_hardware_type)"/>
+			</xacro:unless>
+			<xacro:if value="${is_real_hardware}">
+				<xacro:marvin_hardware_block
+					arm_type="${selected_arm_config}"
+					arm_ctrl_mode="$(arg arm_ctrl_mode)"
+					max_joint_speed="$(arg max_joint_speed)"
+					max_joint_acceleration="$(arg max_joint_acceleration)"
+					device_ip="$(arg device_ip)"
+					left_dyn_param="$(arg left_dyn_param)"
+					right_dyn_param="$(arg right_dyn_param)"
+					selected_gripper_type="${selected_gripper_type}"/>
+			</xacro:if>
 		</hardware>
 		<xacro:if value="${selected_arm_config == 'dual'}">
-			<xacro:dual_arm_ee_block mode="sim"/>
+			<xacro:dual_arm_ee_block mode="${ee_block_mode}"/>
 		</xacro:if>
 		<xacro:unless value="${selected_arm_config == 'dual'}">
-			<xacro:single_arm_ee_block mode="sim" gripper_type="${selected_gripper_type}"/>
+			<xacro:single_arm_ee_block mode="${ee_block_mode}" gripper_type="${selected_gripper_type}"/>
 		</xacro:unless>
+		<xacro:marvin_ft_sensor_interfaces/>
 	</ros2_control>
+	<xacro:if value="${is_real_hardware and selected_arm_config == 'dual'}">
+		<!-- 外接 usb / usb_can：由 m6 external_ee_systems 分发（其内部已调用 ft_sensor_systems） -->
+		<xacro:if value="${has_external_ee}">
+			<xacro:external_ee_systems
+				usb_left_port="$(arg usb_left_port)"
+				usb_right_port="$(arg usb_right_port)"
+				left_ee_can_interface="$(arg left_ee_can_interface)"
+				right_ee_can_interface="$(arg right_ee_can_interface)"
+				left_read_tactile="$(arg left_read_tactile)"
+				right_read_tactile="$(arg right_read_tactile)"
+				left_ee_rw_rate="$(arg left_ee_rw_rate)"
+				right_ee_rw_rate="$(arg right_ee_rw_rate)"/>
+		</xacro:if>
+		<!-- 臂体总线（marvin / tianji_can）：只需力传感器系统 -->
+		<xacro:unless value="${has_external_ee}">
+			<xacro:ft_sensor_systems
+				left_ft="$(arg left_ft)"
+				right_ft="$(arg right_ft)"
+				usb_left_ft_port="$(arg usb_left_ft_port)"
+				usb_right_ft_port="$(arg usb_right_ft_port)"/>
+		</xacro:unless>
+	</xacro:if>
+	<xacro:arg name="gazebo" default="false"/>
+	<xacro:if value="$(arg gazebo)">
+		<gazebo>
+			<plugin filename="gz_ros2_control-system" name="gz_ros2_control::GazeboSimROS2ControlPlugin">
+				<xacro:if value="${selected_arm_config == 'dual'}">
+					<parameters>$(find m20s_ccs_description)/config/ros2_control/ros2_controllers.yaml</parameters>
+				</xacro:if>
+				<xacro:if value="${selected_arm_config == 'left'}">
+					<parameters>$(find m20s_ccs_description)/config/ros2_control/left.yaml</parameters>
+				</xacro:if>
+				<xacro:if value="${selected_arm_config == 'right'}">
+					<parameters>$(find m20s_ccs_description)/config/ros2_control/right.yaml</parameters>
+				</xacro:if>
+			</plugin>
+		</gazebo>
+	</xacro:if>
 </robot>
