Commit message: 新增：m20s不再依赖m6

File: m20s_ccs_description/xacro/robot.xacro (robot description, xacro)
@@ -53,5 +53,5 @@
 	</xacro:if>
 	<xacro:include filename="$(find m20s_ccs_description)/xacro/arm.xacro"/>
-	<xacro:include filename="$(find m6_ccs_description)/xacro/arm_mount.xacro"/>
+	<xacro:include filename="$(find m20s_ccs_description)/xacro/arm_mount.xacro"/>
 	<!-- 单左臂 -->
 	<xacro:if value="${selected_arm_config == 'left'}">

File: m20s_ccs_description/xacro/ros2_control/robot.xacro (robot description, xacro)
@@ -32,33 +32,12 @@
 	<xacro:include filename="$(find m20s_ccs_description)/xacro/robot.xacro"/>
 	<xacro:include filename="$(find robot_common_launch)/xacro/ros2_control/simulation_hardware.xacro"/>
-	<!-- ===== 复用 m6_ccs 的硬件 / 力传感器 / 外接末端宏（不改动 m6 包） =====
-	     m6 侧有两个会干扰本包的 eager include，因此顺序与条件受约束：
-	       1. marvin_hardware.xacro 会 include m6 的 eefs.xacro → 同名宏覆盖本包；
-	       2. external_ee_systems.xacro 会 include m6 的 end_effector_interfaces.xacro
-	          → side_gripper_joint / dual_arm_ee_block 同名覆盖本包；且它无条件
-	          include 各 side_systems.xacro，而这些文件在 linkerhand / jodell /
-	          changingtek / theohand 中尚不存在，故只能按外接驱动条件加载
-	          （加载后 external_ee_systems 宏才存在，调用点也须同样加条件）。
-	     ft_sensor_systems.xacro 自带宏、无 include，可安全直接引入。
-	     结论：m6 文件之后必须重新引入本包 eefs / end_effector_interfaces 夺回宏定义。 -->
-	<xacro:property name="has_external_ee"
-		value="${left_drive_type == 'usb' or right_drive_type == 'usb' or left_drive_type == 'usb_can' or right_drive_type == 'usb_can'}"/>
-	<xacro:include filename="$(find m6_ccs_description)/xacro/ros2_control/marvin_hardware.xacro"/>
-	<xacro:include filename="$(find m6_ccs_description)/xacro/ros2_control/ft_sensor_systems.xacro"/>
-	<xacro:if value="${has_external_ee}">
-		<xacro:include filename="$(find m6_ccs_description)/xacro/ros2_control/external_ee_systems.xacro"/>
-	</xacro:if>
-	<!-- 以下两个 include 必须在上面 m6 的 include 之后，职责不同：
-	    - xacro/eefs.xacro：夺回被 m6 覆盖的同名宏，主要是 ee_dyn_param（负载参数表）。
-	       另需注意单臂时 xacro/robot.xacro 走的是非 dual 分支、不会引入 eefs，故此处必须显式 include。
-	    - ros2_control/end_effector_interfaces.xacro：双重职责
-	        a) 非外接驱动（marvin / tianji_can / mock）时，m6 的 external_ee_systems 未被引入，
-	            本行是 dual_arm_ee_block / single_arm_ee_block / side_gripper_joint 的唯一来源；
-	        b) 外接驱动（usb / usb_can）时，m6 的 external_ee_systems 会引入 m6 版同名宏并覆盖，
-	            本行负责夺回。m6 版 side_gripper_joint 没有 gripper_type 形参，被覆盖会直接报
-	            "Invalid parameter gripper_type"。
-	     综上：这两个 include 不可删除，也不可上移到 m6 include 之前。 -->
-	<xacro:include filename="$(find m20s_ccs_description)/xacro/eefs.xacro"/>
-	<xacro:include filename="$(find m20s_ccs_description)/xacro/ros2_control/end_effector_interfaces.xacro"/>
+	<xacro:include filename="$(find m20s_ccs_description)/xacro/ros2_control/marvin_hardware.xacro"/>
+	<!-- 本包自有的末端接口 / 力传感器 / 外接末端宏，不再依赖 m6_ccs_description。
+	     external_ee_systems.xacro 内部会引入：
+	       - end_effector_interfaces.xacro → dual_arm_ee_block / single_arm_ee_block / side_gripper_joint；
+	       - ft_sensor_systems.xacro      → ft_sensor_systems / side_ft_sensor_system；
+	     并自包含外接 usb / usb_can 的 side system 定义。因此它可无条件引入，既不会覆盖本包
+	     同名宏，也不必再按驱动类型条件加载（旧方案必须按 usb/usb_can 条件包含 m6 文件并回夺宏）。 -->
+	<xacro:include filename="$(find m20s_ccs_description)/xacro/ros2_control/external_ee_systems.xacro"/>
 	<xacro:property name="ee_block_mode" value="${'real' if is_real_hardware else 'sim'}"/>
 	<ros2_control name="M20S_CCS_System" type="system">
@@ -88,24 +67,19 @@
 	</ros2_control>
 	<xacro:if value="${is_real_hardware and selected_arm_config == 'dual'}">
-		<!-- 外接 usb / usb_can：由 m6 external_ee_systems 分发（其内部已调用 ft_sensor_systems） -->
-		<xacro:if value="${has_external_ee}">
-			<xacro:external_ee_systems
-				usb_left_port="$(arg usb_left_port)"
-				usb_right_port="$(arg usb_right_port)"
-				left_ee_can_interface="$(arg left_ee_can_interface)"
-				right_ee_can_interface="$(arg right_ee_can_interface)"
-				left_read_tactile="$(arg left_read_tactile)"
-				right_read_tactile="$(arg right_read_tactile)"
-				left_ee_rw_rate="$(arg left_ee_rw_rate)"
-				right_ee_rw_rate="$(arg right_ee_rw_rate)"/>
-		</xacro:if>
-		<!-- 臂体总线（marvin / tianji_can）：只需力传感器系统 -->
-		<xacro:unless value="${has_external_ee}">
-			<xacro:ft_sensor_systems
-				left_ft="$(arg left_ft)"
-				right_ft="$(arg right_ft)"
-				usb_left_ft_port="$(arg usb_left_ft_port)"
-				usb_right_ft_port="$(arg usb_right_ft_port)"/>
-		</xacro:unless>
+		<!-- 外接 usb / usb_can 由本包 external_ee_systems 分发；其内部无条件调用
+		     ft_sensor_systems，故臂体总线（marvin / tianji_can）亦由此路径覆盖。 -->
+		<xacro:external_ee_systems
+			usb_left_port="$(arg usb_left_port)"
+			usb_right_port="$(arg usb_right_port)"
+			left_ee_can_interface="$(arg left_ee_can_interface)"
+			right_ee_can_interface="$(arg right_ee_can_interface)"
+			left_read_tactile="$(arg left_read_tactile)"
+			right_read_tactile="$(arg right_read_tactile)"
+			left_ee_rw_rate="$(arg left_ee_rw_rate)"
+			right_ee_rw_rate="$(arg right_ee_rw_rate)"
+			left_ft="$(arg left_ft)"
+			right_ft="$(arg right_ft)"
+			usb_left_ft_port="$(arg usb_left_ft_port)"
+			usb_right_ft_port="$(arg usb_right_ft_port)"/>
 	</xacro:if>
 	<xacro:arg name="gazebo" default="false"/>

Commit message: Feature/add m20s hardware (#20)
* 新增：添加了 m20s real hardware

* 新增：m20s不再依赖m6

File: m20s_ccs_description/xacro/robot.xacro (robot description, xacro)
@@ -9,4 +9,6 @@
 	<xacro:arg name="right_tcp_offset_xyz" default="0 0 0"/>
 	<xacro:arg name="right_tcp_offset_rpy" default="0 0 0"/>
+	<!-- eef_fixed_joints: declared in arm.xacro (included below); used by EndEffectors -->
+	<!-- 从 type 参数解析 arm_config / 对称末端 -->
 	<xacro:property name="type_arg" value="$(arg type)"/>
 	<xacro:property name="left_type_arg" value="$(arg left_type)"/>
@@ -14,7 +16,10 @@
 	<xacro:property name="effective_left_type" value="${left_type_arg if left_type_arg != '' else type_arg}"/>
 	<xacro:property name="effective_right_type" value="${right_type_arg if right_type_arg != '' else type_arg}"/>
+	<!-- 默认值 -->
 	<xacro:property name="selected_arm_config" value="dual"/>
 	<xacro:property name="selected_gripper_type" value="none"/>
 	<xacro:property name="selected_gripper_pad" value="default"/>
+	<!-- 从 type 解析 arm_config 和 gripper_type -->
+	<!-- 单臂配置 -->
 	<xacro:if value="${type_arg == 'left'}">
 		<xacro:property name="selected_arm_config" value="left"/>
@@ -23,4 +28,6 @@
 		<xacro:property name="selected_arm_config" value="right"/>
 	</xacro:if>
+	<!-- 双臂配置 -->
+	<!-- 适用于人形机器人的配置 -->
 	<xacro:if value="${type_arg == 'ag2f90'}">
 		<xacro:property name="selected_gripper_type" value="ag2f90_d"/>
@@ -46,5 +53,6 @@
 	</xacro:if>
 	<xacro:include filename="$(find m20s_ccs_description)/xacro/arm.xacro"/>
-	<xacro:include filename="$(find m6_ccs_description)/xacro/arm_mount.xacro"/>
+	<xacro:include filename="$(find m20s_ccs_description)/xacro/arm_mount.xacro"/>
+	<!-- 单左臂 -->
 	<xacro:if value="${selected_arm_config == 'left'}">
 		<xacro:M20S_CCS side="left"
@@ -60,4 +68,5 @@
 		</xacro:if>
 	</xacro:if>
+	<!-- 单右臂 -->
 	<xacro:if value="${selected_arm_config == 'right'}">
 		<xacro:M20S_CCS side="right"
@@ -65,4 +74,5 @@
 			tcp_offset_rpy="$(arg right_tcp_offset_rpy)"/>
 	</xacro:if>
+	<!-- 双臂配置 -->
 	<xacro:if value="${selected_arm_config == 'dual'}">
 		<link name="base_link"/>
@@ -79,5 +89,9 @@
 			<child link="arm_base"/>
 		</joint>
-		<xacro:DualArmMount parent="arm_base"/>
+		<!-- 65度角，98.785mm间距 -->
+		<xacro:DualArmMount parent="arm_base"
+			left_xyz="0 0.0494 0" right_xyz="0 -0.0494 0"
+			left_rpy="-1.1345 0 0" right_rpy="1.1345 0 0"
+		/>
 		<xacro:M20S_CCS name="left"
 			tcp_offset_xyz="$(arg left_tcp_offset_xyz)"

File: m20s_ccs_description/xacro/ros2_control/robot.xacro (robot description, xacro)
@@ -2,5 +2,26 @@
 <robot xmlns:xacro="http://www.ros.org/wiki/xacro" name="M20S_CCS">
 	<xacro:arg name="ros2_control_hardware_type" default="mock_components"/>
+	<xacro:arg name="arm_ctrl_mode" default="position"/>
+	<xacro:arg name="device_ip" default=""/>
 	<xacro:arg name="type" default="dual"/>
+	<xacro:arg name="left_ee_drive_type" default=""/>
+	<xacro:arg name="right_ee_drive_type" default=""/>
+	<xacro:property name="is_real_hardware" value="${'$(arg ros2_control_hardware_type)' == 'real'}"/>
+	<xacro:property name="ee_drive_type" value="${'marvin' if is_real_hardware else ''}"/>
+	<xacro:property name="left_drive_type" value="${'$(arg left_ee_drive_type)' if '$(arg left_ee_drive_type)' != '' else ee_drive_type}"/>
+	<xacro:property name="right_drive_type" value="${'$(arg right_ee_drive_type)' if '$(arg right_ee_drive_type)' != '' else ee_drive_type}"/>
+	<xacro:arg name="left_dyn_param" default=""/>
+	<xacro:arg name="right_dyn_param" default=""/>
+	<xacro:arg name="max_joint_speed" default="100"/>
+	<xacro:arg name="max_joint_acceleration" default="100"/>
+	<xacro:arg name="usb_left_port" default="/dev/ttyUSB0"/>
+	<xacro:arg name="usb_right_port" default="/dev/ttyUSB2"/>
+	<xacro:arg name="left_ee_can_interface" default="can0"/>
+	<xacro:arg name="right_ee_can_interface" default="can1"/>
+	<xacro:arg name="left_read_tactile" default="false"/>
+	<xacro:arg name="right_read_tactile" default="false"/>
+	<xacro:arg name="left_ee_rw_rate" default=""/>
+	<xacro:arg name="right_ee_rw_rate" default=""/>
+	<!-- left_ft / right_ft / usb_*_ft_port: see marvin_hardware.xacro -->
 	<link name="world"/>
 	<joint name="world_fixed" type="fixed">
@@ -11,15 +32,70 @@
 	<xacro:include filename="$(find m20s_ccs_description)/xacro/robot.xacro"/>
 	<xacro:include filename="$(find robot_common_launch)/xacro/ros2_control/simulation_hardware.xacro"/>
-	<xacro:include filename="$(find m20s_ccs_description)/xacro/ros2_control/end_effector_interfaces.xacro"/>
+	<xacro:include filename="$(find m20s_ccs_description)/xacro/ros2_control/marvin_hardware.xacro"/>
+	<!-- 本包自有的末端接口 / 力传感器 / 外接末端宏，不再依赖 m6_ccs_description。
+	     external_ee_systems.xacro 内部会引入：
+	       - end_effector_interfaces.xacro → dual_arm_ee_block / single_arm_ee_block / side_gripper_joint；
+	       - ft_sensor_systems.xacro      → ft_sensor_systems / side_ft_sensor_system；
+	     并自包含外接 usb / usb_can 的 side system 定义。因此它可无条件引入，既不会覆盖本包
+	     同名宏，也不必再按驱动类型条件加载（旧方案必须按 usb/usb_can 条件包含 m6 文件并回夺宏）。 -->
+	<xacro:include filename="$(find m20s_ccs_description)/xacro/ros2_control/external_ee_systems.xacro"/>
+	<xacro:property name="ee_block_mode" value="${'real' if is_real_hardware else 'sim'}"/>
 	<ros2_control name="M20S_CCS_System" type="system">
 		<hardware>
-			<xacro:simulation_hardware_plugin hardware_type="$(arg ros2_control_hardware_type)"/>
+			<xacro:unless value="${is_real_hardware}">
+				<xacro:simulation_hardware_plugin hardware_type="$(arg ros2_control_hardware_type)"/>
+			</xacro:unless>
+			<xacro:if value="${is_real_hardware}">
+				<xacro:marvin_hardware_block
+					arm_type="${selected_arm_config}"
+					arm_ctrl_mode="$(arg arm_ctrl_mode)"
+					max_joint_speed="$(arg max_joint_speed)"
+					max_joint_acceleration="$(arg max_joint_acceleration)"
+					device_ip="$(arg device_ip)"
+					left_dyn_param="$(arg left_dyn_param)"
+					right_dyn_param="$(arg right_dyn_param)"
+					selected_gripper_type="${selected_gripper_type}"/>
+			</xacro:if>
 		</hardware>
 		<xacro:if value="${selected_arm_config == 'dual'}">
-			<xacro:dual_arm_ee_block mode="sim"/>
+			<xacro:dual_arm_ee_block mode="${ee_block_mode}"/>
 		</xacro:if>
 		<xacro:unless value="${selected_arm_config == 'dual'}">
-			<xacro:single_arm_ee_block mode="sim" gripper_type="${selected_gripper_type}"/>
+			<xacro:single_arm_ee_block mode="${ee_block_mode}" gripper_type="${selected_gripper_type}"/>
 		</xacro:unless>
+		<xacro:marvin_ft_sensor_interfaces/>
 	</ros2_control>
+	<xacro:if value="${is_real_hardware and selected_arm_config == 'dual'}">
+		<!-- 外接 usb / usb_can 由本包 external_ee_systems 分发；其内部无条件调用
+		     ft_sensor_systems，故臂体总线（marvin / tianji_can）亦由此路径覆盖。 -->
+		<xacro:external_ee_systems
+			usb_left_port="$(arg usb_left_port)"
+			usb_right_port="$(arg usb_right_port)"
+			left_ee_can_interface="$(arg left_ee_can_interface)"
+			right_ee_can_interface="$(arg right_ee_can_interface)"
+			left_read_tactile="$(arg left_read_tactile)"
+			right_read_tactile="$(arg right_read_tactile)"
+			left_ee_rw_rate="$(arg left_ee_rw_rate)"
+			right_ee_rw_rate="$(arg right_ee_rw_rate)"
+			left_ft="$(arg left_ft)"
+			right_ft="$(arg right_ft)"
+			usb_left_ft_port="$(arg usb_left_ft_port)"
+			usb_right_ft_port="$(arg usb_right_ft_port)"/>
+	</xacro:if>
+	<xacro:arg name="gazebo" default="false"/>
+	<xacro:if value="$(arg gazebo)">
+		<gazebo>
+			<plugin filename="gz_ros2_control-system" name="gz_ros2_control::GazeboSimROS2ControlPlugin">
+				<xacro:if value="${selected_arm_config == 'dual'}">
+					<parameters>$(find m20s_ccs_description)/config/ros2_control/ros2_controllers.yaml</parameters>
+				</xacro:if>
+				<xacro:if value="${selected_arm_config == 'left'}">
+					<parameters>$(find m20s_ccs_description)/config/ros2_control/left.yaml</parameters>
+				</xacro:if>
+				<xacro:if value="${selected_arm_config == 'right'}">
+					<parameters>$(find m20s_ccs_description)/config/ros2_control/right.yaml</parameters>
+				</xacro:if>
+			</plugin>
+		</gazebo>
+	</xacro:if>
 </robot>
